File: dcdc-regulator-test/dcdc-regulator-test.kicad_pcb (KiCad board)
At the start: 2 copper layers, 8 parts, among them U1 AP63205WU, U2 MIC5504-3.3YM5

Commit message: example layout
Parts:
- U2: footprint Package_TO_SOT_SMD:SOT-23-5_HandSoldering -> Package_TO_SOT_SMD:SOT-23-5
- moved U1 43.0 mm to (76.2, 76.2)
- moved C1 35.1 mm to (76.2, 79.2), turned to 180 degrees
- moved L1 32.5 mm to (83.2, 74.9)
- moved C3 30.8 mm to (77.5, 73.0)
- moved C2 30.4 mm to (80.0, 79.2)
- moved C5 12.1 mm to (118.1, 69.8), turned to 90 degrees
- moved C4 4.59 mm to (110.5, 69.8), turned to 90 degrees
- moved U2 1.59 mm to (114.3, 71.1)
Routing:
- net +5V: track 0.00 -> 26.8 mm, vias 0 -> 2
- net Net-(U1-SW): track 0.00 -> 7.54 mm
- net +3V3: track 0.00 -> 3.02 mm
- net Net-(U1-BST): track 0.00 -> 2.71 mm
- added copper zone on F.Cu, net GND
