File: Libraries/design_blocks_library.kicad_blocks/LINREG_3V3_300mA.kicad_block/LINREG_3V3_300mA.kicad_sch (KiCad schematic)
At the start: 3 parts, among them U2 MIC5504-3.3YM5

Commit message: Fixed design block formatting
Other:
- company: (none) -> Formula Slug
- title: (none) -> Linear Regulator 3.3V 300mA
Changed lines of the file:
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@@
 	(generator_version "9.0")
 	(paper "B")
+	(title_block
+		(title "Linear Regulator 3.3V 300mA")
+		(date "2025-08-23")
+		(rev "1.0")
+		(company "Formula Slug")
+	)
 	(junction
 		(at 165.1 54.61)
@@
 		(dnp no)
 		(fields_autoplaced yes)
-		(property "Reference" "U2"
+		(property "Reference" "U?"
 			(at 184.15 46.99 0)
 			(effects
@@
 				(path "/1eaf6089-efbb-4c23-ad74-83bc24c8d4ef"
 					(reference "U2")
+					(unit 1)
+				)
+			)
+			(project "LINREG_3V3_300mA"
+				(path "/80430d07-2ce8-4c8d-ad3b-445ca3ced0f3"
+					(reference "U?")
 					(unit 1)
 				)
@@
 		(on_board yes)
 		(dnp no)
-		(property "Reference" "C5"
+		(property "Reference" "C?"
 			(at 199.39 58.42 0)
 			(effects
@@
 				(path "/1eaf6089-efbb-4c23-ad74-83bc24c8d4ef"
 					(reference "C5")
+					(unit 1)
+				)
+			)
+			(project "LINREG_3V3_300mA"
+				(path "/80430d07-2ce8-4c8d-ad3b-445ca3ced0f3"
+					(reference "C?")
 					(unit 1)
 				)
@@
 		(on_board yes)
 		(dnp no)
-		(property "Reference" "C4"
+		(property "Reference" "C?"
 			(at 167.64 58.42 0)
 			(effects
@@
 				(path "/1eaf6089-efbb-4c23-ad74-83bc24c8d4ef"
 					(reference "C4")
+					(unit 1)
+				)
+			)
+			(project "LINREG_3V3_300mA"
+				(path "/80430d07-2ce8-4c8d-ad3b-445ca3ced0f3"
+					(reference "C?")
 					(unit 1)
 				)
@@
 		(dnp no)
 		(fields_autoplaced yes)
-		(property "Reference" "#PWR03"
+		(property "Reference" "#PWR?"
 			(at 184.15 71.12 0)
 			(effects
@@
 				(path "/1eaf6089-efbb-4c23-ad74-83bc24c8d4ef"
 					(reference "#PWR03")
+					(unit 1)
+				)
+			)
+			(project "LINREG_3V3_300mA"
+				(path "/80430d07-2ce8-4c8d-ad3b-445ca3ced0f3"
+					(reference "#PWR?")
 					(unit 1)
 				)
@@
 		(dnp no)
 		(fields_autoplaced yes)
-		(property "Reference" "#PWR02"
+		(property "Reference" "#PWR?"
 			(at 196.85 58.42 0)
 			(effects
@@
 				(path "/1eaf6089-efbb-4c23-ad74-83bc24c8d4ef"
 					(reference "#PWR02")
+					(unit 1)
+				)
+			)
+			(project "LINREG_3V3_300mA"
+				(path "/80430d07-2ce8-4c8d-ad3b-445ca3ced0f3"
+					(reference "#PWR?")
 					(unit 1)
 				)
@@
 		(dnp no)
 		(fields_autoplaced yes)
-		(property "Reference" "#PWR01"
+		(property "Reference" "#PWR?"
 			(at 165.1 58.42 0)
 			(effects
@@
 				)
 			)
-		)
-	)
+			(project "LINREG_3V3_300mA"
+				(path "/80430d07-2ce8-4c8d-ad3b-445ca3ced0f3"
+					(reference "#PWR?")
+					(unit 1)
+				)
+			)
+		)
+	)
+	(sheet_instances
+		(path "/"
+			(page "1")
+		)
+	)
+	(embedded_fonts no)
 )
