File: stm32-test/stm32-test.kicad_pcb (KiCad board)
At the start: 2 copper layers, 12 parts, among them J2 Conn_01x04_Pin, SW2 SW_Push, U1 STM32G441KBTx, U2 AP63205WU, U3 MIC5504-3.3YM5, U4 ISO1050DUB

Commit message: working on pcb now
Parts:
- added C1: 10uF, Capacitor_SMD:C_0805_2012Metric_Pad1.18x1.45mm_HandSolder, F.Cu at (131.5, 85.5)
- added C15: 100nF, Capacitor_SMD:C_0805_2012Metric_Pad1.18x1.45mm_HandSolder, F.Cu at (165.6, 104.7)
- added C16: 100nF, Capacitor_SMD:C_0805_2012Metric_Pad1.18x1.45mm_HandSolder, F.Cu at (165.6, 107.7)
- added C2: 100nF, Capacitor_SMD:C_0805_2012Metric_Pad1.18x1.45mm_HandSolder, F.Cu at (131.5, 82.0)
- added C3: 10uF, Capacitor_SMD:C_0805_2012Metric_Pad1.18x1.45mm_HandSolder, F.Cu at (143.0, 95.5)
- added C4: 100nF, Capacitor_SMD:C_0805_2012Metric_Pad1.18x1.45mm_HandSolder, F.Cu at (143.1, 97.5)
- added C5: 100nF, Capacitor_SMD:C_0805_2012Metric_Pad1.18x1.45mm_HandSolder, F.Cu at (139.0, 97.5)
- added C6: 1uF, Capacitor_SMD:C_0805_2012Metric_Pad1.18x1.45mm_HandSolder, F.Cu at (139.0, 99.5)
- added C7: 100nF, Capacitor_SMD:C_0805_2012Metric_Pad1.18x1.45mm_HandSolder, F.Cu at (160.7, 98.7)
- added C8: 6.8pF, Capacitor_SMD:C_0805_2012Metric_Pad1.18x1.45mm_HandSolder, F.Cu at (160.7, 101.7)
- added C9: 6.8pF, Capacitor_SMD:C_0805_2012Metric_Pad1.18x1.45mm_HandSolder, F.Cu at (160.7, 104.7)
- added J1: Conn_01x04, Connector_Molex:Molex_Nano-Fit_105309-xx04_1x04_P2.50mm_Vertical, F.Cu at (184.5, 111.3)
- added J3: Conn_02x04_Top_Bottom, Connector_Molex:Molex_Nano-Fit_105310-xx08_2x04_P2.50mm_Vertical, F.Cu at (173.6, 111.3)
- added J4: Conn_01x02_Pin, Connector_PinSocket_2.54mm:PinSocket_1x02_P2.54mm_Vertical, F.Cu at (155.8, 117.6)
- added J5: Conn_01x02_Pin, Connector_PinSocket_2.54mm:PinSocket_1x02_P2.54mm_Vertical, F.Cu at (160.4, 117.6)
- added J6: Conn_01x02_Pin, Connector_PinSocket_2.54mm:PinSocket_1x02_P2.54mm_Vertical, F.Cu at (165.1, 117.6)
- added R1: 10k, Resistor_SMD:R_0805_2012Metric_Pad1.20x1.40mm_HandSolder, F.Cu at (183.8, 123.1)
- added R2: 4.7k, Resistor_SMD:R_0805_2012Metric_Pad1.20x1.40mm_HandSolder, F.Cu at (183.8, 126.0)
- added R3: 4.7k, Resistor_SMD:R_0805_2012Metric_Pad1.20x1.40mm_HandSolder, F.Cu at (183.8, 129.0)
- added Y1: 24MHz, Crystal:Crystal_SMD_2012-2Pin_2.0x1.2mm_HandSoldering, F.Cu at (184.6, 102.0)
- added Y2: 24MHz, Crystal:Crystal_SMD_2016-4Pin_2.0x1.6mm, F.Cu at (181.8, 105.5)
- moved U1 47.1 mm to (137.5, 91.0)
- moved C13 24.5 mm to (165.6, 98.7)
- moved C14 24.5 mm to (165.6, 101.7)
- moved J2 21.6 mm to (188.5, 123.9)
- moved L1 20.7 mm to (172.0, 131.4)
- moved U4 16.0 mm to (160.0, 127.8)
- moved SW2 14.9 mm to (172.1, 124.8)
- moved C12 9.50 mm to (160.7, 113.7)
- moved C10 9.50 mm to (160.7, 107.7)
- moved C11 9.50 mm to (160.7, 110.7)
- moved U2 7.28 mm to (178.9, 124.0)
- moved U3 7.28 mm to (178.9, 128.6)
Connections:
- J2 pad 1: unconnected-(J2-Pin_1-Pad1) -> /SPI_MOSI
- J2 pad 2: unconnected-(J2-Pin_2-Pad2) -> /SPI_MISO
- J2 pad 3: unconnected-(J2-Pin_3-Pad3) -> /SPI_CLK
- J2 pad 4: unconnected-(J2-Pin_4-Pad4) -> /SPI_CS
- U1 pad 2: Net-(U1-PF0) -> /OSC_IN
- U1 pad 3: Net-(U1-PF1) -> /OSC_OUT
- U1 pad 31: Net-(U1-PB8) -> /BOOT0

Commit message: stm32-test progress; added global symbol & footprint libraries
Parts:
- removed Y1: 24MHz, Crystal:Crystal_SMD_2012-2Pin_2.0x1.2mm_HandSoldering
- added SW1: TL3302AF180QJ, fs_4_footprint_library:SW_TL3302AF180QJ_EWI, F.Cu at (125.0, 88.5)
- SW2: footprint Button_Switch_SMD:SW_SPST_PTS647_Sx50 -> Button_Switch_SMD:SW_SPST_PTS647_Sx38
- moved J2 70.5 mm to (121.4, 102.4), turned to 180 degrees
- moved L1 69.8 mm to (103.3, 119.2)
- moved U2 69.8 mm to (110.2, 111.8)
- moved U3 69.8 mm to (110.2, 116.4)
- moved SW2 62.7 mm to (125.0, 83.4)
- moved C13 62.1 mm to (104.6, 110.8)
- moved C14 62.1 mm to (104.6, 113.8)
- moved R1 58.6 mm to (140.7, 83.3), turned to 90 degrees
- moved Y2 53.3 mm to (133.1, 83.8)
- moved R3 52.8 mm to (140.7, 98.6), turned to 90 degrees
- moved R2 49.4 mm to (142.7, 98.6), turned to 90 degrees
- moved J3 46.3 mm to (149.2, 71.9)
- moved C12 45.2 mm to (116.9, 124.4)
- moved C10 45.2 mm to (116.9, 118.4)
- moved C11 45.2 mm to (116.9, 121.4)
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Connections:
- U1 pad 7: unconnected-(U1-PA2-Pad7) -> /UART_TX
- U1 pad 8: unconnected-(U1-PA3-Pad8) -> /UART_RX
Routing:
- net GND: track 0.00 -> 20.6 mm
- net +3V3: track 0.00 -> 11.6 mm, vias 0 -> 3
- net /NRST: track 0.00 -> 8.79 mm
- net /OSC_OUT: track 0.00 -> 6.88 mm
- net /OSC_IN: track 0.00 -> 6.45 mm
- net Net-(U1-VDDA): track 0.00 -> 5.87 mm
- net /I2C_SCL: track 0.00 -> 4.14 mm
- net /I2C_SDA: track 0.00 -> 2.88 mm
- net /BOOT0: track 0.00 -> 2.88 mm
- added copper zone on In1.Cu, net +3V3
- added copper zone on B.Cu, net GND
- added copper zone on F.Cu, net GND
- added copper zone on In2.Cu, net GND
Other:
- copper layers 2 -> 4
