File: stm32-test/stm32-test.kicad_sch (KiCad schematic)
At the start: 15 parts, among them J1 Conn_01x04, J2 Conn_02x03_Top_Bottom, SW1 SW_SPST, U1 STM32G441KBTx, Y1 24MHz

Commit message: save (wip)
Parts:
- removed J2: Conn_02x03_Top_Bottom, symbol Connector_Generic:Conn_02x03_Top_Bottom
- removed SW1: SW_SPST, symbol Switch:SW_SPST
- added C10: 10uF, Capacitor_SMD:C_0805_2012Metric_Pad1.18x1.45mm_HandSolder, symbol Device:C
- added C11: 100nF, Capacitor_SMD:C_0805_2012Metric_Pad1.18x1.45mm_HandSolder, symbol Device:C
- added C12: 47uF, Capacitor_SMD:C_0805_2012Metric_Pad1.18x1.45mm_HandSolder, symbol Device:C
- added C13, C14: 1uF, Capacitor_SMD:C_0805_2012Metric_Pad1.18x1.45mm_HandSolder, symbol Device:C
- added C15, C16: 100nF, symbol Device:C
- added J2: Conn_01x04_Pin, Connector_PinHeader_2.54mm:PinHeader_1x04_P2.54mm_Vertical, symbol Connector:Conn_01x04_Pin
- added J3: Conn_02x04_Top_Bottom, symbol Connector_Generic:Conn_02x04_Top_Bottom
- added L1: 4.7uF, Inductor_SMD:L_Bourns_SRP5030T, symbol Device:L
- added R2, R3: 4.7k, symbol Device:R
- added SW2: SW_Push, Button_Switch_SMD:SW_SPST_PTS647_Sx50, symbol Switch:SW_Push
- added U2: AP63205WU, Package_TO_SOT_SMD:TSOT-23-6, symbol Regulator_Switching:AP63205WU
- added U3: MIC5504-3.3YM5, Package_TO_SOT_SMD:SOT-23-5, symbol Regulator_Linear:MIC5504-3.3YM5
- added U4: ISO1050DUB, Package_SO:SOP-8_6.62x9.15mm_P2.54mm, symbol Interface_CAN_LIN:ISO1050DUB
Connections:
- net +3V3: now also C14.2, J3.1 (Pin_1), R2.1, R3.1, U3.5 (VOUT)
- net CANH: now also U4.7 (CANH)
- net CANL: now also U4.6 (CANL)
- net GND: now also C10.1, C12.1, C13.1, C14.1, J3.4 (Pin_4), SW2.1, U2.4 (GND), U3.2 (GND)
- net NRST: now also J3.8 (Pin_8), SW2.2
- net STLINK_SWCLK: now also J3.2 (Pin_2)
- net STLINK_SWDIO: now also J3.3 (Pin_3)
- net STLINK_SWO: now also J3.7 (Pin_7)
- net SPI_CLK: now reaches U1.10 (PA5)
- net SPI_MISO: now reaches U1.11 (PA6)
- net SPI_MOSI: now reaches U1.12 (PA7)
- net SPI_MOSI: now also J2.2 (Pin_2)
- net I2C_SDA: now reaches U1.18 (PA8)
- net I2C_SDA: now also R3.2
- net I2C_SCL: now reaches U1.19 (PA9)
- net I2C_SCL: now also R2.2
- net at U1.2 (PF0): now also C8.1, Y1.2
- net CAN_RX: now reaches U1.21 (PA11)
- net CAN_RX: now also U4.2 (RXD)
- net CAN_TX: now reaches U1.22 (PA12)
- net CAN_TX: now also U4.3 (TXD)
- net at U1.3 (PF1): now also C9.1, Y1.1
- net SPI_CS: now reaches U1.9 (PA4)
- new net: C15.1, U4.1 (VCC1)
- new net: C15.2, U4.4 (GND1)
- new net: C11.1, L1.1, U2.5 (SW)
- new net: C11.2, U2.6 (BST)
- new net: C16.2, U4.5 (GND2)
- new net: C16.1, U4.8 (VCC2)
- new net +12V: C10.2, U2.2 (EN), U2.3 (IN)
- new net +5V: C12.2, C13.2, L1.2, U2.1 (FB), U3.1 (VIN), U3.3 (EN)
- new net UART_RX: J3.6 (Pin_6)
- new net UART_TX: J3.5 (Pin_5)
- no-connect marks 0 -> 10
Other:
- note added: "CAN Tranceiver"
- note added: "MCU"
- note added: "Power Circuitry"
- moved on the sheet: C1, C2, C3, C4, C5, C6, C7, C8, C9, J1, R1, U1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

Commit message: working on pcb now
Parts:
- removed Y1: 24MHz, symbol Device:Crystal
- added J4, J5, J6: Conn_01x02_Pin, Connector_PinSocket_2.54mm:PinSocket_1x02_P2.54mm_Vertical, symbol Connector:Conn_01x02_Pin
- added Y2: 24MHz, Crystal:Crystal_SMD_2016-4Pin_2.0x1.6mm, symbol Device:Crystal_GND24
- C1, C15, C16, C2, C3, C4, C5, C6, C7, C8, C9: footprint (none) -> Capacitor_SMD:C_0805_2012Metric_Pad1.18x1.45mm_HandSolder
- J1: footprint (none) -> Connector_Molex:Molex_Nano-Fit_105309-xx04_1x04_P2.50mm_Vertical
- J3: footprint (none) -> Connector_Molex:Molex_Nano-Fit_105310-xx08_2x04_P2.50mm_Vertical
- R1, R2, R3: footprint (none) -> Resistor_SMD:R_0805_2012Metric_Pad1.20x1.40mm_HandSolder
Connections:
- net +3V3: now also J4.1 (Pin_1), J6.1 (Pin_1)
- net GND: now also J4.2 (Pin_2), J6.2 (Pin_2), Y2.2, Y2.4
- net I2C_SDA: now also J5.1 (Pin_1), J5.2 (Pin_2)
- net SPI_CLK: now also J2.3 (Pin_3)
- net SPI_CS: now also J2.4 (Pin_4)
- net SPI_MISO: now also J2.2 (Pin_2)
- net SPI_MOSI: now also J2.1 (Pin_1); no longer J2.2 (Pin_2)
- net OSC_IN: now reaches C8.1, U1.2 (PF0)
- net OSC_IN: now also Y2.3
- net OSC_OUT: now reaches C9.1, U1.3 (PF1)
- net OSC_OUT: now also Y2.1
- net BOOT0: now reaches R1.1, U1.31 (PB8)
Other:
- note added: "Connectors and Test Points"
- moved on the sheet: J1, J2, J3

Commit message: stm32-test progress; added global symbol & footprint libraries
Parts:
- added SW1: TL3302AF180QJ, SW_TL3302AF180QJ_EWI, symbol fs_4_schematic_library:TL3302AF180QJ
- SW2: footprint Button_Switch_SMD:SW_SPST_PTS647_Sx50 -> Button_Switch_SMD:SW_SPST_PTS647_Sx38
Connections:
- net GND: now also SW1.1
- net NRST: now also SW1.2
- net UART_RX: now also U1.8 (PA3)
- net UART_TX: now also U1.7 (PA2)
- no-connect marks 10 -> 9
Other:
- moved on the sheet: SW2
Changed lines of the file:
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@@
 	(text "Decoupling capacitors pairs need to be\nplaced as close to respective Vdd/Vss as\npossible (pins 16&17, 1&32, 14&15). Note\nthat VSS contains all VSS mcu pins for\neach VDD/VSS pair."
 		(exclude_from_sim no)
-		(at 83.82 35.56 0)
+		(at 83.82 29.21 0)
 		(effects
 			(font
@@
 	)
 	(junction
+		(at 106.68 50.8)
+		(diameter 0)
+		(color 0 0 0 0)
+	)
+	(junction
 		(at 118.11 55.88)
 		(diameter 0)
@@
 	)
 	(junction
+		(at 118.11 50.8)
+		(diameter 0)
+		(color 0 0 0 0)
+	)
+	(junction
 		(at 210.82 35.56)
 		(diameter 0)
@@
 	)
 	(no_connect
-		(at 156.21 69.85)
-	)
-	(no_connect
 		(at 130.81 87.63)
 	)
@@
 	)
 	(no_connect
-		(at 156.21 72.39)
+		(at 156.21 102.87)
 	)
 	(no_connect
@@
 	(wire
 		(pts
-			(xy 156.21 82.55) (xy 167.64 82.55)
+			(xy 118.11 45.72) (xy 118.11 50.8)
 		)
 		(stroke
@@
 	(wire
 		(pts
-			(xy 106.68 55.88) (xy 106.68 52.07)
+			(xy 156.21 82.55) (xy 167.64 82.55)
 		)
 		(stroke
@@
 	(wire
 		(pts
+			(xy 106.68 50.8) (xy 106.68 55.88)
+		)
+		(stroke
+			(width 0)
+			(type default)
+		)
+	)
+	(wire
+		(pts
 			(xy 156.21 95.25) (xy 173.99 95.25)
 		)
@@
 	(wire
 		(pts
-			(xy 148.59 36.83) (xy 154.94 36.83)
+			(xy 106.68 45.72) (xy 106.68 50.8)
 		)
 		(stroke
@@
 	(wire
 		(pts
-			(xy 106.68 55.88) (xy 109.22 55.88)
+			(xy 148.59 36.83) (xy 154.94 36.83)
 		)
 		(stroke
@@
 	(wire
 		(pts
-			(xy 156.21 80.01) (xy 167.64 80.01)
+			(xy 106.68 55.88) (xy 109.22 55.88)
 		)
 		(stroke
@@
 	(wire
 		(pts
-			(xy 140.97 25.4) (xy 140.97 29.21)
+			(xy 156.21 80.01) (xy 167.64 80.01)
 		)
 		(stroke
@@
 	(wire
 		(pts
-			(xy 24.13 39.37) (xy 38.1 39.37)
+			(xy 140.97 25.4) (xy 140.97 29.21)
 		)
 		(stroke
@@
 	(wire
 		(pts
-			(xy 118.11 68.58) (xy 118.11 69.85)
+			(xy 24.13 39.37) (xy 38.1 39.37)
 		)
 		(stroke
@@
 	(wire
 		(pts
-			(xy 156.21 87.63) (xy 180.34 87.63)
+			(xy 118.11 68.58) (xy 118.11 69.85)
 		)
 		(stroke
@@
 	(wire
 		(pts
-			(xy 118.11 55.88) (xy 118.11 52.07)
+			(xy 156.21 87.63) (xy 180.34 87.63)
 		)
 		(stroke
@@
 	(wire
 		(pts
-			(xy 106.68 52.07) (xy 107.95 52.07)
+			(xy 106.68 50.8) (xy 107.95 50.8)
 		)
 		(stroke
@@
 	(wire
 		(pts
+			(xy 156.21 69.85) (xy 167.64 69.85)
+		)
+		(stroke
+			(width 0)
+			(type default)
+		)
+	)
+	(wire
+		(pts
 			(xy 54.61 107.95) (xy 66.04 107.95)
 		)
@@
 	(wire
 		(pts
+			(xy 118.11 50.8) (xy 118.11 55.88)
+		)
+		(stroke
+			(width 0)
+			(type default)
+		)
+	)
+	(wire
+		(pts
 			(xy 203.2 35.56) (xy 203.2 36.83)
 		)
@@
 	(wire
 		(pts
+			(xy 156.21 72.39) (xy 167.64 72.39)
+		)
+		(stroke
+			(width 0)
+			(type default)
+		)
+	)
+	(wire
+		(pts
 			(xy 123.19 55.88) (xy 118.11 55.88)
 		)
@@
 	(wire
 		(pts
+			(xy 107.95 45.72) (xy 106.68 45.72)
+		)
+		(stroke
+			(width 0)
+			(type default)
+		)
+	)
+	(wire
+		(pts
 			(xy 140.97 25.4) (xy 143.51 25.4)
 		)
@@
 		)
 	)
+	(label "UART_RX"
+		(at 167.64 72.39 180)
+		(effects
+			(font
+				(size 1.27 1.27)
+			)
+			(justify right bottom)
+		)
+	)
 	(label "SPI_MISO"
 		(at 66.04 82.55 180)
@@
 		)
 	)
+	(label "UART_TX"
+		(at 167.64 69.85 180)
+		(effects
+			(font
+				(size 1.27 1.27)
+			)
+			(justify right bottom)
+		)
+	)
 	(label "STLINK_SWO"
 		(at 110.49 80.01 0)
@@
 	)
 	(symbol
+		(lib_id "fs_4_schematic_library:TL3302AF180QJ")
+		(at 105.41 44.45 0)
+		(unit 1)
+		(exclude_from_sim no)
+		(in_bom yes)
+		(on_board yes)
+		(dnp no)
+		(property "Reference" "SW1"
+			(at 101.6 40.64 0)
+			(effects
+				(font
+					(size 1.524 1.524)
+				)
+			)
+		)
+		(property "Value" "TL3302AF180QJ"
+			(at 101.6 43.18 0)
+			(effects
+				(font
+					(size 1.524 1.524)
+				)
+			)
+		)
+		(property "Footprint" "SW_TL3302AF180QJ_EWI"
+			(at 109.22 33.782 0)
+			(effects
+				(font
+					(size 1.27 1.27)
+					(italic yes)
+				)
+				(hide yes)
+			)
+		)
+		(property "Datasheet" "https://configured-product-images.s3.amazonaws.com/Datasheets/TL3302.pdf"
+			(at 112.776 30.734 0)
+			(effects
+				(font
+					(size 1.27 1.27)
+					(italic yes)
+				)
+				(hide yes)
+			)
+		)
+		(property "Description" ""
+			(at 105.41 44.45 0)
+			(effects
+				(font
+					(size 1.27 1.27)
+				)
+				(hide yes)
+			)
+		)
+		(pin "1"
+		)
+		(pin "2"
+		)
+		(instances
+			(project ""
+				(path "/f1fb9b18-14c7-4eb6-8c96-349425b1ffb6"
+					(reference "SW1")
+					(unit 1)
+				)
+			)
+		)
+	)
+	(symbol
 		(lib_id "Device:C")
 		(at 154.94 33.02 0)
@@
 	(symbol
 		(lib_id "Switch:SW_Push")
-		(at 113.03 52.07 0)
+		(at 113.03 50.8 0)
 		(unit 1)
 		(exclude_from_sim no)
@@
 		(on_board yes)
 		(dnp no)
-		(fields_autoplaced yes)
 		(property "Reference" "SW2"
-			(at 113.03 44.45 0)
+			(at 101.6 49.53 0)
 			(effects
 				(font
@@
 		)
 		(property "Value" "SW_Push"
-			(at 113.03 46.99 0)
+			(at 101.6 52.07 0)
 			(effects
 				(font
@@
 			)
 		)
-		(property "Footprint" "Button_Switch_SMD:SW_SPST_PTS647_Sx50"
-			(at 113.03 46.99 0)
+		(property "Footprint" "Button_Switch_SMD:SW_SPST_PTS647_Sx38"
+			(at 113.03 45.72 0)
 			(effects
 				(font
@@
 		)
 		(property "Datasheet" "https://www.ckswitches.com/media/2567/pts647.pdf"
-			(at 113.03 46.99 0)
+			(at 113.03 45.72 0)
 			(effects
 				(font
@@
 		)
 		(property "Description" "Push button switch, generic, two pins"
-			(at 113.03 52.07 0)
+			(at 113.03 50.8 0)
 			(effects
 				(font

Commit message: save (not quite sure what the diff is?); update stm32 project version; add gerbers
Parts:
- removed J1: Conn_01x04, Connector_Molex:Molex_Nano-Fit_105309-xx04_1x04_P2.50mm_Vertical, symbol Connector_Generic:Conn_01x04
- removed J3: Conn_02x04_Top_Bottom, Connector_Molex:Molex_Nano-Fit_105310-xx08_2x04_P2.50mm_Vertical, symbol Connector_Generic:Conn_02x04_Top_Bottom
- removed U4: ISO1050DUB, Package_SO:SOP-8_6.62x9.15mm_P2.54mm, symbol Interface_CAN_LIN:ISO1050DUB
- added J1: Conn_01x04_Pin, Connector_PinHeader_2.54mm:PinHeader_1x04_P2.54mm_Vertical, symbol Connector:Conn_01x04_Pin
- added J7: Conn_02x07_Odd_Even, Connector_PinHeader_1.27mm:PinHeader_2x07_P1.27mm_Vertical_SMD, symbol Connector_Generic:Conn_02x07_Odd_Even
- added U5: ISO1044BD, Package_SO:SOIC-8_3.9x4.9mm_P1.27mm, symbol Interface_CAN_LIN:ISO1044BD
- C1, C3: Digi PN (none) -> 1276-6455-1-ND; MFG (none) -> Samsung Electro-Mechanics; MFG PN (none) -> CL21A106KOQNNNG
- C10: Digi PN (none) -> 1276-6455-1-ND; MFG (none) -> Samsung Electro-Mechanics; MFG PN (none) -> CL21A106KOQNNNG; Manufacturer Samsung Electro-Mechanics -> (none); PN CL21A106KOQNNNG -> (none)
- C11: Digi PN (none) -> 311-1140-1-ND; MFG (none) -> Yageo; MFG PN (none) -> CC0805KRX7R9BB104; Manufacturer Yageo -> (none); PN CC0805KRX7R9BB104 -> (none)
- C12: Digi PN (none) -> 1276-1852-1-ND; MFG (none) -> Samsung Electro-Mechanics; MFG PN (none) -> CL21A476MQYNNNE; Manufacturer Samsung Electro-Mechanics -> (none); PN CL21A476MQYNNNE -> (none)
- C13, C14: Digi PN (none) -> 1276-1029-1-ND; MFG (none) -> Samsung Electro-Mechanics; MFG PN (none) -> CL21B105KBFNNNE; Manufacturer Samsung Electro-Mechanics -> (none); PN CL21B105KBFNNNE -> (none)
- C15, C16, C2, C4, C5, C7: Digi PN (none) -> 311-1140-1-ND; MFG (none) -> Yageo; MFG PN (none) -> CC0805KRX7R9BB104
- C6: Digi PN (none) -> 1276-1029-1-ND; MFG (none) -> Samsung Electro-Mechanics; MFG PN (none) -> CL21B105KBFNNNE
- C8, C9: Digi PN (none) -> 311-4155-1-ND; MFG (none) -> Yageo; MFG PN (none) -> CC0805DRNPO9BN6R8
- L1: Digi PN (none) -> SRP5030TA-4R7MCT-ND; MFG (none) -> Bourns; MFG PN (none) -> SRP5030TA-4R7M; Manufacturer Bourns -> (none); PN SRP5030TA-4R7M -> (none)
- R1: Digi PN (none) -> 311-10KLGCT-ND; MFG (none) -> Yageo; MFG PN (none) -> AC0805FR-0710KL
- R2, R3: Digi PN (none) -> YAG3738CT-ND; MFG (none) -> Yageo; MFG PN (none) -> AC0805FR-074K7L
- SW1: footprint SW_TL3302AF180QJ_EWI -> FS_4_FOOTPRINTS_LIBRARY:SW_TL3302AF180QJ_EWI-L; Digi PN (none) -> EG4576CT-ND; MFG (none) -> E-Switch; MFG PN (none) -> TL3302AF180QJ
- SW2: Digi PN (none) -> PTS647SK38SMTR2LFSCT-ND; MFG (none) -> C&K; MFG PN (none) -> PTS647SK38SMTR2 LFS
- U1: Digi PN (none) -> 497-STM32G441KBT6-ND; MFG (none) -> STM; MFG PN (none) -> STM32G441KBT6
- U2: Digi PN (none) -> AP63205WU-7DICT-ND; MFG (none) -> Diodes Inc; MFG PN (none) -> AP63205WU-7
- U3: Digi PN (none) -> 576-4764-1-ND; MFG (none) -> Microchip Technology; MFG PN (none) -> MIC5504-3.3YM5-TR
- Y2: Digi PN (none) -> XC3063CT-ND; MFG (none) -> ECS; MFG PN (none) -> ECS-240-8-37B-CKY-TR
Connections:
- net +12V: now also J1.1 (Pin_1)
- net +3V3: now also C15.1, J7.3 (Pin_3), U5.1 (VCC1)
- net +5V: now also C16.1, U5.8 (VCC2)
- net CANH: now also J1.2 (Pin_2), U5.6 (CANH)
- net CANL: now also J1.3 (Pin_3), U5.5 (CANL)
- net CAN_RX: now also U5.3 (RXD)
- net CAN_TX: now also U5.2 (TXD)
- net GND: now also C15.2, C16.2, J1.4 (Pin_4), J7.5 (Pin_5), J7.7 (Pin_7), U5.4 (GND1), U5.7 (GND2)
- net I2C_SCL: now also J5.2 (Pin_2)
- net I2C_SDA: no longer J5.2 (Pin_2)
- net NRST: now also J7.12 (Pin_12)
- net STLINK_SWCLK: now also J7.6 (Pin_6)
- net STLINK_SWDIO: now also J7.4 (Pin_4)
- net STLINK_SWO: now also J7.8 (Pin_8)
- net UART_RX: now also J7.13 (Pin_13)
- net UART_TX: now also J7.14 (Pin_14)
- new net GNDDETECT: J7.11 (Pin_11)
- no-connect marks 9 -> 13
