File: mcu-designblocks/tractive-battery-mcu/tractive-battery-mcu.kicad_sch (KiCad schematic)
At the start: 28 parts, among them J1 Conn_01x04_Pin, J4 Conn_01x02_Pin, J6 Conn_01x02_Pin, J7 Conn_02x07_Odd_Even, SW2 SW_Push, U1 STM32G441KBTx, U2 AP63205WU, U3 MIC5504-3.3YM5, U5 ISO1044BD, Y2 24MHz

Commit message: remove connectors
Parts:
- removed C10: 10uF, Capacitor_SMD:C_0805_2012Metric_Pad1.18x1.45mm_HandSolder, symbol Device:C
- removed C11: 100nF, Capacitor_SMD:C_0805_2012Metric_Pad1.18x1.45mm_HandSolder, symbol Device:C
- removed C12: 47uF, Capacitor_SMD:C_0805_2012Metric_Pad1.18x1.45mm_HandSolder, symbol Device:C
- removed C13, C14: 1uF, Capacitor_SMD:C_0805_2012Metric_Pad1.18x1.45mm_HandSolder, symbol Device:C
- removed J4, J6: Conn_01x02_Pin, Connector_PinSocket_2.54mm:PinSocket_1x02_P2.54mm_Vertical, symbol Connector:Conn_01x02_Pin
- removed L1: 4.7uF, Inductor_SMD:L_Bourns_SRP5030T, symbol Device:L
- removed U2: AP63205WU, Package_TO_SOT_SMD:TSOT-23-6, symbol Regulator_Switching:AP63205WU
- removed U3: MIC5504-3.3YM5, Package_TO_SOT_SMD:SOT-23-5, symbol Regulator_Linear:MIC5504-3.3YM5
Connections:
- net +3V3: now also C5.2, C6.2
- net GND: no longer C5.2, C6.2
Other:
- note removed: "Power Circuitry"
- moved on the sheet: C15, C16, U5
