File: Telemetry-Logging-Board/audio.kicad_sch (KiCad schematic)
At the start: 1 part, among them J8 AudioJack4

Commit message: CAN: wire MCP2518FD↔ISO1044, add power blocks on CAN sheet + audio touch-ups
Parts:
- added U11: TLV320AIC23BPW, Package_SO:TSSOP-28_4.4x9.7mm_P0.65mm, symbol Audio:TLV320AIC23BPW
Changed lines of the file:
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@@
+		)
+	)
+	(symbol
+		(lib_id "Audio:TLV320AIC23BPW")
+		(at 142.24 100.33 0)
+		(unit 1)
+		(exclude_from_sim no)
+		(in_bom yes)
+		(on_board yes)
+		(dnp no)
+		(fields_autoplaced yes)
+		(property "Reference" "U11"
+			(at 152.0033 125.73 0)
+			(effects
+				(font
+					(size 1.27 1.27)
+				)
+				(justify left)
+			)
+		)
+		(property "Value" "TLV320AIC23BPW"
+			(at 152.0033 128.27 0)
+			(effects
+				(font
+					(size 1.27 1.27)
+				)
+				(justify left)
+			)
+		)
+		(property "Footprint" "Package_SO:TSSOP-28_4.4x9.7mm_P0.65mm"
+			(at 142.24 100.33 0)
+			(effects
+				(font
+					(size 1.27 1.27)
+					(italic yes)
+				)
+				(hide yes)
+			)
+		)
+		(property "Datasheet" "http://www.ti.com/lit/ds/symlink/tlv320aic23b.pdf"
+			(at 142.24 100.33 0)
+			(effects
+				(font
+					(size 1.27 1.27)
+				)
+				(hide yes)
+			)
+		)
+		(property "Description" "Stero Audio CODEC, 8- to 96-kHz, With Integrated Headphone Amplifier, TSSOP-28"
+			(at 142.24 100.33 0)
+			(effects
+				(font
+					(size 1.27 1.27)
+				)
+				(hide yes)
+			)
+		)
+		(pin "4"
+		)
+		(pin "1"
+		)
+		(pin "7"
+		)
+		(pin "19"
+		)
+		(pin "18"
+		)
+		(pin "8"
+		)
+		(pin "21"
+		)
+		(pin "11"
+		)
+		(pin "23"
+		)
+		(pin "26"
+		)
+		(pin "12"
+		)
+		(pin "5"
+		)
+		(pin "6"
+		)
+		(pin "24"
+		)
+		(pin "25"
+		)
+		(pin "28"
+		)
+		(pin "3"
+		)
+		(pin "27"
+		)
+		(pin "14"
+		)
+		(pin "2"
+		)
+		(pin "15"
+		)
+		(pin "13"
+		)
+		(pin "22"
+		)
+		(pin "10"
+		)
+		(pin "20"
+		)
+		(pin "9"
+		)
+		(pin "17"
+		)
+		(pin "16"
+		)
+		(instances
+			(project ""
+				(path "/5c64cdbc-39cd-49c8-9a12-12e4867a5d0b/0d9b0337-e460-4e79-9ba1-c2085a495d38"
+					(reference "U11")
+					(unit 1)
+				)
+			)
 		)
 	)
