File: Telemetry-Logging-Board/ftdi.kicad_sch (KiCad schematic)
At the start: 2 parts, among them P1 USB_C_Plug_USB2.0, U8 FT230XQ

Commit message: FTDI
Parts:
- added C10: 4.7uF, symbol Device:C
- added C11, C12, C13: 100nF, symbol Device:C_Small
- added C6: 10nF, symbol Device:C
- added C7, C8: 47pF, symbol Device:C
- added C9: 100nF, symbol Device:C
- added FB1: FerriteBead, symbol Device:FerriteBead
- added R1, R2: 27Ω, symbol Device:R
Connections:
- net FTDI_RX: now also U8.2 (RXD)
- net FTDI_TX: now also U8.15 (TXD)
- net GND: now also C10.1, C11.2, C12.2, C13.2, C6.1, C7.2, C8.2, C9.1
- net +3V3: now reaches U8.1 (VCCIO)
- net +3V3: now also U8.8 (3V3OUT), U8.9 (~{RESET}), C11.1, C12.1, C13.1
- net at U8.10 (VCC): now also C10.2, C9.2, FB1.2
- net at U8.6 (USBDP): now also R2.2
- net at U8.7 (USBDM): now also R1.2
- net at P1.A4 (VBUS), P1.A9 (VBUS), P1.B4 (VBUS)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: now also C6.2, FB1.1
- net at P1.A6 (D+): now also C7.1, R2.1
- net at P1.A7 (D-): now also C8.1, R1.1
Other:
- moved on the sheet: U8

Commit message: FTDI's usb CC pin
Parts:
- added R4: 5.1kΩ, symbol Device:R
Connections:
- net GND: now also R4.2
- net at P1.A5 (CC): now also R4.1
Changed lines of the file:
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@@
+	(wire
+		(pts
+			(xy 106.68 76.2) (xy 102.87 76.2)
+		)
+		(stroke
+			(width 0)
+			(type default)
+		)
+	)
 	(wire
 		(pts
@@
 		(pts
 			(xy 143.51 58.42) (xy 146.05 58.42)
+		)
+		(stroke
+			(width 0)
+			(type default)
+		)
+	)
+	(wire
+		(pts
+			(xy 116.84 76.2) (xy 114.3 76.2)
 		)
 		(stroke
@@
 	)
 	(symbol
+		(lib_id "Device:R")
+		(at 110.49 76.2 90)
+		(unit 1)
+		(exclude_from_sim no)
+		(in_bom yes)
+		(on_board yes)
+		(dnp no)
+		(property "Reference" "R4"
+			(at 110.998 78.74 90)
+			(effects
+				(font
+					(size 1.27 1.27)
+				)
+			)
+		)
+		(property "Value" "5.1kΩ"
+			(at 110.998 81.28 90)
+			(effects
+				(font
+					(size 1.27 1.27)
+				)
+			)
+		)
+		(property "Footprint" ""
+			(at 110.49 77.978 90)
+			(effects
+				(font
+					(size 1.27 1.27)
+				)
+				(hide yes)
+			)
+		)
+		(property "Datasheet" "~"
+			(at 110.49 76.2 0)
+			(effects
+				(font
+					(size 1.27 1.27)
+				)
+				(hide yes)
+			)
+		)
+		(property "Description" "Resistor"
+			(at 110.49 76.2 0)
+			(effects
+				(font
+					(size 1.27 1.27)
+				)
+				(hide yes)
+			)
+		)
+		(pin "1"
+		)
+		(pin "2"
+		)
+		(instances
+			(project "Telemetry-Logging-Board"
+				(path "/5c64cdbc-39cd-49c8-9a12-12e4867a5d0b/09aa2675-e127-459f-bbca-5f705be2e41d"
+					(reference "R4")
+					(unit 1)
+				)
+			)
+		)
+	)
+	(symbol
 		(lib_id "Device:FerriteBead")
 		(at 127 71.12 90)
@@
 					(unit 1)
 				)
+			)
+		)
+	)
+	(symbol
+		(lib_id "power:GND")
+		(at 116.84 76.2 0)
+		(unit 1)
+		(exclude_from_sim no)
+		(in_bom yes)
+		(on_board yes)
+		(dnp no)
+		(fields_autoplaced yes)
+		(property "Reference" "#PWR033"
+			(at 116.84 82.55 0)
+			(effects
+				(font
+					(size 1.27 1.27)
+				)
+				(hide yes)
+			)
+		)
+		(property "Value" "GND"
+			(at 116.84 81.28 0)
+			(effects
+				(font
+					(size 1.27 1.27)
+				)
+			)
+		)
+		(property "Footprint" ""
+			(at 116.84 76.2 0)
+			(effects
+				(font
+					(size 1.27 1.27)
+				)
+				(hide yes)
+			)
+		)
+		(property "Datasheet" ""
+			(at 116.84 76.2 0)
+			(effects
+				(font
+					(size 1.27 1.27)
+				)
+				(hide yes)
+			)
+		)
+		(property "Description" "Power symbol creates a global label with name \"GND\" , ground"
+			(at 116.84 76.2 0)
+			(effects
+				(font
+					(size 1.27 1.27)
+				)
+				(hide yes)
+			)
+		)
+		(pin "1"
+		)
+		(instances
+			(project ""
+				(path "/5c64cdbc-39cd-49c8-9a12-12e4867a5d0b/09aa2675-e127-459f-bbca-5f705be2e41d"
+					(reference "#PWR033")
+					(unit 1)
+				)

Commit message: varius cleanup, despec audio
Parts:
- removed FB1: FerriteBead, symbol Device:FerriteBead
Connections:
- net at C6.2, P1.A4 (VBUS), P1.A9 (VBUS)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: now also C10.2, C9.2, U8.10 (VCC)
Changed lines of the file:
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@@
 	(wire
 		(pts
-			(xy 107.95 71.12) (xy 123.19 71.12)
+			(xy 107.95 71.12) (xy 143.51 71.12)
 		)
 		(stroke
@@
 		(pts
 			(xy 166.37 106.68) (xy 168.91 106.68)
-		)
-		(stroke
-			(width 0)
-			(type default)
-		)
-	)
-	(wire
-		(pts
-			(xy 130.81 71.12) (xy 143.51 71.12)
 		)
 		(stroke
@@
 					(unit 1)
 				)
-			)
-		)
-	)
-	(symbol
-		(lib_id "Device:FerriteBead")
-		(at 127 71.12 90)
-		(unit 1)
-		(exclude_from_sim no)
-		(in_bom yes)
-		(on_board yes)
-		(dnp no)
-		(fields_autoplaced yes)
-		(property "Reference" "FB1"
-			(at 126.9492 63.5 90)
-			(effects
-				(font
-					(size 1.27 1.27)
-				)
-			)
-		)
-		(property "Value" "FerriteBead"
-			(at 126.9492 66.04 90)
-			(effects
-				(font
-					(size 1.27 1.27)
-				)
-			)
-		)
-		(property "Footprint" ""
-			(at 127 72.898 90)
-			(effects
-				(font
-					(size 1.27 1.27)
-				)
-				(hide yes)
-			)
-		)
-		(property "Datasheet" "~"
-			(at 127 71.12 0)
-			(effects
-				(font
-					(size 1.27 1.27)
-				)
-				(hide yes)
-			)
-		)
-		(property "Description" "Ferrite bead"
-			(at 127 71.12 0)
-			(effects
-				(font
-					(size 1.27 1.27)
-				)
-				(hide yes)
-			)
-		)
-		(pin "2"
-		)
-		(pin "1"
-		)
-		(instances
-			(project ""
-				(path "/5c64cdbc-39cd-49c8-9a12-12e4867a5d0b/09aa2675-e127-459f-bbca-5f705be2e41d"
-					(reference "FB1")
-					(unit 1)
-				)

Commit message: chose footprints
Parts:
- removed P1: USB_C_Plug_USB2.0, symbol Connector:USB_C_Plug_USB2.0
- added J8: USB_C_Receptacle_USB2.0_16P, Connector_USB:USB_C_Receptacle_GCT_USB4105-xx-A_16P_TopMnt_Horizontal, symbol Connector:USB_C_Receptacle_USB2.0_16P
- added R10: 5.1kΩ, Resistor_SMD:R_0805_2012Metric, symbol Device:R
- C16: renamed from C6; footprint (none) -> Capacitor_SMD:C_0805_2012Metric_Pad1.18x1.45mm_HandSolder
- C17: renamed from C7; footprint (none) -> Capacitor_SMD:C_0805_2012Metric_Pad1.18x1.45mm_HandSolder
- C18: renamed from C8; footprint (none) -> Capacitor_SMD:C_0805_2012Metric_Pad1.18x1.45mm_HandSolder
- C19: renamed from C9; footprint (none) -> Capacitor_SMD:C_0805_2012Metric_Pad1.18x1.45mm_HandSolder
- C20: renamed from C11; footprint (none) -> Capacitor_SMD:C_0805_2012Metric_Pad1.18x1.45mm_HandSolder
- C21: renamed from C12; footprint (none) -> Capacitor_SMD:C_0805_2012Metric_Pad1.18x1.45mm_HandSolder
- C22: renamed from C10; footprint (none) -> Capacitor_SMD:C_0805_2012Metric_Pad1.18x1.45mm_HandSolder
- C23: renamed from C13; footprint (none) -> Capacitor_SMD:C_0805_2012Metric_Pad1.18x1.45mm_HandSolder
- R7: renamed from R4; footprint (none) -> Resistor_SMD:R_0805_2012Metric
- R8: renamed from R1; footprint (none) -> Resistor_SMD:R_0805_2012Metric
- R9: renamed from R2; footprint (none) -> Resistor_SMD:R_0805_2012Metric
- renumbered U8 to U10
Connections:
- net GND: now also J8.A1 (GND), J8.A12 (GND), J8.B1 (GND), J8.B12 (GND), R10.2
- net at C17.1, R9.1: now also J8.A6 (D+), J8.B6 (D+)
- net at R7.1: now also J8.A5 (CC1)
- net at C16.2, C19.2, C22.2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: now also J8.A4 (VBUS), J8.A9 (VBUS), J8.B4 (VBUS), J8.B9 (VBUS)
- net at C18.1, R8.1: now also J8.A7 (D-), J8.B7 (D-)
- new net: J8.B5 (CC2), R10.1
Other:
- moved on the sheet: R7

Commit message: Change to same m.2 footprint as teledatics, fix some crystals, mess with layout
Parts:
- removed C20: 100nF, Capacitor_SMD:C_0805_2012Metric_Pad1.18x1.45mm_HandSolder, symbol Device:C_Small
- removed U10: FT230XQ, Package_DFN_QFN:QFN-16-1EP_4x4mm_P0.65mm_EP2.1x2.1mm, symbol Interface_USB:FT230XQ
- added U10: FT234XD, Package_DFN_QFN:WDFN-12-1EP_3x3mm_P0.45mm_EP1.7x2.5mm, symbol Interface_USB:FT234XD
Connections:
- net +3V3: now also U10.2 (~{RESET}), U10.9 (VCCIO)
- net FTDI_RX: now also U10.10 (RXD/D1)
- net FTDI_TX: now also U10.7 (TXD/D0)
- net GND: now also U10.13 (GND), U10.5 (GND)
- net at R9.2: now also U10.12 (USBDP)
- net at C16.2, C19.2, C22.2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: now also U10.4 (VCC)
- net at R8.2: now also U10.1 (USBDM)
- no-connect marks 0 -> 1
Other:
- moved on the sheet: C21, C23

Commit message: route, no drc
Connections:
- net +3V3 renamed VCCIO
Changed lines of the file:
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@@
-	)
-	(junction
-		(at 172.72 58.42)
-		(diameter 0)
-		(color 0 0 0 0)
 	)
 	(junction
@@
 		(color 0 0 0 0)
 	)
-	(junction
-		(at 147.32 96.52)
-		(diameter 0)
-		(color 0 0 0 0)
-	)
 	(no_connect
 		(at 153.67 83.82)
@@
 			(width 0)
 			(type default)
+		)
+	)
+	(hierarchical_label "VCCIO"
+		(shape input)
+		(at 147.32 96.52 90)
+		(effects
+			(font
+				(size 1.27 1.27)
+			)
+			(justify left)
+		)
+	)
+	(hierarchical_label "VCCIO"
+		(shape input)
+		(at 172.72 58.42 90)
+		(effects
+			(font
+				(size 1.27 1.27)
+			)
+			(justify left)
 		)
 	)
@@
 	)
 	(symbol
-		(lib_id "power:+3V3")
-		(at 147.32 96.52 0)
-		(unit 1)
-		(exclude_from_sim no)
-		(in_bom yes)
-		(on_board yes)
-		(dnp no)
-		(property "Reference" "#PWR047"
-			(at 147.32 100.33 0)
-			(effects
-				(font
-					(size 1.27 1.27)
-				)
-				(hide yes)
-			)
-		)
-		(property "Value" "+3V3"
-			(at 143.51 94.742 0)
-			(effects
-				(font
-					(size 1.27 1.27)
-				)
-			)
-		)
-		(property "Footprint" ""
-			(at 147.32 96.52 0)
-			(effects
-				(font
-					(size 1.27 1.27)
-				)
-				(hide yes)
-			)
-		)
-		(property "Datasheet" ""
-			(at 147.32 96.52 0)
-			(effects
-				(font
-					(size 1.27 1.27)
-				)
-				(hide yes)
-			)
-		)
-		(property "Description" "Power symbol creates a global label with name \"+3V3\""
-			(at 147.32 96.52 0)
-			(effects
-				(font
-					(size 1.27 1.27)
-				)
-				(hide yes)
-			)
-		)
-		(pin "1"
-		)
-		(instances
-			(project "Telemetry-Logging-Board"
-				(path "/5c64cdbc-39cd-49c8-9a12-12e4867a5d0b/09aa2675-e127-459f-bbca-5f705be2e41d"
-					(reference "#PWR047")
-					(unit 1)
-				)
-			)
-		)
-	)
-	(symbol
 		(lib_id "Device:R")
 		(at 114.3 72.39 90)
@@
 					(unit 1)
 				)
-			)
-		)
-	)
-	(symbol
-		(lib_id "power:+3V3")
-		(at 172.72 58.42 0)
-		(unit 1)
-		(exclude_from_sim no)
-		(in_bom yes)
-		(on_board yes)
-		(dnp no)
-		(property "Reference" "#PWR050"
-			(at 172.72 62.23 0)
-			(effects
-				(font
-					(size 1.27 1.27)
-				)
-				(hide yes)
-			)
-		)
-		(property "Value" "+3V3"
-			(at 176.53 56.896 0)
-			(effects
-				(font
-					(size 1.27 1.27)
-				)
-			)
-		)
-		(property "Footprint" ""
-			(at 172.72 58.42 0)
-			(effects
-				(font
-					(size 1.27 1.27)
-				)
-				(hide yes)
-			)
-		)
-		(property "Datasheet" ""
-			(at 172.72 58.42 0)
-			(effects
-				(font
-					(size 1.27 1.27)
-				)
-				(hide yes)
-			)
-		)
-		(property "Description" "Power symbol creates a global label with name \"+3V3\""
-			(at 172.72 58.42 0)
-			(effects
-				(font
-					(size 1.27 1.27)
-				)
-				(hide yes)
-			)
-		)
-		(pin "1"
-		)
-		(instances
-			(project "Telemetry-Logging-Board"
-				(path "/5c64cdbc-39cd-49c8-9a12-12e4867a5d0b/09aa2675-e127-459f-bbca-5f705be2e41d"
-					(reference "#PWR050")
-					(unit 1)
-				)
