File: Telemetry-Logging-Board/Telemetry-Logging-Board.kicad_pcb (KiCad board)
At the start: 4 copper layers, 43.8 x 66.3 mm, 57 parts, among them J1 Raspberry_Pi_4, J2 Heltec Thingimagiger, J3 Main, J4 BATT_CO, J6 AUX_CAN, U1 PCF8523T, U10 BQ25172DSGR, U2 AP63205WU, U3 MIC5504-3.3YM5, U4 MCP2518FD-xQBB, U5 ISO1044BD, U6 MCP2518FD-xQBB, U7 ISO1044BD, U8 MCP2518FD-xQBB, U9 ISO1044BD, Y1 32.768 kHz Quartz Crystal, Y2 ECS-200-12-33Q-JES-TR, Y3 ECS-200-12-33Q-JES-TR, Y4 ECS-200-12-33Q-JES-TR

Commit message: cleanup silkscreen
Parts:
- added G***: , formula_slug_footprint_library:FORMULA SLUG TITLE, F.Cu at (160.1, 91.2)
Changed lines of the file:
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@@
 		(embedded_fonts no)
 	)
+	(footprint "formula_slug_footprint_library:FORMULA SLUG TITLE"
+		(layer "F.Cu")
+		(at 160.05742 91.191457 180)
+		(descr "Cosmetic Logo With Title Text")
+		(tags "logo, title")
+		(property "Reference" "G***"
+			(at 0 0 0)
+			(layer "F.SilkS")
+			(hide yes)
+			(effects
+				(font
+					(size 1.5 1.5)
+					(thickness 0.3)
+				)
+			)
+		)
+		(property "Value" ""
+			(at 0.75 0 0)
+			(layer "F.SilkS")
+			(hide yes)
+			(effects
+				(font
+					(size 1.5 1.5)
+					(thickness 0.3)
+				)
+			)
+		)
+		(property "Datasheet" ""
+			(at 0 0 180)
+			(unlocked yes)
+			(layer "F.Fab")
+			(hide yes)
+			(effects
+				(font
+					(size 1.27 1.27)
+					(thickness 0.15)
+				)
+			)
+		)
+		(property "Description" ""
+			(at 0 0 180)
+			(unlocked yes)
+			(layer "F.Fab")
+			(hide yes)
+			(effects
+				(font
+					(size 1.27 1.27)
+					(thickness 0.15)
+				)
+			)
+		)
+		(attr board_only exclude_from_pos_files exclude_from_bom)
+		(fp_poly
+			(pts
+				(xy -2.978538 -1.18802) (xy -2.983976 -1.1638) (xy -2.997969 -1.146607) (xy -3.029051 -1.135011)
+				(xy -3.085756 -1.12758) (xy -3.176619 -1.122883) (xy -3.310176 -1.119489) (xy -3.39732 -1.117802)
+				(xy -3.564909 -1.1128) (xy -3.692359 -1.105064) (xy -3.774696 -1.095029) (xy -3.806943 -1.083133)
+				(xy -3.807221 -1.081855) (xy -3.794554 -1.047871) (xy -3.759992 -0.975661) (xy -3.708692 -0.87555)
+				(xy -3.645813 -0.757863) (xy -3.640482 -0.74808) (xy -3.559231 -0.597402) (xy -3.505712 -0.488519)
+				(xy -3.480657 -0.414643) (xy -3.484796 -0.368987) (xy -3.518859 -0.344766) (xy -3.583579 -0.335193)
+				(xy -3.679686 -0.33348) (xy -3.68514 -0.333479) (xy -3.792282 -0.332066) (xy -3.853894 -0.326265)
+				(xy -3.879986 -0.313737) (xy -3.880569 -0.292141) (xy -3.879137 -0.288135) (xy -3.859129 -0.254652)
+				(xy -3.810992 -0.181981) (xy -3.738892 -0.076171) (xy -3.64699 0.056732) (xy -3.539453 0.210679)
+				(xy -3.420443 0.379621) (xy -3.382892 0.432652) (xy -2.904048 1.108095) (xy -2.896242 0.792952)
+				(xy -2.889488 0.633907) (xy -2.876955 0.524137) (xy -2.856434 0.45745) (xy -2.825717 0.427656) (xy -2.782596 0.428564)
+				(xy -2.768006 0.433473) (xy -2.751673 0.445088) (xy -2.739984 0.470553) (xy -2.732378 0.517495)
+				(xy -2.728298 0.59354) (xy -2.727182 0.706311) (xy -2.728471 0.863435) (xy -2.729747 0.954656) (xy -2.733 1.135545)
+				(xy -2.737037 1.268249) (xy -2.74262 1.360161) (xy -2.75051 1.418676) (xy -2.761469 1.451189) (xy -2.776258 1.465093)
+				(xy -2.782515 1.466939) (xy -2.826862 1.451253) (xy -2.88518 1.399229) (xy -2.909682 1.370032) (xy -2.987567 1.267154)
+				(xy -3.083166 1.13683) (xy -3.192391 0.985003) (xy -3.311155 0.817616) (xy -3.435368 0.640612) (xy -3.560942 0.459936)
+				(xy -3.683791 0.28153) (xy -3.799825 0.111337) (xy -3.904957 -0.044698) (xy -3.995098 -0.180633)
+				(xy -4.066161 -0.290525) (xy -4.114057 -0.368429) (xy -4.134698 -0.408403) (xy -4.13516 -0.411609)
+				(xy -4.12066 -0.436378) (xy -4.081382 -0.452174) (xy -4.006396 -0.461682) (xy -3.911132 -0.466651)
+				(xy -3.809759 -0.472504) (xy -3.734104 -0.480736) (xy -3.697537 -0.48978) (xy -3.696061 -0.491833)
+				(xy -3.70842 -0.521472) (xy -3.742186 -0.590206) (xy -3.792395 -0.688202) (xy -3.854083 -0.80563)
+				(xy -3.862801 -0.822025) (xy -3.926298 -0.94564) (xy -3.978662 -1.055906) (xy -4.014757 -1.1414)
+				(xy -4.029444 -1.190697) (xy -4.029541 -1.192849) (xy -4.027655 -1.212848) (xy -4.017105 -1.227595)
+				(xy -3.990548 -1.237889) (xy -3.940641 -1.24453) (xy -3.860043 -1.248318) (xy -3.741411 -1.250051)
+				(xy -3.577404 -1.250528) (xy -3.499599 -1.250547) (xy -2.969657 -1.250547)
+			)
+			(stroke
+				(width 0)
+				(type solid)
+			)
+			(fill yes)
+			(layer "F.SilkS")
+		)
+		(fp_poly
+			(pts
+				(xy -2.788263 -1.56467) (xy -2.778994 -1.529389) (xy -2.766898 -1.463828) (xy -2.737018 -1.388231)
+				(xy -2.698962 -1.321398) (xy -2.662339 -1.282125) (xy -2.650665 -1.278337) (xy -2.61524 -1.301406)
+				(xy -2.598411 -1.333753) (xy -2.560999 -1.408084) (xy -2.512444 -1.449615) (xy -2.46491 -1.448785)
+				(xy -2.458117 -1.444004) (xy -2.434541 -1.398362) (xy -2.448633 -1.353116) (xy -2.490172 -1.333917)
+				(xy -2.524233 -1.317017) (xy -2.524036 -1.280438) (xy -2.493003 -1.245357) (xy -2.474525 -1.23704)
+				(xy -2.411633 -1.198295) (xy -2.347304 -1.131401) (xy -2.297658 -1.056289) (xy -2.278775 -0.995027)
+				(xy -2.296398 -0.940177) (xy -2.340673 -0.869722) (xy -2.362145 -0.843347) (xy -2.412674 -0.778381)
+				(xy -2.442288 -0.725963) (xy -2.445514 -0.712386) (xy -2.43322 -0.66912) (xy -2.40161 -0.596283)
+				(xy -2.373203 -0.539666) (xy -2.300939 -0.401477) (xy -2.251324 -0.300887) (xy -2.220165 -0.226828)
+				(xy -2.203269 -0.16823) (xy -2.196441 -0.114026) (xy -2.195405 -0.070409) (xy -2.203501 0.021962)
+				(xy -2.235816 0.092973) (xy -2.285722 0.152829) (xy -2.392706 0.232287) (xy -2.539714 0.291482)
+				(xy -2.713537 0.326128) (xy -2.842345 0.333479) (xy -2.922925 0.331154) (xy -2.961255 0.319792)
+				(xy -2.970612 0.292813) (xy -2.968508 0.270952) (xy -2.958854 0.238553) (xy -2.933158 0.217909)
+				(xy -2.87939 0.204636) (xy -2.785518 0.194346) (xy -2.750238 0.191389) (xy -2.568212 0.164483) (xy -2.436787 0.117181)
+				(xy -2.354635 0.048897) (xy -2.33162 0.006701) (xy -2.315465 -0.066428) (xy -2.325412 -0.145948)
+				(xy -2.364791 -0.243749) (xy -2.436932 -0.371722) (xy -2.438171 -0.373754) (xy -2.521938 -0.542703)
+				(xy -2.555677 -0.692421) (xy -2.539253 -0.821431) (xy -2.487231 -0.911962) (xy -2.44141 -0.972466)
+				(xy -2.430368 -1.011524) (xy -2.449222 -1.046623) (xy -2.449522 -1.046985) (xy -2.500892 -1.088963)
+				(xy -2.573915 -1.128633) (xy -2.578151 -1.130435) (xy -2.670371 -1.151155) (xy -2.740898 -1.126072)
+				(xy -2.790345 -1.053828) (xy -2.819324 -0.933065) (xy -2.828448 -0.762423) (xy -2.821911 -0.58979)
+				(xy -2.814805 -0.418247) (xy -2.821674 -0.285793) (xy -2.845746 -0.176984) (xy -2.89025 -0.076379)
+				(xy -2.948893 0.017655) (xy -3.016632 0.097772) (xy -3.105241 0.177523) (xy -3.199866 0.245958)
+				(xy -3.285654 0.292126) (xy -3.339557 0.305689) (xy -3.384583 0.291405) (xy -3.387109 0.253564)
+				(xy -3.35072 0.199683) (xy -3.278997 0.137278) (xy -3.249635 0.117041) (xy -3.150799 0.037865) (xy -3.060628 -0.058414)
+				(xy -3.027744 -0.103884) (xy -2.995354 -0.156452) (xy -2.973012 -0.202032) (xy -2.959073 -0.252029)
+				(xy -2.951886 -0.317844) (xy -2.949806 -0.410882) (xy -2.951184 -0.542547) (xy -2.95261 -0.623879)
+				(xy -2.953548 -0.807423) (xy -2.947433 -0.945212) (xy -2.932173 -1.046848) (xy -2.905678 -1.121934)
+				(xy -2.865854 -1.180073) (xy -2.822511 -1.221237) (xy -2.785256 -1.269093) (xy -2.789732 -1.324585)
+				(xy -2.837599 -1.398923) (xy -2.851284 -1.415565) (xy -2.898631 -1.491215) (xy -2.903143 -1.548819)
+				(xy -2.865568 -1.580415) (xy -2.835446 -1.584026)
+			)
+			(stroke
+				(width 0)
+				(type solid)
+			)
+			(fill yes)
+			(layer "F.SilkS")
+		)
+		(fp_text user "Architect: ${COMMENT4}"
+			(at -2.032 1.524 180)
+			(unlocked yes)
+			(layer "F.SilkS")
+			(effects
+				(font
+					(size 0.9906 0.9906)
+					(thickness 0.1524)
+					(bold yes)
+				)
+				(justify left)
+			)
+		)
+		(fp_text user "${COMPANY}"
+			(at -2.032 -1.524 180)
+			(unlocked yes)
+			(layer "F.SilkS")
+			(effects
+				(font
+					(size 0.9906 0.9906)
+					(thickness 0.1524)
+					(bold yes)
+				)
+				(justify left)
+			)
+		)
+		(fp_text user "FS-4 ${TITLE} V3.0"
+			(at -2.032 0 180)
+			(unlocked yes)
+			(layer "F.SilkS")
+			(effects
+				(font
+					(size 0.9906 0.9906)
+					(thickness 0.1524)
+					(bold yes)
+				)
+				(justify left)
+			)
+		)
+		(embedded_fonts no)
+	)
 	(footprint "Battery:BatteryHolder_Keystone_2998_1x6.8mm"
 		(layer "F.Cu")
@@
 		(tags "capacitor handsolder")
 		(property "Reference" "C9"
-			(at -2.5 0 0)
+			(at 1.25 1.75 0)
 			(layer "B.SilkS")
 			(effects
@@
 		(tags "SOT TO_SOT_SMD")
 		(property "Reference" "U3"
-			(at -1.75 -2 0)
+			(at 2.5 0 0)
 			(layer "B.SilkS")
 			(effects
@@
 		(tags "solder jumper open")
 		(property "Reference" "JP1"
-			(at 1.5 2 0)
+			(at 2.75 0 0)
 			(layer "B.SilkS")
 			(effects
@@
 	)
 	(via
-		(at 149.5 90.15)
+		(at 149.5 90.75)
 		(size 0.6)
 		(drill 0.3)
@@
 	)
 	(segment
-		(start 152.05 90.15)
-		(end 152.2 90.3)
-		(width 0.5)
-		(layer "B.Cu")
-		(net 2)
-	)
-	(segment
 		(start 139 83.4)
 		(end 139 84.8)
@@
 	)
 	(segment
-		(start 146.65 90.15)
-		(end 149.5 90.15)
+		(start 152.2 90.3)
+		(end 152.05 90.15)
 		(width 0.5)
 		(layer "B.Cu")
@@
 	)
 	(segment
+		(start 150.1 90.15)
+		(end 149.5 90.75)
+		(width 0.5)
+		(layer "B.Cu")
+		(net 2)
+	)
+	(segment
 		(start 144.15 85.25)
 		(end 144.6 84.8)
@@
 	)
 	(segment
-		(start 152.2 90.3)
-		(end 152.2 91.6)
+		(start 146.6 90.2)
+		(end 146.65 90.15)
 		(width 0.5)
 		(layer "B.Cu")
@@
 	)
 	(segment
-		(start 160.6375 64.395072)
-		(end 160.500001 64.257573)
+		(start 152.2 90.3)
+		(end 152.2 91.6)
 		(width 0.5)
 		(layer "B.Cu")
@@
 	)
 	(segment
-		(start 149.5 90.15)
-		(end 152.05 90.15)
+		(start 160.6375 64.395072)
+		(end 160.500001 64.257573)
 		(width 0.5)
 		(layer "B.Cu")
@@
 	)
 	(segment
+		(start 148.9 90.15)
+		(end 149.5 90.75)
+		(width 0.5)
+		(layer "B.Cu")
+		(net 2)
+	)
+	(segment
 		(start 140.595 54.405)
 		(end 139.75 55.25)
@@
 	)
 	(segment
+		(start 152.05 90.15)
+		(end 150.1 90.15)
+		(width 0.5)
+		(layer "B.Cu")
+		(net 2)
+	)
+	(segment
 		(start 133.094311 54.724311)
 		(end 133.094311 55.25)
@@
 	)
 	(segment
+		(start 146.65 90.15)
+		(end 148.9 90.15)
+		(width 0.5)
+		(layer "B.Cu")
+		(net 2)
+	)
+	(segment
 		(start 139.25 65.7875)
 		(end 140.25 64.7875)
@@
 		(layer "B.Cu")
 		(net 2)
-	)
-	(segment
-		(start 146.6 90.2)
-		(end 146.65 90.15)
-		(width 0.5)
-		(layer "B.Cu")
-		(net 2)
