File: mcu-designblocks/STM32F446RETx/STM32F446RETx.kicad_sch (KiCad schematic)
At the start: 18 parts

Commit message: fix footprint for ferrite bead
Parts:
- FB?: footprint Inductor_SMD:L_0201_0603Metric_Pad0.64x0.40mm_HandSolder -> Inductor_SMD:L_0603_1608Metric_Pad1.05x0.95mm_HandSolder
Changed lines of the file:
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@@
 			)
 		)
-		(property "Footprint" "Inductor_SMD:L_0201_0603Metric_Pad0.64x0.40mm_HandSolder"
+		(property "Footprint" "Inductor_SMD:L_0603_1608Metric_Pad1.05x0.95mm_HandSolder"
 			(at 173.99 30.988 90)
 			(effects
