File: mcu-designblocks/STM32G441KBTx/STM32G441KBTx.kicad_sch (KiCad schematic)
At the start: 14 parts

Commit message: ground GNDDETECT
Connections:
- net GNDDETECT is gone; now on net GND: J?.11 (Pin_11)
Changed lines of the file:
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@@
+	(wire
+		(pts
+			(xy 92.71 113.03) (xy 109.22 113.03)
+		)
+		(stroke
+			(width 0)
+			(type default)
+		)
+	)
 	(wire
 		(pts
@@
 		(pts
 			(xy 161.29 48.26) (xy 161.29 53.34)
-		)
-		(stroke
-			(width 0)
-			(type default)
-		)
-	)
-	(wire
-		(pts
-			(xy 95.25 113.03) (xy 109.22 113.03)
 		)
 		(stroke
@@
 					(unit 1)
 				)
+			)
+		)
+	)
+	(symbol
+		(lib_id "power:GND")
+		(at 92.71 113.03 0)
+		(unit 1)
+		(exclude_from_sim no)
+		(in_bom yes)
+		(on_board yes)
+		(dnp no)
+		(property "Reference" "#PWR01"
+			(at 92.71 119.38 0)
+			(effects
+				(font
+					(size 1.27 1.27)
+				)
+				(hide yes)
+			)
+		)
+		(property "Value" "GND"
+			(at 90.17 113.03 0)
+			(effects
+				(font
+					(size 1.27 1.27)
+				)
+			)
+		)
+		(property "Footprint" ""
+			(at 92.71 113.03 0)
+			(effects
+				(font
+					(size 1.27 1.27)
+				)
+				(hide yes)
+			)
+		)
+		(property "Datasheet" ""
+			(at 92.71 113.03 0)
+			(effects
+				(font
+					(size 1.27 1.27)
+				)
+				(hide yes)
+			)
+		)
+		(property "Description" "Power symbol creates a global label with name \"GND\" , ground"
+			(at 92.71 113.03 0)
+			(effects
+				(font
+					(size 1.27 1.27)
+				)
+				(hide yes)
+			)
+		)
+		(pin "1"
+		)
+		(instances
+			(project "STM32G441KBTx"
+				(path "/c6f349be-f072-4c68-bea9-9d1d80db7efc"
+					(reference "#PWR01")
+					(unit 1)
+				)

Commit message: redo G441KB with VDDA net + create F4
Other:
- note added: "ST-Link Programming/Debugging Connector"
- note removed: "Connectors and Test Points"
Changed lines of the file:
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@@
 		)
 	)
-	(text "Connectors and Test Points\n"
+	(text "ST-Link Programming/Debugging Connector"
 		(exclude_from_sim no)
 		(at 90.17 88.9 0)

Commit message: fix G441KB caps
Parts:
- removed C?: 10uF, Capacitor_SMD:C_0805_2012Metric_Pad1.18x1.45mm_HandSolder, symbol Device:C
- removed C? (x2): 100nF, Capacitor_SMD:C_0805_2012Metric_Pad1.18x1.45mm_HandSolder, symbol Device:C
- removed FB?: FerriteBead_Small, Inductor_SMD:L_0805_2012Metric_Pad1.05x1.20mm_HandSolder, symbol Device:FerriteBead_Small
- added C? (x2): 100nF, Capacitor_SMD:C_0805_2012Metric_Pad1.18x1.45mm_HandSolder, symbol Device:C
- added C?: 10uF, Capacitor_SMD:C_0805_2012Metric_Pad1.18x1.45mm_HandSolder, symbol Device:C
- added FB?: FerriteBead, Inductor_SMD:L_0805_2012Metric_Pad1.05x1.20mm_HandSolder, symbol Device:FerriteBead
Connections:
- net +3V3: now also C?.2, C?.2, C?.2, FB?.1; no longer C?.2, C?.2, U?.15 (VDDA)
- net GND: now also C?.2, C?.2, C?.1, C?.1, C?.1; no longer C?.1, C?.1
- new net VDDA: C?.1, C?.1, FB?.2, U?.15 (VDDA)
- no-connect marks 21 -> 4
Other:
- moved on the sheet: C?

Commit message: change ferrite bead and update design blocks
Parts:
- FB?: footprint Inductor_SMD:L_0805_2012Metric_Pad1.05x1.20mm_HandSolder -> Inductor_SMD:L_0201_0603Metric_Pad0.64x0.40mm_HandSolder; Digi PN 240-2393-1-ND -> 4816-FCM1608KF-601T03CT-ND; MFG Laird-Signal Integrity Products -> TAI-TECH Advanced Electronics Co., Ltd.; MFG PN HI0805O121R-10 -> FCM 1608KF-601T03
Changed lines of the file:
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@@
 			)
 		)
-		(property "Footprint" "Inductor_SMD:L_0805_2012Metric_Pad1.05x1.20mm_HandSolder"
+		(property "Footprint" "Inductor_SMD:L_0201_0603Metric_Pad0.64x0.40mm_HandSolder"
 			(at 178.562 50.8 90)
 			(effects
@@
 			)
 		)
-		(property "Datasheet" "https://www.laird.com/sites/default/files/hi0805o121r-10-datasheet.pdf"
+		(property "Datasheet" "https://mm.digikey.com/Volume0/opasdata/d220001/medias/docus/6383/FCM%20Series.pdf"
 			(at 180.34 50.8 0)
 			(effects
@@
 			)
 		)
-		(property "Digi PN" "240-2393-1-ND"
+		(property "Digi PN" "4816-FCM1608KF-601T03CT-ND"
 			(at 180.34 50.8 0)
 			(effects
@@
 			)
 		)
-		(property "MFG" "Laird-Signal Integrity Products"
+		(property "MFG" "TAI-TECH Advanced Electronics Co., Ltd."
 			(at 180.34 50.8 0)
 			(effects
@@
 			)
 		)
-		(property "MFG PN" "HI0805O121R-10"
+		(property "MFG PN" "FCM 1608KF-601T03"
 			(at 180.34 50.8 0)
 			(effects

Commit message: make ferrite bead cleaner
Connections:
- net VDDA renamed +3V3_A
Other:
- moved on the sheet: C?, FB?

Commit message: fix footprint for ferrite bead
Parts:
- FB?: footprint Inductor_SMD:L_0201_0603Metric_Pad0.64x0.40mm_HandSolder -> Inductor_SMD:L_0603_1608Metric_Pad1.05x0.95mm_HandSolder
Changed lines of the file:
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@@
 			)
 		)
-		(property "Footprint" "Inductor_SMD:L_0201_0603Metric_Pad0.64x0.40mm_HandSolder"
+		(property "Footprint" "Inductor_SMD:L_0603_1608Metric_Pad1.05x0.95mm_HandSolder"
 			(at 173.99 32.258 90)
 			(effects
