File: Libraries/formula_slug_design_blocks_library.kicad_blocks/STM32G473RCTx.kicad_block/STM32G473RCTx.kicad_sch (KiCad schematic)
At the start: 16 parts

Commit message: finish touches add as design blocks
Other:
- note removed: "STM32G473RCTx"
Changed lines of the file:
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@@
 		)
 	)
-	(text "STM32G473RCTx"
-		(exclude_from_sim no)
-		(at 144.272 17.526 0)
-		(effects
-			(font
-				(size 2.54 2.54)
-			)
-		)
-	)
 	(text "Decoupling capacitors pairs need to be\nplaced as close to respective Vdd/Vss as\npossible (pins 16&17, 1&32, 14&15). Note\nthat VSS contains all VSS mcu pins for\neach VDD/VSS pair."
 		(exclude_from_sim no)
@@
 		)
 	)
-	(sheet_instances
-		(path "/"
-			(page "1")
-		)
-	)
-	(embedded_fonts no)
 )

Commit message: add digi num
Parts:
- U?: Digi PN (none) -> 497-15376-ND; MFG (none) -> STMicroelectronics; MFG PN (none) -> STM32F446RET6
Changed lines of the file:
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@@
+			)
+		)
+		(property "Digi PN" "497-15376-ND"
+			(at 157.48 97.79 0)
+			(effects
+				(font
+					(size 1.27 1.27)
+				)
+				(hide yes)
+			)
+		)
+		(property "MFG" "STMicroelectronics"
+			(at 157.48 97.79 0)
+			(effects
+				(font
+					(size 1.27 1.27)
+				)
+				(hide yes)
+			)
+		)
+		(property "MFG PN" "STM32F446RET6"
+			(at 157.48 97.79 0)
+			(effects
+				(font
+					(size 1.27 1.27)
+				)
+				(hide yes)
 			)
 		)

Commit message: ground GNDDETECT
Connections:
- net GNDDETECT is gone; now on net GND: J?.11 (Pin_11)
Changed lines of the file:
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@@
+	(wire
+		(pts
+			(xy 96.52 151.13) (xy 113.03 151.13)
+		)
+		(stroke
+			(width 0)
+			(type default)
+		)
+	)
 	(wire
 		(pts
@@
 		(pts
 			(xy 127 69.85) (xy 139.7 69.85)
-		)
-		(stroke
-			(width 0)
-			(type default)
-		)
-	)
-	(wire
-		(pts
-			(xy 99.06 151.13) (xy 113.03 151.13)
 		)
 		(stroke
@@
 					(unit 1)
 				)
+			)
+		)
+	)
+	(symbol
+		(lib_id "power:GND")
+		(at 96.52 151.13 0)
+		(unit 1)
+		(exclude_from_sim no)
+		(in_bom yes)
+		(on_board yes)
+		(dnp no)
+		(property "Reference" "#PWR01"
+			(at 96.52 157.48 0)
+			(effects
+				(font
+					(size 1.27 1.27)
+				)
+				(hide yes)
+			)
+		)
+		(property "Value" "GND"
+			(at 93.98 151.13 0)
+			(effects
+				(font
+					(size 1.27 1.27)
+				)
+			)
+		)
+		(property "Footprint" ""
+			(at 96.52 151.13 0)
+			(effects
+				(font
+					(size 1.27 1.27)
+				)
+				(hide yes)
+			)
+		)
+		(property "Datasheet" ""
+			(at 96.52 151.13 0)
+			(effects
+				(font
+					(size 1.27 1.27)
+				)
+				(hide yes)
+			)
+		)
+		(property "Description" "Power symbol creates a global label with name \"GND\" , ground"
+			(at 96.52 151.13 0)
+			(effects
+				(font
+					(size 1.27 1.27)
+				)
+				(hide yes)
+			)
+		)
+		(pin "1"
+		)
+		(instances
+			(project "STM32G473RCTx"
+				(path "/be8abe95-fa0e-434f-bf97-73945cc728ef"
+					(reference "#PWR01")
+					(unit 1)
+				)

Commit message: change ferrite bead and update design blocks
Parts:
- removed C?: 1uF, Capacitor_SMD:C_0805_2012Metric_Pad1.18x1.45mm_HandSolder, symbol Device:C
- removed C? (x5): 100nF, Capacitor_SMD:C_0805_2012Metric_Pad1.18x1.45mm_HandSolder, symbol Device:C
- removed C?: 10uF, Capacitor_SMD:C_0805_2012Metric_Pad1.18x1.45mm_HandSolder, symbol Device:C
- removed FB?: FerriteBead_Small, Inductor_SMD:L_0805_2012Metric_Pad1.05x1.20mm_HandSolder, symbol Device:FerriteBead_Small
- added C?: 10uF, Capacitor_SMD:C_0805_2012Metric_Pad1.18x1.45mm_HandSolder, symbol Device:C
- added C? (x6): 100nF, Capacitor_SMD:C_0805_2012Metric_Pad1.18x1.45mm_HandSolder, symbol Device:C
- added C? (x2): 1uF, Capacitor_SMD:C_0805_2012Metric_Pad1.18x1.45mm_HandSolder, symbol Device:C
- added FB?: FerriteBead, Inductor_SMD:L_0201_0603Metric_Pad0.64x0.40mm_HandSolder, symbol Device:FerriteBead
Connections:
- net +3V3: now also C?.1, C?.1, C?.1, C?.1, C?.2, FB?.1; no longer U?.28 (VREF+), U?.29 (VDDA)
- net GND: now also C?.1, C?.2, C?.2, C?.2, C?.2, C?.2, C?.2, C?.2, C?.2
- new net VDDA: C?.1, C?.1, C?.1, C?.1, FB?.2, U?.28 (VREF+), U?.29 (VDDA)
- no-connect marks 47 -> 4
Other:
- note added: "Decoupling capacitors pairs need to be placed as close to respective Vdd/Vss as possible. Note that VSS contains all VSS mcu pins for each VDD/VSS pair."
- note added: "ST-Link Programming/Debugging Connector"
- note removed: "Connectors and Test Points"
- note removed: "Decoupling capacitors pairs need to be placed as close to respective Vdd/Vss as possible (pins 16&17, 1&32, 14&15). Note that VSS contains all VSS mcu pins for each VDD/VSS pair."

Commit message: make ferrite bead cleaner
Connections:
- net VDDA renamed +3V3_A
Other:
- moved on the sheet: C?, FB?

Commit message: fix footprint for ferrite bead
Parts:
- FB?: footprint Inductor_SMD:L_0201_0603Metric_Pad0.64x0.40mm_HandSolder -> Inductor_SMD:L_0603_1608Metric_Pad1.05x0.95mm_HandSolder
Changed lines of the file:
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@@
 			)
 		)
-		(property "Footprint" "Inductor_SMD:L_0201_0603Metric_Pad0.64x0.40mm_HandSolder"
+		(property "Footprint" "Inductor_SMD:L_0603_1608Metric_Pad1.05x0.95mm_HandSolder"
 			(at 181.61 30.988 90)
 			(effects

Commit message: Fix issues
Parts:
- removed C? (x2): 6.8pF, Capacitor_SMD:C_0805_2012Metric_Pad1.18x1.45mm_HandSolder, symbol Device:C
- removed C?: 100nF, Capacitor_SMD:C_0805_2012Metric_Pad1.18x1.45mm_HandSolder, symbol Device:C
- removed SW?: SW_Push, Button_Switch_SMD:SW_SPST_PTS647_Sx38, symbol Switch:SW_Push
- removed U?: STM32G473RCTx, Package_QFP:LQFP-64_10x10mm_P0.5mm, symbol MCU_ST_STM32G4:STM32G473RCTx
- removed Y?: 24MHz, Crystal:Crystal_SMD_2016-4Pin_2.0x1.6mm, symbol Device:Crystal_GND24
- added C? (x2): 6.8pF, Capacitor_SMD:C_0805_2012Metric_Pad1.18x1.45mm_HandSolder, symbol Device:C
- added C?: 100nF, Capacitor_SMD:C_0805_2012Metric_Pad1.18x1.45mm_HandSolder, symbol Device:C
- added SW?: Y97KT23B5NAFP, Button_Switch_SMD:SW_SPST_PTS647_Sx38, symbol Switch:SW_Push
- added U?: STM32G473RCTx, Package_QFP:LQFP-64_10x10mm_P0.5mm, symbol MCU_ST_STM32G4:STM32G473RCTx
- added Y?: ECS-240-8-37B-CKY-TR, Crystal:Crystal_SMD_2016-4Pin_2.0x1.6mm, symbol Device:Crystal_GND24
- C? (x3): Digi URL (none) -> https://www.digikey.com/en/products/detail/samsung-electro-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
- C? (x6): Digi URL (none) -> https://www.digikey.com/en/products/detail/yageo/CC0805KRX7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
- FB?: value FerriteBead -> FCM 1608KF-601T03; Digi URL (none) -> https://www.digikey.com/en/products/detail/tai-tech-advance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
- J?: value Conn_02x07_Odd_Even -> FTSH-107-01-F-DV-K-P-TR; Digi URL (none) -> https://www.digikey.com/en/products/detail/samtec-inc/FTSH-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; MFG (none) -> Samtec Inc.
- R?: Digi URL (none) -> https://www.digikey.com/en/products/detail/yageo/AC0805FR-0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
Connections:
- net +3V3: now also U?.1 (VBAT), U?.16 (VDD), U?.32 (VDD), U?.48 (VDD), U?.64 (VDD)
- net +3V3_A: now also U?.28 (VREF+), U?.29 (VDDA)
- net BOOT0: now also U?.61 (PB8)
- net GND: now also C?.1, C?.2, C?.2, SW?.1, U?.15 (VSS), U?.27 (VSSA), U?.31 (VSS), U?.47 (VSS), U?.63 (VSS), Y?.2, Y?.4
- net NRST: now also C?.2, SW?.2, U?.7 (PG10)
- net OSC_IN: now also C?.1, U?.5 (PF0), Y?.3
- net OSC_OUT: now also C?.1, U?.6 (PF1), Y?.1
- net STLINK_SWDIO: now also U?.49 (PA13)
- net STLINK_SWO: now also U?.56 (PB3)
- net UART_RX: now also U?.60 (PB7)
- net UART_TX: now also U?.59 (PB6)
- new net STLINK_SWCLOCK: U?.50 (PA14)
Other:
- note added: "Decoupling 100nF capacitors need to be placed as close to respective Vdd/Vss as possible. Note that VSS contains all VSS mcu pins for each VDD/VSS pair."
- note added: "STM32G473RCTx"
- note removed: "Decoupling capacitors pairs need to be placed as close to respective Vdd/Vss as possible. Note that VSS contains all VSS mcu pins for each VDD/VSS pair."
- moved on the sheet: FB?, J?, R?

Commit message: fixes
Parts:
- C?: footprint Capacitor_SMD:C_0805_2012Metric_Pad1.18x1.45mm_HandSolder -> Capacitor_SMD:C_0603_1608Metric_Pad1.08x0.95mm_HandSolder; Digi PN 1276-6455-1-ND -> 1276-CL10A106KO8NQNCCT-ND; Digi URL https://www.digikey.com/en/products/detail/samsung-electro-mechanics/CL21A106KOQNNNG/3894417 -> https://www.digikey.com/en/products/detail/samsung-electro-mechanics/CL10A106KO8NQNC/10479038; MFG PN CL21A106KOQNNNG -> CL10A106KO8NQNC
- C? (x7): footprint Capacitor_SMD:C_0805_2012Metric_Pad1.18x1.45mm_HandSolder -> Capacitor_SMD:C_0603_1608Metric_Pad1.08x0.95mm_HandSolder; Digi PN 311-1140-1-ND -> 311-1344-1-ND; Digi URL https://www.digikey.com/en/products/detail/yageo/CC0805KRX7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 -> https://www.digikey.com/en/products/detail/yageo/CC0603KRX7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; MFG PN CC0805KRX7R9BB104 -> CC0603KRX7R9BB104
- C? (x2): footprint Capacitor_SMD:C_0805_2012Metric_Pad1.18x1.45mm_HandSolder -> Capacitor_SMD:C_0603_1608Metric_Pad1.08x0.95mm_HandSolder; Digi PN 1276-1029-1-ND -> 1276-CL10B105KB9VPJCCT-ND; Digi URL https://www.digikey.com/en/products/detail/samsung-electro-mechanics/CL21B105KBFNNNE/3886687 -> https://www.digikey.com/en/products/detail/samsung-electro-mechanics/cl10b105kb9vpjc/20498526; MFG PN CL21B105KBFNNNE -> CL10B105KB9VPJC
- C? (x2): footprint Capacitor_SMD:C_0805_2012Metric_Pad1.18x1.45mm_HandSolder -> Capacitor_SMD:C_0603_1608Metric_Pad1.08x0.95mm_HandSolder; Digi PN 311-4155-1-ND -> 311-3874-1-ND; Digi URL https://www.digikey.com/en/products/detail/yageo/CC0805DRNP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 -> https://www.digikey.com/en/products/detail/yageo/CC0603DRNP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; MFG PN CC0805DRNPO9BN6R8 -> CC0603DRNPO9BN6R8
- R?: footprint Resistor_SMD:R_0805_2012Metric_Pad1.20x1.40mm_HandSolder -> Resistor_SMD:R_0603_1608Metric_Pad0.98x0.95mm_HandSolder; Digi PN 311-10KLGCT-ND -> 311-10KLDCT-ND; Digi URL https://www.digikey.com/en/products/detail/yageo/AC0805FR-0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 -> https://www.digikey.com/en/products/detail/yageo/AC0603FR-0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; MFG PN AC0805FR-0710KL -> AC0603FR-0710KL
Connections:
- net STLINK_SWCLOCK is gone; now on net STLINK_SWCLK: U?.50 (PA14)
- net UART_RX renamed VCP_UART_RX
- net UART_TX renamed VCP_UART_TX
Other:
- note added: "24MHz"
- note removed: "STM32G473RCTx"
- moved on the sheet: C?, FB?, R?, SW?
