File: Shutdown Circuitry/Shutdown Design.kicad_sch (KiCad schematic)
At the start: 60 parts, among them J1 J1772 Prox and Cntrl Pilot Co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, J2 CAN COTS Charger Connector, J3 Battery_HV_Conn Interlock, J4 Power Electronics HV Interlock, J5 Energy Meter Interlock, J6 MSD Interlock, J7 Power Electronics HV Interlock, K1 G6BK-1114P-US, K2 G6BK-1114P-US, K3 G6BK-1114P-US, K4 JQC-3FF-005-1H, K6 JQC-3FF-005-1H, K7 JQC-3FF-005-1H, Q1 NMOS, Q10 AO3400A, Q2 NMOS, Q3 NMOS, Q8 AO3400A, SW1 SW_Push, SW2 SW_Push_Open, SW3 SW_Push_Open, SW4 SW_Push_Open, SW7 SW_Push, SW8 SW_Push, U1 74HC14, U10 NUCLEO-L432KC, U2 MCP6004, U3 SN74HCS08DR, U7 LM7809_TO220, U8 SN74HCS08DR, U9 ISO1050DUB

Commit message: Updated Schematic
Parts:
- removed D1, D2, D5: 1N4148WT, Diode_SMD:D_SOD-523, symbol Diode:1N4148WT
- removed D3: 1N4148, Diode_THT:D_DO-35_SOD27_P7.62mm_Horizontal, symbol Diode:1N4148
- removed SW7: SW_Push, symbol Switch:SW_Push
- removed unit 1 of U8
- added C5: 1.0μF, Capacitor_SMD:C_0805_2012Metric_Pad1.18x1.45mm_HandSolder, symbol Device:C
- added D2: D, Diode_SMD:D_2010_5025Metric_Pad1.52x2.65mm_HandSolder, symbol Device:D
- added D3: 1N4148WT, Diode_SMD:D_SOD-523, symbol Diode:1N4148WT
- added Q4, Q5, Q6: Relay Driver, Package_TO_SOT_SMD:SOT-23-3, symbol Simulation_SPICE:NMOS
- added R21: 430k, Resistor_SMD:R_0805_2012Metric_Pad1.20x1.40mm_HandSolder, symbol Device:R
- added R25: 10k, Resistor_SMD:R_0805_2012Metric_Pad1.20x1.40mm_HandSolder, symbol Device:R
- added R26: 5.23k, Resistor_SMD:R_0805_2012Metric_Pad1.20x1.40mm_HandSolder, symbol Device:R
- added unit 7 of U1
- added unit 3 of U2
- added unit 4 of U3
- added U5: 74HC14, Package_SO:SOIC-14_3.9x8.7mm_P1.27mm, symbol 74xx:74HC14
- C1: value 1.0μF -> 1uF
- K2: footprint FS_3_Global_Footprint_Library:RELAY_G6BK-1114P-US_OMR -> FS_4_Global_Footprint_Library:RELAY_G6BK-1114P-US_OMR
- Q1, Q2, Q3: value NMOS -> Relay Driver; footprint (none) -> Package_TO_SOT_SMD:SOT-23-3
- R2: value 430k -> 422k
- U2: footprint (none) -> Package_SO:SOIC-14_3.9x8.7mm_P1.27mm
Connections:
- net nBSPD_Set is gone; now on net +12V: K2.6
- net +12V: now also K1.6, K3.6
- net +5V: now also R2.1, D3.1 (K), R25.2, U1.14 (VCC); no longer U1.14 (VCC)
- net GND: now also C5.2, Q4.3 (S), Q5.3 (S), Q6.3 (S), R26.1, U1.7 (GND), U2.9 (-); no longer K1.1, K1.2, K2.1, K2.2, K3.1, K3.2, Q1.1 (D), Q2.1 (D), Q3.1 (D), U1.7 (GND), U2.9 (-)
- net Vreg: now also U2.10 (+); no longer U2.10 (+)
- net nBMS_Fault: now also U1.9, U3.5, U3.11
- net nBMS_Nucleo_Fault_Pin: now also U3.12; no longer U3.12
- net nBSPD_FAULT: now also U5.2, U5.6; no longer Q1.2 (G), U2.7
- net nIMD_Fault: now also U1.6; no longer Q2.2 (G), U1.6
- net nIMD_Set: now also Q5.2 (G); no longer K3.6
- net at R3.1, R4.2: now also U2.13 (-); no longer U2.6 (-)
- net at R2.2: now also C1.1, U2.12 (+), D3.2 (A); no longer U1.4
- net IMD_Fault: now reaches U3.8
- net IMD_Fault: now also Q2.2 (G), U1.5; no longer U1.5
- removed net BSPD_Logic_Output: U1.3
- net BSPD_Shutdown_In renamed Inertia_Shutdown
- net nBMS_Set renamed BMS_Set
- net BMS_Set: now also Q4.2 (G); no longer K1.6
- new net: R25.1, R26.2, U2.6 (-)
- new net: K2.1, Q1.1 (D)
- new net: K2.2, Q6.1 (D)
- new net: K1.2, Q3.1 (D)
- new net: K1.1, Q4.1 (D)
- new net: C5.1, D2.2 (A), R21.1, U2.5 (+)
- new net: U1.8, U3.1
- new net: U2.14, U3.2
- new net: U2.8, U3.13
- new net: K3.1, Q5.1 (D)
- new net: K3.2, Q2.1 (D)
- new net BMS_Fault: Q3.2 (G), U3.3
- new net BSPD_FAULT: Q6.2 (G), U2.7, U5.5
- new net BSPD_Fault_Raw: D2.1 (K), R21.2
- new net BSPD_Set: Q1.2 (G), U5.3
- new net Set_Button_Neg: U5.1
Other:
- note added: ".473 Second Delay"
- note removed: "4.73 Second Delay"
- moved on the sheet: Q3, U1D, U2D, U3A

Commit message: Shutdown update design
Updated footprints on shutdown circuit
Parts:
- removed D7, D9: 1N4148WT, Diode_SMD:D_SOD-523, symbol Diode:1N4148WT
- removed Q10, Q8: AO3400A, Package_TO_SOT_SMD:SOT-23, symbol Transistor_FET:AO3400A
- added Q7, Q8: Relay Driver, Package_TO_SOT_SMD:SOT-23-3, symbol Simulation_SPICE:NMOS
Connections:
- net CAN signal: now also Q7.2 (G)
- net CAN_Signal: now also Q8.2 (G)
- net GND: now also Q7.3 (S), Q8.3 (S)
- net at K6.A2: now also Q8.1 (D)
- net at K4.A2: now also Q7.1 (D)
