File: VCU/Position_Pedals_Filt_Buff.kicad_sch (KiCad schematic)
At the start: 10 parts, among them U15 MCP6004

Commit message: VCU Schematic Update
Documented schematic in more detail. Added and removed certain components based on feedback.
Parts:
- removed C24, C25, C26: 40nF, Capacitor_SMD:C_0603_1608Metric_Pad1.08x0.95mm_HandSolder, symbol Device:C
- removed R93, R95, R97: 100k, Resistor_SMD:R_0603_1608Metric_Pad0.98x0.95mm_HandSolder, symbol Device:R
- removed R94, R96, R98: 200k, Resistor_SMD:R_0603_1608Metric_Pad0.98x0.95mm_HandSolder, symbol Device:R
- removed U15: MCP6004, Package_SO:SOIC-14_3.9x8.7mm_P1.27mm, symbol Amplifier_Operational:MCP6004
Other:
- note removed: "1.67 V"
- note removed: "3.33 V"
- note removed: "APPS + BPPS Buffer + Filter"
