File: VCU/TSSI.kicad_sch (KiCad schematic)
At the start: 40 parts, among them Q10 NMOS, Q11 NMOS, Q3 NMOS, Q4 NMOS, Q5 NMOS, Q6 NMOS, Q7 NMOS, Q8 NMOS, Q9 NMOS, U4 SN74HCS08DR, U8 74HC14, U9 LM555xM

Commit message: VCU Schematic Update
Documented schematic in more detail. Added and removed certain components based on feedback.
Parts:
- removed R45, R46, R52, R53: 330, Resistor_SMD:R_0603_1608Metric_Pad0.98x0.95mm_HandSolder, symbol Device:R
- added C32, C41: 1uF, Capacitor_SMD:C_0603_1608Metric_Pad1.08x0.95mm_HandSolder, symbol Device:C
- added unit 5 of U4
- added unit 7 of U8
- C6, C7: Digi PN (none) -> 311-3874-1-ND; Digi URL (none) -> https://www.digikey.com/en/products/detail/yageo/CC0603DRNP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; MFG (none) -> Yageo; MFG PN (none) -> CC0603DRNPO9BN6R8
- R29, R30, R31, R32, R33, R34, R37, R38, R41, R42, R43, R44, R48, R49, R50, R51: Digi PN (none) -> 311-10KLDCT-ND; Digi URL (none) -> https://www.digikey.com/en/products/detail/yageo/AC0603FR-0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; MFG (none) -> Yageo; MFG PN (none) -> AC0603FR-0710KL
- R35, R36, R39, R40: value 330 -> 200; Digi PN (none) -> 311-10KLDCT-ND; Digi URL (none) -> https://www.digikey.com/en/products/detail/yageo/AC0603FR-0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; MFG (none) -> Yageo; MFG PN (none) -> AC0603FR-0710KL
- R45: renamed from R47; Digi PN (none) -> 311-10KLDCT-ND; Digi URL (none) -> https://www.digikey.com/en/products/detail/yageo/AC0603FR-0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; MFG (none) -> Yageo; MFG PN (none) -> AC0603FR-0710KL
Connections:
- net +5V: now also C32.2, C41.2, U4.14 (VCC), U8.14 (VCC)
- net GND: now also C32.1, C41.1, U4.7 (GND), U8.7 (GND)
Other:
- note added: "Power Supply"

Commit message: VCU Documentation Update
footprint, annotations, and more!
Parts:
- removed Q10, Q11, Q3, Q4, Q7, Q8, Q9: NMOS, Package_TO_SOT_SMD:SOT-23_Handsoldering, symbol Simulation_SPICE:NMOS
- added D14: 1092QC1-125VAC, symbol Device:LED
- added Q10, Q11, Q12, Q3, Q4, Q7, Q8: AO3400A, Package_TO_SOT_SMD:SOT-23, symbol Transistor_FET:AO3400A
- C32, C41: Digi PN 311-3874-1-ND -> 311-3484-1-ND; Digi URL https://www.digikey.com/en/products/detail/yageo/CC0603DRNP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 -> https://www.digikey.com/en/products/detail/yageo/CC0603JRX7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; MFG PN CC0603DRNPO9BN6R8 -> CC0603JRX7R6BB105
- C6: value 10µF -> 10uF; Digi PN 311-3874-1-ND -> 311-3484-1-ND
- C7: Digi PN 311-3874-1-ND -> 311-1778-1-ND; Digi URL https://www.digikey.com/en/products/detail/yageo/CC0603DRNP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 -> https://www.digikey.com/en/products/detail/yageo/CC0603JRX7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; MFG PN CC0603DRNPO9BN6R8 -> CC0603JRX7R9BB103
- R35, R36, R39, R40: value 200 -> 300
- R49: value 330 -> 300
Connections:
- net +5V: no longer R35.2, R36.2
- net BMS_LED_Cathode: now also Q7.3 (D)
- net BSPD_LED_Cathode: now also Q10.3 (D)
- net Brake_LED_Cathode: now also Q12.3 (D)
- net GND: now also Q10.2 (S), Q11.2 (S), Q12.2 (S), Q3.2 (S), Q4.2 (S), Q7.2 (S), Q8.2 (S)
- net IMD_LED_Cathode: now also Q8.3 (D)
- net LED_Strip_Cathode: now also Q4.3 (D)
- net RTD_Buzzer_Neg: now also Q3.3 (D)
- net RTD_LED: now also Q11.1 (G)
- net RTD_LED_Cathode: now also Q11.3 (D)
- net at R48.1: now also Q4.1 (G)
- net at R34.1: now also Q12.1 (G)
- net at R44.1: now also Q8.1 (G)
- net at R43.1: now also Q7.1 (G)
- net at R33.1: now also Q3.1 (G)
- net at R51.1: now also Q10.1 (G)
- new net +12V: R35.2, R36.2
Other:
- moved on the sheet: C32

Commit message: Documentation of VCu
Documentation of components
Parts:
- removed Q5, Q6: NMOS, Package_TO_SOT_SMD:SOT-23_Handsoldering, symbol Simulation_SPICE:NMOS
- added Q5, Q6: AO3400A, Package_TO_SOT_SMD:SOT-23, symbol Transistor_FET:AO3400A
- D7: value D -> ACGRAT105L-HF; Digi PN (none) -> 641-1631-1-ND; Digi URL (none) -> https://www.digikey.com/en/products/detail/comchip-technolo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; MFG PN (none) -> ACGRAT105L-HF
- Q10, Q11, Q12, Q3, Q4, Q7, Q8: Digi PN (none) -> 785-1000-1-ND; Digi URL (none) -> https://www.digikey.com/en/products/detail/alpha-omega-semi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; MFG (none) -> A&O; MFG PN (none) -> AO3400A
- R29, R30: Digi PN 311-10KLDCT-ND -> 13-AC0603FR-0718K7LCT-ND; Digi URL https://www.digikey.com/en/products/detail/yageo/AC0603FR-0710KL/2827814 -> https://www.digikey.com/en/products/detail/yageo/AC0603FR-0718K7L/5895835; MFG PN AC0603FR-0710KL -> AC0603FR-0718K7L
- R31, R32, R37, R38, R41, R42, R45, R50: Digi PN 311-10KLDCT-ND -> 13-AC0603FR-13100KLCT-ND; Digi URL https://www.digikey.com/en/products/detail/yageo/AC0603FR-0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 -> https://www.digikey.com/en/products/detail/yageo/AC0603FR-1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; MFG PN AC0603FR-0710KL -> AC0603FR-13100KL
- R33, R34, R43, R44, R48, R51: Digi PN 311-10KLDCT-ND -> 13-AC0603FR-1010KLCT-ND; Digi URL https://www.digikey.com/en/products/detail/yageo/AC0603FR-0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 -> https://www.digikey.com/en/products/detail/yageo/AC0603FR-1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; MFG PN AC0603FR-0710KL -> AC0603FR-1010KL
- R35, R36, R39, R40, R49: Digi PN 311-10KLDCT-ND -> YAG5330CT-ND; Digi URL https://www.digikey.com/en/products/detail/yageo/AC0603FR-0710KL/2827814 -> https://www.digikey.com/en/products/detail/yageo/AC0603FR-07300RL/5896018; MFG PN AC0603FR-0710KL -> AC0603FR-07300RL
- U4: Digi PN (none) -> 296-SN74HCS08DRCT-ND; Digi URL (none) -> https://www.digikey.com/en/products/detail/texas-instrument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; MFG (none) -> TI; MFG PN (none) -> SN74HCS08DR
- U8: Digi PN (none) -> 296-1194-1-ND; Digi URL (none) -> https://www.digikey.com/en/products/detail/texas-instrument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; MFG (none) -> TI; MFG PN (none) -> SN74HC14DR
- U9: value LM555xM -> LM555CMX; Digi PN (none) -> LM555CMX/NOPBCT-ND; Digi URL (none) -> https://www.digikey.com/en/products/detail/texas-instrument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; MFG (none) -> TI; MFG PN (none) -> LM555CMX/NOPB
Connections:
- net 5v_Oscillation: now also Q6.1 (G)
- net GND: now also Q5.2 (S), Q6.2 (S)
- net TSSI_Fault: now also Q5.1 (G)
- net TSSI_GREEN_Cathode: now also Q5.3 (D)
- net TSSI_RED_Cathode: now also Q6.3 (D)

Commit message: Pin Connections
Updated pin connections and pin headers
Parts:
- removed Q4: AO3400A, Package_TO_SOT_SMD:SOT-23, symbol Transistor_FET:AO3400A
- removed R45: 100k, Resistor_SMD:R_0603_1608Metric_Pad0.98x0.95mm_HandSolder, symbol Device:R
- removed R48: 10k, Resistor_SMD:R_0603_1608Metric_Pad0.98x0.95mm_HandSolder, symbol Device:R
- removed R49: 300, Resistor_SMD:R_0603_1608Metric_Pad0.98x0.95mm_HandSolder, symbol Device:R
Other:
- note removed: "LED Strip Driver"
- moved on the sheet: C32, U4E

Commit message: Documentation
Added test points to unconnected mcu pins, rtd button, and more documentation
Parts:
- removed R36: 300, Resistor_SMD:R_0603_1608Metric_Pad0.98x0.95mm_HandSolder, symbol Device:R
- added D15, D17: 1092QC1-125VAC, symbol Device:LED
- added D16: 1092QC5-125VAC, symbol Device:LED
- added R80, R81, R83: 10k, Resistor_SMD:R_0603_1608Metric_Pad0.98x0.95mm_HandSolder, symbol Device:R
- added R82: 100k, Resistor_SMD:R_0603_1608Metric_Pad0.98x0.95mm_HandSolder, symbol Device:R
Connections:
- net +12V: now also D14.2 (A), D15.2 (A), D16.2 (A), D17.2 (A)
- net 5v_Oscillation: now also R80.2; no longer Q6.1 (G)
- net BMS_LED_Cathode: now also D14.1 (K)
- net BSPD_LED_Cathode: now also D17.1 (K)
- net GND: now also R82.1
- net IMD_LED_Cathode: now also D15.1 (K)
- net RTD_LED: now also R82.2, R83.2; no longer Q11.1 (G)
- net RTD_LED_Cathode: now also D16.1 (K)
- net TSSI_Fault: now also R81.2; no longer Q5.1 (G)
- net BPPS_1_Buff_Filt renamed Brake_Light_Signal
- new net: Q5.1 (G), R81.1
- new net: Q11.1 (G), R83.1
- new net: Q6.1 (G), R80.1
Other:
- moved on the sheet: C41, D14, R31, R32, R37, R38, U8G

Commit message: Documentation
More documentatino of LEDS
Parts:
- removed R39, R40: 300, Resistor_SMD:R_0603_1608Metric_Pad0.98x0.95mm_HandSolder, symbol Device:R
- added C52: 0.1uF, Capacitor_SMD:C_0603_1608Metric_Pad1.08x0.95mm_HandSolder, symbol Device:C
- added D18: 1092QC1-125VAC, symbol Device:LED
- added D19: PCL2212V500B, symbol Device:LED
- added D20: PCL2212V100B, symbol Device:LED
- added LS1: CPT-1625-80-SMT-TR, CPT-1625-80-SMT-TR:XDCR_CPT-1625-80-SMT-TR, symbol RTD_Buzzer:CPT-1625-80-SMT-TR
Connections:
- net +12V: now also D18.2 (A), D19.2 (A), D20.2 (A); no longer R35.2
- net +5V: now also R35.2, C52.1
- net Brake_LED_Cathode: now also D18.1 (K)
- net GND: now also C52.2
- net RTD_Buzzer_Neg: now also LS1.N
- net RTD_Buzzer_Pos: now also LS1.P
- net TSSI_GREEN_Cathode: now also D19.1 (K)
- net TSSI_RED_Cathode: now also D20.1 (K)
- net TSSI_Active_Inverted renamed TSSI_Red_Logic
- net TSSI_Fault renamed TSSI_Status
Other:
- moved on the sheet: C32, C6, C7, D7, Q12, Q3, Q5, Q6, R29, R30, R31, R32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

Commit message: Documentation
Parts:
- removed R83: 10k, Resistor_SMD:R_0603_1608Metric_Pad0.98x0.95mm_HandSolder, symbol Device:R
Connections:
- net RTD_LED: now also Q11.1 (G)
Other:
- note added: "Resistor on MCU page"
Changed lines of the file:
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@@
 		)
 	)
+	(text "Resistor on MCU page\n"
+		(exclude_from_sim no)
+		(at 334.518 68.072 0)
+		(effects
+			(font
+				(size 1.27 1.27)
+			)
+		)
+	)
 	(junction
 		(at 157.48 55.88)
@@
 	(wire
 		(pts
-			(xy 332.74 72.39) (xy 335.28 72.39)
+			(xy 332.74 72.39) (xy 342.9 72.39)
 		)
 		(stroke
@@
 					(unit 1)
 				)
-			)
-		)
-	)
-	(symbol
-		(lib_id "Device:R")
-		(at 339.09 72.39 270)
-		(unit 1)
-		(exclude_from_sim no)
-		(in_bom yes)
-		(on_board yes)
-		(dnp no)
-		(fields_autoplaced yes)
-		(property "Reference" "R83"
-			(at 339.09 66.04 90)
-			(effects
-				(font
-					(size 1.27 1.27)
-				)
-			)
-		)
-		(property "Value" "10k"
-			(at 339.09 68.58 90)
-			(effects
-				(font
-					(size 1.27 1.27)
-				)
-			)
-		)
-		(property "Footprint" "Resistor_SMD:R_0603_1608Metric_Pad0.98x0.95mm_HandSolder"
-			(at 339.09 70.612 90)
-			(effects
-				(font
-					(size 1.27 1.27)
-				)
-				(hide yes)
-			)
-		)
-		(property "Datasheet" "https://www.yageogroup.com/content/datasheet/asset/file/PYU-AC_51_ROHS_L"
-			(at 339.09 72.39 0)
-			(effects
-				(font
-					(size 1.27 1.27)
-				)
-				(hide yes)
-			)
-		)
-		(property "Description" "Resistor"
-			(at 339.09 72.39 0)
-			(effects
-				(font
-					(size 1.27 1.27)
-				)
-				(hide yes)
-			)
-		)
-		(property "Digi PN" "13-AC0603FR-1010KLCT-ND"
-			(at 339.09 72.39 90)
-			(effects
-				(font
-					(size 1.27 1.27)
-				)
-				(hide yes)
-			)
-		)
-		(property "Digi URL" "https://www.digikey.com/en/products/detail/yageo/AC0603FR-1010KL/13694182"
-			(at 339.09 72.39 90)
-			(effects
-				(font
-					(size 1.27 1.27)
-				)
-				(hide yes)
-			)
-		)
-		(property "MFG" "Yageo"
-			(at 339.09 72.39 90)
-			(effects
-				(font
-					(size 1.27 1.27)
-				)
-				(hide yes)
-			)
-		)
-		(property "MFG PN" "AC0603FR-1010KL"
-			(at 339.09 72.39 90)
-			(effects
-				(font
-					(size 1.27 1.27)
-				)
-				(hide yes)
-			)
-		)
-		(property "MANUFACTURER" ""
-			(at 339.09 72.39 90)
-			(effects
-				(font
-					(size 1.27 1.27)
-				)
-				(hide yes)
-			)
-		)
-		(pin "1"
-		)
-		(pin "2"
-		)
-		(instances
-			(project "VCU"
-				(path "/d46cfebc-cd32-4ec9-981b-3f67fe44510e/c0e3a50f-b7e7-4c20-a214-f82a0e3821e9"
-					(reference "R83")
-					(unit 1)
-				)
