File: VCU/VCU_Enclosure_LED.kicad_sch (KiCad schematic)
At the start: 18 parts, among them Q12 NMOS, U10 74HC14

Commit message: VCU Schematic Update
Documented schematic in more detail. Added and removed certain components based on feedback.
Parts:
- added C43: 1uF, Capacitor_SMD:C_0603_1608Metric_Pad1.08x0.95mm_HandSolder, symbol Device:C
- added D10, D11, D12, D13, D8, D9: LTST-S270KRKT, LED_SMD:LED_0603_1608Metric_Pad1.05x0.95mm_HandSolder, symbol Device:LED
- added unit 7 of U10
- R54, R55, R56, R57, R61, R62, R63, R64, R65, R66: Digi PN (none) -> 311-10KLDCT-ND; Digi URL (none) -> https://www.digikey.com/en/products/detail/yageo/AC0603FR-0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; MFG (none) -> Yageo; MFG PN (none) -> AC0603FR-0710KL
- R58, R59, R60, R67, R68, R69: value 330 -> 200; Digi PN (none) -> 311-10KLDCT-ND; Digi URL (none) -> https://www.digikey.com/en/products/detail/yageo/AC0603FR-0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; MFG (none) -> Yageo; MFG PN (none) -> AC0603FR-0710KL
Connections:
- net +5V: now also C43.2, U10.14 (VCC)
- net BOTS_Shutdown: now also R54.1; no longer R54.2
- net BSPD_Shutdown_Out: now also R65.1; no longer R65.2
- net E_Stop_Shutdown: now also R62.1; no longer R62.2
- net GND: now also C43.1, D10.1 (K), D11.1 (K), D13.1 (K), D8.1 (K), D9.1 (K), U10.7 (GND)
- net Inertia_Shutdown: now also R55.1; no longer R55.2
- net Shutdown_In: now also R61.1; no longer R61.2
- net at R56.1, U10.11: now also R54.2; no longer R54.1
- net at R57.1, U10.3: now also R55.2; no longer R55.1
- net at R66.1, U10.1: now also R65.2; no longer R65.1
- net at R64.1, U10.5: now also R62.2; no longer R62.1
- net at R63.1, U10.9: now also R61.2; no longer R61.1
- net BOTS_LED_Anode: no longer names the net of R59.1
- net BOTS_LED_Anode: now also D8.2 (A)
- net E_Stop_Shutdown_LED_Anode: no longer names the net of R68.1
- net E_Stop_Shutdown_LED_Anode: now also D10.2 (A)
- net Inertia_LED_Anode: no longer names the net of R60.1
- net Inertia_LED_Anode: now also D9.2 (A)
- net RTD_LED_Enclosure_Anode: no longer names the net of R58.2
- net RTD_LED_Enclosure_Anode: now also D12.2 (A)
- net RTD_LED_Enclosure_Cathode: no longer names the net of Q12.1 (D)
- net RTD_LED_Enclosure_Cathode: now also D12.1 (K)
- net Shutdown_In_LED_Anode: no longer names the net of R67.1
- net Shutdown_In_LED_Anode: now also D11.2 (A)
- net Shutdown_Out_LED_Anode: no longer names the net of R69.1
- net Shutdown_Out_LED_Anode: now also D13.2 (A)
Other:
- note added: "Power Supply"
- moved on the sheet: R54, R55, R61, R62, R65

Commit message: VCU Documentation Update
footprint, annotations, and more!
Parts:
- removed Q12: NMOS, Package_TO_SOT_SMD:SOT-23_Handsoldering, symbol Simulation_SPICE:NMOS
- removed R67, R68, R69: 200, Resistor_SMD:R_0603_1608Metric_Pad0.98x0.95mm_HandSolder, symbol Device:R
- added R47, R52, R53: 300, Resistor_SMD:R_0603_1608Metric_Pad0.98x0.95mm_HandSolder, symbol Device:R
- added TP3, TP4, TP5, TP6, TP7: TestPoint, TestPoint:TestPoint_Pad_1.5x1.5mm, symbol Connector:TestPoint
- C43: Digi PN 311-3874-1-ND -> 311-3484-1-ND; Digi URL https://www.digikey.com/en/products/detail/yageo/CC0603DRNP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 -> https://www.digikey.com/en/products/detail/yageo/CC0603JRX7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; MFG PN CC0603DRNPO9BN6R8 -> CC0603JRX7R6BB105
- R58, R59, R60: value 200 -> 300
Connections:
- net +5V: no longer R58.1
- net GND: now also D12.1 (K)
- net RTD_LED: now also R47.2
- net at D10.2 (A): now also R60.1
- net at D11.2 (A): now also R58.1
- net at R59.2, U10.10: now also TP3.1
- net at U10.2: now also R53.2, TP4.1
- net at R60.2: now also U10.6, TP6.1; no longer U10.4
- net at D9.2 (A): now also R52.1; no longer R60.1
- net at D13.2 (A): now also R53.1
- net at D12.2 (A): now also R47.1; no longer R58.2
- net at U10.8: now also R58.2, TP7.1
- new net: R52.2, TP5.1, U10.4
Other:
- note added: "4V Input"
- moved on the sheet: D12

Commit message: Documentation of VCu
Documentation of components
Parts:
- D10, D11, D12, D13, D8, D9: Digi PN (none) -> 1516-QBLP631-R3ACT-ND; Digi URL (none) -> https://www.digikey.com/en/products/detail/qt-brightek-qtb/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; MFG (none) -> QTB; MFG PN (none) -> QBLP631-R3A
- R47, R52, R53, R58, R59, R60: Digi PN 311-10KLDCT-ND -> YAG5330CT-ND; Digi URL https://www.digikey.com/en/products/detail/yageo/AC0603FR-0710KL/2827814 -> https://www.digikey.com/en/products/detail/yageo/AC0603FR-07300RL/5896018; MFG PN AC0603FR-0710KL -> AC0603FR-07300RL
- R54, R55, R61, R62, R65: Digi PN 311-10KLDCT-ND -> YAG3575CT-ND; Digi URL https://www.digikey.com/en/products/detail/yageo/AC0603FR-0710KL/2827814 -> https://www.digikey.com/en/products/detail/yageo/AC0603FR-07200KL/5895902; MFG PN AC0603FR-0710KL -> AC0603FR-07200KL
- R56, R57, R63, R64, R66: Digi PN 311-10KLDCT-ND -> 13-AC0603FR-13100KLCT-ND; Digi URL https://www.digikey.com/en/products/detail/yageo/AC0603FR-0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 -> https://www.digikey.com/en/products/detail/yageo/AC0603FR-1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; MFG PN AC0603FR-0710KL -> AC0603FR-13100KL
- U10: Digi PN (none) -> 296-1194-1-ND; Digi URL (none) -> https://www.digikey.com/en/products/detail/texas-instrument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; MFG (none) -> TI; MFG PN (none) -> SN74HC14DR

Commit message: Documentation
Added test points to unconnected mcu pins, rtd button, and more documentation
Connections:
- net BOTS_Shutdown: now also TP3.1
- net BSPD_Shutdown_Out: now also TP4.1
- net E_Stop_Shutdown: now also TP6.1
- net Inertia_Shutdown: now also TP5.1
- net Shutdown_In: now also TP7.1
- net at R60.2, U10.6: no longer TP6.1
- net at R53.2, U10.2: no longer TP4.1
- net at R59.2, U10.10: no longer TP3.1
- net at R52.2, U10.4: no longer TP5.1
- net at R58.2, U10.8: no longer TP7.1
Other:
- moved on the sheet: TP3, TP4, TP5, TP6, TP7
Changed lines of the file:
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@@
 	)
 	(junction
-		(at 220.98 119.38)
+		(at 110.49 148.59)
 		(diameter 0)
 		(color 0 0 0 0)
 	)
 	(junction
-		(at 210.82 198.12)
+		(at 210.82 187.96)
 		(diameter 0)
 		(color 0 0 0 0)
 	)
 	(junction
-		(at 231.14 198.12)
+		(at 220.98 119.38)
 		(diameter 0)
 		(color 0 0 0 0)
 	)
 	(junction
-		(at 110.49 198.12)
+		(at 210.82 198.12)
 		(diameter 0)
 		(color 0 0 0 0)
 	)
 	(junction
-		(at 229.87 160.02)
+		(at 110.49 198.12)
 		(diameter 0)
 		(color 0 0 0 0)
@@
 	)
 	(junction
-		(at 209.55 160.02)
+		(at 110.49 187.96)
 		(diameter 0)
 		(color 0 0 0 0)
 	)
 	(junction
-		(at 110.49 160.02)
+		(at 209.55 160.02)
 		(diameter 0)
 		(color 0 0 0 0)
 	)
 	(junction
-		(at 241.3 119.38)
+		(at 110.49 160.02)
 		(diameter 0)
 		(color 0 0 0 0)
 	)
 	(junction
-		(at 129.54 160.02)
+		(at 220.98 107.95)
 		(diameter 0)
 		(color 0 0 0 0)
@@
 	)
 	(junction
-		(at 129.54 198.12)
+		(at 203.2 149.86)
 		(diameter 0)
 		(color 0 0 0 0)
@@
 	(wire
 		(pts
-			(xy 129.54 149.86) (xy 129.54 160.02)
+			(xy 110.49 138.43) (xy 110.49 148.59)
 		)
 		(stroke
@@
 	(wire
 		(pts
-			(xy 241.3 109.22) (xy 241.3 119.38)
+			(xy 220.98 97.79) (xy 220.98 107.95)
 		)
 		(stroke
@@
 	(wire
 		(pts
-			(xy 187.96 149.86) (xy 209.55 149.86)
+			(xy 187.96 149.86) (xy 203.2 149.86)
 		)
 		(stroke
@@
 	(wire
 		(pts
-			(xy 231.14 187.96) (xy 231.14 198.12)
+			(xy 210.82 177.8) (xy 210.82 187.96)
 		)
 		(stroke
@@
 	(wire
 		(pts
-			(xy 194.31 187.96) (xy 210.82 187.96)
+			(xy 193.04 187.96) (xy 210.82 187.96)
 		)
 		(stroke
@@
 	(wire
 		(pts
-			(xy 229.87 149.86) (xy 229.87 160.02)
+			(xy 203.2 139.7) (xy 203.2 149.86)
 		)
 		(stroke
@@
 	(wire
 		(pts
-			(xy 129.54 187.96) (xy 129.54 198.12)
+			(xy 110.49 177.8) (xy 110.49 187.96)
 		)
 		(stroke
@@
 	(wire
 		(pts
+			(xy 203.2 149.86) (xy 209.55 149.86)
+		)
+		(stroke
+			(width 0)
+			(type default)
+		)
+	)
+	(wire
+		(pts
 			(xy 147.32 160.02) (xy 152.4 160.02)
 		)
@@
 	)
 	(label "Inertia_Shutdown"
-		(at 93.98 187.96 0)
+		(at 92.71 187.96 0)
 		(effects
 			(font
@@
 	)
 	(label "BOTS_Shutdown"
-		(at 95.25 148.59 0)
+		(at 93.98 148.59 0)
 		(effects
 			(font
@@
 	)
 	(label "E_Stop_Shutdown"
-		(at 194.31 187.96 0)
+		(at 193.04 187.96 0)
 		(effects
 			(font
@@
 	(global_label "E_Stop_Shutdown"
 		(shape input)
-		(at 194.31 187.96 180)
+		(at 193.04 187.96 180)
 		(fields_autoplaced yes)
 		(effects
@@
 		)
 		(property "Intersheetrefs" "${INTERSHEET_REFS}"
-			(at 174.9967 187.96 0)
+			(at 173.7267 187.96 0)
 			(effects
 				(font
@@
 	(symbol
 		(lib_id "Connector:TestPoint")
-		(at 231.14 187.96 0)
+		(at 210.82 177.8 0)
 		(unit 1)
 		(exclude_from_sim no)
@@
 		(fields_autoplaced yes)
 		(property "Reference" "TP6"
-			(at 233.68 183.3879 0)
+			(at 213.36 173.2279 0)
 			(effects
 				(font
@@
 		)
 		(property "Value" "TestPoint"
-			(at 233.68 185.9279 0)
+			(at 213.36 175.7679 0)
 			(effects
 				(font
@@
 		)
 		(property "Footprint" "TestPoint:TestPoint_Pad_1.5x1.5mm"
-			(at 236.22 187.96 0)
+			(at 215.9 177.8 0)
 			(effects
 				(font
@@
 		)
 		(property "Datasheet" "~"
-			(at 236.22 187.96 0)
+			(at 215.9 177.8 0)
 			(effects
 				(font
@@
 		)
 		(property "Description" "test point"
-			(at 231.14 187.96 0)
+			(at 210.82 177.8 0)
 			(effects
 				(font
@@
 	(symbol
 		(lib_id "Connector:TestPoint")
-		(at 129.54 187.96 0)
+		(at 110.49 177.8 0)
 		(unit 1)
 		(exclude_from_sim no)
@@
 		(fields_autoplaced yes)
 		(property "Reference" "TP5"
-			(at 132.08 183.3879 0)
+			(at 113.03 173.2279 0)
 			(effects
 				(font
@@
 		)
 		(property "Value" "TestPoint"
-			(at 132.08 185.9279 0)
+			(at 113.03 175.7679 0)
 			(effects
 				(font
@@
 		)
 		(property "Footprint" "TestPoint:TestPoint_Pad_1.5x1.5mm"
-			(at 134.62 187.96 0)
+			(at 115.57 177.8 0)
 			(effects
 				(font
@@
 		)
 		(property "Datasheet" "~"
-			(at 134.62 187.96 0)
+			(at 115.57 177.8 0)
 			(effects
 				(font
@@
 		)
 		(property "Description" "test point"
-			(at 129.54 187.96 0)
+			(at 110.49 177.8 0)
 			(effects
 				(font
@@
 	(symbol
 		(lib_id "Connector:TestPoint")
-		(at 129.54 149.86 0)
+		(at 110.49 138.43 0)
 		(unit 1)
 		(exclude_from_sim no)
@@
 		(fields_autoplaced yes)
 		(property "Reference" "TP3"
-			(at 132.08 145.2879 0)
+			(at 113.03 133.8579 0)
 			(effects
 				(font
@@
 		)
 		(property "Value" "TestPoint"
-			(at 132.08 147.8279 0)
+			(at 113.03 136.3979 0)
 			(effects
 				(font
@@
 		)
 		(property "Footprint" "TestPoint:TestPoint_Pad_1.5x1.5mm"
-			(at 134.62 149.86 0)
+			(at 115.57 138.43 0)
 			(effects
 				(font
@@
 		)
 		(property "Datasheet" "~"
-			(at 134.62 149.86 0)
+			(at 115.57 138.43 0)
 			(effects
 				(font
@@
 		)
 		(property "Description" "test point"
-			(at 129.54 149.86 0)
+			(at 110.49 138.43 0)
 			(effects
 				(font
@@
 	(symbol
 		(lib_id "Connector:TestPoint")
-		(at 241.3 109.22 0)
+		(at 220.98 97.79 0)
 		(unit 1)
 		(exclude_from_sim no)
@@
 		(fields_autoplaced yes)
 		(property "Reference" "TP4"
-			(at 243.84 104.6479 0)
+			(at 223.52 93.2179 0)
 			(effects
 				(font
@@
 		)
 		(property "Value" "TestPoint"
-			(at 243.84 107.1879 0)
+			(at 223.52 95.7579 0)
 			(effects
 				(font
@@
 		)
 		(property "Footprint" "TestPoint:TestPoint_Pad_1.5x1.5mm"
-			(at 246.38 109.22 0)
+			(at 226.06 97.79 0)
 			(effects
 				(font
@@
 		)
 		(property "Datasheet" "~"
-			(at 246.38 109.22 0)
+			(at 226.06 97.79 0)
 			(effects
 				(font
@@
 		)
 		(property "Description" "test point"
-			(at 241.3 109.22 0)
+			(at 220.98 97.79 0)
 			(effects
 				(font
@@
 	(symbol
 		(lib_id "Connector:TestPoint")
-		(at 229.87 149.86 0)
+		(at 203.2 139.7 0)
 		(unit 1)
 		(exclude_from_sim no)
@@
 		(fields_autoplaced yes)
 		(property "Reference" "TP7"
-			(at 232.41 145.2879 0)
+			(at 205.74 135.1279 0)
 			(effects
 				(font
@@
 		)
 		(property "Value" "TestPoint"
-			(at 232.41 147.8279 0)
+			(at 205.74 137.6679 0)
 			(effects
 				(font
@@
 		)
 		(property "Footprint" "TestPoint:TestPoint_Pad_1.5x1.5mm"
-			(at 234.95 149.86 0)
+			(at 208.28 139.7 0)
 			(effects
 				(font
@@
 		)
 		(property "Datasheet" "~"
-			(at 234.95 149.86 0)
+			(at 208.28 139.7 0)
 			(effects
 				(font
@@
 		)
 		(property "Description" "test point"
-			(at 229.87 149.86 0)
+			(at 203.2 139.7 0)
 			(effects
 				(font

Commit message: Documentation
Other:
- note added: "12V"
- note added: "3.3V"
Changed lines of the file:
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@@
+		)
+	)
+	(text "12V\n"
+		(exclude_from_sim no)
+		(at 82.296 184.912 0)
+		(effects
+			(font
+				(size 1.27 1.27)
+			)
+		)
+	)
+	(text "3.3V\n"
+		(exclude_from_sim no)
+		(at 109.728 118.872 0)
+		(effects
+			(font
+				(size 1.27 1.27)
+			)
+		)
+	)
+	(text "12V\n"
+		(exclude_from_sim no)
+		(at 179.832 146.05 0)
+		(effects
+			(font
+				(size 1.27 1.27)
+			)
+		)
+	)
+	(text "12V\n"
+		(exclude_from_sim no)
+		(at 182.626 184.404 0)
+		(effects
+			(font
+				(size 1.27 1.27)
+			)
 		)
 	)
@@
 		)
 	)
+	(text "12V\n"
+		(exclude_from_sim no)
+		(at 182.88 104.394 0)
+		(effects
+			(font
+				(size 1.27 1.27)
+			)
+		)
+	)
 	(text "4V Input\n"
 		(exclude_from_sim no)
@@
 		(effects
 			(font
+				(size 1.27 1.27)
+			)
+		)
+	)
+	(text "12V\n"
+		(exclude_from_sim no)
+		(at 84.582 145.542 0)
+		(effects
+			(font

Commit message: LED Strip Level Shifter
Parts:
- renumbered C43 to C22, D12 to D15, D8 to D16, D9 to D17, D11 to D18, D10 to D19, D13 to D20, R54 to R47, R56 to R48, R55 to R49, R57 to R50, R47 to R51, R59 to R52, R52 to R53, R61 to R54, R63 to R55, R62 to R56, R64 to R57, R65 to R58, R66 to R59, R58 to R60, R60 to R61, R53 to R62, TP5 to TP4, TP7 to TP5, TP4 to TP7, U10 to U12
