File: VCU/VCU.kicad_pcb (KiCad board)
At the start: 4 copper layers, 229 parts, among them J1 ATS13-34P-BM01, J2 AMPHENOL_MRJR538001, J3 ATS13-34P-BM01, J4 FTSH-107-01-F-DV-K-P-TR, K1 G6BK-1114P-US, Q1 AO3400A, Q2 AO3400A, Q3 AO3400A, Q4 AO3400A, Q5 AO3400A, Q6 AO3400A, Q7 AO3400A, Q8 AO3400A, Q9 AO3400A, SW5 Y97KT23B5NAFP, U1 AP63205WU, U10 MCP6004, U11 MCP6004, U12 74LS32, U13 74HC14, U14 SZNUD3124DMT1G, U15 74HC14, U16 LM555CMX, U2 MIC5504-3.3YM5, U20 ISO1044BD, U21 ISO1044BD, U22 ISO1044BD, U23 ISO1044BD, U24 MCP6004, U26 STLINK-V3MODS, U27 STM32F446RETx, U28 BME688, U29 BNO086, U6 MCP6004, U7 MCP6004, U8 74LS32, U9 SN74HCS08DR, Y1 ECS-240-8-37B-CKY-TR

Commit message: updated schematic and pcb
Parts:
- removed BOTS_Shutdown1, BSPD_Shutdown_Out1, E_Stop_Shutdown1, Inertia_Shutdown1, Shutdown_In1, TSSI_Red_Logic1, TSSI_Status1: TestPoint, TestPoint:TestPoint_Pad_1.5x1.5mm
- removed D20, D21, D25, D26: CMOZ3L3 TR PBFREE, Diode_SMD:D_SOD-523
- removed D22: LTST-S270KRKT, LED_SMD:LED_0603_1608Metric_Pad1.05x0.95mm_HandSolder
- removed R90: 100k, Resistor_SMD:R_0603_1608Metric_Pad0.98x0.95mm_HandSolder
- removed R91: 200k, Resistor_SMD:R_0603_1608Metric_Pad0.98x0.95mm_HandSolder
- removed R92: 4.7k, Resistor_SMD:R_0603_1608Metric_Pad0.98x0.95mm_HandSolder
- removed XTAL1: ABS07-120-32.768KHZ-T, ABS07-32.768KHZ-T_Footprint:XTAL_ABS07-120_ABR
- added TP15: TestPoint, TestPoint:TestPoint_Pad_1.5x1.5mm, F.Cu at (138.8, -30.3)
- added TP16: TestPoint, TestPoint:TestPoint_Pad_1.5x1.5mm, F.Cu at (142.3, -37.4)
- added TP17: TestPoint, TestPoint:TestPoint_Pad_1.5x1.5mm, F.Cu at (142.3, -33.8)
- added TP18: TestPoint, TestPoint:TestPoint_Pad_1.5x1.5mm, F.Cu at (142.3, -30.3)
- added TP19: TestPoint, TestPoint:TestPoint_Pad_1.5x1.5mm, F.Cu at (145.9, -37.4)
- added TP20: TestPoint, TestPoint:TestPoint_Pad_1.5x1.5mm, F.Cu at (145.9, -33.8)
- added TP21: TestPoint, TestPoint:TestPoint_Pad_1.5x1.5mm, F.Cu at (145.9, -30.3)
- added XTAL2: ABS07-120-32.768KHZ-T, FS_4_Global_Footprint_Library:XTAL_ABS07-120_ABR, F.Cu at (252.9, -26.6)
- C1, C5: footprint Capacitor_SMD:C_0603_1608Metric_Pad1.08x0.95mm_HandSolder -> Capacitor_SMD:C_0805_2012Metric_Pad1.18x1.45mm_HandSolder
- C10, C11, C12, C13, C14, C15, C17, C18, C19, C49: value 1uF -> 0.1uF
- D19: value CMOZ3L3 TR PBFREE -> LTST-S270KRKT; footprint Diode_SMD:D_SOD-523 -> LED_SMD:LED_0603_1608Metric_Pad1.05x0.95mm_HandSolder
- J1: value ATS13-34P-BM01 -> ATS13-34PB2-BM01
- J2: value AMPHENOL_MRJR538001 -> Conn_01x08_Shielded; footprint FS_4_Global_Footprint_Library:AMPHENOL_MRJR538001 -> FS_4_Global_Footprint_Library:SS-60400-023
- J3: value ATS13-34P-BM01 -> ATS13-34PA2-BM01
- L1: value 4.7uF -> 4.7uH
- R55, R57: value 120k -> 12k
- R56, R58: value 200k -> 20k
- R59: value 200k -> 12k
- R60: value 120k -> 20k
- R63: value 1k -> 120
- R64, R65: value 1k -> 100k
- R66: value 120 -> 300k
- R67: value 100k -> 300k
- R69: value 300k -> 300
- R71, R78: value 100k -> 10k
- R72, R82: value 300 -> 10k
- R73: value 300k -> 10k
- R75, R76: value 10k -> 100k
- R79: value 100k -> 300
- R81: value 10k -> 20k
- R84: value 10k -> 36k
- R85: value 100k -> 20k
- R87: value 360k -> 100k
- R88: value 10k -> 200k
- R89: value 10k -> 4.7k
- TP1: value TestPoint -> BSPD_Fault_nDelayed
- TP3: value TestPoint -> BOTS_Shutdown
- TP4: value TestPoint -> Inertia_Shutdown
- TP5: value TestPoint -> Shutdown_In
- TP6: value TestPoint -> E_Stop_Shutdown
- TP7: value TestPoint -> BSPD_Shutdown_Out
- TP8: value TestPoint -> TSSI_Status
- TP9: value TestPoint -> TSSI_Red_Logic
- U12, U8: value 74LS32 -> SN74HCS32DR
- U13, U15: value 74HC14 -> SN74HC14DR
- moved R36 278.7 mm to (261.0, -64.8)
- moved J1 242.7 mm to (268.9, 120.2), turned to 90 degrees
- moved D2 223.9 mm to (248.0, -67.2)
- moved U24 212.5 mm to (108.6, -28.5)
- moved C50 212.4 mm to (247.9, -32.7)
- moved C51 212.4 mm to (247.9, -30.2)
- moved C52 212.4 mm to (247.9, -27.7)
- moved J4 210.7 mm to (99.6, -28.3)
- moved J2 209.4 mm to (238.4, 145.7)
- moved R49 207.9 mm to (265.4, -57.2)
- moved R50 207.9 mm to (265.4, -54.7)
- moved R51 207.9 mm to (265.4, -52.2)
- moved R52 207.9 mm to (265.4, -49.7)
- moved U15 207.9 mm to (271.8, -41.0)
- moved R82 204.8 mm to (138.0, -60.5)
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Connections:
- C10 pad 1: GND -> +5V
- C10 pad 2: +5V -> GND
- C11 pad 1: GND -> +5V
- C11 pad 2: +5V -> GND
- C12 pad 1: GND -> +5V
- C12 pad 2: +5V -> GND
- C13 pad 1: GND -> +5V
- C13 pad 2: +5V -> GND
- C14 pad 1: GND -> +5V
- C14 pad 2: +5V -> GND
- C15 pad 1: GND -> +5V
- C15 pad 2: +5V -> GND
- C17 pad 1: GND -> +5V
- C17 pad 2: +5V -> GND
- C18 pad 1: GND -> +5V
- C18 pad 2: +5V -> GND
- C19 pad 1: GND -> +5V
- C19 pad 2: +5V -> GND
- C28 pad 1: Net-(U24C-+) -> APPS_1_Buff_Filt
- C29 pad 1: Net-(U24D-+) -> APPS_2_Buff_Filt
- C30 pad 1: Net-(U24B-+) -> BPPS_1_Buff_Filt
- C35 pad 1: GND -> Dash_Launch_Filtered
- C35 pad 2: Dash_Launch_Filtered -> GND
- C36 pad 1: GND -> Dash_Lap_Filtered
- C36 pad 2: Dash_Lap_Filtered -> GND
- C39 pad 1: GND -> Driverless_Signal_Filtered
- C39 pad 2: Driverless_Signal_Filtered -> GND
- C49 pad 1: GND -> +5V
- C49 pad 2: +5V -> GND
- D19 pad 1: BPPS_1_Buff_Filt -> GND
- D19 pad 2: GND -> Net-(D19-A)
- J1 pad 1: +12V -> /CAN_Data_L
- J1 pad 10: +12V -> unconnected-(J1-Pin_10-Pad10)
- J1 pad 11: GND -> /Reset_Button
- J1 pad 12: /Rear_Brake_Raw -> /Brake_LED_Cathode
- J1 pad 13: +12V -> /RTD_Buzzer_Neg
- J1 pad 14: GND -> /Driverless_Signal
- J1 pad 15: nIMD_Fault -> /Rear_Brake_Raw
- J1 pad 16: nBMS_Fault -> /Front_Brake_Raw
- J1 pad 17: /Reset_Button -> /nIMD_Fault
- J1 pad 2: GND -> /CAN_Data_H
- J1 pad 20: CAN_Data_H -> +12V
- J1 pad 21: CAN_Data_L -> /RTD_Buzzer_Pos
- J1 pad 22: /CAN_Powertrain_H -> /TSSI_RED_Cathode
- J1 pad 23: /CAN_Powertrain_L -> /TSSI_GREEN_Cathode
- J1 pad 25: /Brake_LED_Cathode -> +12V
- J1 pad 26: /RTD_Buzzer_Pos -> +12V
- J1 pad 27: /RTD_Buzzer_Neg -> GND
- J1 pad 28: /Driverless_Signal -> unconnected-(J1-Pin_28-Pad28)
- J1 pad 29: /UART5_TX -> unconnected-(J1-Pin_29-Pad29)
- J1 pad 3: /Current_Vref_Raw -> /CAN_Powertrain_L
- J1 pad 30: /UART5_RX -> unconnected-(J1-Pin_30-Pad30)
- J1 pad 31: unconnected-(J1-Pin_31-Pad31) -> +12V
- J1 pad 32: unconnected-(J1-Pin_32-Pad32) -> +12V
- J1 pad 33: unconnected-(J1-Pin_33-Pad33) -> GND
- J1 pad 34: unconnected-(J1-Pin_34-Pad34) -> GND
- J1 pad 4: /Current_Analog_Raw -> /CAN_Powertrain_H
- J1 pad 5: +12V -> /UART5_RX
- J1 pad 6: /TSSI_GREEN_Cathode -> /UART5_TX
- J1 pad 7: +12V -> /Current_Analog_Raw
- J1 pad 8: /TSSI_RED_Cathode -> /Current_Vref_Raw
- J1 pad 9: /Front_Brake_Raw -> /nBMS_Fault
- J2 pad 1: unconnected-(J2-Pin_1-Pad1) -> +12V
- J2 pad 2: +12V -> GND
- J2 pad 3: GND -> /Dash_Launch
- J2 pad 4: /Aux_CAN_CTLR_Jumper -> /Dash_Lap
- J2 pad 5: /CAN_Dash_H -> unconnected-(J2-Pin_5-Pad5)
- J2 pad 6: /CAN_Dash_L -> /CAN_Dash_H
- J2 pad 7: /Dash_Lap -> /CAN_Dash_L
- J2 pad 8: /Dash_Launch -> /Aux_CAN_CTLR_Jumper
- J3 pad 1: unconnected-(J3-Pin_1-Pad1) -> /APPS_1_Raw
- J3 pad 10: Inertia_Shutdown -> +5V
- J3 pad 11: BOTS_Shutdown -> +5V
- J3 pad 12: E_Stop_Shutdown -> +5V
- J3 pad 13: Shutdown_In -> +5V
- J3 pad 14: BOTS_Shutdown -> +12V
- J3 pad 15: +5V -> +12V
- J3 pad 16: GND -> +12V
- J3 pad 17: /Status_Indicator_Strip -> +12V
- J3 pad 18: +12V -> GND
- J3 pad 19: /RTD_LED_Cathode -> GND
- J3 pad 2: unconnected-(J3-Pin_2-Pad2) -> /APPS_2_Raw
- J3 pad 20: +3V3 -> GND
- J3 pad 21: /RTD_Button_Neg -> GND
- J3 pad 22: /APPS_1_Raw -> E_Stop_Shutdown
- J3 pad 23: +5V -> E_Stop_Shutdown
- J3 pad 24: GND -> Inertia_Shutdown
- J3 pad 25: /APPS_2_Raw -> +3V3
- J3 pad 26: +5V -> unconnected-(J3-Pin_26-Pad26)
- J3 pad 27: GND -> unconnected-(J3-Pin_27-Pad27)
- J3 pad 28: /BPPS_1_Raw -> Shutdown_In
- J3 pad 29: +5V -> BOTS_Shutdown
- J3 pad 3: +12V -> /BPPS_1_Raw
- J3 pad 30: GND -> BOTS_Shutdown
- J3 pad 4: /BMS_LED_Cathode -> /Status_Indicator_Strip
- J3 pad 5: +12V -> /BMS_LED_Cathode
- J3 pad 7: +12V -> /BSPD_LED_Cathode
- J3 pad 8: /BSPD_LED_Cathode -> /RTD_Button_Neg
- J3 pad 9: E_Stop_Shutdown -> /RTD_LED_Cathode
- R21 pad 2: BSPD_Fault -> /MCU/BSDP_Fault
- R51 pad 2: BSPD_Fault -> /MCU/BSDP_Fault
- R52 pad 2: BSPD_Fault -> /MCU/BSDP_Fault
- R55 pad 1: Net-(U24C-+) -> APPS_1_Buff_Filt
- R55 pad 2: /BPPS_1_Raw -> Net-(U24D--)
- R56 pad 1: Net-(U24C-+) -> APPS_1_Buff_Filt
- R57 pad 1: Net-(U24D-+) -> GND
- R57 pad 2: /APPS_1_Raw -> APPS_2_Buff_Filt
- R58 pad 1: Net-(U24D-+) -> Net-(U24B--)
- R58 pad 2: GND -> APPS_2_Buff_Filt
- R59 pad 1: /APPS_2_Raw -> BPPS_1_Buff_Filt
- R59 pad 2: Net-(U24B-+) -> Net-(U24C--)
- R60 pad 1: GND -> BPPS_1_Buff_Filt
- R60 pad 2: Net-(U24B-+) -> GND
- R62 pad 1: CAN_Data_L -> /CAN_Data_L
- R62 pad 2: CAN_Data_H -> /CAN_Data_H
- R63 pad 1: Net-(U24C--) -> /CAN_Powertrain_L
- R63 pad 2: BPPS_1_Buff_Filt -> /CAN_Powertrain_H
- R64 pad 1: Net-(U24D--) -> /Dash_Launch
- R64 pad 2: APPS_1_Buff_Filt -> GND
- R65 pad 1: Net-(U24B--) -> /Dash_Lap
- R65 pad 2: APPS_2_Buff_Filt -> GND
- R66 pad 1: /CAN_Powertrain_L -> Dash_Launch_Filtered
- R66 pad 2: /CAN_Powertrain_H -> /Dash_Launch
- R67 pad 1: /Dash_Lap -> Dash_Lap_Filtered
- R67 pad 2: GND -> /Dash_Lap
- R68 pad 1: /Dash_Launch -> /Driverless_Signal
- R69 pad 1: Dash_Launch_Filtered -> Net-(D19-A)
- R69 pad 2: /Dash_Lap -> RTD_LED
- R70 pad 1: Dash_Lap_Filtered -> Driverless_Signal_Filtered
- R70 pad 2: /Dash_Launch -> /Driverless_Signal
- R71 pad 1: /Driverless_Signal -> +5V
- R71 pad 2: GND -> /Status_Indicator_Strip
- R72 pad 1: Net-(D22-A) -> /MCU/Status_Indicator_Strip_3V
- R72 pad 2: RTD_LED -> +3V3
- R73 pad 1: Driverless_Signal_Filtered -> /MCU/BOOT0
- R73 pad 2: /Driverless_Signal -> GND
- R74 pad 1: +5V -> RTD_LED
- R74 pad 2: /Status_Indicator_Strip -> Net-(Q7-G)
- R75 pad 1: +3V3 -> GND
- R75 pad 2: /MCU/Status_Indicator_Strip_3V -> RTD_Buzzer
- R76 pad 2: /MCU/BOOT0 -> Brake_Light_Signal
- R77 pad 1: RTD_LED -> Net-(Q8-G)
- R77 pad 2: Net-(Q7-G) -> RTD_Buzzer
- R78 pad 1: GND -> Net-(Q9-G)
- R78 pad 2: RTD_Buzzer -> Brake_Light_Signal
- R79 pad 1: GND -> /RTD_Buzzer_Pos
- R79 pad 2: Brake_Light_Signal -> +5V
- R80 pad 1: Net-(Q8-G) -> /MCU/BOOT1
- R80 pad 2: RTD_Buzzer -> GND
- R81 pad 1: Net-(Q9-G) -> GND
- R81 pad 2: Brake_Light_Signal -> /MCU/Rear_Brake_Buff_Filtered_3V
- R82 pad 1: /RTD_Buzzer_Pos -> /MCU/BSPD_Shutdown_Out_3V04
- R82 pad 2: +5V -> GND
- R83 pad 1: /MCU/BOOT1 -> Rear_Brake_Buff_Filtered
- R83 pad 2: GND -> /MCU/Rear_Brake_Buff_Filtered_3V
- R84 pad 1: Net-(D25-K) -> BSPD_Shutdown_Out
- R84 pad 2: /MCU/Rear_Brake_Buff_Filtered_2.25V -> /MCU/BSPD_Shutdown_Out_3V04
- R85 pad 1: /MCU/BSPD_Shutdown_Out_3V04 -> GND
- R85 pad 2: GND -> /MCU/Front_Brake_Buff_Filtered_3V
- R86 pad 1: /MCU/Rear_Brake_Buff_Filtered_2.25V -> Front_Brake_Buff_Filtered
- R86 pad 2: Rear_Brake_Buff_Filtered -> /MCU/Front_Brake_Buff_Filtered_3V
- R87 pad 1: BSPD_Shutdown_Out -> /MCU/BSDP_Fault
- R87 pad 2: /MCU/BSPD_Shutdown_Out_3V04 -> /MCU/BSPD_Fault_3V3
- R88 pad 1: Net-(D26-K) -> /MCU/BSPD_Fault_3V3
- R88 pad 2: /MCU/Front_Brake_Buff_Filtered_2.25V -> GND
- R89 pad 1: /MCU/Front_Brake_Buff_Filtered_2.25V -> +3V3
- R89 pad 2: Front_Brake_Buff_Filtered -> BNO_BOOTN
- TP10 pad 1: Net-(U27-PB7) -> Net-(U27-PC5)
- TP11 pad 1: Net-(U27-PB13) -> Net-(U27-PC6)
- TP12 pad 1: Net-(U27-PB10) -> Net-(U27-PA9)
- TP13 pad 1: Net-(U27-PA7) -> Net-(U27-PB1)
- TP14 pad 1: Net-(U27-PA12) -> Net-(U27-PA8)
- TP2 pad 1: BSPD_Fault -> /MCU/BSDP_Fault
- TP3 pad 1: Net-(U27-PC5) -> BOTS_Shutdown
- TP4 pad 1: Net-(U27-PC6) -> Inertia_Shutdown
- TP5 pad 1: Net-(U27-PA9) -> Shutdown_In
- TP6 pad 1: Net-(U27-PB1) -> E_Stop_Shutdown
- TP7 pad 1: Net-(U27-PA8) -> BSPD_Shutdown_Out
- TP8 pad 1: Net-(U27-PA10) -> /Shutdown_VCU/Shutdown_LEDS/TSSI_Status
- TP9 pad 1: Net-(U27-PA15) -> /Shutdown_VCU/Shutdown_LEDS/TSSI_Red_Logic
- U11 pad 8: BSPD_Fault -> /MCU/BSDP_Fault
- U13 pad 11: nIMD_Fault -> /nIMD_Fault
- U13 pad 13: BSPD_Fault -> /MCU/BSDP_Fault
- U13 pad 9: nBMS_Fault -> /nBMS_Fault
- U14 pad 5: BSPD_Fault -> /MCU/BSDP_Fault
- U22 pad 5: CAN_Data_L -> /CAN_Data_L
- U22 pad 6: CAN_Data_H -> /CAN_Data_H
- U23 pad 5: CAN_Data_L -> /CAN_Data_L
- U23 pad 6: CAN_Data_H -> /CAN_Data_H
- U24 pad 10: Net-(U24C-+) -> /BPPS_1_Raw
- U24 pad 12: Net-(U24D-+) -> /APPS_1_Raw
- U24 pad 5: Net-(U24B-+) -> /APPS_2_Raw
- U27 pad 14: /MCU/Rear_Brake_Buff_Filtered_2.25V -> /MCU/Rear_Brake_Buff_Filtered_3V
- U27 pad 15: /MCU/Front_Brake_Buff_Filtered_2.25V -> /MCU/Front_Brake_Buff_Filtered_3V
- U27 pad 23: Net-(U27-PA7) -> RTD_Buzzer
- U27 pad 24: RTD_Buzzer -> Brake_Light_Signal
- U27 pad 44: Brake_Light_Signal -> Net-(U27-PA11)
- U9 pad 10: nBMS_Fault -> /nBMS_Fault
- U9 pad 9: nIMD_Fault -> /nIMD_Fault
Routing:
- net +5V: vias 0 -> 28
Other:
- board outline added: 152.4 x 50.8 mm

Commit message: Update VCU.kicad_pcb
Parts:
- moved R5 161.9 mm to (265.6, 102.4)
- moved R10 151.3 mm to (264.4, 85.9)
- moved R9 151.3 mm to (264.4, 83.4)
- moved C6 151.3 mm to (255.7, 75.8)
- moved C7 151.3 mm to (255.7, 78.3)
- moved R4 151.3 mm to (260.0, 90.9)
- moved R35 88.9 mm to (239.3, 18.9)
- moved R36 88.9 mm to (239.3, 21.4)
- moved R37 88.9 mm to (239.3, 23.9)
- moved R38 88.9 mm to (239.3, 26.4)
- moved R39 88.9 mm to (239.3, 28.9)
- moved R40 88.9 mm to (239.3, 31.4)
- moved R41 88.9 mm to (239.3, 34.0)
- moved R42 88.9 mm to (239.3, 36.5)
- moved R43 88.9 mm to (239.3, 39.0)
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Routing:
- removed copper zone on In2.Cu, net +3V3
- removed copper zone on In2.Cu, net +5V
- removed copper zone on In1.Cu, net GND
- removed copper zone on In2.Cu, net Net-(U24C--)

Commit message: PCB and Schematic Changes
Layed out pcb components and removed some test points, changed gates for chips.
Parts:
- removed TP12, TP13, TP15, TP16, TP19, TP20: TestPoint, TestPoint:TestPoint_Pad_1.5x1.5mm
- removed XTAL2: ABS07-120-32.768KHZ-T, FS_4_Global_Footprint_Library:XTAL_ABS07-120_ABR
- added XTAL1: ABS07-120-32.768KHZ-T, FS_4_Global_Footprint_Library:XTAL_ABS07-120_ABR, F.Cu at (231.0, 146.9)
- R57: value 12k -> 20k
- R58: value 20k -> 12k
- TP1: value BSPD_Fault_nDelayed -> TestPoint; footprint TestPoint:TestPoint_Pad_1.5x1.5mm -> TestPoint:TestPoint_Pad_D1.0mm
- TP10, TP11, TP14, TP17, TP18, TP2, TP21, TP3, TP4, TP5, TP6, TP7, TP8, TP9: footprint TestPoint:TestPoint_Pad_1.5x1.5mm -> TestPoint:TestPoint_Pad_D1.0mm
- U10: value MCP6004 -> SN74HCS08DR
- U8: value SN74HCS32DR -> MCP6004
- U9: value SN74HCS08DR -> SN74HCS32DR
- moved C36 180.2 mm to (269.1, 153.2)
- moved C35 174.8 mm to (269.1, 143.1)
- moved R65 168.8 mm to (269.1, 158.3), turned to 180 degrees
- moved C24 168.0 mm to (255.1, 143.1)
- moved R67 163.4 mm to (269.1, 155.8)
- moved R64 163.4 mm to (269.1, 148.1), turned to 180 degrees
- moved R62 158.8 mm to (265.3, 140.5)
- moved R66 158.2 mm to (269.1, 145.6)
- moved C31 156.5 mm to (261.5, 135.4)
- moved C26 154.1 mm to (255.1, 127.8), turned to 180 degrees
- moved R76 153.3 mm to (237.3, 167.2), turned to 180 degrees
- moved C34 152.8 mm to (258.9, 118.9), turned to 180 degrees
- moved C45 152.2 mm to (247.5, 134.2)
- moved R75 151.1 mm to (237.3, 162.1), turned to 180 degrees
- moved C32 149.4 mm to (248.8, 143.1)
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Connections:
- C6 pad 1: Net-(U7C-+) -> Net-(U8C-+)
- C7 pad 1: Net-(U7D-+) -> Net-(U8D-+)
- C8 pad 1: Net-(U7A-+) -> Net-(U8B-+)
- C9 pad 1: Net-(U7B-+) -> Net-(U8A-+)
- R10 pad 1: Net-(U7D-+) -> Net-(U8D-+)
- R11 pad 2: Net-(U7B-+) -> Net-(U8A-+)
- R12 pad 2: Net-(U7A-+) -> Net-(U8B-+)
- R55 pad 2: Net-(U24D--) -> Net-(U24C--)
- R57 pad 1: GND -> Net-(U24D--)
- R58 pad 1: Net-(U24B--) -> GND
- R59 pad 2: Net-(U24C--) -> Net-(U24A--)
- R9 pad 2: Net-(U7C-+) -> Net-(U8C-+)
- RV1 pad 2: Net-(U6C--) -> Net-(U7B--)
- RV2 pad 2: Net-(U6D--) -> Net-(U7A--)
- TP14 pad 1: Net-(U27-PA8) -> Net-(U27-PB1)
- TP17 pad 1: Net-(U27-PB7) -> Net-(U27-PA15)
- TP18 pad 1: Net-(U27-PB13) -> Net-(U27-PB7)
- U10 pad 1: /Shutdown_VCU/Current_Sensor_Short -> /Reset_Button
- U10 pad 10: Rear_Brake_Buff_Filtered -> /nBMS_Fault
- U10 pad 11: GND -> unconnected-(U10-Pad11)
- U10 pad 12: /Shutdown_VCU/Open_Threshold -> unconnected-(U10-Pad12)
- U10 pad 13: Rear_Brake_Buff_Filtered -> unconnected-(U10-Pad13)
- U10 pad 14: /Shutdown_VCU/Rear_Brake_Open -> +5V
- U10 pad 2: /Shutdown_VCU/Short_Threshold -> /Shutdown_VCU/nBSPD_Fault
- U10 pad 3: Current_Analog_Buff_Filtered -> /Shutdown_VCU/BSPD_Set
- U10 pad 4: +5V -> /Shutdown_VCU/High_Current_Output
- U10 pad 5: /Shutdown_VCU/Open_Threshold -> /Shutdown_VCU/Hard_Braking
- U10 pad 6: Current_Analog_Buff_Filtered -> Hard_Braking_High_Current
- U10 pad 7: /Shutdown_VCU/Current_Sensor_Open -> GND
- U10 pad 8: /Shutdown_VCU/Rear_Brake_Short -> /Shutdown_VCU/Shutdown_LEDS/TSSI_Status
- U10 pad 9: /Shutdown_VCU/Short_Threshold -> /nIMD_Fault
- U24 pad 1: unconnected-(U24-Pad1) -> Net-(U24A--)
- U24 pad 10: /BPPS_1_Raw -> /APPS_1_Raw
- U24 pad 12: /APPS_1_Raw -> /APPS_2_Raw
- U24 pad 2: unconnected-(U24A---Pad2) -> Net-(U24A--)
- U24 pad 3: unconnected-(U24A-+-Pad3) -> /BPPS_1_Raw
- U24 pad 5: /APPS_2_Raw -> unconnected-(U24B-+-Pad5)
- U24 pad 6: Net-(U24B--) -> unconnected-(U24B---Pad6)
- U24 pad 7: Net-(U24B--) -> unconnected-(U24-Pad7)
- U27 pad 29: Net-(U27-PB10) -> unconnected-(U27-PB10-Pad29)
- U27 pad 34: Net-(U27-PB13) -> unconnected-(U27-PB13-Pad34)
- U27 pad 41: Net-(U27-PA8) -> unconnected-(U27-PA8-Pad41)
- U27 pad 42: Net-(U27-PA9) -> unconnected-(U27-PA9-Pad42)
- U27 pad 43: Net-(U27-PA10) -> unconnected-(U27-PA10-Pad43)
- U27 pad 44: Net-(U27-PA11) -> unconnected-(U27-PA11-Pad44)
- U6 pad 10: Rear_Brake_Buff_Filtered -> Current_Analog_Buff_Filtered
- U6 pad 12: Front_Brake_Buff_Filtered -> /Shutdown_VCU/Open_Threshold
- U6 pad 13: Net-(U6D--) -> Current_Analog_Buff_Filtered
- U6 pad 14: /Shutdown_VCU/Hard_Front_Brake -> /Shutdown_VCU/Current_Sensor_Open
- U6 pad 8: /Shutdown_VCU/Hard_Rear_Brake -> /Shutdown_VCU/Current_Sensor_Short
- U6 pad 9: Net-(U6C--) -> /Shutdown_VCU/Short_Threshold
- U7 pad 1: Current_Vref_Buff_Filtered -> /Shutdown_VCU/Hard_Front_Brake
- U7 pad 10: Net-(U7C-+) -> Rear_Brake_Buff_Filtered
- U7 pad 12: Net-(U7D-+) -> /Shutdown_VCU/Open_Threshold
- U7 pad 13: Front_Brake_Buff_Filtered -> Rear_Brake_Buff_Filtered
- U7 pad 14: Front_Brake_Buff_Filtered -> /Shutdown_VCU/Rear_Brake_Open
- U7 pad 2: Current_Vref_Buff_Filtered -> Net-(U7A--)
- U7 pad 3: Net-(U7A-+) -> Front_Brake_Buff_Filtered
- U7 pad 5: Net-(U7B-+) -> Rear_Brake_Buff_Filtered
- U7 pad 6: Current_Analog_Buff_Filtered -> Net-(U7B--)
- U7 pad 7: Current_Analog_Buff_Filtered -> /Shutdown_VCU/Hard_Rear_Brake
- U7 pad 8: Rear_Brake_Buff_Filtered -> /Shutdown_VCU/Rear_Brake_Short
- U7 pad 9: Rear_Brake_Buff_Filtered -> /Shutdown_VCU/Short_Threshold
- U8 pad 1: Rear_Brake_Fault -> Current_Analog_Buff_Filtered
- U8 pad 10: /Shutdown_VCU/Brake_Current_Sensor_Fault -> Net-(U8C-+)
- U8 pad 11: /Shutdown_VCU/Brake_Current_Sensor_Fault -> GND
- U8 pad 12: Current_Sensor_Fault -> Net-(U8D-+)
- U8 pad 13: Net-(U8-Pad13) -> Front_Brake_Buff_Filtered
- U8 pad 14: +5V -> Front_Brake_Buff_Filtered
- U8 pad 2: Front_Brake_Fault -> Current_Analog_Buff_Filtered
- U8 pad 3: Net-(U8-Pad13) -> Net-(U8A-+)
- U8 pad 4: /Shutdown_VCU/Hard_Rear_Brake -> +5V
- U8 pad 5: /Shutdown_VCU/Hard_Front_Brake -> Net-(U8B-+)
- U8 pad 6: /Shutdown_VCU/Hard_Braking -> Current_Vref_Buff_Filtered
- U8 pad 7: GND -> Current_Vref_Buff_Filtered
- U8 pad 8: /Shutdown_VCU/BSPD_Fault_nDelayed -> Rear_Brake_Buff_Filtered
- U8 pad 9: Hard_Braking_High_Current -> Rear_Brake_Buff_Filtered
- U9 pad 1: /Reset_Button -> Rear_Brake_Fault
- U9 pad 10: /nBMS_Fault -> /Shutdown_VCU/Brake_Current_Sensor_Fault
- U9 pad 11: unconnected-(U9-Pad11) -> /Shutdown_VCU/Brake_Current_Sensor_Fault
- U9 pad 12: unconnected-(U9-Pad12) -> Current_Sensor_Fault
- U9 pad 13: unconnected-(U9-Pad13) -> Net-(U9-Pad13)
- U9 pad 2: /Shutdown_VCU/nBSPD_Fault -> Front_Brake_Fault
- U9 pad 3: /Shutdown_VCU/BSPD_Set -> Net-(U9-Pad13)
- U9 pad 4: /Shutdown_VCU/High_Current_Output -> /Shutdown_VCU/Hard_Rear_Brake
- U9 pad 5: /Shutdown_VCU/Hard_Braking -> /Shutdown_VCU/Hard_Front_Brake
- U9 pad 6: Hard_Braking_High_Current -> /Shutdown_VCU/Hard_Braking
- U9 pad 8: /Shutdown_VCU/Shutdown_LEDS/TSSI_Status -> /Shutdown_VCU/BSPD_Fault_nDelayed
- U9 pad 9: /nIMD_Fault -> Hard_Braking_High_Current
Other:
- board size 152.4 x 50.8 mm -> 98.8 x 101.6 mm

Commit message: pcb layout
Parts:
- moved Q3 42.5 mm to (253.8, 115.7), turned to 0 degrees
- moved TP8 40.4 mm to (252.6, 112.6), turned to 0 degrees
- moved R49 37.5 mm to (250.0, 116.9), turned to 0 degrees
- moved Q4 37.4 mm to (248.8, 111.3), turned to 0 degrees
- moved R47 37.0 mm to (250.0, 114.5), turned to 0 degrees
- moved R48 32.5 mm to (244.9, 110.0), turned to 180 degrees
- moved R50 31.8 mm to (244.9, 112.6), turned to 180 degrees
- moved Q8 25.0 mm to (262.7, 148.1)
- moved R76 25.0 mm to (258.9, 154.5)
- moved R78 25.0 mm to (258.9, 151.9)
- moved Q9 25.0 mm to (262.7, 153.2)
- moved R75 25.0 mm to (258.9, 149.4)
- moved R77 25.0 mm to (258.9, 146.9)
- moved Q2 19.3 mm to (222.1, 139.2)
- moved R42 19.3 mm to (225.9, 138.0)
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
Commit message: footprint relay spst
Parts:
- added K2: G6SK-2G, Relay_SMD:Relay_DPDT_Omron_G6SK-2G, F.Cu at (299.0, 66.8)
- added K3: G6DN-1A, FS_4_Global_Footprint_Library:RELAY_G6DN-1A, F.Cu at (292.0, 60.3)
- moved C13 0.80 mm to (239.4, 79.3)
- moved R17 0.51 mm to (244.4, 80.8)
- moved U11 0.36 mm to (238.3, 74.7)
- moved R25 0.25 mm to (218.5, 118.9)

Commit message: footprijt update
Parts:
- removed K1: G6BK-1114P-US, FS_4_Global_Footprint_Library:RELAY_G6BK-1114P-US_OMR
- added D22: ACGRAT105L-HF, Diode_SMD:D_2010_5025Metric_Pad1.52x2.65mm_HandSolder, F.Cu at (151.0, 179.1)
- added H1: MountingHole_Pad, MountingHole:MountingHole_3.2mm_M3_Pad, F.Cu at (202.4, 73.2)
- added H2: MountingHole_Pad, MountingHole:MountingHole_3.2mm_M3_Pad, F.Cu at (194.8, 167.2)
- added H3: MountingHole_Pad, MountingHole:MountingHole_3.2mm_M3_Pad, F.Cu at (281.5, 132.9)
- added H4: MountingHole_Pad, MountingHole:MountingHole_3.2mm_M3_Pad, F.Cu at (273.9, 73.2)
- J1: footprint FS_4_Global_Footprint_Library:ATS13-34P-BM01 -> FS_4_Global_Footprint_Library:ATS13-34PB2-BM01
- J3: footprint FS_4_Global_Footprint_Library:ATS13-34P-BM01 -> FS_4_Global_Footprint_Library:ATS13-34PA2-BM01
- moved K3 195.1 mm to (129.4, 168.2), turned to 90 degrees
- moved K2 188.4 mm to (136.0, 161.2), turned to 90 degrees
- moved C23 111.0 mm to (144.2, 138.0)
- moved C24 111.0 mm to (144.2, 145.6)
- moved C26 111.0 mm to (144.2, 130.3)
- moved C34 111.0 mm to (148.0, 121.5)
- moved C6 111.0 mm to (155.6, 85.9)
- moved C7 111.0 mm to (151.8, 85.9)
- moved C8 111.0 mm to (148.0, 97.3)
- moved C9 111.0 mm to (148.0, 105.0)
- moved L1 111.0 mm to (159.4, 135.4)
- moved Q8 111.0 mm to (151.8, 150.7)
- moved Q9 111.0 mm to (151.8, 155.8)
- moved R10 111.0 mm to (151.8, 89.1)
- moved R11 111.0 mm to (148.0, 107.5)
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Connections:
- K2 pad 1: unconnected-(K2-Pad1) -> +12V
- K2 pad 12: unconnected-(K2-Pad12) -> Net-(K2-Pad12)
- K2 pad 6: unconnected-(K2-Pad6) -> +12V
- K2 pad 7: unconnected-(K2-Pad7) -> Net-(K2-Pad7)
- K2 pad 8: unconnected-(K2-Pad8) -> Net-(D22-K)
- K2 pad 9: unconnected-(K2-Pad9) -> +12V
- K3 pad 1: unconnected-(K3-Pad1) -> GND
- K3 pad 2: unconnected-(K3-Pad2) -> Net-(D22-K)
- K3 pad 5: unconnected-(K3-Pad5) -> BSPD_Shutdown_Out
- K3 pad 8: unconnected-(K3-Pad8) -> Inertia_Shutdown
- U14 pad 3: Net-(K1-Pad2) -> Net-(K2-Pad7)
- U14 pad 6: Net-(K1-Pad1) -> Net-(K2-Pad12)
Other:
- board size 98.8 x 101.6 mm -> 94.4 x 101.6 mm

Commit message: PCB Layout and Documentation
Parts:
- moved C20 208.5 mm to (323.4, 121.0)
- moved C27 208.5 mm to (323.4, 108.3)
- moved R41 208.5 mm to (323.4, 138.7)
- moved R42 208.5 mm to (323.4, 133.7)
- moved R43 208.5 mm to (323.4, 141.3)
- moved R44 208.5 mm to (323.4, 136.2)
- moved R53 208.5 mm to (323.4, 103.2)
- moved R54 208.5 mm to (323.4, 105.7)
- moved R74 208.5 mm to (323.4, 145.1)
- moved TP11 208.5 mm to (331.0, 131.1)
- moved TP3 208.5 mm to (311.3, 98.1)
- moved C39 208.5 mm to (336.1, 103.2)
- moved D19 208.5 mm to (347.5, 95.6)
- moved Q1 208.5 mm to (319.6, 140.0)
- moved Q2 208.5 mm to (319.6, 134.9)
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Connections:
- net /MCU/3V3_A renamed +3V3A
- U10 pad 1: /Reset_Button -> unconnected-(U10-Pad1)
- U10 pad 11: unconnected-(U10-Pad11) -> /Shutdown_VCU/BSPD_Set
- U10 pad 12: unconnected-(U10-Pad12) -> /Reset_Button
- U10 pad 13: unconnected-(U10-Pad13) -> /Shutdown_VCU/nBSPD_Fault
- U10 pad 2: /Shutdown_VCU/nBSPD_Fault -> unconnected-(U10-Pad2)
- U10 pad 3: /Shutdown_VCU/BSPD_Set -> unconnected-(U10-Pad3)
- U7 pad 10: Rear_Brake_Buff_Filtered -> /Shutdown_VCU/Open_Threshold
- U7 pad 12: /Shutdown_VCU/Open_Threshold -> Rear_Brake_Buff_Filtered
- U7 pad 13: Rear_Brake_Buff_Filtered -> /Shutdown_VCU/Short_Threshold
- U7 pad 14: /Shutdown_VCU/Rear_Brake_Open -> /Shutdown_VCU/Rear_Brake_Short
- U7 pad 8: /Shutdown_VCU/Rear_Brake_Short -> /Shutdown_VCU/Rear_Brake_Open
- U7 pad 9: /Shutdown_VCU/Short_Threshold -> Rear_Brake_Buff_Filtered
- U9 pad 1: Rear_Brake_Fault -> Current_Sensor_Fault
- U9 pad 11: /Shutdown_VCU/Brake_Current_Sensor_Fault -> /Shutdown_VCU/Hard_Braking
- U9 pad 12: Current_Sensor_Fault -> /Shutdown_VCU/Hard_Rear_Brake
- U9 pad 13: Net-(U9-Pad13) -> /Shutdown_VCU/Hard_Front_Brake
- U9 pad 2: Front_Brake_Fault -> Net-(U9-Pad2)
- U9 pad 3: Net-(U9-Pad13) -> /Shutdown_VCU/Brake_Current_Sensor_Fault
- U9 pad 4: /Shutdown_VCU/Hard_Rear_Brake -> Rear_Brake_Fault
- U9 pad 5: /Shutdown_VCU/Hard_Front_Brake -> Front_Brake_Fault
- U9 pad 6: /Shutdown_VCU/Hard_Braking -> Net-(U9-Pad2)
Routing:
- net Hard_Braking_High_Current: track 0.00 -> 19.3 mm
- net Current_Sensor_Fault: track 0.00 -> 18.7 mm
- net +12V: track 0.00 -> 18.4 mm
- net Front_Brake_Fault: track 0.00 -> 10.5 mm
- net Rear_Brake_Fault: track 0.00 -> 8.46 mm
- net Net-(D3-A): track 0.00 -> 4.24 mm
- net Net-(D4-A): track 0.00 -> 2.05 mm
- net /Aux_CAN_CTLR_Jumper: vias 0 -> 1
Other:
- board size 94.4 x 101.6 mm -> 92.5 x 101.6 mm

Commit message: Changed Pin Numbers on Connector
Parts:
- moved R3 123.3 mm to (219.3, 74.0), turned to 0 degrees
- moved TP3 119.2 mm to (197.0, 131.9)
- moved R14 117.0 mm to (216.8, 80.1), turned to -90 degrees
- moved R2 116.4 mm to (229.0, 70.9), turned to 180 degrees
- moved R8 114.0 mm to (220.3, 71.4), turned to 90 degrees
- moved R13 111.7 mm to (218.3, 80.1), turned to -90 degrees
- moved TP14 111.1 mm to (224.9, 154.7), turned to 0 degrees
- moved TP8 109.5 mm to (241.7, 123.7)
- moved R53 108.7 mm to (214.8, 108.5)
- moved R54 108.7 mm to (214.8, 111.0)
- moved C27 108.7 mm to (214.8, 113.1)
- moved R48 106.9 mm to (238.4, 130.4)
- moved Q4 106.9 mm to (242.2, 131.4)
- moved R50 106.7 mm to (238.4, 132.1)
- moved TP11 104.7 mm to (229.0, 154.7), turned to 0 degrees
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Connections:
- J1 pad 1: /CAN_Data_L -> /CAN_Powertrain_L
- J1 pad 2: /CAN_Data_H -> /CAN_Powertrain_H
- J1 pad 3: /CAN_Powertrain_L -> /CAN_Data_L
- J1 pad 4: /CAN_Powertrain_H -> /CAN_Data_H
Routing:
- net +12V: track 18.4 -> 0.00 mm
