File: steering-wheel-board/steering_wheel.kicad_sch (KiCad schematic)
At the start: 12 parts, among them J1 Connector Type TBD, U1 AP63205WU, U2 MIC5504-3.3YM5, U3 ISO1044BD

Commit message: added some notes
Parts:
- added J3: Conn_01x40, symbol Connector_Generic:Conn_01x40
Other:
- note added: "TODO: Include test points/debug points for the following items: Backlight_PWM LED_High LED_Low Digital buses for all the rotary switches UART/some way to connect MCU to laptop for debug"
- note added: "TODO: add in ribbon cable connections"
- note added: "TODO: add part number of specific ribbon cable connector we'll use verify correct pitch, try to get one with both top and bottom contacts to make assembly easier"
Changed lines of the file:
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@@
+		)
+	)
+	(text "TODO: Include test points/debug points\nfor the following items:\nBacklight_PWM\nLED_High\nLED_Low\nDigital buses for all the rotary switches\nUART/some way to  connect MCU to laptop for debug\n"
+		(exclude_from_sim no)
+		(at 22.098 68.58 0)
+		(effects
+			(font
+				(size 1.27 1.27)
+			)
+			(justify left)
 		)
 	)
@@
 			)
 			(justify left)
+		)
+	)
+	(text "TODO: add part number of \nspecific ribbon cable connector we'll use\nverify correct pitch, \ntry to get one with both top\nand bottom contacts to make assembly easier"
+		(exclude_from_sim no)
+		(at 369.062 102.362 0)
+		(effects
+			(font
+				(size 1.27 1.27)
+			)
+			(justify left)
+		)
+	)
+	(text "TODO: add in ribbon cable connections\n"
+		(exclude_from_sim no)
+		(at 359.41 183.642 0)
+		(effects
+			(font
+				(size 1.27 1.27)
+			)
 		)
 	)
@@
 					(unit 1)
 				)
+			)
+		)
+	)
+	(symbol
+		(lib_id "Connector_Generic:Conn_01x40")
+		(at 363.22 123.19 0)
+		(unit 1)
+		(exclude_from_sim no)
+		(in_bom yes)
+		(on_board yes)
+		(dnp no)
+		(fields_autoplaced yes)
+		(property "Reference" "J3"
+			(at 365.76 123.1899 0)
+			(effects
+				(font
+					(size 1.27 1.27)
+				)
+				(justify left)
+			)
+		)
+		(property "Value" "Conn_01x40"
+			(at 365.76 125.7299 0)
+			(effects
+				(font
+					(size 1.27 1.27)
+				)
+				(justify left)
+			)
+		)
+		(property "Footprint" ""
+			(at 363.22 123.19 0)
+			(effects
+				(font
+					(size 1.27 1.27)
+				)
+				(hide yes)
+			)
+		)
+		(property "Datasheet" "~"
+			(at 363.22 123.19 0)
+			(effects
+				(font
+					(size 1.27 1.27)
+				)
+				(hide yes)
+			)
+		)
+		(property "Description" "Generic connector, single row, 01x40, script generated (kicad-library-utils/schlib/autogen/connector/)"
+			(at 363.22 123.19 0)
+			(effects
+				(font
+					(size 1.27 1.27)
+				)
+				(hide yes)
+			)
+		)
+		(pin "38"
+		)
+		(pin "35"
+		)
+		(pin "24"
+		)
+		(pin "18"
+		)
+		(pin "26"
+		)
+		(pin "16"
+		)
+		(pin "33"
+		)
+		(pin "22"
+		)
+		(pin "25"
+		)
+		(pin "29"
+		)
+		(pin "32"
+		)
+		(pin "37"
+		)
+		(pin "4"
+		)
+		(pin "3"
+		)
+		(pin "31"
+		)
+		(pin "23"
+		)
+		(pin "15"
+		)
+		(pin "39"
+		)
+		(pin "2"
+		)
+		(pin "1"
+		)
+		(pin "40"
+		)
+		(pin "21"
+		)
+		(pin "19"
+		)
+		(pin "34"
+		)
+		(pin "20"
+		)
+		(pin "7"
+		)
+		(pin "6"
+		)
+		(pin "5"
+		)
+		(pin "28"
+		)
+		(pin "8"
+		)
+		(pin "14"
+		)
+		(pin "27"
+		)
+		(pin "13"
+		)
+		(pin "17"
+		)
+		(pin "12"
+		)
+		(pin "11"
+		)
+		(pin "9"
+		)
+		(pin "30"
+		)
+		(pin "10"
+		)
+		(pin "36"
+		)
+		(instances
+			(project ""
+				(path "/553a23ec-442a-4f98-939d-2d5634a662f5"
+					(reference "J3")
+					(unit 1)
+				)

Commit message: ribbon cable connection added
Parts:
- removed J3: Conn_01x40, symbol Connector_Generic:Conn_01x40
Connections:
- net Lap Signal renamed Lap_Signal
- net Launch Control Signal renamed Launch_Control_Signal
Other:
- added sheet Ribbon Cable Connector (ribboncable.kicad_sch)
- sheet MCU ports: added Drive_Mode_Encoder[0..1], Regen_Encoder[0..1], TC_Encoder[0..1]; removed Drive_Mode_Encoder[0..2], Regen_Encoder[0..2], TC_Encoder[0..2]
- note added: "Out"
- note added: "Primary connector will be the pigtail connector that connects the steering wheel to the rest of the car Needs to be something strong and waterproof and there needs to be enough slack in the cable for the wheel to be able to be taken off and put to the side The cable should be coiled so the extra slack doesn't get in the way while driving"
- note removed: "TODO: add in ribbon cable connections"
- note removed: "TODO: add part number of specific ribbon cable connector we'll use verify correct pitch, try to get one with both top and bottom contacts to make assembly easier"
- moved on the sheet: C1, C2, C3, C4, C5, C6, C7, L1, U1, U2, U3

Commit message: started work on dial encoders
Parts:
- added J4, J5, J6: 2x3 Nanofit, symbol Connector:Conn_01x06_Pin
Connections:
- net +3V3: now also J4.1 (Pin_1), J5.1 (Pin_1), J6.1 (Pin_1)
- new net Mode_Dial0: J6.2 (Pin_2)
- new net Mode_Dial1: J6.3 (Pin_3)
- new net Mode_Dial2: J6.4 (Pin_4)
- new net Mode_Dial3: J6.5 (Pin_5)
- new net Regen_Dial0: J5.2 (Pin_2)
- new net Regen_Dial1: J5.3 (Pin_3)
- new net Regen_Dial2: J5.4 (Pin_4)
- new net Regen_Dial3: J5.5 (Pin_5)
- new net TC_Dial0: J4.2 (Pin_2)
- new net TC_Dial1: J4.3 (Pin_3)
- new net TC_Dial2: J4.4 (Pin_4)
- new net TC_Dial3: J4.5 (Pin_5)
- no-connect marks 0 -> 3
Other:
- note added: "Drive Mode Dial Connector"
- note added: "Regen Dial Connector"
- note added: "TC Dial Connector"
- note removed: "TODO Secondary Connector Internal connections for all the buttons TBD until we source specific encoders and buttons because I don't know how many pins we'll need"
