File: steering-wheel-board/bridgetek.kicad_sch (KiCad schematic)
At the start: 9 parts, among them U4 BT817Q

Commit message: MCU page of steering wheel schematic
Changed lines of the file:
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@@
-	(wire
-		(pts
-			(xy 149.86 168.91) (xy 86.36 168.91)
-		)
-		(stroke
-			(width 0)
-			(type default)
-		)
-	)
 	(wire
 		(pts
@@
 		(pts
 			(xy 217.17 214.63) (xy 270.51 214.63)
+		)
+		(stroke
+			(width 0)
+			(type default)
+		)
+	)
+	(wire
+		(pts
+			(xy 217.17 220.98) (xy 270.51 220.98)
 		)
 		(stroke
@@
 	)
 	(label "Driver_Interrupt"
-		(at 107.95 168.91 0)
-		(effects
-			(font
-				(size 1.27 1.27)
-			)
-			(justify left bottom)
+		(at 236.22 220.98 180)
+		(effects
+			(font
+				(size 1.27 1.27)
+			)
+			(justify right bottom)
 		)
 	)
@@
 	(hierarchical_label "Driver_Interrupt"
 		(shape tri_state)
-		(at 86.36 168.91 180)
-		(effects
-			(font
-				(size 1.27 1.27)
-			)
-			(justify right)
-		)
-	)
+		(at 270.51 220.98 0)
+		(effects
+			(font
+				(size 1.27 1.27)
+			)
+			(justify left)
+		)
+	)

Commit message: added some notes
Other:
- note added: "Possible TODO: explore possibility of using flash memory or audio in future revisions talk to firmware to determine if we'll do this"
- note added: "TODO: clean this up it looks like shit"
Changed lines of the file:
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@@
 		(comment 6 "Display Driver")
+	)
+	(text "Possible TODO: explore possibility of \nusing flash memory or audio in future revisions\ntalk to firmware to determine if we'll do this"
+		(exclude_from_sim no)
+		(at 90.424 229.362 0)
+		(effects
+			(font
+				(size 1.27 1.27)
+			)
+		)
+	)
+	(text "TODO:\nclean this up it looks like shit"
+		(exclude_from_sim no)
+		(at 162.56 72.644 0)
+		(effects
+			(font
+				(size 1.27 1.27)
+			)
+		)
 	)
 	(junction

Commit message: ribbon cable connection added
Other:
- note added: "All filtering capacitor values are taken from BT817Q datasheet"
- note removed: "TODO: clean this up it looks like shit"
- moved on the sheet: C10, C11, C12, C13, C14, C15, C8, C9, U4

Commit message: page numbers added to datasheet references
Other:
- note added: "Note: using single SPI because firmware has decided that SPI data rate is not the primary performance bottleneck and the QSPI compatible STM32 is much larger see https://fsae.slack.com/archives/C07NHPGM5EE/p1766291511492069"
Changed lines of the file:
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@@
+		)
+	)
+	(text "Note: using single SPI\nbecause firmware has decided that \nSPI data rate is not  the primary performance bottleneck\nand the QSPI compatible STM32 is much larger\nsee \nhttps://fsae.slack.com/archives/C07NHPGM5EE/p1766291511492069 "
+		(exclude_from_sim no)
+		(at 28.702 113.284 0)
+		(effects
+			(font
+				(size 1.27 1.27)
+			)
+			(justify left)
 		)
 	)

Commit message: encoders added to steering wheel schematic
Changed lines of the file:
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@@
 	)
 	(junction
-		(at 212.09 85.09)
-		(diameter 0)
-		(color 0 0 0 0)
-	)
-	(junction
 		(at 212.09 185.42)
 		(diameter 0)
@@
 	(wire
 		(pts
-			(xy 212.09 85.09) (xy 212.09 92.71)
-		)
-		(stroke
-			(width 0)
-			(type default)
-		)
-	)
-	(wire
-		(pts
 			(xy 243.84 113.03) (xy 275.59 113.03)
 		)
@@
 	(wire
 		(pts
-			(xy 212.09 69.85) (xy 212.09 85.09)
+			(xy 212.09 69.85) (xy 212.09 92.71)
 		)
 		(stroke
@@
 					(unit 1)
 				)
-			)
-		)
-	)
-	(symbol
-		(lib_id "power:PWR_FLAG")
-		(at 212.09 85.09 90)
-		(unit 1)
-		(exclude_from_sim no)
-		(in_bom yes)
-		(on_board yes)
-		(dnp no)
-		(property "Reference" "#FLG03"
-			(at 210.185 85.09 0)
-			(effects
-				(font
-					(size 1.27 1.27)
-				)
-				(hide yes)
-			)
-		)
-		(property "Value" "PWR_FLAG"
-			(at 208.28 85.0899 90)
-			(effects
-				(font
-					(size 1.27 1.27)
-				)
-				(justify left)
-			)
-		)
-		(property "Footprint" ""
-			(at 212.09 85.09 0)
-			(effects
-				(font
-					(size 1.27 1.27)
-				)
-				(hide yes)
-			)
-		)
-		(property "Datasheet" "~"
-			(at 212.09 85.09 0)
-			(effects
-				(font
-					(size 1.27 1.27)
-				)
-				(hide yes)
-			)
-		)
-		(property "Description" "Special symbol for telling ERC where power comes from"
-			(at 212.09 85.09 0)
-			(effects
-				(font
-					(size 1.27 1.27)
-				)
-				(hide yes)
-			)
-		)
-		(pin "1"
-		)
-		(instances
-			(project ""
-				(path "/553a23ec-442a-4f98-939d-2d5634a662f5/abdb237b-4b87-473b-94a9-df050f5c08e4"
-					(reference "#FLG03")
-					(unit 1)
-				)

Commit message: added notes
Other:
- note added: "TODO: double check voltage and temp ratings against Bridgetek datasheet"
Changed lines of the file:
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@@
 	(title_block
 		(title "Steering Wheel Board")
-		(date "2026-01-07")
+		(date "2026-01-11")
 		(rev "1.0")
 		(company "Formula Slug")
@@
 		(comment 6 "Display Driver")
 	)
+	(text "TODO: double check voltage and temp ratings against Bridgetek datasheet\n"
+		(exclude_from_sim no)
+		(at 160.02 43.434 0)
+		(effects
+			(font
+				(size 1.27 1.27)
+			)
+		)
+	)
 	(text "All filtering capacitor values are taken from BT817Q datasheet"
