File: steering-wheel-board/ribboncable.kicad_sch (KiCad schematic)
At the start: 1 part, among them J3 Conn_01x40

Commit message: page numbers added to datasheet references
Other:
- note added: "Pin assignments given on page 5 of Crystalfontz CFAF800480H0-043Sx datasheet"
Changed lines of the file:
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@@
 		(comment 6 "Ribbon Cable Connector")
+	)
+	(text "Pin assignments given on page 5 of Crystalfontz\nCFAF800480H0-043Sx datasheet"
+		(exclude_from_sim no)
+		(at 258.826 108.458 0)
+		(effects
+			(font
+				(size 1.27 1.27)
+			)
+		)
 	)
 	(text "Pins 37-40 are resistive touch pins \nUnused for our application"

Commit message: encoders added to steering wheel schematic
Parts:
- J3: footprint (none) -> FS_4_Footprint_Library:CONN_F32D-1A7Y1-21040_AMP; symbol Connector_Generic:Conn_01x40 -> Connector_Generic_MountingPin:Conn_01x40_MountingPin; Digikey Link (none) -> https://www.digikey.com/en/products/detail/amphenol-cs-fci/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; Digikey Part Number (none) -> 609-F32D-1A7Y1-21040CT-ND; Manufacturer Part Number (none) -> F32D-1A7Y1-21040; Name (none) -> F32D-1A7Y1-21040 40 Pin ZIF Connector
Connections:
- no-connect marks 5 -> 6
Other:
- note removed: "TODO: add part number of specific ribbon cable connector we'll use verify correct pitch, try to get one with both top and bottom contacts to make assembly easier"
Changed lines of the file:
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@@
 		)
 	)
-	(text "TODO: add part number of \nspecific ribbon cable connector we'll use\nverify correct pitch, \ntry to get one with both top\nand bottom contacts to make assembly easier"
-		(exclude_from_sim no)
-		(at 223.012 136.652 0)
-		(effects
-			(font
-				(size 1.27 1.27)
-			)
-			(justify left)
-		)
+	(no_connect
+		(at 217.17 213.36)
 	)
 	(no_connect
@@
 	)
 	(symbol
-		(lib_id "Connector_Generic:Conn_01x40")
+		(lib_id "Connector_Generic_MountingPin:Conn_01x40_MountingPin")
 		(at 217.17 157.48 0)
 		(unit 1)
@@
 		(fields_autoplaced yes)
 		(property "Reference" "J3"
-			(at 219.71 157.4799 0)
+			(at 219.71 157.8355 0)
 			(effects
 				(font
@@
 		)
 		(property "Value" "Conn_01x40"
-			(at 219.71 160.0199 0)
+			(at 219.71 160.3755 0)
 			(effects
 				(font
@@
 			)
 		)
-		(property "Footprint" ""
+		(property "Footprint" "FS_4_Footprint_Library:CONN_F32D-1A7Y1-21040_AMP"
 			(at 217.17 157.48 0)
 			(effects
@@
 			)
 		)
-		(property "Description" "Generic connector, single row, 01x40, script generated (kicad-library-utils/schlib/autogen/connector/)"
+		(property "Description" "Generic connectable mounting pin connector, single row, 01x40, script generated (kicad-library-utils/schlib/autogen/connector/)"
 			(at 217.17 157.48 0)
 			(effects
@@
 			)
 		)
+		(property "Digikey Part Number" "609-F32D-1A7Y1-21040CT-ND"
+			(at 217.17 157.48 0)
+			(effects
+				(font
+					(size 1.27 1.27)
+				)
+				(hide yes)
+			)
+		)
+		(property "Name" "F32D-1A7Y1-21040 40 Pin ZIF Connector"
+			(at 217.17 157.48 0)
+			(effects
+				(font
+					(size 1.27 1.27)
+				)
+				(hide yes)
+			)
+		)
+		(property "Digikey Link" "https://www.digikey.com/en/products/detail/amphenol-cs-fci/F32D-1A7Y1-21040/11564657"
+			(at 217.17 157.48 0)
+			(effects
+				(font
+					(size 1.27 1.27)
+				)
+				(hide yes)
+			)
+		)
+		(property "Manufacturer Part Number" "F32D-1A7Y1-21040"
+			(at 217.17 157.48 0)
+			(effects
+				(font
+					(size 1.27 1.27)
+				)
+				(hide yes)
+			)
+		)
 		(pin "38"
 		)
@@
 		(pin "36"
 		)
+		(pin "MP"
+		)
 		(instances

Commit message: formatting changes, updated resistor ladder and CAN termination/aux can jumper
Parts:
- removed J3: Conn_01x40, FS_4_Footprint_Library:CONN_F32D-1A7Y1-21040_AMP, symbol Connector_Generic_MountingPin:Conn_01x40_MountingPin
Connections:
- no-connect marks 6 -> 0
Other:
- note removed: "Pin assignments given on page 5 of Crystalfontz CFAF800480H0-043Sx datasheet"
- note removed: "Pins 37-40 are resistive touch pins Unused for our application"
