File: steering-wheel-board/switches.kicad_sch (KiCad schematic)
At the start: 15 parts, among them SW2 SW_SPST, SW3 SW_SPST, SW4 SW_SPST

Commit message: formatting changes, updated resistor ladder and CAN termination/aux can jumper
Parts:
- removed R8: 100k, symbol Device:R
Connections:
- net Analog_0V83 is gone; now on net GND: R7.2, S1.4 (NO_3), S2.4 (NO_3), S3.4 (NO_3)
- net Analog_1V65 renamed Analog_1V1
- net Analog_2V5 renamed Analog_2V2
Other:
- note added: "Buttons"
- note added: "NOTE: filtering and pulldowns for Lap and launch are on VCU"
- note added: "Rotary Dials PCB mount 4-position rotary switches Using a resistor divider to read dial position as analog signal"
- note added: "V = (1/3)*3.3 = 1.1V"
- note added: "V = (2/3)*3.3 = 2.2V"
- note removed: "Rotary Dials PCB mount dials Using a resistor divider to read dial position as analog signal"
- note removed: "V = (1/4)*3.3 = ~0.825V"
- note removed: "V = (2/4)*3.3 = ~1.65V"
- note removed: "V = (3/4)*3.3 = ~2.5V"
- moved on the sheet: C26, R10, R17, R4, R5, R6, R7, R9, S1, S2, S3, SW2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

Commit message: added footprints and digikey info for all components other than pushbuttons
Parts:
- removed R10, R9: 10k, symbol Device:R
- added R3: 100k, Resistor_SMD:R_0603_1608Metric, symbol Device:R
- added R8: 10k, Resistor_SMD:R_0603_1608Metric, symbol Device:R
- C26: footprint (none) -> Capacitor_SMD:C_0603_1608Metric; Digikey Link (none) -> https://www.digikey.com/en/products/detail/samsung-electro-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; Digikey Part Number (none) -> 1276-1946-1-ND; Manufacturer (none) -> Samsung Electro-Mechanics; Manufacturer Part Number (none) -> CL10B105KP8NNNC; Name (none) -> CL10B105KP8NNNC
- R17: footprint (none) -> Resistor_SMD:R_0603_1608Metric; Digikey Link (none) -> https://www.digikey.com/en/products/detail/stackpole-electr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; Digikey Part Number (none) -> RMCF0603FT3K00CT-ND; Manufacturer (none) -> Stackpole Electronics Inc; Manufacturer Part Number (none) -> RMCF0603FT3K00; Name (none) -> RMCF0603FT3K00CT-ND
- R4: footprint (none) -> Resistor_SMD:R_0603_1608Metric; Digikey Link (none) -> https://www.digikey.com/en/products/detail/yageo/RC0603FR-0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; Digikey Part Number (none) -> 311-10.0KHRCT-ND; Manufacturer (none) -> YAGEO; Manufacturer Part Number (none) -> RC0603FR-0710KL; Name (none) -> Resistor
- R5, R6: footprint (none) -> Resistor_SMD:R_0603_1608Metric; Digikey Link (none) -> https://www.digikey.com/en/products/detail/stackpole-electr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; Digikey Part Number (none) -> RMCF0603FT100KCT-ND; Manufacturer (none) -> Stackpole Electronics Inc; Manufacturer Part Number (none) -> RMCF0603FT100K; Name (none) -> Resistor
- R7: value 100k -> 10k; footprint (none) -> Resistor_SMD:R_0603_1608Metric; Digikey Link (none) -> https://www.digikey.com/en/products/detail/yageo/RC0603FR-0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; Digikey Part Number (none) -> 311-10.0KHRCT-ND; Manufacturer (none) -> YAGEO; Manufacturer Part Number (none) -> RC0603FR-0710KL; Name (none) -> Resistor
- S1, S2, S3: Digikey Link (none) -> https://www.digikey.com/en/products/detail/e-switch/KC14A10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; Digikey Part Number (none) -> KC14A10.001NPS-ND; Height 32.2 -> (none); Manufacturer (none) -> E-Switch; Manufacturer Part Number (none) -> KC14A10.001NPS; Manufacturer_Name E-Switch -> (none); Manufacturer_Part_Number KC14A10.001NPS -> (none); Mouser Part Number 612-KC14A10.001NPS -> (none); Mouser Price/Stock https://www.mouser.co.uk/ProductDetail/E-Switch/KC14A10.001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 -> (none); Name (none) -> Rotary Switch
Connections:
- net Analog_1V1: now also R6.1, R3.2; no longer R6.2, R7.1
- net Analog_2V2: now also R3.1; no longer R6.1
- net GND: now also R6.2, R8.2
- net Launch_Control: now also R7.1
- net Layout_Cycle_Unfiltered: now also R8.1

Commit message: backup to make sure nothing breaks
Parts:
- SW3, SW4: now left out of the parts list
Other:
- note added: "Buttons are panel mount and connect to the board externally"
Changed lines of the file:
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@@
 		)
 	)
+	(text "Buttons are panel mount and connect to the board\nexternally"
+		(exclude_from_sim no)
+		(at 102.616 200.152 0)
+		(effects
+			(font
+				(size 1.27 1.27)
+			)
+			(justify left)
+		)
+	)
 	(text "V = (2/3)*3.3 = 2.2V"
 		(exclude_from_sim no)
@@
 		(unit 1)
 		(exclude_from_sim no)
-		(in_bom yes)
-		(on_board yes)
+		(in_bom no)
+		(on_board no)
 		(dnp no)
 		(fields_autoplaced yes)
@@
 			)
 		)
+		(property "Digikey Part Number" ""
+			(at 49.53 181.61 0)
+			(effects
+				(font
+					(size 1.27 1.27)
+				)
+				(hide yes)
+			)
+		)
+		(property "Digikey Link" ""
+			(at 49.53 181.61 0)
+			(effects
+				(font
+					(size 1.27 1.27)
+				)
+				(hide yes)
+			)
+		)
+		(property "Manufacturer Part Number" ""
+			(at 49.53 181.61 0)
+			(effects
+				(font
+					(size 1.27 1.27)
+				)
+				(hide yes)
+			)
+		)
+		(property "Manufacturer" ""
+			(at 49.53 181.61 0)
+			(effects
+				(font
+					(size 1.27 1.27)
+				)
+				(hide yes)
+			)
+		)
 		(pin "2"
 		)
@@
 		(unit 1)
 		(exclude_from_sim no)
-		(in_bom yes)
-		(on_board yes)
+		(in_bom no)
+		(on_board no)
 		(dnp no)
 		(fields_autoplaced yes)
@@
 			(at 46.99 207.01 0)
 			(effects
+				(font
+					(size 1.27 1.27)
+				)
+				(hide yes)
+			)
+		)
+		(property "Digikey Part Number" ""
+			(at 46.99 207.01 0)
+			(effects
+				(font
+					(size 1.27 1.27)
+				)
+				(hide yes)
+			)
+		)
+		(property "Digikey Link" ""
+			(at 46.99 207.01 0)
+			(effects
+				(font
+					(size 1.27 1.27)
+				)
+				(hide yes)
+			)
+		)
+		(property "Manufacturer Part Number" ""
+			(at 46.99 207.01 0)
+			(effects
+				(font
+					(size 1.27 1.27)
+				)
+				(hide yes)
+			)
+		)
+		(property "Manufacturer" ""
+			(at 46.99 207.01 0)
+			(effects

Commit message: updated symbol fields
Parts:
- C26: Digi PN (none) -> 1276-1946-1-ND; Digi URL (none) -> https://www.digikey.com/en/products/detail/samsung-electro-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; Digikey Link https://www.digikey.com/en/products/detail/samsung-electro-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 -> (none); Digikey Part Number 1276-1946-1-ND -> (none); MFG (none) -> Samsung Electro-Mechanics; MFG PN (none) -> CL10B105KP8NNNC; Manufacturer Samsung Electro-Mechanics -> (none); Manufacturer Part Number CL10B105KP8NNNC -> (none)
- R17: Digi PN (none) -> RMCF0603FT3K00CT-ND; Digi URL (none) -> https://www.digikey.com/en/products/detail/stackpole-electr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; Digikey Link https://www.digikey.com/en/products/detail/stackpole-electr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 -> (none); Digikey Part Number RMCF0603FT3K00CT-ND -> (none); MFG (none) -> Stackpole Electronics Inc; MFG PN (none) -> RMCF0603FT3K00; Manufacturer Stackpole Electronics Inc -> (none); Manufacturer Part Number RMCF0603FT3K00 -> (none)
- R3, R5, R6: Digi PN (none) -> RMCF0603FT100KCT-ND; Digi URL (none) -> https://www.digikey.com/en/products/detail/stackpole-electr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; Digikey Link https://www.digikey.com/en/products/detail/stackpole-electr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 -> (none); Digikey Part Number RMCF0603FT100KCT-ND -> (none); MFG (none) -> Stackpole Electronics Inc; MFG PN (none) -> RMCF0603FT100K; Manufacturer Stackpole Electronics Inc -> (none); Manufacturer Part Number RMCF0603FT100K -> (none)
- R4, R7, R8: Digi PN (none) -> 311-10.0KHRCT-ND; Digi URL (none) -> https://www.digikey.com/en/products/detail/yageo/RC0603FR-0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; Digikey Link https://www.digikey.com/en/products/detail/yageo/RC0603FR-0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 -> (none); Digikey Part Number 311-10.0KHRCT-ND -> (none); MFG (none) -> YAGEO; MFG PN (none) -> RC0603FR-0710KL; Manufacturer YAGEO -> (none); Manufacturer Part Number RC0603FR-0710KL -> (none)
- S1, S2, S3: Digi PN (none) -> KC14A10.001NPS-ND; Digi URL (none) -> https://www.digikey.com/en/products/detail/e-switch/KC14A10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; Digikey Link https://www.digikey.com/en/products/detail/e-switch/KC14A10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 -> (none); Digikey Part Number KC14A10.001NPS-ND -> (none); MFG (none) -> E-Switch; MFG PN (none) -> KC14A10.001NPS; Manufacturer E-Switch -> (none); Manufacturer Part Number KC14A10.001NPS -> (none)

Commit message: added nanofits for buttons
Other:
- note added: "Analog_GND"
- moved on the sheet: C26, R17, R3, R4, R5, R6, R7, R8, S1, S2, S3, SW2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

Commit message: fixed symbol library names
Parts:
- removed S2, S3: KC14A10.001NPS, FS_4_Footprint_Library:KC14A10001NPS, symbol FS_4_Global_Schematics_Library:KC14A10.001NPS
- added S2, S3: KC14A10.001NPS, FS_4_Global_Footprint_Library:KC14A10001NPS, symbol FS_4_Global_Symbol_Library:KC14A10.001NPS
- S1: footprint FS_4_Footprint_Library:KC14A10001NPS -> FS_4_Global_Footprint_Library:KC14A10001NPS; symbol FS_4_Global_Schematics_Library:KC14A10.001NPS -> FS_4_Global_Symbol_Library:KC14A10.001NPS; Height (none) -> 32.2; Manufacturer_Name (none) -> E-Switch; Manufacturer_Part_Number (none) -> KC14A10.001NPS; Mouser Part Number (none) -> 612-KC14A10.001NPS; Mouser Price/Stock (none) -> https://www.mouser.co.uk/ProductDetail/E-Switch/KC14A10.001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
Connections:
- net +3V3: now also S2.1 (NC), S3.1 (NC)
- net Analog_1V1: now also S2.3 (NO_2), S3.3 (NO_2)
- net Analog_2V2: now also S2.2 (NO_1), S3.2 (NO_1)
- net GND: now also S2.4 (NO_3), S3.4 (NO_3)
- net Mode_Analog: now also S2.10 (A_-_COM)
- net Regen_Analog: now also S3.10 (A_-_COM)

Commit message: added digikey part information for pushbuttons
Parts:
- removed SW3, SW4: SW_SPST, symbol Switch:SW_SPST
- added SW3, SW4: SW_SPST, symbol Switch:SW_Push
- SW2: symbol Switch:SW_SPST -> Switch:SW_Push; Digi PN (none) -> EG2025-ND; Digi URL (none) -> https://www.digikey.com/en/products/detail/e-switch/ps1024a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; MFG (none) -> E-Switch; MFG PN (none) -> PS1024ALRED
Connections:
- net +3V3: now also SW3.1, SW4.1
- net Lap: now also SW3.2
- net Launch_Control: now also SW4.2
Other:
- note removed: "Lap button part TBD normally open board mount momentary on"
- note removed: "Launch control button part TBD normally open board mount momentary on"
- note removed: "Layout cycle button exact part TBD some sort of board mount normally open button"

Commit message: - changed 47u and 10u caps for DCDC to 0805 per Cole's request - added low pass filters to rotary switches - changed rotary switch symbols per Cole's request - made panel mount button symbols DNP - removed the CAN termination stuff that Sam said wouldn't work - set junction size to default per Wesley's request - minor styling/readability fixes
Parts:
- removed S2, S3: KC14A10.001NPS, FS_4_Global_Footprint_Library:KC14A10001NPS, symbol FS_4_Global_Symbol_Library:KC14A10.001NPS
- added C27, C28, C29: 68n, Capacitor_SMD:C_0603_1608Metric, symbol Device:C
- added R10, R12, R9: 11k, Resistor_SMD:R_0603_1608Metric, symbol Device:R
- added S2, S3: KC14A10.001NPS, FS_4_Global_Footprint_Library:KC14A10001NPS, symbol Switch:SW_Rotary_1x4_MP
- S1: symbol FS_4_Global_Symbol_Library:KC14A10.001NPS -> Switch:SW_Rotary_1x4_MP; Height 32.2 -> (none); Manufacturer_Name E-Switch -> (none); Manufacturer_Part_Number KC14A10.001NPS -> (none); Mouser Part Number 612-KC14A10.001NPS -> (none); Mouser Price/Stock https://www.mouser.co.uk/ProductDetail/E-Switch/KC14A10.001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 -> (none)
- SW2, SW3, SW4: now not fitted
Connections:
- net +3V3: now also S2.1, S3.1
- net Analog_1V1: now also S2.3, S3.3
- net Analog_2V2: now also S2.2, S3.2
- net GND: now also C27.2, C28.2, C29.2, S2.4, S3.4
- net Mode_Analog: now also C28.1, R10.2
- net Regen_Analog: now also C29.1, R12.2
- net TC_Analog: now also C27.1, R9.2; no longer S1.10 (A_-_COM)
- new net Mode_Unfiltered: R10.1, S2.5
- new net Regen_Unfiltered: R12.1, S3.5
- new net TC_Unfiltered: R9.1, S1.5
Other:
- note added: "11k resistor and 68n cap: cutoff freq. = 1/2piRC = 1/((2pi)(11k)(68n)) = 212 Hz cutoff"
- note added: "3k resistor and 1u cap cutoff freq = 1/2piRC = 1/((2pi)(3k)(1u)) = 53 Hz cutoff"
- note removed: "3k resistor and 1u cap = 53 Hz cutoff"
- moved on the sheet: C26, R17, R3, R4, R5, R6, R7, R8
