File: steering-wheel-board/MCU.kicad_sch (KiCad schematic)
At the start: 15 parts, among them J2 FTSH-107-01-F-DV-K-P-TR, SW1 Y97KT23B5NAFP, U5 STM32G441KBTx, Y1 ECS-240-8-37B-CKY-TR

Commit message: revised steering wheel board schematic to address PR comments; replaced encoders with resistor ladders for dials, and added dials into schematic
Parts:
- added C6, C7: 100nF, Capacitor_SMD:C_0805_2012Metric_Pad1.18x1.45mm_HandSolder, symbol Device:C
- added U3: ISO1044BD, Package_SO:SOIC-8_3.9x4.9mm_P1.27mm, symbol Interface_CAN_LIN:ISO1044BD
Connections:
- net +3V3: now also C7.1, U3.1 (VCC1)
- net CAN_RX: now also U3.3 (RXD)
- net CAN_TX: now also U3.2 (TXD)
- net GND: now also C6.2, C7.2, U3.4 (GND1), U3.7 (GND2)
- net Layout_Cycle: now also U5.27 (PB4); no longer U5.13 (PB0)
- net Drive_Mode_Encoder0 renamed Regen_Analog
- net Drive_Mode_Encoder1 renamed Mode_Analog
- net Regen_Encoder0: no longer names the net of U5.19 (PA9)
- net Regen_Encoder1: no longer names the net of U5.20 (PA10)
- net TC_Encoder0: no longer names the net of U5.28 (PB5)
- net TC_Encoder1: no longer names the net of U5.29 (PB6)
- new net +5V: C6.1, U3.8 (VCC2)
- new net CAN_H: U3.6 (CANH)
- new net CAN_L: U3.5 (CANL)
- new net TC_Analog: U5.13 (PB0)
- no-connect marks 6 -> 9
Other:
- note added: "CAN"
- moved on the sheet: C16, C17, C18, C19, C20, C21, C22, C23, FB1, J2, R1, R2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

Commit message: added footprints and digikey info for all components other than pushbuttons
Parts:
- C16, C17: Digi PN 311-3874-1-ND -> (none); Digi URL https://www.digikey.com/en/products/detail/yageo/CC0603DRNP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 -> (none); Digikey Link (none) -> https://www.digikey.com/en/products/detail/yageo/CC0603DRNP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; Digikey Part Number (none) -> 311-3874-1-ND; MFG Yageo -> (none); MFG PN CC0603DRNPO9BN6R8 -> (none); Manufacturer (none) -> Yageo; Manufacturer Part Number (none) -> CC0603DRNPO9BN6R8
- C18: value 100nF -> 100n; footprint Capacitor_SMD:C_0603_1608Metric_Pad1.08x0.95mm_HandSolder -> Capacitor_SMD:C_0603_1608Metric; Digi PN 311-1344-1-ND -> (none); Digi URL https://www.digikey.com/en/products/detail/yageo/CC0603KRX7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 -> (none); Digikey Link (none) -> https://www.digikey.com/en/products/detail/murata-electroni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; Digikey Part Number (none) -> 490-5798-1-ND; MFG Yageo -> (none); MFG PN CC0603KRX7R9BB104 -> (none); Manufacturer (none) -> Murata Electronics; Manufacturer Part Number (none) -> GCJ188R71H104KA12D
- C19: value 10uF -> 10u; Digi PN 1276-CL10A106KO8NQNCCT-ND -> (none); Digi URL https://www.digikey.com/en/products/detail/samsung-electro-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 -> (none); Digikey Link (none) -> https://www.digikey.com/en/products/detail/samsung-electro-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; Digikey Part Number (none) -> 1276-CL10A106KO8NQNCCT-ND; MFG Samsung Electro-Mechanics -> (none); MFG PN CL10A106KO8NQNC -> (none); Manufacturer (none) -> Samsung Electro-Mechanics; Manufacturer Part Number (none) -> CL10A106KO8NQNC
- C20, C21: value 100nF -> 100n; Digi PN 311-1344-1-ND -> (none); Digi URL https://www.digikey.com/en/products/detail/yageo/CC0603KRX7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 -> (none); Digikey Link (none) -> https://www.digikey.com/en/products/detail/yageo/CC0603KRX7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; Digikey Part Number (none) -> 311-1344-1-ND; MFG Yageo -> (none); MFG PN CC0603KRX7R9BB104 -> (none); Manufacturer (none) -> Yageo; Manufacturer Part Number (none) -> CC0603KRX7R9BB104
- C22: value 1uF -> 1u; Digi PN 1276-CL10B105KB9VPJCCT-ND -> (none); Digi URL https://www.digikey.com/en/products/detail/samsung-electro-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 -> (none); Digikey Link (none) -> https://www.digikey.com/en/products/detail/samsung-electro-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; Digikey Part Number (none) -> 1276-CL10B105KB9VPJCCT-ND; MFG Samsung Electro-Mechanics -> (none); MFG PN CL10B105KB9VPJC -> (none); Manufacturer (none) -> Samsung Electro-Mechanics; Manufacturer Part Number (none) -> CL10B105KB9VPJC
- C23: Digi PN 311-1344-1-ND -> (none); Digi URL https://www.digikey.com/en/products/detail/yageo/CC0603KRX7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 -> (none); Digikey Link (none) -> https://www.digikey.com/en/products/detail/yageo/CC0603KRX7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; Digikey Part Number (none) -> 311-1344-1-ND; MFG Yageo -> (none); MFG PN CC0603KRX7R9BB104 -> (none); Manufacturer (none) -> Yageo; Manufacturer Part Number (none) -> CC0603KRX7R9BB104
- C6, C7: value 100nF -> 100n; footprint Capacitor_SMD:C_0805_2012Metric_Pad1.18x1.45mm_HandSolder -> Capacitor_SMD:C_0603_1608Metric; Digi PN 311-1140-1-ND -> (none); Digikey Link (none) -> https://www.digikey.com/en/products/detail/murata-electroni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; Digikey Part Number (none) -> 490-5798-1-ND; MFG Yageo -> (none); MFG PN CC0805KRX7R9BB104 -> (none); Manufacturer (none) -> Murata Electronics; Manufacturer Part Number (none) -> GCJ188R71H104KA12D
- FB1: Digi PN 4816-FCM1608KF-601T03CT-ND -> (none); Digi URL https://www.digikey.com/en/products/detail/tai-tech-advance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 -> (none); Digikey Link (none) -> https://www.digikey.com/en/products/detail/tai-tech-advance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; Digikey Part Number (none) -> 4816-FCM1608KF-601T03CT-ND; MFG TAI-TECH Advanced Electronics Co., Ltd. -> (none); MFG PN FCM 1608KF-601T03 -> (none); Manufacturer (none) -> TAI-TECH Advanced Electronics Co., Ltd.; Manufacturer Part Number (none) -> FCM 1608KF-601T03
- J2: Digi PN SAM13170CT-ND -> (none); Digi URL https://www.digikey.com/en/products/detail/samtec-inc/FTSH-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 -> (none); Digikey Link (none) -> https://www.digikey.com/en/products/detail/samtec-inc/FTSH-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; Digikey Part Number (none) -> SAM13170CT-ND; MFG Samtec Inc. -> (none); MFG PN FTSH-107-01-F-DV-K-P-TR -> (none); Manufacturer (none) -> Samtec Inc.; Manufacturer Part Number (none) -> FTSH-107-01-F-DV-K-P-TR
- R1: footprint Resistor_SMD:R_0603_1608Metric_Pad0.98x0.95mm_HandSolder -> Resistor_SMD:R_0603_1608Metric; Digi PN 311-10KLDCT-ND -> (none); Digi URL https://www.digikey.com/en/products/detail/yageo/AC0603FR-0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 -> (none); Digikey Link (none) -> https://www.digikey.com/en/products/detail/yageo/RC0603FR-0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; Digikey Part Number (none) -> 311-10.0KHRCT-ND; MFG Yageo -> (none); MFG PN AC0603FR-0710KL -> (none); Manufacturer (none) -> YAGEO; Manufacturer Part Number (none) -> RC0603FR-0710KL; Name (none) -> Resistor
- R2: footprint (none) -> Resistor_SMD:R_0603_1608Metric; Digikey Link (none) -> https://www.digikey.com/en/products/detail/yageo/RC0603FR-0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; Digikey Part Number (none) -> 311-4.70KHRCT-ND; Manufacturer (none) -> YAGEO; Manufacturer Part Number (none) -> RC0603FR-074K7L
- SW1: Digi PN 108-Y97KT23B5NAFPCT-ND -> (none); Digi URL https://www.digikey.com/en/products/detail/c-k/y97kt23b5naf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 -> (none); Digikey Link (none) -> https://www.digikey.com/en/products/detail/c-k/y97kt23b5naf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; Digikey Part Number (none) -> 108-Y97KT23B5NAFPCT-ND; MFG C&K -> (none); MFG PN Y97KT23B5NAFP -> (none); Manufacturer (none) -> C&K; Manufacturer Part Number (none) -> Y97KT23B5NAFP; Name (none) -> Push button switch, generic, two pins
- U3: Digi PN 296-ISO1044BDRCT-ND -> (none); Digikey Link (none) -> https://www.digikey.com/en/products/detail/texas-instrument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; Digikey Part Number (none) -> 296-ISO1044BDRCT-ND; MFG Texas Instruments -> (none); MFG PN ISO1044BDR -> (none); Manufacturer (none) -> Texas Instruments; Manufacturer Part Number (none) -> ISO1044BDR
- U5: Digi PN 497-STM32G441KBT6-ND -> (none); Digi URL https://www.digikey.com/en/products/detail/stmicroelectroni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 -> (none); Digikey Link (none) -> https://www.digikey.com/en/products/detail/stmicroelectroni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; Digikey Part Number (none) -> 497-STM32G441KBT6-ND; MFG STM -> (none); MFG PN STM32G441KBT6 -> (none); Manufacturer (none) -> STMicroelectronics; Manufacturer Part Number (none) -> STM32G441KBT6; Name (none) -> STM32G441KBT6
- Y1: Digi PN XC3063CT-ND -> (none); Digi URL https://www.digikey.com/en/products/detail/ecs-inc/ECS-240-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 -> (none); Digikey Link (none) -> https://www.digikey.com/en/products/detail/ecs-inc/ECS-240-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; Digikey Part Number (none) -> XC3063CT-ND; MFG ECS -> (none); MFG PN ECS-240-8-37B-CKY-TR -> (none); Manufacturer (none) -> ECS; Manufacturer Part Number (none) -> ECS-240-8-37B-CKY-TR; Name (none) -> Crystal

Commit message: updated symbol fields
Parts:
- C16, C17: Digi PN (none) -> 311-3874-1-ND; Digi URL (none) -> https://www.digikey.com/en/products/detail/yageo/CC0603DRNP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; Digikey Link https://www.digikey.com/en/products/detail/yageo/CC0603DRNP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 -> (none); Digikey Part Number 311-3874-1-ND -> (none); MFG (none) -> Yageo; MFG PN (none) -> CC0603DRNPO9BN6R8; Manufacturer Yageo -> (none); Manufacturer Part Number CC0603DRNPO9BN6R8 -> (none)
- C18, C6, C7: Digi PN (none) -> 490-5798-1-ND; Digi URL (none) -> https://www.digikey.com/en/products/detail/murata-electroni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; Digikey Link https://www.digikey.com/en/products/detail/murata-electroni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 -> (none); Digikey Part Number 490-5798-1-ND -> (none); MFG (none) -> Murata Electronics; MFG PN (none) -> GCJ188R71H104KA12D; Manufacturer Murata Electronics -> (none); Manufacturer Part Number GCJ188R71H104KA12D -> (none)
- C19: Digi PN (none) -> 1276-CL10A106KO8NQNCCT-ND; Digi URL (none) -> https://www.digikey.com/en/products/detail/samsung-electro-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; Digikey Link https://www.digikey.com/en/products/detail/samsung-electro-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 -> (none); Digikey Part Number 1276-CL10A106KO8NQNCCT-ND -> (none); MFG (none) -> Samsung Electro-Mechanics; MFG PN (none) -> CL10A106KO8NQNC; Manufacturer Samsung Electro-Mechanics -> (none); Manufacturer Part Number CL10A106KO8NQNC -> (none)
- C20, C21, C23: Digi PN (none) -> 311-1344-1-ND; Digi URL (none) -> https://www.digikey.com/en/products/detail/yageo/CC0603KRX7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; Digikey Link https://www.digikey.com/en/products/detail/yageo/CC0603KRX7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 -> (none); Digikey Part Number 311-1344-1-ND -> (none); MFG (none) -> Yageo; MFG PN (none) -> CC0603KRX7R9BB104; Manufacturer Yageo -> (none); Manufacturer Part Number CC0603KRX7R9BB104 -> (none)
- C22: Digi PN (none) -> 1276-CL10B105KB9VPJCCT-ND; Digi URL (none) -> https://www.digikey.com/en/products/detail/samsung-electro-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; Digikey Link https://www.digikey.com/en/products/detail/samsung-electro-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 -> (none); Digikey Part Number 1276-CL10B105KB9VPJCCT-ND -> (none); MFG (none) -> Samsung Electro-Mechanics; MFG PN (none) -> CL10B105KB9VPJC; Manufacturer Samsung Electro-Mechanics -> (none); Manufacturer Part Number CL10B105KB9VPJC -> (none)
- FB1: Digi PN (none) -> 4816-FCM1608KF-601T03CT-ND; Digi URL (none) -> https://www.digikey.com/en/products/detail/tai-tech-advance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; Digikey Link https://www.digikey.com/en/products/detail/tai-tech-advance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 -> (none); Digikey Part Number 4816-FCM1608KF-601T03CT-ND -> (none); MFG (none) -> TAI-TECH Advanced Electronics Co., Ltd.; MFG PN (none) -> FCM 1608KF-601T03; Manufacturer TAI-TECH Advanced Electronics Co., Ltd. -> (none); Manufacturer Part Number FCM 1608KF-601T03 -> (none)
- J2: Digi PN (none) -> SAM13170CT-ND; Digi URL (none) -> https://www.digikey.com/en/products/detail/samtec-inc/FTSH-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; Digikey Link https://www.digikey.com/en/products/detail/samtec-inc/FTSH-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 -> (none); Digikey Part Number SAM13170CT-ND -> (none); MFG (none) -> Samtec Inc.; MFG PN (none) -> FTSH-107-01-F-DV-K-P-TR; Manufacturer Samtec Inc. -> (none); Manufacturer Part Number FTSH-107-01-F-DV-K-P-TR -> (none)
- R1: Digi PN (none) -> 311-10.0KHRCT-ND; Digi URL (none) -> https://www.digikey.com/en/products/detail/yageo/RC0603FR-0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; Digikey Link https://www.digikey.com/en/products/detail/yageo/RC0603FR-0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 -> (none); Digikey Part Number 311-10.0KHRCT-ND -> (none); MFG (none) -> YAGEO; MFG PN (none) -> RC0603FR-0710KL; Manufacturer YAGEO -> (none); Manufacturer Part Number RC0603FR-0710KL -> (none)
- R2: Digi PN (none) -> 311-4.70KHRCT-ND; Digi URL (none) -> https://www.digikey.com/en/products/detail/yageo/RC0603FR-0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; Digikey Link https://www.digikey.com/en/products/detail/yageo/RC0603FR-0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 -> (none); Digikey Part Number 311-4.70KHRCT-ND -> (none); MFG (none) -> YAGEO; MFG PN (none) -> RC0603FR-074K7L; Manufacturer YAGEO -> (none); Manufacturer Part Number RC0603FR-074K7L -> (none)
- SW1: Digikey Link https://www.digikey.com/en/products/detail/c-k/y97kt23b5naf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 -> (none); Digikey Part Number 108-Y97KT23B5NAFPCT-ND -> (none); MFG PN (none) -> Y97KT23B5NAFP; Manufacturer C&K -> (none); Manufacturer Part Number Y97KT23B5NAFP -> (none)
- U3: Digi PN (none) -> 296-ISO1044BDRCT-ND; Digi URL (none) -> https://www.digikey.com/en/products/detail/texas-instrument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; Digikey Link https://www.digikey.com/en/products/detail/texas-instrument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 -> (none); Digikey Part Number 296-ISO1044BDRCT-ND -> (none); MFG (none) -> Texas Instruments; MFG PN (none) -> ISO1044BDR; Manufacturer Texas Instruments -> (none); Manufacturer Part Number ISO1044BDR -> (none)
- U5: Digi PN (none) -> 497-STM32G441KBT6-ND; Digi URL (none) -> https://www.digikey.com/en/products/detail/stmicroelectroni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; Digikey Link https://www.digikey.com/en/products/detail/stmicroelectroni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 -> (none); Digikey Part Number 497-STM32G441KBT6-ND -> (none); MFG (none) -> STMicroelectronics; MFG PN (none) -> STM32G441KBT6; Manufacturer STMicroelectronics -> (none); Manufacturer Part Number STM32G441KBT6 -> (none)
- Y1: Digi PN (none) -> XC3063CT-ND; Digi URL (none) -> https://www.digikey.com/en/products/detail/ecs-inc/ECS-240-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; Digikey Link https://www.digikey.com/en/products/detail/ecs-inc/ECS-240-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 -> (none); Digikey Part Number XC3063CT-ND -> (none); MFG (none) -> ECS; MFG PN (none) -> ECS-240-8-37B-CKY-TR; Manufacturer ECS -> (none); Manufacturer Part Number ECS-240-8-37B-CKY-TR -> (none)

Commit message: added nanofits for buttons
Other:
- note added: "GNDDETECT"
Changed lines of the file:
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@@
+		)
+	)
+	(text "GNDDETECT"
+		(exclude_from_sim no)
+		(at 158.496 138.176 0)
+		(effects
+			(font
+				(size 1.27 1.27)
+			)
+			(justify left bottom)
 		)
 	)
@@
 		(effects
 			(font
-				(size 1.27 1.27)
-			)
-			(justify left bottom)
-		)
-	)
-	(label "GNDDETECT"
-		(at 158.75 138.43 0)
-		(effects
-			(font

Commit message: - changed 47u and 10u caps for DCDC to 0805 per Cole's request - added low pass filters to rotary switches - changed rotary switch symbols per Cole's request - made panel mount button symbols DNP - removed the CAN termination stuff that Sam said wouldn't work - set junction size to default per Wesley's request - minor styling/readability fixes
Other:
- note added: "MCU"
- moved on the sheet: C6, C7, U3

Commit message: added test points to MCU, layout work
Parts:
- added TP1, TP2, TP3, TP4, TP5: TestPoint, TestPoint:TestPoint_Pad_1.0x1.0mm, symbol Connector:TestPoint
Connections:
- net at U5.18 (PA8): now also TP1.1
- net at U5.19 (PA9): now also TP2.1
- net at U5.20 (PA10): now also TP3.1
- net at U5.28 (PB5): now also TP4.1
- net at U5.29 (PB6): now also TP5.1
- no-connect marks 9 -> 4
