File: steering-wheel-board/steering_wheel.kicad_pcb (KiCad board)
At the start: 2 copper layers, 0 parts

Commit message: started pcb work
Parts:
- added C1: 10u, Capacitor_SMD:C_0805_2012Metric_Pad1.18x1.45mm_HandSolder, F.Cu at (-38.7, 6.73)
- added C10: 10u, Capacitor_SMD:C_0603_1608Metric, F.Cu at (-50.4, 2.77)
- added C11: 100n, Capacitor_SMD:C_0603_1608Metric, F.Cu at (-50.4, 5.29)
- added C12: 100n, Capacitor_SMD:C_0603_1608Metric, F.Cu at (-50.4, 7.79)
- added C13: 100n, Capacitor_SMD:C_0603_1608Metric, F.Cu at (-46.4, -2.25)
- added C14: 100n, Capacitor_SMD:C_0603_1608Metric, F.Cu at (-46.4, 0.27)
- added C15: 100n, Capacitor_SMD:C_0603_1608Metric, F.Cu at (-46.4, 2.77)
- added C16: 6.8pF, Capacitor_SMD:C_0603_1608Metric_Pad1.08x0.95mm_HandSolder, F.Cu at (133.9, 2.95)
- added C17: 6.8pF, Capacitor_SMD:C_0603_1608Metric_Pad1.08x0.95mm_HandSolder, F.Cu at (133.9, 5.46)
- added C18: 100n, Capacitor_SMD:C_0603_1608Metric, F.Cu at (138.1, 19.4)
- added C19: 10u, Capacitor_SMD:C_0603_1608Metric_Pad1.08x0.95mm_HandSolder, F.Cu at (133.9, 7.97)
- added C2: 100n, Capacitor_SMD:C_0603_1608Metric, F.Cu at (-39.1, 12.5)
- added C20: 100n, Capacitor_SMD:C_0603_1608Metric_Pad1.08x0.95mm_HandSolder, F.Cu at (133.9, 10.5)
- added C21: 100n, Capacitor_SMD:C_0603_1608Metric_Pad1.08x0.95mm_HandSolder, F.Cu at (133.9, 13.0)
- added C22: 1u, Capacitor_SMD:C_0603_1608Metric_Pad1.08x0.95mm_HandSolder, F.Cu at (133.9, 15.5)
- added C23: 100nF, Capacitor_SMD:C_0603_1608Metric_Pad1.08x0.95mm_HandSolder, F.Cu at (133.9, 18.0)
- added C24: 220n, Capacitor_SMD:C_0603_1608Metric, F.Cu at (-46.4, 5.29)
- added C25: 1u, Capacitor_SMD:C_0603_1608Metric, F.Cu at (-46.4, 7.79)
- added C26: 1u, Capacitor_SMD:C_0603_1608Metric, F.Cu at (131.3, 35.5)
- added C27: 68n, Capacitor_SMD:C_0603_1608Metric, F.Cu at (131.3, 38.0)
- added C28: 68n, Capacitor_SMD:C_0603_1608Metric, F.Cu at (131.3, 40.5)
- added C29: 68n, Capacitor_SMD:C_0603_1608Metric, F.Cu at (131.3, 43.0)
- added C3: 47u, Capacitor_SMD:C_0805_2012Metric_Pad1.18x1.45mm_HandSolder, F.Cu at (-38.7, 9.74)
- added C4: 1u, Capacitor_SMD:C_0603_1608Metric, F.Cu at (-39.1, 15.0)
- added C5: 1u, Capacitor_SMD:C_0603_1608Metric, F.Cu at (-39.1, 17.5)
- added C6: 100n, Capacitor_SMD:C_0603_1608Metric, F.Cu at (138.1, 14.4)
- added C7: 100n, Capacitor_SMD:C_0603_1608Metric, F.Cu at (138.1, 16.9)
- added C8: 100n, Capacitor_SMD:C_0603_1608Metric, F.Cu at (-50.4, -2.25)
- added C9: 1u, Capacitor_SMD:C_0603_1608Metric, F.Cu at (-50.4, 0.27)
- added FB1: FCM 1608KF-601T03, Inductor_SMD:L_0603_1608Metric_Pad1.05x0.95mm_HandSolder, F.Cu at (133.9, 20.5)
- added J1: Keystone 985 RJ45, FS_4_Global_Footprint_Library:Keystone_985, B.Cu at (50.1, 2.18)
- added J10: Test Pad, TestPoint:TestPoint_Plated_Hole_D2.0mm, F.Cu at (-54.8, -1.18)
- added J11: Test Pad, TestPoint:TestPoint_Plated_Hole_D2.0mm, F.Cu at (-54.8, 3.48)
- added J12: Test Pad, TestPoint:TestPoint_Plated_Hole_D2.0mm, F.Cu at (-54.8, 8.12)
- added J2: FTSH-107-01-F-DV-K-P-TR, Connector_PinHeader_1.27mm:PinHeader_2x07_P1.27mm_Vertical_SMD, F.Cu at (152.3, 7.17)
- added J3: Nanofit 01x02 Right Angle, FS_4_Global_Footprint_Library:Nanofit-1054301202-1x2SMD90Deg, F.Cu at (-39.0, 56.3)
- added J4: Conn_01x40, FS_4_Global_Footprint_Library:CONN_F32D-1A7Y1-21040_AMP, F.Cu at (78.2, 16.0)
- added J5: Nanofit 01x02 Right Angle, FS_4_Global_Footprint_Library:Nanofit-1054301202-1x2SMD90Deg, F.Cu at (-27.5, 56.3)
- added J6: Nanofit 01x02 Right Angle, FS_4_Global_Footprint_Library:Nanofit-1054301202-1x2SMD90Deg, F.Cu at (118.8, -9.98)
- added L1: 4.7uF, Inductor_SMD:L_Bourns_SRP5030T, F.Cu at (-29.5, 19.0)
- added L2: 22u, FS_4_Global_Footprint_Library:CDRH5D28NP-220NC, F.Cu at (-52.7, 22.8)
- added R1: 10k, Resistor_SMD:R_0603_1608Metric, F.Cu at (138.1, 21.9)
- added R10: 11k, Resistor_SMD:R_0603_1608Metric, F.Cu at (139.3, 38.0)
- added R11: 4.99, Resistor_SMD:R_1210_3225Metric, F.Cu at (-44.7, 26.8)
- added R12: 11k, Resistor_SMD:R_0603_1608Metric, F.Cu at (139.3, 40.5)
- added R17: 3k, Resistor_SMD:R_0603_1608Metric, F.Cu at (139.3, 43.0)
- added R18: 120, Resistor_SMD:R_0603_1608Metric, F.Cu at (-39.1, 20.0)
- added R2: 4.7k, Resistor_SMD:R_0603_1608Metric, F.Cu at (138.1, 24.4)
- added R3: 100k, Resistor_SMD:R_0603_1608Metric, F.Cu at (131.3, 45.5)
- added R4: 10k, Resistor_SMD:R_0603_1608Metric, F.Cu at (135.3, 35.5)
- added R5: 100k, Resistor_SMD:R_0603_1608Metric, F.Cu at (135.3, 38.0)
- added R6: 100k, Resistor_SMD:R_0603_1608Metric, F.Cu at (135.3, 40.5)
- added R7: 10k, Resistor_SMD:R_0603_1608Metric, F.Cu at (135.3, 43.0)
- added R8: 10k, Resistor_SMD:R_0603_1608Metric, F.Cu at (135.3, 45.5)
- added R9: 11k, Resistor_SMD:R_0603_1608Metric, F.Cu at (139.3, 35.5)
- added S1: KC14A10.001NPS, FS_4_Global_Footprint_Library:KC14A10001NPS, F.Cu at (2.03, 95.5)
- added S2: KC14A10.001NPS, FS_4_Global_Footprint_Library:KC14A10001NPS, F.Cu at (91.5, 101.5)
- added S3: KC14A10.001NPS, FS_4_Global_Footprint_Library:KC14A10001NPS, F.Cu at (49.5, 121.5)
- added SW1: Y97KT23B5NAFP, Button_Switch_SMD:SW_SPST_PTS647_Sx38, F.Cu at (152.8, 16.3)
- added U1: AP63205WU, Package_TO_SOT_SMD:TSOT-23-6, F.Cu at (-38.5, -1.62)
- added U2: MIC5504-3.3YM5, Package_TO_SOT_SMD:SOT-23-5, F.Cu at (-38.5, 3.00)
- added U3: ISO1044BD, Package_SO:SOIC-8_3.9x4.9mm_P1.27mm, F.Cu at (144.4, 16.5)
- added U4: BT817Q, Package_DFN_QFN:VQFN-64-1EP_9x9mm_P0.5mm_EP7.15x7.15mm, F.Cu at (76.4, 7.00)
- added U5: STM32G441KBTx, Package_QFP:LQFP-32_7x7mm_P0.8mm, F.Cu at (141.8, 7.40)
- added U7: AP3019AKTR, Package_TO_SOT_SMD:SOT-23-6, F.Cu at (-49.9, 11.4)
- added Y1: ECS-240-8-37B-CKY-TR, Crystal:Crystal_SMD_2016-4Pin_2.0x1.6mm, F.Cu at (150.6, 21.4)
Other:
- board text added: "${REFERENCE}"
- board text added: "16.88mm from edge of screen to ribbon cable pin 1"

Commit message: layout work
Parts:
- moved U7 135.4 mm to (85.5, 12.5), turned to 90 degrees
- moved R11 135.2 mm to (90.0, 14.5)
- moved L2 131.9 mm to (79.0, 14.0), turned to 90 degrees
- moved C24 131.7 mm to (85.2, 8.50), turned to 180 degrees
- moved C25 128.1 mm to (81.7, 8.50), turned to 180 degrees
- moved U5 103.9 mm to (39.0, -7.50)
- moved S1 13.3 mm to (12.2, 104.1)
- moved J4 11.8 mm to (78.2, 4.18)
- moved U4 11.4 mm to (76.2, -4.44)
- moved J6 11.3 mm to (114.8, -20.5)
- moved S2 3.99 mm to (88.0, 103.5)
- moved J1 2.59 mm to (52.6, 1.50)
- moved S3 0.75 mm to (50.2, 121.1)
Other:
- board outline added: 106.5 x 142 mm

Commit message: added test points to MCU, layout work
Parts:
- added TP1: TestPoint, TestPoint:TestPoint_Pad_1.0x1.0mm, F.Cu at (-13.5, 7.50)
- added TP2: TestPoint, TestPoint:TestPoint_Pad_1.0x1.0mm, F.Cu at (-13.5, 10.6)
- added TP3: TestPoint, TestPoint:TestPoint_Pad_1.0x1.0mm, F.Cu at (-13.5, 13.6)
- added TP4: TestPoint, TestPoint:TestPoint_Pad_1.0x1.0mm, F.Cu at (-13.5, 16.6)
- added TP5: TestPoint, TestPoint:TestPoint_Pad_1.0x1.0mm, F.Cu at (-13.5, 19.7)
- J2, SW1: moved to B.Cu
- moved J2 138.2 mm to (15.0, -8.55), turned to -90 degrees
- moved Y1 123.3 mm to (31.2, -9.55)
- moved SW1 121.7 mm to (31.1, 13.9), turned to 180 degrees
- moved R18 93.1 mm to (53.5, 10.0), turned to 180 degrees
- moved J6 47.1 mm to (99.5, 24.0)
- moved C26 45.6 mm to (176.7, 39.0)
- moved C27 45.6 mm to (176.7, 41.5)
- moved C28 45.6 mm to (176.7, 44.0)
- moved C29 45.6 mm to (176.7, 46.5)
- moved L1 33.1 mm to (-19.2, -12.5)
- moved R10 33.0 mm to (172.2, 41.5)
- moved R12 33.0 mm to (172.2, 44.0)
- moved R17 33.0 mm to (172.2, 46.5)
- moved R9 33.0 mm to (172.2, 39.0)
- moved C1 22.7 mm to (-30.5, -14.5)
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Connections:
- U5 pad 18: unconnected-(U5-PA8-Pad18) -> Net-(U5-PA8)
- U5 pad 19: unconnected-(U5-PA9-Pad19) -> Net-(U5-PA9)
- U5 pad 20: unconnected-(U5-PA10-Pad20) -> Net-(U5-PA10)
- U5 pad 28: unconnected-(U5-PB5-Pad28) -> Net-(U5-PB5)
- U5 pad 29: unconnected-(U5-PB6-Pad29) -> Net-(U5-PB6)

Commit message: - fixed units and DRC rules for steering wheel PCB - layout pretty much done except for dial placement
Parts:
- C18, TP1, TP2, TP3, TP4, TP5: moved to B.Cu
- moved R17 158.6 mm to (18.5, 7.50), turned to -90 degrees
- moved C26 158.4 mm to (21.5, 7.50), turned to 90 degrees
- moved C27 144.6 mm to (33.5, 21.2), turned to 90 degrees
- moved J11 142.7 mm to (87.0, 20.0), turned to 180 degrees
- moved C29 141.5 mm to (37.5, 21.2), turned to 90 degrees
- moved R9 139.4 mm to (33.5, 24.8), turned to 90 degrees
- moved R8 139.2 mm to (16.5, 7.50), turned to 90 degrees
- moved C28 138.1 mm to (40.5, 21.2), turned to 90 degrees
- moved R4 137.8 mm to (15.8, 19.5)
- moved R12 136.0 mm to (37.5, 24.8), turned to 90 degrees
- moved J12 135.8 mm to (80.5, 20.5), turned to 180 degrees
- moved R10 132.7 mm to (40.5, 24.8), turned to 90 degrees
- moved C8 132.5 mm to (81.5, -14.5)
- moved C9 132.5 mm to (81.5, -11.5)
- moved C15 130.1 mm to (83.5, -4.50)
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Routing:
- net +3V3: track 0.00 -> 271.6 mm, vias 0 -> 9
- net GND: track 0.00 -> 89.3 mm, vias 0 -> 31
- net /MCU/CAN_RX: track 0.00 -> 63.3 mm
- net /Launch_Control: track 0.00 -> 62.8 mm, vias 0 -> 1
- net /MCU/CAN_TX: track 0.00 -> 59.4 mm
- net /Lap: track 0.00 -> 52.1 mm, vias 0 -> 2
- net +12V: track 0.00 -> 51.0 mm, vias 0 -> 2
- net /Display Interface/SPI.MOSI: track 0.00 -> 48.7 mm
- net /MCU/Driver_Interrupt: track 0.00 -> 48.1 mm, vias 0 -> 4
- net /Display Interface/SPI.CLK: track 0.00 -> 45.9 mm
- net /Display Interface/Driver_Power: track 0.00 -> 45.3 mm, vias 0 -> 4
- net /Display Interface/SPI.MISO: track 0.00 -> 44.5 mm, vias 0 -> 2
- net /Display Interface/Backlight_PWM: track 0.00 -> 40.1 mm
- net /Display Interface/SPI.CS: track 0.00 -> 39.3 mm, vias 0 -> 2
- net +1V2: track 0.00 -> 38.7 mm, vias 0 -> 3
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- added copper zone on B.Cu, net GND
- added copper zone on F.Cu, net GND
Other:
- board text removed: "${REFERENCE}"

Commit message: pcb work
Parts:
- added REF**: MountingHole_5.3mm_M5, MountingHole:MountingHole_5.3mm_M5, F.Cu at (7.87, -7.62)
- added REF**: MountingHole_5.3mm_M5, MountingHole:MountingHole_5.3mm_M5, F.Cu at (21.3, 117.9)
- added REF**: MountingHole_5.3mm_M5, MountingHole:MountingHole_5.3mm_M5, F.Cu at (84.1, 117.9)
- added REF**: MountingHole_5.3mm_M5, MountingHole:MountingHole_5.3mm_M5, F.Cu at (97.0, -7.62)
- moved R10 1.87 mm to (38.9, 23.9), turned to 0 degrees
- moved R12 1.26 mm to (36.3, 24.4)
- moved R2 1.12 mm to (32.0, -6.00)
- moved S3 0.67 mm to (49.7, 120.6)
Routing:
- net /MCU/CAN_TX: track 59.4 -> 56.6 mm
- net /MCU/CAN_RX: track 63.3 -> 60.6 mm
- net /CAN_L: track 5.92 -> 4.09 mm
- net +3V3: track 271.6 -> 270.0 mm
- net +12V: track 51.0 -> 52.2 mm
- net /MCU/Layout_Cycle: track 37.9 -> 36.8 mm
- net /Display Interface/SPI.MOSI: track 48.7 -> 47.7 mm
- net GND: track 89.3 -> 88.6 mm, vias 31 -> 30
- net /MCU/Driver_Interrupt: track 48.1 -> 47.4 mm
- net Net-(U5-PA8): track 22.4 -> 23.1 mm
- net /Display Interface/Driver_Power: track 45.3 -> 44.6 mm
- net Net-(U5-PA10): track 14.6 -> 15.2 mm
- net STLINK_SWO: track 30.3 -> 29.7 mm
Other:
- board size 106.5 x 142 mm -> 106.4 x 142 mm

Commit message: steering wheel board layout rev 1 done hopefully unless i missed something
Parts:
- added REF**: MountingHole_5.3mm_M5, MountingHole:MountingHole_5.3mm_M5, F.Cu at (7.87, 34.0)
- added REF**: MountingHole_5.3mm_M5, MountingHole:MountingHole_5.3mm_M5, F.Cu at (97.0, 34.0)
- moved S1 75.9 mm to (88.0, 103.5)
- moved S2 42.0 mm to (49.7, 120.6)
- moved S3 41.0 mm to (12.2, 104.1)
- moved C7 20.2 mm to (55.1, -2.04), turned to -90 degrees
- moved C2 18.4 mm to (57.3, 16.0), turned to 0 degrees
- moved C1 15.6 mm to (58.4, 10.2)
- moved U1 15.4 mm to (58.2, 13.2)
- moved R6 14.2 mm to (14.7, 28.9), turned to -90 degrees
- moved U3 13.8 mm to (51.3, 0.25), turned to -90 degrees
- moved L1 13.6 mm to (52.1, 14.0), turned to 180 degrees
- moved C4 11.3 mm to (47.0, 11.5), turned to 90 degrees
- moved C5 11.1 mm to (41.2, 10.9)
- moved U2 11.1 mm to (44.2, 10.9)
- moved R3 10.4 mm to (14.7, 25.9), turned to -90 degrees
- moved C6 10.1 mm to (55.6, 3.30), turned to 0 degrees
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Connections:
- J1 pad 1: +12V -> /CAN_L
- J1 pad 2: GND -> /CAN_H
- J1 pad 5: /CAN_H -> unconnected-(J1-Pad5)
- J1 pad 6: /CAN_L -> unconnected-(J1-Pad6)
- J1 pad 7: unconnected-(J1-Pad7) -> +12V
- J1 pad 8: unconnected-(J1-Pad8) -> GND
- R18 pad 1: /CAN_H -> /CAN_L
- R18 pad 2: /CAN_L -> /CAN_H
Routing:
- net +3V3: track 270.0 -> 445.3 mm, vias 9 -> 19
- net /Switches/Analog_2V2: track 1.35 -> 174.3 mm, vias 0 -> 1
- net /Switches/Analog_1V1: track 1.35 -> 171.2 mm, vias 0 -> 1
- net /Switches/Mode_Unfiltered: track 0.00 -> 121.9 mm
- net /Switches/TC_Unfiltered: track 0.00 -> 110.3 mm
- net /Switches/Regen_Unfiltered: track 0.00 -> 81.4 mm
- net GND: track 88.6 -> 134.6 mm, vias 30 -> 33
- net /MCU/CAN_RX: track 60.6 -> 18.8 mm, vias 0 -> 2
- net /MCU/CAN_TX: track 56.6 -> 22.5 mm, vias 0 -> 2
- net +12V: track 52.2 -> 35.2 mm, vias 2 -> 0
- net /Display Interface/Backlight_PWM: track 40.1 -> 51.3 mm, vias 0 -> 2
- net Net-(U1-SW): track 10.2 -> 2.67 mm
- net +5V: track 37.6 -> 31.9 mm
- net NRST: track 30.2 -> 25.1 mm, vias 1 -> 3
- net /CAN_L: track 4.09 -> 9.05 mm
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- added copper zone on F.Cu, net +12V
- added copper zone on F.Cu, net +3V3
- added copper zone on F.Cu, net +5V
- added copper zone on F.Cu, net Net-(U1-SW)
Other:
- outline, holes or cut-outs redrawn

Commit message: added title block
Parts:
- added G***: , FS_3_Global_Footprint_Library:FORMULA SLUG TITLE, F.Cu at (4.99, -0.20)
Changed lines of the file:
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@@
 		)
 	)
+	(property "COMMENT4" "Nova Mondal")
+	(property "REVISION" "1.2")
+	(property "TITLE" "Steering Wheel")
 	(net 0 "")
 	(net 1 "GND")
@@
 			(effects
 				(font
-					(size 1 1)
-					(thickness 0.15)
+					(size 1.016 1.016)
+					(thickness 0.1524)
 				)
 			)
@@
 			(effects
 				(font
-					(size 1.27 1.27)
-					(thickness 0.254)
+					(size 1.016 1.016)
+					(thickness 0.1524)
 				)
 			)
@@
 			(effects
 				(font
-					(size 1 1)
-					(thickness 0.15)
+					(size 1.016 1.016)
+					(thickness 0.1524)
 				)
 			)
@@
 			(effects
 				(font
-					(size 1 1)
-					(thickness 0.15)
+					(size 1.016 1.016)
+					(thickness 0.1524)
 				)
 			)
@@
 			(effects
 				(font
-					(size 1.27 1.27)
-					(thickness 0.254)
+					(size 1.016 1.016)
+					(thickness 0.1524)
 				)
 			)
@@
 			(effects
 				(font
-					(size 1 1)
-					(thickness 0.15)
+					(size 1.016 1.016)
+					(thickness 0.1524)
 				)
 			)
@@
 			(effects
 				(font
-					(size 1.27 1.27)
-					(thickness 0.254)
+					(size 1.016 1.016)
+					(thickness 0.1524)
 				)
 			)
@@
 		)
 	)
+	(footprint "FS_3_Global_Footprint_Library:FORMULA SLUG TITLE"
+		(layer "F.Cu")
+		(at 4.99058 -0.195456)
+		(descr "Cosmetic Logo With Title Text")
+		(tags "logo, title")
+		(property "Reference" "G***"
+			(at 0 0 0)
+			(layer "F.SilkS")
+			(hide yes)
+			(effects
+				(font
+					(size 1.016 1.016)
+					(thickness 0.1524)
+				)
+			)
+		)
+		(property "Value" ""
+			(at 0.75 0 0)
+			(layer "F.SilkS")
+			(hide yes)
+			(effects
+				(font
+					(size 1.016 1.016)
+					(thickness 0.1524)
+				)
+			)
+		)
+		(property "Datasheet" ""
+			(at 0 0 0)
+			(unlocked yes)
+			(layer "F.Fab")
+			(hide yes)
+			(effects
+				(font
+					(size 1.27 1.27)
+					(thickness 0.15)
+				)
+			)
+		)
+		(property "Description" ""
+			(at 0 0 0)
+			(unlocked yes)
+			(layer "F.Fab")
+			(hide yes)
+			(effects
+				(font
+					(size 1.27 1.27)
+					(thickness 0.15)
+				)
+			)
+		)
+		(attr board_only exclude_from_pos_files exclude_from_bom)
+		(fp_poly
+			(pts
+				(xy -2.978538 -1.18802) (xy -2.983976 -1.1638) (xy -2.997969 -1.146607) (xy -3.029051 -1.135011)
+				(xy -3.085756 -1.12758) (xy -3.176619 -1.122883) (xy -3.310176 -1.119489) (xy -3.39732 -1.117802)
+				(xy -3.564909 -1.1128) (xy -3.692359 -1.105064) (xy -3.774696 -1.095029) (xy -3.806943 -1.083133)
+				(xy -3.807221 -1.081855) (xy -3.794554 -1.047871) (xy -3.759992 -0.975661) (xy -3.708692 -0.87555)
+				(xy -3.645813 -0.757863) (xy -3.640482 -0.74808) (xy -3.559231 -0.597402) (xy -3.505712 -0.488519)
+				(xy -3.480657 -0.414643) (xy -3.484796 -0.368987) (xy -3.518859 -0.344766) (xy -3.583579 -0.335193)
+				(xy -3.679686 -0.33348) (xy -3.68514 -0.333479) (xy -3.792282 -0.332066) (xy -3.853894 -0.326265)
+				(xy -3.879986 -0.313737) (xy -3.880569 -0.292141) (xy -3.879137 -0.288135) (xy -3.859129 -0.254652)
+				(xy -3.810992 -0.181981) (xy -3.738892 -0.076171) (xy -3.64699 0.056732) (xy -3.539453 0.210679)
+				(xy -3.420443 0.379621) (xy -3.382892 0.432652) (xy -2.904048 1.108095) (xy -2.896242 0.792952)
+				(xy -2.889488 0.633907) (xy -2.876955 0.524137) (xy -2.856434 0.45745) (xy -2.825717 0.427656) (xy -2.782596 0.428564)
+				(xy -2.768006 0.433473) (xy -2.751673 0.445088) (xy -2.739984 0.470553) (xy -2.732378 0.517495)
+				(xy -2.728298 0.59354) (xy -2.727182 0.706311) (xy -2.728471 0.863435) (xy -2.729747 0.954656) (xy -2.733 1.135545)
+				(xy -2.737037 1.268249) (xy -2.74262 1.360161) (xy -2.75051 1.418676) (xy -2.761469 1.451189) (xy -2.776258 1.465093)
+				(xy -2.782515 1.466939) (xy -2.826862 1.451253) (xy -2.88518 1.399229) (xy -2.909682 1.370032) (xy -2.987567 1.267154)
+				(xy -3.083166 1.13683) (xy -3.192391 0.985003) (xy -3.311155 0.817616) (xy -3.435368 0.640612) (xy -3.560942 0.459936)
+				(xy -3.683791 0.28153) (xy -3.799825 0.111337) (xy -3.904957 -0.044698) (xy -3.995098 -0.180633)
+				(xy -4.066161 -0.290525) (xy -4.114057 -0.368429) (xy -4.134698 -0.408403) (xy -4.13516 -0.411609)
+				(xy -4.12066 -0.436378) (xy -4.081382 -0.452174) (xy -4.006396 -0.461682) (xy -3.911132 -0.466651)
+				(xy -3.809759 -0.472504) (xy -3.734104 -0.480736) (xy -3.697537 -0.48978) (xy -3.696061 -0.491833)
+				(xy -3.70842 -0.521472) (xy -3.742186 -0.590206) (xy -3.792395 -0.688202) (xy -3.854083 -0.80563)
+				(xy -3.862801 -0.822025) (xy -3.926298 -0.94564) (xy -3.978662 -1.055906) (xy -4.014757 -1.1414)
+				(xy -4.029444 -1.190697) (xy -4.029541 -1.192849) (xy -4.027655 -1.212848) (xy -4.017105 -1.227595)
+				(xy -3.990548 -1.237889) (xy -3.940641 -1.24453) (xy -3.860043 -1.248318) (xy -3.741411 -1.250051)
+				(xy -3.577404 -1.250528) (xy -3.499599 -1.250547) (xy -2.969657 -1.250547)
+			)
+			(stroke
+				(width 0)
+				(type solid)
+			)
+			(fill yes)
+			(layer "F.SilkS")
+		)
+		(fp_poly
+			(pts
+				(xy -2.788263 -1.56467) (xy -2.778994 -1.529389) (xy -2.766898 -1.463828) (xy -2.737018 -1.388231)
+				(xy -2.698962 -1.321398) (xy -2.662339 -1.282125) (xy -2.650665 -1.278337) (xy -2.61524 -1.301406)
+				(xy -2.598411 -1.333753) (xy -2.560999 -1.408084) (xy -2.512444 -1.449615) (xy -2.46491 -1.448785)
+				(xy -2.458117 -1.444004) (xy -2.434541 -1.398362) (xy -2.448633 -1.353116) (xy -2.490172 -1.333917)
+				(xy -2.524233 -1.317017) (xy -2.524036 -1.280438) (xy -2.493003 -1.245357) (xy -2.474525 -1.23704)
+				(xy -2.411633 -1.198295) (xy -2.347304 -1.131401) (xy -2.297658 -1.056289) (xy -2.278775 -0.995027)
+				(xy -2.296398 -0.940177) (xy -2.340673 -0.869722) (xy -2.362145 -0.843347) (xy -2.412674 -0.778381)
+				(xy -2.442288 -0.725963) (xy -2.445514 -0.712386) (xy -2.43322 -0.66912) (xy -2.40161 -0.596283)
+				(xy -2.373203 -0.539666) (xy -2.300939 -0.401477) (xy -2.251324 -0.300887) (xy -2.220165 -0.226828)
+				(xy -2.203269 -0.16823) (xy -2.196441 -0.114026) (xy -2.195405 -0.070409) (xy -2.203501 0.021962)
+				(xy -2.235816 0.092973) (xy -2.285722 0.152829) (xy -2.392706 0.232287) (xy -2.539714 0.291482)
+				(xy -2.713537 0.326128) (xy -2.842345 0.333479) (xy -2.922925 0.331154) (xy -2.961255 0.319792)
+				(xy -2.970612 0.292813) (xy -2.968508 0.270952) (xy -2.958854 0.238553) (xy -2.933158 0.217909)
+				(xy -2.87939 0.204636) (xy -2.785518 0.194346) (xy -2.750238 0.191389) (xy -2.568212 0.164483) (xy -2.436787 0.117181)
+				(xy -2.354635 0.048897) (xy -2.33162 0.006701) (xy -2.315465 -0.066428) (xy -2.325412 -0.145948)
+				(xy -2.364791 -0.243749) (xy -2.436932 -0.371722) (xy -2.438171 -0.373754) (xy -2.521938 -0.542703)
+				(xy -2.555677 -0.692421) (xy -2.539253 -0.821431) (xy -2.487231 -0.911962) (xy -2.44141 -0.972466)
+				(xy -2.430368 -1.011524) (xy -2.449222 -1.046623) (xy -2.449522 -1.046985) (xy -2.500892 -1.088963)
+				(xy -2.573915 -1.128633) (xy -2.578151 -1.130435) (xy -2.670371 -1.151155) (xy -2.740898 -1.126072)
+				(xy -2.790345 -1.053828) (xy -2.819324 -0.933065) (xy -2.828448 -0.762423) (xy -2.821911 -0.58979)
+				(xy -2.814805 -0.418247) (xy -2.821674 -0.285793) (xy -2.845746 -0.176984) (xy -2.89025 -0.076379)
+				(xy -2.948893 0.017655) (xy -3.016632 0.097772) (xy -3.105241 0.177523) (xy -3.199866 0.245958)
+				(xy -3.285654 0.292126) (xy -3.339557 0.305689) (xy -3.384583 0.291405) (xy -3.387109 0.253564)
+				(xy -3.35072 0.199683) (xy -3.278997 0.137278) (xy -3.249635 0.117041) (xy -3.150799 0.037865) (xy -3.060628 -0.058414)
+				(xy -3.027744 -0.103884) (xy -2.995354 -0.156452) (xy -2.973012 -0.202032) (xy -2.959073 -0.252029)
+				(xy -2.951886 -0.317844) (xy -2.949806 -0.410882) (xy -2.951184 -0.542547) (xy -2.95261 -0.623879)
+				(xy -2.953548 -0.807423) (xy -2.947433 -0.945212) (xy -2.932173 -1.046848) (xy -2.905678 -1.121934)
+				(xy -2.865854 -1.180073) (xy -2.822511 -1.221237) (xy -2.785256 -1.269093) (xy -2.789732 -1.324585)
+				(xy -2.837599 -1.398923) (xy -2.851284 -1.415565) (xy -2.898631 -1.491215) (xy -2.903143 -1.548819)
+				(xy -2.865568 -1.580415) (xy -2.835446 -1.584026)
+			)
+			(stroke
+				(width 0)
+				(type solid)
+			)
+			(fill yes)
+			(layer "F.SilkS")
+		)
+		(fp_text user "Architect: ${COMMENT4}"
+			(at -2.032 1.524 0)
+			(unlocked yes)
+			(layer "F.SilkS")
+			(effects
+				(font
+					(size 1.016 1.016)
+					(thickness 0.1524)
+					(bold yes)
+				)
+				(justify left)
+			)
+		)
+		(fp_text user "${COMPANY}"
+			(at -2.032 -1.524 0)
+			(unlocked yes)
+			(layer "F.SilkS")
+			(effects
+				(font
+					(size 1.016 1.016)
+					(thickness 0.1524)
+					(bold yes)
+				)
+				(justify left)
+			)
+		)
+		(fp_text user "FS-4 ${TITLE} V${REVISION}"
+			(at -2.032 0 0)
+			(unlocked yes)
+			(layer "F.SilkS")
+			(effects
+				(font
+					(size 1.016 1.016)
+					(thickness 0.1524)
+					(bold yes)
+				)
+				(justify left)
+			)
+		)
+		(embedded_fonts no)
+	)
 	(footprint "Resistor_SMD:R_0603_1608Metric"
 		(layer "F.Cu")
@@
 			(effects
 				(font
-					(size 1 1)
-					(thickness 0.15)
+					(size 1.016 1.016)
+					(thickness 0.1524)
 				)
 			)
@@
 			(effects
 				(font
-					(size 1 1)
-					(thickness 0.15)
+					(size 1.016 1.016)
+					(thickness 0.1524)
 				)
 			)
