File: steering-wheel-board/steering_wheel.kicad_pcb (KiCad board)
At the start: 2 copper layers, 106.4 x 142 mm, 78 parts, among them J1 Keystone 985 RJ45, J10 Test Pad, J11 Test Pad, J12 Test Pad, J2 FTSH-107-01-F-DV-K-P-TR, J3 Nanofit 01x02 Right Angle, J4 Conn_01x40, J5 Nanofit 01x02 Right Angle, J6 Nanofit 01x02 Right Angle, SW1 Y97KT23B5NAFP, U1 AP63205WU, U2 MIC5504-3.3YM5, U3 ISO1044BD, U4 BT817Q, U5 STM32G441KBTx, U7 AP3019AKTR, Y1 ECS-240-8-37B-CKY-TR

Commit message: added missing BOM fields and added company to title block
Parts:
- L1: value 4.7uF -> 4.7u
- moved G*** 1.05 mm to (4.74, 0.82)
Changed lines of the file:
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@@
 	)
 	(property "COMMENT4" "Nova Mondal")
+	(property "COMPANY" "Formula Slug")
 	(property "REVISION" "1.2")
 	(property "TITLE" "Steering Wheel")
@@
 	(footprint "FS_3_Global_Footprint_Library:FORMULA SLUG TITLE"
 		(layer "F.Cu")
-		(at 4.99058 -0.195456)
+		(at 4.73658 0.820544)
 		(descr "Cosmetic Logo With Title Text")
 		(tags "logo, title")
@@
 		(sheetname "/Display Interface/")
 		(sheetfile "display.kicad_sch")
-		(attr exclude_from_pos_files)
+		(attr exclude_from_pos_files exclude_from_bom dnp)
 		(fp_circle
 			(center 0 0)
@@
 			)
 		)
+		(property "Digi URL" "https://www.digikey.com/en/products/detail/diodes-incorporated/AP63205WU-7/9858424?s=N4IgTCBcDaIIIAUBsBmMAGArAdQKogF0BfIA"
+			(at 0 0 180)
+			(unlocked yes)
+			(layer "F.Fab")
+			(hide yes)
+			(effects
+				(font
+					(size 1 1)
+					(thickness 0.15)
+				)
+			)
+		)
+		(property "Digi PN" "AP63205WU-7DICT-ND"
+			(at 0 0 180)
+			(unlocked yes)
+			(layer "F.Fab")
+			(hide yes)
+			(effects
+				(font
+					(size 1 1)
+					(thickness 0.15)
+				)
+			)
+		)
+		(property "MFG" "Diodes Incorporated"
+			(at 0 0 180)
+			(unlocked yes)
+			(layer "F.Fab")
+			(hide yes)
+			(effects
+				(font
+					(size 1 1)
+					(thickness 0.15)
+				)
+			)
+		)
+		(property "MFG PN" "AP63205WU-7"
+			(at 0 0 180)
+			(unlocked yes)
+			(layer "F.Fab")
+			(hide yes)
+			(effects
+				(font
+					(size 1 1)
+					(thickness 0.15)
+				)
+			)
+		)
 		(property ki_fp_filters "TSOT?23*")
 		(sheetname "/")
@@
 			)
 		)
-		(property "Value" "4.7uF"
+		(property "Value" "4.7u"
 			(at 0 3.55 0)
 			(layer "F.Fab")
@@
 			)
 		)
+		(property "Digi URL" "https://www.digikey.com/en/products/detail/bourns-inc/SRP5030TA-4R7M/5429673?s=N4IgTCBcDaIMoCUAKBWADAZjQFQIIFoAWBAdgFkQBdAXyA"
+			(at 0 0 180)
+			(unlocked yes)
+			(layer "F.Fab")
+			(hide yes)
+			(effects
+				(font
+					(size 1 1)
+					(thickness 0.15)
+				)
+			)
+		)
+		(property "Digi PN" "SRP5030TA-4R7MCT-ND"
+			(at 0 0 180)
+			(unlocked yes)
+			(layer "F.Fab")
+			(hide yes)
+			(effects
+				(font
+					(size 1 1)
+					(thickness 0.15)
+				)
+			)
+		)
+		(property "MFG" "Bourns"
+			(at 0 0 180)
+			(unlocked yes)
+			(layer "F.Fab")
+			(hide yes)
+			(effects
+				(font
+					(size 1 1)
+					(thickness 0.15)
+				)
+			)
+		)
+		(property "MFG PN" "SRP5030TA-4R7M"
+			(at 0 0 180)
+			(unlocked yes)
+			(layer "F.Fab")
+			(hide yes)
+			(effects
+				(font
+					(size 1 1)
+					(thickness 0.15)
+				)
+			)
+		)
 		(property ki_fp_filters "Choke_* *Coil* Inductor_* L_*")
 		(sheetname "/")
@@
 		(sheetname "/Display Interface/")
 		(sheetfile "display.kicad_sch")
-		(attr exclude_from_pos_files)
+		(attr exclude_from_pos_files exclude_from_bom dnp)
 		(fp_circle
 			(center 0 0)
@@
 		(sheetname "/Display Interface/")
 		(sheetfile "display.kicad_sch")
-		(attr exclude_from_pos_files)
+		(attr exclude_from_pos_files exclude_from_bom dnp)
 		(fp_circle
 			(center 0 0)
@@
 			)
 		)
-		(property "Digi PN" ""
+		(property "Digi PN" "576-4764-1-ND"
 			(at 0 0 180)
 			(unlocked yes)
@@
 			)
 		)
-		(property "Digi URL" ""
+		(property "Digi URL" "https://www.digikey.com/en/products/detail/microchip-technology/MIC5504-3-3YM5-TR/4864018"
 			(at 0 0 180)
 			(unlocked yes)
@@
 			)
 		)
-		(property "MFG" ""
+		(property "MFG" "Microchip Technology"
 			(at 0 0 180)
 			(unlocked yes)
@@
 		(sheetname "/MCU/")
 		(sheetfile "MCU.kicad_sch")
-		(attr exclude_from_pos_files)
+		(attr exclude_from_pos_files exclude_from_bom dnp)
 		(fp_line
 			(start -0.7 -0.7)
@@
 		(sheetname "/MCU/")
 		(sheetfile "MCU.kicad_sch")
-		(attr exclude_from_pos_files)
+		(attr exclude_from_pos_files exclude_from_bom dnp)
 		(fp_line
 			(start -0.7 -0.7)
@@
 		(sheetname "/MCU/")
 		(sheetfile "MCU.kicad_sch")
-		(attr exclude_from_pos_files)
+		(attr exclude_from_pos_files exclude_from_bom dnp)
 		(fp_line
 			(start -0.7 -0.7)
@@
 		(sheetname "/MCU/")
 		(sheetfile "MCU.kicad_sch")
-		(attr exclude_from_pos_files)
+		(attr exclude_from_pos_files exclude_from_bom dnp)
 		(fp_line
 			(start -0.7 -0.7)
@@
 		(sheetname "/MCU/")
 		(sheetfile "MCU.kicad_sch")
-		(attr exclude_from_pos_files)
+		(attr exclude_from_pos_files exclude_from_bom dnp)
 		(fp_line
 			(start -0.7 -0.7)
