File: Vicor_DCDC/DCDC/DCDC.kicad_pcb (KiCad board)
At the start: 4 copper layers, 7 parts

Commit message: GLV Protection Circuit
- Added undervoltage protection circuit and reverse polarity protection circuit schematics
- Added three footprints to the library related to circuits listed
Connections:
- PS1 pad 2: Net-(PS1-PC) -> unconnected-(PS1-PC-Pad2)
Routing:
- net -IN: track 29.3 -> 30.1 mm
Changed lines of the file:
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@@
 	(net 4 "+OUT")
 	(net 5 "-OUT")
-	(net 6 "Net-(PS1-PC)")
-	(net 7 "unconnected-(PS1-PR-Pad3)")
-	(net 8 "Net-(PS1-SC)")
+	(net 6 "unconnected-(PS1-PR-Pad3)")
+	(net 7 "Net-(PS1-SC)")
+	(net 8 "unconnected-(PS1-PC-Pad2)")
 	(footprint "Capacitor_SMD:C_0805_2012Metric_Pad1.18x1.45mm_HandSolder"
 		(layer "F.Cu")
@@
 			(layers "F.Cu" "F.Mask" "F.Paste")
 			(roundrect_rratio 0.208333)
-			(net 8 "Net-(PS1-SC)")
+			(net 7 "Net-(PS1-SC)")
 			(pintype "passive")
 		)
@@
 			(layers "*.Cu" "*.Mask")
 			(remove_unused_layers no)
-			(net 6 "Net-(PS1-PC)")
+			(net 8 "unconnected-(PS1-PC-Pad2)")
 			(pinfunction "PC")
 			(pintype "passive")
@@
 			(layers "*.Cu" "*.Mask")
 			(remove_unused_layers no)
-			(net 7 "unconnected-(PS1-PR-Pad3)")
+			(net 6 "unconnected-(PS1-PR-Pad3)")
 			(pinfunction "PR")
 			(pintype "passive")
@@
 			(layers "*.Cu" "*.Mask")
 			(remove_unused_layers no)
-			(net 8 "Net-(PS1-SC)")
+			(net 7 "Net-(PS1-SC)")
 			(pinfunction "SC")
 			(pintype "passive")
@@
 	)
 	(segment
+		(start 109.215936 99.38)
+		(end 109.94 99.38)
+		(width 0.2)
+		(layer "F.Cu")
+		(net 1)
+	)
+	(segment
 		(start 102 99.5)
 		(end 103 99.5)
@@
 		(width 0.2)
 		(layer "F.Cu")
-		(net 8)
+		(net 7)
 	)
 	(segment
@@
 		(width 0.2)
 		(layer "F.Cu")
-		(net 8)
+		(net 7)
 	)
 	(zone
