File: Tractive_Battery_Board/precharge_relay_n_notch_example.kicad_pcb (KiCad board)
At the start: 2 copper layers, 71.5 x 40 mm, 1 part

Commit message: minor tweaks
Other:
- outline, holes or cut-outs redrawn
Changed lines of the file:
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@@
 		)
 		(fp_line
-			(start 2.159 3.2135)
-			(end 1.524 3.2135)
-			(stroke
-				(width 0.12)
-				(type solid)
-			)
-			(layer "F.SilkS")
-		)
-		(fp_line
-			(start 1.524 3.2135)
-			(end 1.524 3.8735)
-			(stroke
-				(width 0.12)
-				(type solid)
-			)
-			(layer "F.SilkS")
-		)
-		(fp_line
-			(start 2.032 3.8735)
-			(end 1.016 3.8735)
-			(stroke
-				(width 0.12)
-				(type solid)
-			)
-			(layer "F.SilkS")
-		)
-		(fp_line
-			(start 1.016 3.8735)
-			(end 1.016 5.7785)
-			(stroke
-				(width 0.12)
-				(type solid)
-			)
-			(layer "F.SilkS")
-		)
-		(fp_line
-			(start 2.032 5.3975)
-			(end 1.016 4.7625)
-			(stroke
-				(width 0.12)
-				(type solid)
-			)
-			(layer "F.SilkS")
-		)
-		(fp_line
-			(start 2.032 5.7785)
-			(end 2.032 3.8735)
-			(stroke
-				(width 0.12)
-				(type solid)
-			)
-			(layer "F.SilkS")
-		)
-		(fp_line
-			(start 2.032 5.7785)
-			(end 1.016 5.7785)
-			(stroke
-				(width 0.12)
-				(type solid)
-			)
-			(layer "F.SilkS")
-		)
-		(fp_line
-			(start 2.159 6.4135)
-			(end 1.524 6.4135)
-			(stroke
-				(width 0.12)
-				(type solid)
-			)
-			(layer "F.SilkS")
-		)
-		(fp_line
-			(start 1.524 6.4135)
-			(end 1.524 5.7785)
+			(start 2.635 3.451)
+			(end 2 3.451)
+			(stroke
+				(width 0.12)
+				(type solid)
+			)
+			(layer "F.SilkS")
+		)
+		(fp_line
+			(start 2 3.451)
+			(end 2 4.111)
+			(stroke
+				(width 0.12)
+				(type solid)
+			)
+			(layer "F.SilkS")
+		)
+		(fp_line
+			(start 2.508 4.111)
+			(end 1.492 4.111)
+			(stroke
+				(width 0.12)
+				(type solid)
+			)
+			(layer "F.SilkS")
+		)
+		(fp_line
+			(start 1.492 4.111)
+			(end 1.492 6.016)
+			(stroke
+				(width 0.12)
+				(type solid)
+			)
+			(layer "F.SilkS")
+		)
+		(fp_line
+			(start 2.508 5.635)
+			(end 1.492 5)
+			(stroke
+				(width 0.12)
+				(type solid)
+			)
+			(layer "F.SilkS")
+		)
+		(fp_line
+			(start 2.508 6.016)
+			(end 2.508 4.111)
+			(stroke
+				(width 0.12)
+				(type solid)
+			)
+			(layer "F.SilkS")
+		)
+		(fp_line
+			(start 2.508 6.016)
+			(end 1.492 6.016)
+			(stroke
+				(width 0.12)
+				(type solid)
+			)
+			(layer "F.SilkS")
+		)
+		(fp_line
+			(start 2.635 6.651)
+			(end 2 6.651)
+			(stroke
+				(width 0.12)
+				(type solid)
+			)
+			(layer "F.SilkS")
+		)
+		(fp_line
+			(start 2 6.651)
+			(end 2 6.016)
 			(stroke
 				(width 0.12)
@@
 			(members "a0b3f04c-a298-4c2d-8ce5-cacb473bd286" "fb5a1cdb-d4ee-40be-a115-65e17d68d697")
 		)
+		(group ""
+			(members "03969a20-f497-418e-8632-d9d787fd17cb" "063bec82-3d92-493d-9b53-40a855f9b679"
+				"2ca4daae-7524-42a1-9abc-b567137524c1" "3183e544-2379-484b-92df-572ab5307a6d"
+				"731611f6-f447-467d-bf8d-5b208204b9bd" "a005f20e-f189-4526-9fac-34e8bec24487"
+				"ccb0175b-0b9b-4ffa-9023-33cc50ed4738" "fb72ee25-b32b-469e-ab42-696359527e47"
+				"ff01f92a-a396-4302-a975-8f81995c0e58"
+			)
+		)
 		(embedded_fonts no)
 	)
 	(gr_line
-		(start 122.2 82.3)
-		(end 129.7 82.3)
-		(stroke
-			(width 0.05)
-			(type default)
-		)
-		(layer "Edge.Cuts")
-	)
-	(gr_arc
-		(start 129.7 82.3)
-		(mid 132.2 84.8)
-		(end 129.7 87.3)
-		(stroke
-			(width 0.05)
-			(type default)
-		)
-		(layer "Edge.Cuts")
-	)
-	(gr_line
-		(start 129.7 87.3)
-		(end 119.7 87.3)
+		(start 131.95 77.8)
+		(end 131.95 70.8)
+		(stroke
+			(width 0.05)
+			(type default)
+		)
+		(layer "Edge.Cuts")
+	)
+	(gr_line
+		(start 120.25 86.95)
+		(end 129.25 86.95)
+		(stroke
+			(width 0.05)
+			(type default)
+		)
+		(layer "Edge.Cuts")
+	)
+	(gr_line
+		(start 118.65 78)
+		(end 118.65 78.5)
+		(stroke
+			(width 0.05)
+			(type default)
+		)
+		(layer "Edge.Cuts")
+	)
+	(gr_arc
+		(start 118.65 78)
+		(mid 120.25 76.4)
+		(end 121.85 78)
+		(stroke
+			(width 0.05)
+			(type default)
+		)
+		(layer "Edge.Cuts")
+	)
+	(gr_line
+		(start 118.65 78.5)
+		(end 118.65 85.35)
+		(stroke
+			(width 0.05)
+			(type default)
+		)
+		(layer "Edge.Cuts")
+	)
+	(gr_arc
+		(start 133.7 79.55)
+		(mid 132.462563 79.037437)
+		(end 131.95 77.8)
+		(stroke
+			(width 0.05)
+			(type default)
+		)
+		(layer "Edge.Cuts")
+	)
+	(gr_line
+		(start 135.45 76.05)
+		(end 135.45 70.8)
 		(stroke
 			(width 0.05)
@@
 	)
 	(gr_arc
-		(start 117.2 74.8)
-		(mid 119.7 72.3)
-		(end 122.2 74.8)
-		(stroke
-			(width 0.05)
-			(type default)
-		)
-		(layer "Edge.Cuts")
-	)
-	(gr_arc
-		(start 119.7 87.3)
-		(mid 117.932233 86.567767)
-		(end 117.2 84.8)
-		(stroke
-			(width 0.05)
-			(type default)
-		)
-		(layer "Edge.Cuts")
-	)
-	(gr_line
-		(start 117.2 74.8)
-		(end 117.2 84.8)
-		(stroke
-			(width 0.05)
-			(type default)
-		)
-		(layer "Edge.Cuts")
-	)
-	(gr_line
-		(start 122.2 74.8)
-		(end 122.2 82.3)
-		(stroke
-			(width 0.05)
-			(type default)
-		)
-		(layer "Edge.Cuts")
+		(start 129.25 83.75)
+		(mid 130.85 85.35)
+		(end 129.25 86.95)
+		(stroke
+			(width 0.05)
+			(type default)
+		)
+		(layer "Edge.Cuts")
+	)
+	(gr_arc
+		(start 131.95 70.8)
+		(mid 133.7 69.05)
+		(end 135.45 70.8)
+		(stroke
+			(width 0.05)
+			(type default)
+		)
+		(layer "Edge.Cuts")
+	)
+	(gr_arc
+		(start 142.7 76.05)
+		(mid 144.45 77.8)
+		(end 142.7 79.55)
+		(stroke
+			(width 0.05)
+			(type default)
+		)
+		(layer "Edge.Cuts")
+	)
+	(gr_arc
+		(start 120.25 86.95)
+		(mid 119.118629 86.481371)
+		(end 118.65 85.35)
+		(stroke
+			(width 0.05)
+			(type default)
+		)
+		(layer "Edge.Cuts")
+	)
+	(gr_line
+		(start 142.7 76.05)
+		(end 135.45 76.05)
+		(stroke
+			(width 0.05)
+			(type default)
+		)
+		(layer "Edge.Cuts")
+	)
+	(gr_line
+		(start 129.25 83.75)
+		(end 121.85 83.75)
+		(stroke
+			(width 0.05)
+			(type default)
+		)
+		(layer "Edge.Cuts")
+	)
+	(gr_line
+		(start 142.7 79.55)
+		(end 133.7 79.55)
+		(stroke
+			(width 0.05)
+			(type default)
+		)
+		(layer "Edge.Cuts")
+	)
+	(gr_line
+		(start 121.85 83.75)
+		(end 121.85 78)
+		(stroke
+			(width 0.05)
+			(type default)
+		)
+		(layer "Edge.Cuts")
+	)
+	(dimension
+		(type orthogonal)
+		(layer "Edge.Cuts")
+		(pts
+			(xy 141.2 76.05) (xy 141.25 79.55)
+		)
+		(height 5.8)
+		(orientation 1)
+		(format
+			(prefix "")
+			(suffix "")
+			(units 3)
+			(units_format 0)
+			(precision 4)
+			(suppress_zeroes yes)
+		)
+		(style
+			(thickness 0.05)
+			(arrow_length 1.27)
+			(text_position_mode 0)
+			(arrow_direction outward)
+			(extension_height 0.58642)
+			(extension_offset 0.5)
+			(keep_text_aligned yes)
+		)
+		(gr_text "3.5"
+			(at 145.85 77.8 90)
+			(layer "Edge.Cuts")
+			(effects
+				(font
+					(size 1 1)
+					(thickness 0.15)
+				)
+			)
+		)
+	)
+	(dimension
+		(type orthogonal)
+		(layer "Edge.Cuts")
+		(pts
+			(xy 128.1 83.75) (xy 128.3 86.95)
+		)
+		(height 4.75)
+		(orientation 1)
+		(format
+			(prefix "")
+			(suffix "")
+			(units 3)
+			(units_format 0)
+			(precision 4)
+			(suppress_zeroes yes)
+		)
+		(style
+			(thickness 0.05)
+			(arrow_length 1.27)
+			(text_position_mode 0)
+			(arrow_direction outward)
+			(extension_height 0.58642)
+			(extension_offset 0.5)
+			(keep_text_aligned yes)
+		)
+		(gr_text "3.2"
+			(at 131.7 85.35 90)
+			(layer "Edge.Cuts")
+			(effects
+				(font
+					(size 1 1)
+					(thickness 0.15)
+				)
+			)
+		)
 	)
 	(group ""
-		(members "0ae116a1-259c-4e83-b5c3-759f749552a5" "28db7b20-79a4-47a0-87e0-fa39f1109f30"
-			"3b71302a-7aaa-4e4f-9f93-867671b7a8e7" "71d31999-cc3a-4ea6-81fa-2c20f2e39aae"
-			"7287793d-194b-4da5-8a4e-166401bd5c22" "72a528bb-665e-4972-8842-98afb0ba0dab"
-			"d5deed1d-6b4a-4f4a-af85-a8576f567ab0"
-		)
-	)
+		(members "03478599-468d-44b2-9781-6c61a4d54840" "466793f2-7726-44f9-8b62-dd972013ea9a"
+			"4999de1e-b215-4d69-a2e9-49a290a51eb4" "92c84684-ede3-4e38-b815-f26114880a5a"
+			"9416b437-0d04-4c8a-96ea-58c1f22f6385" "99da967d-be8b-4782-ae97-762388fa5e9e"
+			"e7367398-1a4d-4804-9400-66af2bc2f1cb"
+		)
+	)
