File: Tractive_Battery_Board/Tractive_Battery_Board.kicad_sch (KiCad schematic)
At the start: 59 parts, among them J1 TS+/-, J12 Busbar_Temp_Sense, J13 E-Meter, J14 FTSH-107-01-F-DV-K-P-TR, J15 BMS_Temp_Sense, J2 HVIL, J3 Conn_01x12_Pin, J4 Conn_01x16_Pin, J6 IRs Power, J8 Conn_01x03, Q1 NMOS, Q6 PMOS, SW2 Y97KT23B5NAFP, U10 AP63205WU, U11 DS18B20Z, U12 STM32F446RETx, U15 ZXTR2005ZQ-13, U3 ISO1044BD, U9 MIC5504-3.3YM5, Y2 ECS-240-8-37B-CKY-TR

Commit message: small corrections
Parts:
- removed J6: IRs Power, Connector_Molex:Molex_Nano-Fit_105309-xx04_1x04_P2.50mm_Vertical, symbol 1FS_2_Global_Symbol_Library:1053091204
- removed SZNUD3124LT1G5: Q4, Package_TO_SOT_SMD:TSOT-23_HandSoldering, symbol FS_4_SCHEMATICS:SZNUD3124LT1G
- added R34: 10k, symbol Device:R
- added R37: 100k, symbol Device:R
- added SW1: SH_RESET_BUTTON, symbol Switch:SW_Push
- R10: value 1.6k -> 1.2k
- R11: value 560 -> 270
Connections:
- net PreChargeControl is gone; now on net PreCharge_Control: U12.14 (PA0)
- net +3.3V: now also Q6.3 (S); no longer Q6.1 (D)
- net +5V: now also SW1.1
- net GND: now also Q1.1 (D), R37.2; no longer Q1.3 (S)
- net SH_Reset-: now also SW1.2
- net Shutdown + IMD Delay/BMS_FAULT_5V: now also Q1.3 (S); no longer Q1.1 (D)
- net Shutdown_TB_In: now also U12.20 (PA4)
- net Shutdown_TB_Out: now also U12.21 (PA5)
- net TS1W: now also Q6.1 (D); no longer Q6.3 (S)
- net BMS_Fault_3.3V: no longer names the net of Q1.2 (G)
- net BMS_Fault_3.3V: now also R34.1; no longer U12.26 (PB0)
- new net nBMS_Fault_3.3V: R34.2, R37.1, U12.26 (PB0)
Other:
- sheet Shutdown + IMD Delay ports: added nBMS_FAULT_DELAYED_5V, nIMD_FAULT_DELAYED_5V; removed nBMS_FAULT, nIMD_FAULT
- note added: "Ask firmware about TS1W pin assignmnet"
- note added: "breadboard to test"
- note added: "include diagraam for IRs"
- note added: "inlcude off-board switch -- . include building maaterials"
- moved on the sheet: R10, R18

Commit message: Shutdown LED logic fixed
Connections:
- net +5V: now also U12.41 (PA8)
- net IMD_FAULT_12V: now reaches J8.1 (Pin_1), R10.1
Other:
- moved on the sheet: R37, SW1

Commit message: more small changes
Connections:
- net +5V: no longer U12.41 (PA8)
- net GND: no longer C1.2, C2.2
- net Shutdown_TB_In: no longer J3.4 (Pin_4)
- net Shutdown_TB_Out: no longer J3.5 (Pin_5)
- net TS-: now also C1.2, C2.2
- net SH_RESET: now reaches U12.50 (PA15)
- net SH_Reset- renamed SH_RESET-
- net V_Curr_VRef renamed V_Curr_Ref
- new net Shutdown_In: J3.4 (Pin_4)
- new net Shutdown_Out: J3.5 (Pin_5)
Other:
- note removed: "inlcude off-board switch -- . include building maaterials"

Commit message: removed duped components
Parts:
- removed R2: 120, symbol Device:R
- added R41: 120, symbol Device:R
Connections:
- net CAN_L1: now also R41.2
- net CAN_L_RES1: now also R41.1
Changed lines of the file:
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@@
 		(dnp no)
 		(fields_autoplaced yes)
-		(property "Reference" "#FLG?"
+		(property "Reference" "#FLG0101"
 			(at 69.85 61.595 0)
 			(effects
@@
 			(project ""
 				(path "/ca333741-5826-495c-b860-5422aa5e17fc"
-					(reference "#FLG?")
+					(reference "#FLG0101")
 					(unit 1)
 				)
@@
 		(on_board yes)
 		(dnp no)
-		(property "Reference" "#PWR042"
+		(property "Reference" "#PWR0101"
 			(at 27.94 227.33 0)
 			(effects
@@
 			(project "Tractive_Battery_Board"
 				(path "/ca333741-5826-495c-b860-5422aa5e17fc"
-					(reference "#PWR042")
+					(reference "#PWR0101")
 					(unit 1)
 				)
@@
 		(dnp no)
 		(fields_autoplaced yes)
-		(property "Reference" "#PWR?"
+		(property "Reference" "#PWR0104"
 			(at 77.47 67.31 0)
 			(effects
@@
 			(project ""
 				(path "/ca333741-5826-495c-b860-5422aa5e17fc"
-					(reference "#PWR?")
+					(reference "#PWR0104")
 					(unit 1)
 				)
@@
 	)
 	(symbol
+		(lib_id "Device:R")
+		(at 228.6 49.53 0)
+		(unit 1)
+		(exclude_from_sim no)
+		(in_bom yes)
+		(on_board yes)
+		(dnp no)
+		(property "Reference" "R41"
+			(at 231.648 48.768 0)
+			(effects
+				(font
+					(size 1.27 1.27)
+				)
+			)
+		)
+		(property "Value" "120"
+			(at 231.902 50.546 0)
+			(effects
+				(font
+					(size 1.27 1.27)
+				)
+			)
+		)
+		(property "Footprint" ""
+			(at 226.822 49.53 90)
+			(effects
+				(font
+					(size 1.27 1.27)
+				)
+				(hide yes)
+			)
+		)
+		(property "Datasheet" "~"
+			(at 228.6 49.53 0)
+			(effects
+				(font
+					(size 1.27 1.27)
+				)
+				(hide yes)
+			)
+		)
+		(property "Description" "Resistor"
+			(at 228.6 49.53 0)
+			(effects
+				(font
+					(size 1.27 1.27)
+				)
+				(hide yes)
+			)
+		)
+		(pin "2"
+		)
+		(pin "1"
+		)
+		(instances
+			(project "Tractive_Battery_Board"
+				(path "/ca333741-5826-495c-b860-5422aa5e17fc"
+					(reference "R41")
+					(unit 1)
+				)
+			)
+		)
+	)
+	(symbol
 		(lib_id "power:GND")
 		(at 285.75 66.04 0)
@@
 		(dnp no)
 		(fields_autoplaced yes)
-		(property "Reference" "#PWR?"
+		(property "Reference" "#PWR0106"
 			(at 46.99 49.53 0)
 			(effects
@@
 			(project ""
 				(path "/ca333741-5826-495c-b860-5422aa5e17fc"
-					(reference "#PWR?")
-					(unit 1)
-				)
-			)
-		)
-	)
-	(symbol
-		(lib_id "Device:R")
-		(at 228.6 49.53 0)
-		(unit 1)
-		(exclude_from_sim no)
-		(in_bom yes)
-		(on_board yes)
-		(dnp no)
-		(property "Reference" "R2"
-			(at 231.648 48.768 0)
-			(effects
-				(font
-					(size 1.27 1.27)
-				)
-			)
-		)
-		(property "Value" "120"
-			(at 231.902 50.546 0)
-			(effects
-				(font
-					(size 1.27 1.27)
-				)
-			)
-		)
-		(property "Footprint" ""
-			(at 226.822 49.53 90)
-			(effects
-				(font
-					(size 1.27 1.27)
-				)
-				(hide yes)
-			)
-		)
-		(property "Datasheet" "~"
-			(at 228.6 49.53 0)
-			(effects
-				(font
-					(size 1.27 1.27)
-				)
-				(hide yes)
-			)
-		)
-		(property "Description" "Resistor"
-			(at 228.6 49.53 0)
-			(effects
-				(font
-					(size 1.27 1.27)
-				)
-				(hide yes)
-			)
-		)
-		(pin "2"
-		)
-		(pin "1"
-		)
-		(instances
-			(project "Tractive_Battery_Board"
-				(path "/ca333741-5826-495c-b860-5422aa5e17fc"
-					(reference "R2")
+					(reference "#PWR0106")
 					(unit 1)
 				)
@@
 		(dnp no)
 		(fields_autoplaced yes)
-		(property "Reference" "#PWR?"
+		(property "Reference" "#PWR0103"
 			(at 27.94 67.31 0)
 			(effects
@@
 			(project ""
 				(path "/ca333741-5826-495c-b860-5422aa5e17fc"
-					(reference "#PWR?")
+					(reference "#PWR0103")
 					(unit 1)
 				)
@@
 		(dnp no)
 		(fields_autoplaced yes)
-		(property "Reference" "#PWR?"
+		(property "Reference" "#PWR0107"
 			(at 59.69 36.83 0)
 			(effects
@@
 			(project ""
 				(path "/ca333741-5826-495c-b860-5422aa5e17fc"
-					(reference "#PWR?")
+					(reference "#PWR0107")
 					(unit 1)
 				)
@@
 		(dnp no)
 		(fields_autoplaced yes)
-		(property "Reference" "#PWR?"
+		(property "Reference" "#PWR0102"
 			(at 46.99 85.09 0)
 			(effects
@@
 			(project ""
 				(path "/ca333741-5826-495c-b860-5422aa5e17fc"
-					(reference "#PWR?")
+					(reference "#PWR0102")
 					(unit 1)
 				)
@@
 		(dnp no)
 		(fields_autoplaced yes)
-		(property "Reference" "#PWR?"
+		(property "Reference" "#PWR0105"
 			(at 27.94 36.83 0)
 			(effects
@@
 			(project ""
 				(path "/ca333741-5826-495c-b860-5422aa5e17fc"
-					(reference "#PWR?")
+					(reference "#PWR0105")
 					(unit 1)
 				)

Commit message: footprint updates + started layout
Parts:
- removed Q6: PMOS, symbol Simulation_SPICE:PMOS
- added Q3: BSS308PE, Package_TO_SOT_SMD:SOT-23_Handsoldering, symbol FS_3_Global_Symbol_Library:BSS308PE
- C1, C2: footprint (none) -> Capacitor_SMD:C_0805_2012Metric_Pad1.18x1.45mm_HandSolder
- D1: value D_Zener -> HPZR-C50-QX; footprint (none) -> Diode_SMD:Nexperia_CFP3_SOD-123W
- J1: footprint (none) -> Connector_Harwin:Harwin_LTek-Male_02_P2.00mm_Vertical; now left out of the parts list
- J12, J13, J15, J2: footprint (none) -> Connector_Harwin:Harwin_LTek-Male_02_P2.00mm_Vertical
- J3: footprint (none) -> Connector_Harwin:Harwin_LTek-Male_2x06_P2.00mm_Vertical
- J4: footprint (none) -> Connector_Harwin:Harwin_LTek-Male_2x08_P2.00mm_Vertical
- J8: footprint (none) -> Connector_Harwin:Harwin_LTek-Male_03_P2.00mm_Vertical
- JP1: footprint (none) -> Jumper:Jumper_Harwin_S1621_P10.9mm
- R10, R11, R12, R15, R17, R18, R33, R34, R37, R41: footprint (none) -> Resistor_SMD:R_0805_2012Metric_Pad1.20x1.40mm_HandSolder
Connections:
- net +3.3V: now also Q3.2 (S)
- net TS1W: now also Q3.3 (D)
- net TS1W_PU_Control: now also Q3.1 (G)
Changed lines of the file:
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@@
 	)
 	(junction
-		(at 222.25 138.43)
-		(diameter 0)
-		(color 0 0 0 0)
-	)
-	(junction
 		(at 91.44 110.49)
 		(diameter 0)
@@
 	(wire
 		(pts
-			(xy 222.25 138.43) (xy 229.87 138.43)
-		)
-		(stroke
-			(width 0)
-			(type default)
-		)
-	)
-	(wire
-		(pts
 			(xy 69.85 191.77) (xy 73.66 191.77)
 		)
@@
 	)
 	(symbol
+		(lib_id "FS_3_Global_Symbol_Library:BSS308PE")
+		(at 200.66 110.49 0)
+		(mirror x)
+		(unit 1)
+		(exclude_from_sim no)
+		(in_bom yes)
+		(on_board yes)
+		(dnp no)
+		(property "Reference" "Q3"
+			(at 199.898 107.442 0)
+			(effects
+				(font
+					(size 1.27 1.27)
+				)
+				(justify right)
+			)
+		)
+		(property "Value" "BSS308PE"
+			(at 199.898 104.902 0)
+			(effects
+				(font
+					(size 1.27 1.27)
+				)
+				(justify right)
+			)
+		)
+		(property "Footprint" "Package_TO_SOT_SMD:SOT-23_Handsoldering"
+			(at 205.74 113.03 0)
+			(effects
+				(font
+					(size 1.27 1.27)
+				)
+				(hide yes)
+			)
+		)
+		(property "Datasheet" "https://www.infineon.com/dgdl/Infineon-BSS308PE-DS-v02_03-en.pdf?fileId=db3a304330f686060131099c80400073"
+			(at 200.66 97.79 0)
+			(effects
+				(font
+					(size 1.27 1.27)
+				)
+				(hide yes)
+			)
+		)
+		(property "Description" "-2A Id, -30V Vds, P-Channel MOSFET, PG-SOT23"
+			(at 200.66 110.49 0)
+			(effects
+				(font
+					(size 1.27 1.27)
+				)
+				(hide yes)
+			)
+		)
+		(property "Sim.Device" "PMOS"
+			(at 200.66 93.345 0)
+			(effects
+				(font
+					(size 1.27 1.27)
+				)
+				(hide yes)
+			)
+		)
+		(property "Sim.Type" "VDMOS"
+			(at 200.66 91.44 0)
+			(effects
+				(font
+					(size 1.27 1.27)
+				)
+				(hide yes)
+			)
+		)
+		(property "Sim.Pins" "1=S 2=G 3=D"
+			(at 200.66 95.25 0)
+			(effects
+				(font
+					(size 1.27 1.27)
+				)
+				(hide yes)
+			)
+		)
+		(pin "2"
+		)
+		(pin "3"
+		)
+		(pin "1"
+		)
+		(instances
+			(project "Tractive_Battery_Board"
+				(path "/ca333741-5826-495c-b860-5422aa5e17fc"
+					(reference "Q3")
+					(unit 1)
+				)
+			)
+		)
+	)
+	(symbol
 		(lib_id "power:GND")
 		(at 134.62 190.5 0)
@@
 			)
 		)
-		(property "Footprint" ""
+		(property "Footprint" "Connector_Harwin:Harwin_LTek-Male_02_P2.00mm_Vertical"
 			(at 260.35 142.24 0)
 			(effects
@@
 			)
 		)
-		(property "Footprint" ""
+		(property "Footprint" "Capacitor_SMD:C_0805_2012Metric_Pad1.18x1.45mm_HandSolder"
 			(at 385.7752 77.47 0)
 			(effects
@@
 			)
 		)
-		(property "Footprint" ""
+		(property "Footprint" "Resistor_SMD:R_0805_2012Metric_Pad1.20x1.40mm_HandSolder"
 			(at 309.372 132.08 90)
 			(effects
@@
 			)
 		)
-		(property "Footprint" ""
+		(property "Footprint" "Resistor_SMD:R_0805_2012Metric_Pad1.20x1.40mm_HandSolder"
 			(at 356.362 184.15 90)
 			(effects
@@
 			)
 		)
-		(property "Footprint" ""
+		(property "Footprint" "Connector_Harwin:Harwin_LTek-Male_02_P2.00mm_Vertical"
 			(at 260.35 127 0)
 			(effects
@@
 			)
 		)
-		(property "Footprint" ""
+		(property "Footprint" "Resistor_SMD:R_0805_2012Metric_Pad1.20x1.40mm_HandSolder"
 			(at 338.582 104.14 90)
 			(effects
@@
 	)
 	(symbol
-		(lib_id "Simulation_SPICE:PMOS")
-		(at 200.66 110.49 0)
-		(mirror x)
-		(unit 1)
-		(exclude_from_sim no)
-		(in_bom yes)
-		(on_board yes)
-		(dnp no)
-		(property "Reference" "Q6"
-			(at 205.994 111.76 0)
-			(effects
-				(font
-					(size 1.27 1.27)
-				)
-				(justify left)
-			)
-		)
-		(property "Value" "PMOS"
-			(at 205.994 109.22 0)
-			(effects
-				(font
-					(size 1.27 1.27)
-				)
-				(justify left)
-			)
-		)
-		(property "Footprint" ""
-			(at 205.74 113.03 0)
-			(effects
-				(font
-					(size 1.27 1.27)
-				)
-				(hide yes)
-			)
-		)
-		(property "Datasheet" "https://ngspice.sourceforge.io/docs/ngspice-html-manual/manual.xhtml#cha_MOSFETs"
-			(at 200.66 97.79 0)
-			(effects
-				(font
-					(size 1.27 1.27)
-				)
-				(hide yes)
-			)
-		)
-		(property "Description" "P-MOSFET transistor, drain/source/gate"
-			(at 200.66 110.49 0)
-			(effects
-				(font
-					(size 1.27 1.27)
-				)
-				(hide yes)
-			)
-		)
-		(property "Sim.Device" "PMOS"
-			(at 200.66 93.345 0)
-			(effects
-				(font
-					(size 1.27 1.27)
-				)
-				(hide yes)
-			)
-		)
-		(property "Sim.Type" "VDMOS"
-			(at 200.66 91.44 0)
-			(effects
-				(font
-					(size 1.27 1.27)
-				)
-				(hide yes)
-			)
-		)
-		(property "Sim.Pins" "1=D 2=G 3=S"
-			(at 200.66 95.25 0)
-			(effects
-				(font
-					(size 1.27 1.27)
-				)
-				(hide yes)
-			)
-		)
-		(pin "2"
-		)
-		(pin "3"
-		)
-		(pin "1"
-		)
-		(instances
-			(project ""
-				(path "/ca333741-5826-495c-b860-5422aa5e17fc"
-					(reference "Q6")
-					(unit 1)
-				)
-			)
-		)
-	)
-	(symbol
 		(lib_id "Connector_Generic:Conn_01x03")
 		(at 294.64 120.65 0)
@@
 			)
 		)
-		(property "Footprint" ""
+		(property "Footprint" "Connector_Harwin:Harwin_LTek-Male_03_P2.00mm_Vertical"
 			(at 294.64 120.65 0)
 			(effects
@@
 			)
 		)
-		(property "Footprint" ""
+		(property "Footprint" "Connector_Harwin:Harwin_LTek-Male_2x08_P2.00mm_Vertical"
 			(at 307.34 187.96 0)
 			(effects
@@
 			)
 		)
-		(property "Footprint" ""
+		(property "Footprint" "Resistor_SMD:R_0805_2012Metric_Pad1.20x1.40mm_HandSolder"
 			(at 194.818 121.92 90)
 			(effects
@@
 			)
 		)
-		(property "Footprint" ""
+		(property "Footprint" "Jumper:Jumper_Harwin_S1621_P10.9mm"
 			(at 236.22 127 0)
 			(effects
@@
 			)
 		)
-		(property "Footprint" ""
+		(property "Footprint" "Connector_Harwin:Harwin_LTek-Male_02_P2.00mm_Vertical"
 			(at 227.33 135.89 0)
 			(effects
@@
 			)
 		)
-		(property "Footprint" ""
+		(property "Footprint" "Resistor_SMD:R_0805_2012Metric_Pad1.20x1.40mm_HandSolder"
 			(at 51.308 182.88 90)
 			(effects
@@
 			)
 		)
-		(property "Datasheet" "https://ngspice.sourceforge.io/docs/ngspice-html-manual/manual.xhtml#cha_MOSFETs"
+		(property "Datasheet" "https://www.onsemi.com/pdf/datasheet/ntb5860nl-d.pdf"
 			(at 337.82 100.33 0)
 			(effects
@@
 			)
 		)
-		(property "Footprint" ""
+		(property "Footprint" "Resistor_SMD:R_0805_2012Metric_Pad1.20x1.40mm_HandSolder"
 			(at 309.372 139.7 90)
 			(effects
@@
 			)
 		)
-		(property "Value" "D_Zener"
+		(property "Value" "HPZR-C50-QX"
 			(at 350.52 63.5 0)
 			(effects
@@
 			)
 		)
-		(property "Footprint" ""
+		(property "Footprint" "Diode_SMD:Nexperia_CFP3_SOD-123W"
 			(at 350.52 67.31 0)
 			(effects
@@
 			)
 		)
-		(property "Datasheet" "~"
+		(property "Datasheet" "https://assets.nexperia.com/documents/data-sheet/HPZR-Q_SER.pdf"
 			(at 350.52 67.31 0)
 			(effects
@@
 			)
 		)
-		(property "Description" "Zener diode"
+		(property "Description" "50V Zener Diode"
 			(at 350.52 67.31 0)
 			(effects
@@
 			)
 		)
-		(property "Footprint" ""
+		(property "Footprint" "Resistor_SMD:R_0805_2012Metric_Pad1.20x1.40mm_HandSolder"
 			(at 309.372 124.46 90)
 			(effects
@@
 			)
 		)
-		(property "Footprint" ""
+		(property "Footprint" "Connector_Harwin:Harwin_LTek-Male_2x06_P2.00mm_Vertical"
 			(at 276.86 182.88 0)
 			(effects
@@
 			)
 		)
-		(property "Footprint" ""
+		(property "Footprint" "Resistor_SMD:R_0805_2012Metric_Pad1.20x1.40mm_HandSolder"
 			(at 226.822 49.53 90)
 			(effects
@@
 			)
 		)
-		(property "Footprint" ""
+		(property "Footprint" "Resistor_SMD:R_0805_2012Metric_Pad1.20x1.40mm_HandSolder"
 			(at 328.93 111.252 90)
 			(effects
@@
 		(unit 1)
 		(exclude_from_sim no)
-		(in_bom yes)
+		(in_bom no)
 		(on_board yes)
 		(dnp no)
@@
 			)
 		)
-		(property "Footprint" ""
+		(property "Footprint" "Connector_Harwin:Harwin_LTek-Male_02_P2.00mm_Vertical"
 			(at 341.63 82.55 0)
 			(effects
@@
 			)
 		)
-		(property "Footprint" ""
+		(property "Footprint" "Capacitor_SMD:C_0805_2012Metric_Pad1.18x1.45mm_HandSolder"
 			(at 357.8352 77.47 0)
 			(effects
@@
 			)
 		)
-		(property "Footprint" ""
+		(property "Footprint" "Resistor_SMD:R_0805_2012Metric_Pad1.20x1.40mm_HandSolder"
 			(at 324.358 116.84 90)
 			(effects
@@
 			)
 		)
-		(property "Footprint" ""
+		(property "Footprint" "Connector_Harwin:Harwin_LTek-Male_02_P2.00mm_Vertical"
 			(at 400.05 85.09 0)
 			(effects
