File: Tractive_Battery_Board/Tractive_Battery_Board.kicad_sch (KiCad schematic)
At the start: 60 parts, among them J1 TS+/-, J12 Busbar_Temp_Sense, J13 E-Meter, J14 FTSH-107-01-F-DV-K-P-TR, J15 BMS_Temp_Sense, J2 HVIL, J3 Conn_01x12_Pin, J4 Conn_01x16_Pin, J8 Conn_01x03, Q1 NMOS, Q3 BSS308PE, SW1 SH_RESET_BUTTON, SW2 Y97KT23B5NAFP, U10 AP63205WU, U11 DS18B20Z, U12 STM32F446RETx, U15 ZXTR2005ZQ-13, U3 ISO1044BD, U9 MIC5504-3.3YM5, Y2 ECS-240-8-37B-CKY-TR

Commit message: mcu block layout
Parts:
- J12, J13, J15: footprint Connector_Harwin:Harwin_LTek-Male_02_P2.00mm_Vertical -> Connector_Molex:Molex_Nano-Fit_105309-xx02_1x02_P2.50mm_Vertical
- J8: value Conn_01x03 -> IMD_Connector
Connections:
- net SH_RESET is gone; now on net +5V: U12.50 (PA15)
- net IMD_Fault_3.3V: now also U12.24 (PC4); no longer U12.27 (PB1)
- net nBMS_Fault_3.3V: now also U12.25 (PC5); no longer U12.26 (PB0)
Other:
- note removed: "peep layout in folder"
- moved on the sheet: Y2
Changed lines of the file:
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@@
 		)
 	)
-	(text "peep layout in folder\n\n\n"
-		(exclude_from_sim no)
-		(at 62.484 83.312 0)
-		(effects
-			(font
-				(size 1.27 1.27)
-			)
-		)
-	)
 	(text "Ask firmware about TS1W pin assignmnet\n\n"
 		(exclude_from_sim no)
@@
 	)
 	(junction
-		(at 101.6 102.87)
+		(at 38.1 175.26)
 		(diameter 0)
 		(color 0 0 0 0)
 	)
 	(junction
-		(at 44.45 175.26)
+		(at 101.6 102.87)
 		(diameter 0)
 		(color 0 0 0 0)
@@
 	)
 	(junction
+		(at 38.1 161.29)
+		(diameter 0)
+		(color 0 0 0 0)
+	)
+	(junction
 		(at 46.99 43.18)
 		(diameter 0)
@@
 	)
 	(junction
-		(at 44.45 161.29)
-		(diameter 0)
-		(color 0 0 0 0)
-	)
-	(junction
 		(at 59.69 33.02)
 		(diameter 0)
@@
 	(wire
 		(pts
+			(xy 49.53 175.26) (xy 49.53 163.83)
+		)
+		(stroke
+			(width 0)
+			(type default)
+		)
+	)
+	(wire
+		(pts
 			(xy 72.39 63.5) (xy 77.47 63.5)
 		)
@@
 	(wire
 		(pts
-			(xy 34.29 161.29) (xy 44.45 161.29)
+			(xy 34.29 161.29) (xy 38.1 161.29)
 		)
 		(stroke
@@
 	(wire
 		(pts
-			(xy 49.53 167.64) (xy 52.07 167.64)
+			(xy 38.1 175.26) (xy 49.53 175.26)
+		)
+		(stroke
+			(width 0)
+			(type default)
+		)
+	)
+	(wire
+		(pts
+			(xy 43.18 167.64) (xy 45.72 167.64)
 		)
 		(stroke
@@
 	(wire
 		(pts
+			(xy 62.23 163.83) (xy 62.23 146.05)
+		)
+		(stroke
+			(width 0)
+			(type default)
+		)
+	)
+	(wire
+		(pts
 			(xy 312.42 190.5) (xy 318.77 190.5)
 		)
@@
 	(wire
 		(pts
-			(xy 44.45 163.83) (xy 44.45 161.29)
+			(xy 38.1 163.83) (xy 38.1 161.29)
 		)
 		(stroke
@@
 	(wire
 		(pts
+			(xy 71.12 166.37) (xy 73.66 166.37)
+		)
+		(stroke
+			(width 0)
+			(type default)
+		)
+	)
+	(wire
+		(pts
 			(xy 237.49 187.96) (xy 241.3 187.96)
 		)
@@
 	(wire
 		(pts
-			(xy 60.96 146.05) (xy 73.66 146.05)
+			(xy 62.23 146.05) (xy 73.66 146.05)
 		)
 		(stroke
@@
 	(wire
 		(pts
-			(xy 34.29 175.26) (xy 44.45 175.26)
+			(xy 34.29 175.26) (xy 38.1 175.26)
 		)
 		(stroke
@@
 	(wire
 		(pts
-			(xy 60.96 175.26) (xy 60.96 146.05)
-		)
-		(stroke
-			(width 0)
-			(type default)
-		)
-	)
-	(wire
-		(pts
 			(xy 59.69 71.12) (xy 57.15 71.12)
 		)
@@
 	(wire
 		(pts
-			(xy 44.45 175.26) (xy 60.96 175.26)
+			(xy 36.83 38.1) (xy 34.29 38.1)
 		)
 		(stroke
@@
 	(wire
 		(pts
-			(xy 36.83 38.1) (xy 34.29 38.1)
+			(xy 38.1 161.29) (xy 59.69 161.29)
 		)
 		(stroke
@@
 	(wire
 		(pts
-			(xy 44.45 171.45) (xy 44.45 175.26)
+			(xy 38.1 171.45) (xy 38.1 175.26)
 		)
 		(stroke
@@
 	(wire
 		(pts
-			(xy 101.6 110.49) (xy 111.76 110.49)
+			(xy 71.12 168.91) (xy 73.66 168.91)
 		)
 		(stroke
@@
 	(wire
 		(pts
-			(xy 248.92 142.24) (xy 248.92 127)
+			(xy 101.6 110.49) (xy 111.76 110.49)
 		)
 		(stroke
@@
 	(wire
 		(pts
-			(xy 27.94 63.5) (xy 27.94 64.77)
+			(xy 248.92 142.24) (xy 248.92 127)
 		)
 		(stroke
@@
 	(wire
 		(pts
-			(xy 114.3 176.53) (xy 118.11 176.53)
+			(xy 27.94 63.5) (xy 27.94 64.77)
 		)
 		(stroke
@@
 	(wire
 		(pts
+			(xy 49.53 163.83) (xy 62.23 163.83)
+		)
+		(stroke
+			(width 0)
+			(type default)
+		)
+	)
+	(wire
+		(pts
 			(xy 72.39 63.5) (xy 72.39 73.66)
 		)
@@
 	(wire
 		(pts
-			(xy 26.67 167.64) (xy 39.37 167.64)
+			(xy 26.67 167.64) (xy 33.02 167.64)
 		)
 		(stroke
@@
 	(wire
 		(pts
-			(xy 114.3 179.07) (xy 118.11 179.07)
-		)
-		(stroke
-			(width 0)
-			(type default)
-		)
-	)
-	(wire
-		(pts
 			(xy 59.69 161.29) (xy 59.69 143.51)
 		)
@@
 	(wire
 		(pts
-			(xy 44.45 161.29) (xy 59.69 161.29)
-		)
-		(stroke
-			(width 0)
-			(type default)
-		)
-	)
-	(wire
-		(pts
 			(xy 39.37 231.14) (xy 41.91 231.14)
 		)
@@
 	(global_label "nBMS_Fault_3.3V"
 		(shape output)
-		(at 118.11 176.53 0)
+		(at 71.12 168.91 180)
 		(fields_autoplaced yes)
 		(effects
@@
 				(size 1.27 1.27)
 			)
-			(justify left)
+			(justify right)
 		)
 		(property "Intersheetrefs" "${INTERSHEET_REFS}"
-			(at 137.0002 176.53 0)
+			(at 52.2298 168.91 0)
 			(effects
 				(font
 					(size 1.27 1.27)
 				)
-				(justify left)
+				(justify right)
 				(hide yes)
 			)
@@
 	(global_label "IMD_Fault_3.3V"
 		(shape input)
-		(at 118.11 179.07 0)
+		(at 71.12 166.37 180)
 		(fields_autoplaced yes)
 		(effects
@@
 				(size 1.27 1.27)
 			)
-			(justify left)
+			(justify right)
 		)
 		(property "Intersheetrefs" "${INTERSHEET_REFS}"
-			(at 135.2465 179.07 0)
+			(at 53.9835 166.37 0)
 			(effects
 				(font
 					(size 1.27 1.27)
 				)
-				(justify left)
+				(justify right)
 				(hide yes)
 			)
@@
 		)
 	)
-	(global_label "SH_RESET"
+	(global_label "SH_RESET+"
 		(shape input)
 		(at 118.11 171.45 0)
@@
 		)
 		(property "Intersheetrefs" "${INTERSHEET_REFS}"
-			(at 130.3479 171.45 0)
+			(at 131.9203 171.45 0)
 			(effects
 				(font
@@
 	(symbol
 		(lib_id "power:GND")
-		(at 52.07 167.64 0)
+		(at 45.72 167.64 0)
 		(unit 1)
 		(exclude_from_sim no)
@@
 		(fields_autoplaced yes)
 		(property "Reference" "#PWR045"
-			(at 52.07 173.99 0)
+			(at 45.72 173.99 0)
 			(effects
 				(font
@@
 		)
 		(property "Value" "GND"
-			(at 52.07 172.72 0)
+			(at 45.72 172.72 0)
 			(effects
 				(font
@@
 		)
 		(property "Footprint" ""
-			(at 52.07 167.64 0)
+			(at 45.72 167.64 0)
 			(effects
 				(font
@@
 		)
 		(property "Datasheet" ""
-			(at 52.07 167.64 0)
+			(at 45.72 167.64 0)
 			(effects
 				(font
@@
 		)
 		(property "Description" "Power symbol creates a global label with name \"GND\" , ground"
-			(at 52.07 167.64 0)
+			(at 45.72 167.64 0)
 			(effects
 				(font
@@
 			)
 		)
-		(property "Footprint" "Connector_Harwin:Harwin_LTek-Male_02_P2.00mm_Vertical"
+		(property "Footprint" "Connector_Molex:Molex_Nano-Fit_105309-xx02_1x02_P2.50mm_Vertical"
 			(at 260.35 142.24 0)
 			(effects
@@
 			)
 		)
-		(property "Footprint" "Connector_Harwin:Harwin_LTek-Male_02_P2.00mm_Vertical"
+		(property "Footprint" "Connector_Molex:Molex_Nano-Fit_105309-xx02_1x02_P2.50mm_Vertical"
 			(at 260.35 127 0)
 			(effects
@@
 			)
 		)
-		(property "Value" "Conn_01x03"
+		(property "Value" "IMD_Connector"
 			(at 294.64 114.3 0)
 			(effects
@@
 			)
 		)
-		(property "Footprint" "Connector_Harwin:Harwin_LTek-Male_02_P2.00mm_Vertical"
+		(property "Footprint" "Connector_Molex:Molex_Nano-Fit_105309-xx02_1x02_P2.50mm_Vertical"
 			(at 227.33 135.89 0)
 			(effects
@@
 	(symbol
 		(lib_id "Device:Crystal_GND24")
-		(at 44.45 167.64 90)
+		(at 38.1 167.64 90)
 		(unit 1)
 		(exclude_from_sim no)
@@
 		(dnp no)
 		(property "Reference" "Y2"
-			(at 43.942 156.972 90)
+			(at 37.592 156.972 90)
 			(effects
 				(font
@@
 		)
 		(property "Value" "ECS-240-8-37B-CKY-TR"
-			(at 45.212 159.512 90)
+			(at 38.862 159.512 90)
 			(effects
 				(font
@@
 		)
 		(property "Footprint" "Crystal:Crystal_SMD_2016-4Pin_2.0x1.6mm"
-			(at 44.45 167.64 0)
+			(at 38.1 167.64 0)
 			(effects
 				(font
@@
 		)
 		(property "Datasheet" "https://ecsxtal.com/store/pdf/ECX-1637B.pdf"
-			(at 44.45 167.64 0)
+			(at 38.1 167.64 0)
 			(effects
 				(font
@@
 		)
 		(property "Description" "Four pin crystal, GND on pins 2 and 4"
-			(at 44.45 167.64 0)
+			(at 38.1 167.64 0)
 			(effects
 				(font
@@
 		)
 		(property "Digi PN" "XC3063CT-ND"
-			(at 44.45 167.64 0)
+			(at 38.1 167.64 0)
 			(effects
 				(font
@@
 		)
 		(property "MFG" "ECS"
-			(at 44.45 167.64 0)
+			(at 38.1 167.64 0)
 			(effects
 				(font
@@
 		)
 		(property "MFG PN" "ECS-240-8-37B-CKY-TR"
-			(at 44.45 167.64 0)
+			(at 38.1 167.64 0)
 			(effects
 				(font
@@
 		)
 		(property "Digi URL" "https://www.digikey.com/en/products/detail/ecs-inc/ECS-240-8-37B-CKY-TR/9838850"
-			(at 44.45 167.64 90)
+			(at 38.1 167.64 90)
 			(effects
 				(font

Commit message: SH_Reset fixes
Parts:
- removed SW1: SH_RESET_BUTTON, symbol Switch:SW_Push
- added R42: 10k, Resistor_SMD:R_0805_2012Metric_Pad1.20x1.40mm_HandSolder, symbol Device:R
- added R43: 4.9k, Resistor_SMD:R_0805_2012Metric_Pad1.20x1.40mm_HandSolder, symbol Device:R
Connections:
- net +5V: now also R42.2; no longer U12.50 (PA15)
- net GND: now also R43.2
- new net SH_RESET+_3.3V: R42.1, R43.1, U12.50 (PA15)
Other:
- moved on the sheet: R18

Commit message: SH_Reset tweaks
Parts:
- added SW1: SW_Push, symbol Switch:SW_Push
- Q1: footprint (none) -> Package_TO_SOT_SMD:SOT-23_Handsoldering
- R18: now not fitted
Connections:
- net +5V: now also SW1.1; no longer R42.2
- net GND: now also R42.1; no longer R43.2
- net SH_RESET-: now also R43.1, SW1.2
- removed net SH_RESET+_3.3V: R42.1, R43.1, U12.50 (PA15)
- new net SH_RESET_3.3V: R42.2, R43.2, U12.50 (PA15)
Other:
- note added: "I am confused </3"
- note added: "am i chud"
- note added: "source digikey part"
- moved on the sheet: R42, R43
