File: Tractive_Battery_Board/Shutdown Logic.kicad_sch (KiCad schematic)
At the start: 29 parts, among them J10 Shutdown IL, K1 G6BK-1114P-US, K2 G6BK-1114P-US, K4 G6SK-2G, U13 SZNUD3124LT1G, U14 SZNUD3124LT1G, U2 74HC14, U4 SZNUD3124LT1G, U5 MCP6004, U6 SN74HCS08DR, U8 SZNUD3124LT1G

Commit message: pin assignments + net naming
Parts:
- added C12: 15nF, symbol Device:C
Connections:
- net GND: now also C12.2; no longer R38.2
- net nIMD_FAULT_DELAYED_5V: no longer K4.5, R38.1
- net BMS_FAULT renamed BMS_FAULT_DELAYED
- net IMD_Fault renamed IMD_FAULT_DELAYED
- net nBMS_FAULT_DELAYED_5V renamed nBMS_FAULT_VCU
- new net: K4.5, R38.1
- new net nIMD_FAULT_VCU: C12.1, R38.2
Other:
- moved on the sheet: R38

Commit message: bms changes
Parts:
- removed K1, K2: G6BK-1114P-US, FS_3_Global_Footprint_Library:RELAY_G6BK-1114P-US_OMR, symbol 1FS_2_Global_Symbol_Library:G6BK-1114P-US
- added C37: 15nF, symbol Device:C
- added D3, D7: D, Diode_SMD:D_2010_5025Metric_Pad1.52x2.65mm_HandSolder, symbol Device:D
- added K1, K5: Fujitsu_FTR-LYAA005x, Relay_THT:Relay_SPST-NO_Fujitsu_FTR-LYAA005x_FormA_Vertical, symbol Relay:Fujitsu_FTR-LYAA005x
- added K2: G6SK-2G, Relay_SMD:Relay_DPDT_Omron_G6SK-2G, symbol Relay:G6SK-2
- added R54: 100k, Resistor_SMD:R_0603_1608Metric_Pad0.98x0.95mm_HandSolder, symbol Device:R
Connections:
- net +12V: now also K4.4, K2.1, K2.4, K2.6
- net +5V: now also K4.9, K2.9; no longer K4.4
- net GND: now also C37.2, D3.2 (A), D7.2 (A), K1.A2, K5.A2
- net Shutdown_TB_In: now also K5.14
- net nBMS_FAULT_VCU: now also C37.1, R54.2; no longer U2.2, U8.1
- net at J10.1 (Pin_1), TP8.1: now also K1.13
- net at U8.3: now also K2.12
- net at U4.3: now also K2.7
- net at TP2.1: now also K1.14, K5.13
- net at K4.5: now also D7.1 (K), K1.A1; no longer R38.1
- net at K4.8: now also R38.1
- new net: D3.1 (K), K2.5, K5.A1
- new net: K2.8, R54.1
- new net nBMS_FAULT_DELAYED_5V: U2.2, U8.1
Other:
- moved on the sheet: C12, C7, C9, D2, D4, J10, K4, R1, R14, R16, R38, R39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

Commit message: updated 2n1 relays
Parts:
- removed U13, U14, U4, U8: SZNUD3124LT1G, Package_TO_SOT_SMD:TSOT-23_HandSoldering, symbol FS_4_Global_Symbol_Library:SZNUD3124LT1G
- added U13, U4: SZNUD3124DMT1G, Package_TO_SOT_SMD:SC-74-6_1.55x2.9mm_P0.95mm, symbol FS_4_Global_Symbol_Library:SZNUD3124DMT1G
Connections:
- net BMS_FAULT_DELAYED: now also U4.5
- net GND: now also U13.1, U13.4, U4.1, U4.4
- net IMD_FAULT_DELAYED: now also U13.5
- net nBMS_FAULT_DELAYED_5V: now also U4.2
- net nIMD_Set: now also U13.2
- net at K2.7: now also U4.3
- net at K2.12: now also U4.6
- net at K4.12: now also U13.6
- net at K4.7: now also U13.3

Commit message: fixed librararies
Parts:
- removed K1, K5: Fujitsu_FTR-LYAA005x, Relay_THT:Relay_SPST-NO_Fujitsu_FTR-LYAA005x_FormA_Vertical, symbol Relay:Fujitsu_FTR-LYAA005x
- added K1, K5: G6DN-1A, FS_4_Global_Footprint_Library:RELAY_G6DN-1A, symbol FS_4_Global_Symbol_Library:G6DN-1A
Connections:
- net GND: now also K1.2, K5.2
- net Shutdown_TB_In: now also K5.5
- net at J10.1 (Pin_1), TP8.1: now also K1.8
- net at D7.1 (K), K4.5: now also K1.1
- net at D3.1 (K), K2.5: now also K5.1
- net at TP2.1: now also K1.5, K5.8
Other:
- moved on the sheet: TP1, TP5, U13B, U2G, U4B, U5E, U6E

Commit message: mcu protections
Parts:
- added C38, C39, C40: 100nF, symbol Device:C
Connections:
- net +5V: now also C38.1, C39.1, C40.1
- net GND: now also C38.2, C39.2, C40.2
- net at R39.1, R40.2: now also U5.6 (-); no longer U5.2 (-)
- net at U5.1: now also U6.2; no longer U6.10
- net at C9.1, D4.2 (A), R1.2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: now also U5.5 (+); no longer U5.3 (+)
- net at U5.7: now also U6.10; no longer U6.2
- net at C7.1, D2.2 (A), R9.2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: now also U5.3 (+); no longer U5.5 (+)
- net at R14.1, R16.2: now also U5.2 (-); no longer U5.6 (-)
Other:
- note added: "BMS NO Relay"
- note added: "IMD NO Relay"
- note added: "~100Hz RC Filter"
- note removed: "BMS_Relay"
- note removed: "IMD Relay"
- moved on the sheet: C12, C37, C7, C9, D2, D3, D4, D7, J10, K1, K2, K4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

Commit message: added nanofit footprints
Parts:
- J10: footprint Connector_Harwin:Harwin_LTek-Male_02_P2.00mm_Vertical -> FS_4_Global_Footprint_Library:CONN_SD-105431-001_02_MOL
Changed lines of the file:
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@@
 			)
 		)
-		(property "Footprint" "Connector_Harwin:Harwin_LTek-Male_02_P2.00mm_Vertical"
+		(property "Footprint" "FS_4_Global_Footprint_Library:CONN_SD-105431-001_02_MOL"
 			(at 361.95 87.63 0)
 			(effects

Commit message: cleanup + IMD voltage divider fix
Parts:
- removed C12, C37: 15nF, symbol Device:C
- removed R38, R54: 100k, Resistor_SMD:R_0603_1608Metric_Pad0.98x0.95mm_HandSolder, symbol Device:R
Connections:
- net nBMS_FAULT_VCU: now also K2.8
- net nIMD_FAULT_VCU: now also K4.8
Other:
- note removed: "~100Hz RC Filter"

Commit message: new HVIL + connector footprint renames
Parts:
- C38, C39, C40: footprint (none) -> Capacitor_SMD:C_0603_1608Metric_Pad1.08x0.95mm_HandSolder
