File: Tractive_Battery_Board/TB_Precharge.kicad_sch (KiCad schematic)
At the start: 6 parts, among them J5 Conn_01x02, J6 IRs Power, K3 J102K1CS324VDC.20, U16 SZNUD3124LT1G, U17 SZNUD3124LT1G, U2 74HC14

Commit message: removed duped components
Parts:
- removed U16, U17: SZNUD3124LT1G, Package_TO_SOT_SMD:TSOT-23_HandSoldering, symbol FS_4_SCHEMATICS:SZNUD3124LT1G
- added U16, U17: SZNUD3124LT1G, Package_TO_SOT_SMD:TSOT-23_HandSoldering, symbol FS_4_Global_Symbol_Library:SZNUD3124LT1G
Connections:
- net GND: now also U16.2, U17.2
- net nPreCharge_Control: now also U17.1
- net at U2.8: now also U16.1
- net at K3.A1: now also U16.3
- net at J6.1: now also U17.3

Commit message: footprint updates + started layout
Parts:
- J5: footprint (none) -> Connector_Harwin:Harwin_LTek-Male_02_P2.00mm_Vertical
- J6: footprint Connector_Molex:Molex_Nano-Fit_105309-xx04_1x04_P2.50mm_Vertical -> Connector_Harwin:Harwin_LTek-Male_04_P2.00mm_Vertical
- U2: footprint (none) -> Package_SO:SOIC-14_3.9x8.7mm_P1.27mm
Changed lines of the file:
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@@
 			)
 		)
-		(property "Footprint" ""
+		(property "Footprint" "Connector_Harwin:Harwin_LTek-Male_02_P2.00mm_Vertical"
 			(at 127 58.42 0)
 			(effects
@@
 			)
 		)
-		(property "Footprint" ""
+		(property "Footprint" "Package_SO:SOIC-14_3.9x8.7mm_P1.27mm"
 			(at 66.04 52.07 0)
 			(effects
@@
 			)
 		)
-		(property "Footprint" "Connector_Molex:Molex_Nano-Fit_105309-xx04_1x04_P2.50mm_Vertical"
+		(property "Footprint" "Connector_Harwin:Harwin_LTek-Male_04_P2.00mm_Vertical"
 			(at 97.79 87.63 0)
 			(effects

Commit message: IR+ relay changed
Parts:
- removed U17: SZNUD3124LT1G, Package_TO_SOT_SMD:TSOT-23_HandSoldering, symbol FS_4_Global_Symbol_Library:SZNUD3124LT1G
- added Q2: NMOS, Package_TO_SOT_SMD:SOT-23_Handsoldering, symbol Simulation_SPICE:NMOS
Connections:
- net GND: now also Q2.1 (D)
- net nPreCharge_Control: now also Q2.2 (G)
- net at J6.1: now also Q2.3 (S)
Other:
- note added: "using a general nmos, double check if correct"
Changed lines of the file:
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@@
+		)
+	)
+	(text "using a general nmos, double check if correct\n"
+		(exclude_from_sim no)
+		(at 59.944 104.648 0)
+		(effects
+			(font
+				(size 1.27 1.27)
+			)
 		)
 	)
@@
 	(wire
 		(pts
+			(xy 59.69 85.09) (xy 59.69 87.63)
+		)
+		(stroke
+			(width 0)
+			(type default)
+		)
+	)
+	(wire
+		(pts
 			(xy 92.71 92.71) (xy 76.2 92.71)
 		)
@@
 	(wire
 		(pts
+			(xy 59.69 97.79) (xy 59.69 100.33)
+		)
+		(stroke
+			(width 0)
+			(type default)
+		)
+	)
+	(wire
+		(pts
 			(xy 53.34 52.07) (xy 58.42 52.07)
 		)
@@
 	(wire
 		(pts
-			(xy 46.99 92.71) (xy 45.72 92.71)
+			(xy 45.72 92.71) (xy 52.07 92.71)
 		)
 		(stroke
@@
 	)
 	(symbol
-		(lib_id "FS_4_Global_Symbol_Library:SZNUD3124LT1G")
-		(at 59.69 92.71 0)
+		(lib_id "Simulation_SPICE:NMOS")
+		(at 57.15 92.71 0)
+		(mirror x)
 		(unit 1)
 		(exclude_from_sim no)
@@
 		(on_board yes)
 		(dnp no)
-		(property "Reference" "U17"
-			(at 61.468 94.488 0)
+		(property "Reference" "Q2"
+			(at 62.23 95.504 0)
 			(effects
 				(font
@@
 			)
 		)
-		(property "Value" "SZNUD3124LT1G"
-			(at 61.468 97.028 0)
+		(property "Value" "NMOS"
+			(at 62.23 92.964 0)
 			(effects
 				(font
@@
 			)
 		)
-		(property "Footprint" "Package_TO_SOT_SMD:TSOT-23_HandSoldering"
-			(at 86.614 76.708 0)
-			(effects
-				(font
-					(size 1.27 1.27)
-					(italic yes)
-				)
-				(hide yes)
-			)
-		)
-		(property "Datasheet" "https://www.onsemi.com/pdf/datasheet/nud3124-d.pdf"
-			(at 91.948 81.788 0)
-			(effects
-				(font
-					(size 1.27 1.27)
-					(italic yes)
-				)
-				(hide yes)
-			)
-		)
-		(property "Description" "Relay Driver"
-			(at 70.358 74.168 0)
-			(effects
-				(font
-					(size 1.27 1.27)
-				)
-				(hide yes)
-			)
-		)
-		(property "Digi PN" "SZNUD3124LT1GOSCT-ND"
-			(at 76.962 71.628 0)
-			(effects
-				(font
-					(size 1.27 1.27)
-				)
-				(hide yes)
-			)
-		)
-		(property "Digi URL" "https://www.digikey.com/en/products/detail/onsemi/SZNUD3124LT1G/3063416"
-			(at 103.632 79.248 0)
-			(effects
-				(font
-					(size 1.27 1.27)
-				)
-				(hide yes)
-			)
-		)
-		(property "MFG" "onsemi"
-			(at 68.072 84.328 0)
-			(effects
-				(font
-					(size 1.27 1.27)
-				)
-				(hide yes)
-			)
-		)
-		(property "MFG PN" "SZNUD3124LT1G"
-			(at 72.39 69.088 0)
+		(property "Footprint" "Package_TO_SOT_SMD:SOT-23_Handsoldering"
+			(at 62.23 95.25 0)
+			(effects
+				(font
+					(size 1.27 1.27)
+				)
+				(hide yes)
+			)
+		)
+		(property "Datasheet" "https://www.onsemi.com/pdf/datasheet/ntb5860nl-d.pdf"
+			(at 57.15 80.01 0)
+			(effects
+				(font
+					(size 1.27 1.27)
+				)
+				(hide yes)
+			)
+		)
+		(property "Description" "N-MOSFET transistor, drain/source/gate"
+			(at 57.15 92.71 0)
+			(effects
+				(font
+					(size 1.27 1.27)
+				)
+				(hide yes)
+			)
+		)
+		(property "Sim.Device" "NMOS"
+			(at 57.15 75.565 0)
+			(effects
+				(font
+					(size 1.27 1.27)
+				)
+				(hide yes)
+			)
+		)
+		(property "Sim.Type" "VDMOS"
+			(at 57.15 73.66 0)
+			(effects
+				(font
+					(size 1.27 1.27)
+				)
+				(hide yes)
+			)
+		)
+		(property "Sim.Pins" "1=D 2=G 3=S"
+			(at 57.15 77.47 0)
 			(effects
 				(font
@@
 		(pin "1"
 		)
+		(pin "2"
+		)
 		(pin "3"
-		)
-		(pin "2"
 		)
 		(instances
 			(project "Tractive_Battery_Board"
 				(path "/ca333741-5826-495c-b860-5422aa5e17fc/fa150f42-0d9b-43a1-bf36-032543240a34"
-					(reference "U17")
+					(reference "Q2")
 					(unit 1)
 				)

Commit message: fixed librararies
Parts:
- removed K3: J102K1CS324VDC.20, FS_4_SCHEMATICS:J102K1CS324VDC.20, symbol FS_4_SCHEMATICS:J102K1CS324VDC.20
- added K3: J102K1CS312VDC.20, FS_4_Global_Footprint_Library:J102K1CS312VDC.20, symbol FS_4_Global_Symbol_Library:J102K1CS312DC.20
Connections:
- net IRs_Final: now also K3.A2
- net at J5.1 (Pin_1): now also K3.4
- net at J5.2 (Pin_2): now also K3.2, K3.3
- net at U16.3: now also K3.A1
Changed lines of the file:
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@@
+	)
+	(symbol
+		(lib_id "FS_4_Global_Symbol_Library:J102K1CS312DC.20")
+		(at 109.22 48.26 270)
+		(unit 1)
+		(exclude_from_sim no)
+		(in_bom yes)
+		(on_board yes)
+		(dnp no)
+		(fields_autoplaced yes)
+		(property "Reference" "K3"
+			(at 109.22 33.02 90)
+			(effects
+				(font
+					(size 1.27 1.27)
+				)
+			)
+		)
+		(property "Value" "J102K1CS312VDC.20"
+			(at 109.22 35.56 90)
+			(effects
+				(font
+					(size 1.27 1.27)
+				)
+			)
+		)
+		(property "Footprint" "FS_4_Global_Footprint_Library:J102K1CS312VDC.20"
+			(at 109.22 48.26 0)
+			(effects
+				(font
+					(size 1.27 1.27)
+				)
+				(hide yes)
+			)
+		)
+		(property "Datasheet" "https://www.citrelay.com/wp-content/uploads/2025/05/Relay-J102.pdf"
+			(at 109.22 48.26 0)
+			(effects
+				(font
+					(size 1.27 1.27)
+				)
+				(hide yes)
+			)
+		)
+		(property "Description" "Precharge Relay"
+			(at 109.22 48.26 0)
+			(effects
+				(font
+					(size 1.27 1.27)
+				)
+				(hide yes)
+			)
+		)
+		(property "Digi PN" "2449-J102K1CS324VDC.20-ND"
+			(at 109.22 48.26 0)
+			(effects
+				(font
+					(size 1.27 1.27)
+				)
+				(hide yes)
+			)
+		)
+		(property "MFG" "CIT Relay and Switch"
+			(at 109.22 48.26 0)
+			(effects
+				(font
+					(size 1.27 1.27)
+				)
+				(hide yes)
+			)
+		)
+		(property "MFG PN" "J102K1CS324VDC.20"
+			(at 109.22 48.26 0)
+			(effects
+				(font
+					(size 1.27 1.27)
+				)
+				(hide yes)
+			)
+		)
+		(property "Digi URL" ""
+			(at 109.22 48.26 0)
+			(effects
+				(font
+					(size 1.27 1.27)
+				)
+				(hide yes)
+			)
+		)
+		(pin "4"
+		)
+		(pin "A2"
+		)
+		(pin "A1"
+		)
+		(pin "1"
+		)
+		(pin "3"
+		)
+		(pin "2"
+		)
+		(instances
+			(project ""
+				(path "/ca333741-5826-495c-b860-5422aa5e17fc/fa150f42-0d9b-43a1-bf36-032543240a34"
+					(reference "K3")
+					(unit 1)
+				)
+			)
+		)
 	)
 	(symbol
@@
 					(unit 1)
 				)
-			)
-		)
-	)
-	(symbol
-		(lib_id "FS_4_SCHEMATICS:J102K1CS324VDC.20")
-		(at 109.22 48.26 270)
-		(unit 1)
-		(exclude_from_sim no)
-		(in_bom yes)
-		(on_board yes)
-		(dnp no)
-		(property "Reference" "K3"
-			(at 109.22 33.528 90)
-			(effects
-				(font
-					(size 1.27 1.27)
-				)
-			)
-		)
-		(property "Value" "J102K1CS324VDC.20"
-			(at 109.22 35.56 90)
-			(effects
-				(font
-					(size 1.27 1.27)
-				)
-			)
-		)
-		(property "Footprint" "FS_4_SCHEMATICS:J102K1CS324VDC.20"
-			(at 109.22 48.26 0)
-			(effects
-				(font
-					(size 1.27 1.27)
-				)
-				(hide yes)
-			)
-		)
-		(property "Datasheet" "https://www.citrelay.com/wp-content/uploads/2025/05/Relay-J102.pdf"
-			(at 109.22 48.26 0)
-			(effects
-				(font
-					(size 1.27 1.27)
-				)
-				(hide yes)
-			)
-		)
-		(property "Description" "Precharge Relay"
-			(at 109.22 48.26 0)
-			(effects
-				(font
-					(size 1.27 1.27)
-				)
-				(hide yes)
-			)
-		)
-		(property "Digi PN" "2449-J102K1CS324VDC.20-ND"
-			(at 109.22 48.26 0)
-			(effects
-				(font
-					(size 1.27 1.27)
-				)
-				(hide yes)
-			)
-		)
-		(property "MFG" "CIT Relay and Switch"
-			(at 109.22 48.26 0)
-			(effects
-				(font
-					(size 1.27 1.27)
-				)
-				(hide yes)
-			)
-		)
-		(property "MFG PN" "J102K1CS324VDC.20"
-			(at 109.22 48.26 0)
-			(effects
-				(font
-					(size 1.27 1.27)
-				)
-				(hide yes)
-			)
-		)
-		(property "Digi URL" "https://www.digikey.com/en/products/detail/cit-relay-and-switch/J102K1CS324VDC-20/14001744"
-			(at 109.22 48.26 0)
-			(effects
-				(font
-					(size 1.27 1.27)
-				)
-				(hide yes)
-			)
-		)
-		(pin "1"
-		)
-		(pin "2"
-		)
-		(pin "4"
-		)
-		(pin "A1"
-		)
-		(pin "A2"
-		)
-		(pin "3"
-		)
-		(instances
-			(project "Tractive_Battery_Board"
-				(path "/ca333741-5826-495c-b860-5422aa5e17fc/fa150f42-0d9b-43a1-bf36-032543240a34"
-					(reference "K3")
-					(unit 1)
-				)

Commit message: mcu protections
Parts:
- removed U16: SZNUD3124LT1G, Package_TO_SOT_SMD:TSOT-23_HandSoldering, symbol FS_4_Global_Symbol_Library:SZNUD3124LT1G
- added U8: SZNUD3124DMT1G, Package_TO_SOT_SMD:SC-74-6_1.55x2.9mm_P0.95mm, symbol FS_4_Global_Symbol_Library:SZNUD3124DMT1G
Connections:
- net GND: now also U8.1
- net at K3.A1: now also U8.6
- net at U2.8: now also U8.2
Other:
- note added: "nPrecharge_Control outputs LOW during precharge"
- note removed: "Precharge_control outputs LOW during precharge"
Changed lines of the file:
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@@
 	(generator_version "9.0")
 	(paper "B")
-	(text "Precharge_control outputs LOW during precharge\n"
+	(text "nPrecharge_Control outputs LOW during precharge\n"
 		(exclude_from_sim no)
 		(at 55.372 80.772 0)
@@
 				(path "/ca333741-5826-495c-b860-5422aa5e17fc/fa150f42-0d9b-43a1-bf36-032543240a34"
 					(reference "J5")
+					(unit 1)
+				)
+			)
+		)
+	)
+	(symbol
+		(lib_id "FS_4_Global_Symbol_Library:SZNUD3124DMT1G")
+		(at 88.9 52.07 0)
+		(unit 1)
+		(exclude_from_sim no)
+		(in_bom yes)
+		(on_board yes)
+		(dnp no)
+		(property "Reference" "U8"
+			(at 83.82 42.418 0)
+			(effects
+				(font
+					(size 1.27 1.27)
+				)
+				(justify right)
+			)
+		)
+		(property "Value" "SZNUD3124DMT1G"
+			(at 83.82 44.958 0)
+			(effects
+				(font
+					(size 1.27 1.27)
+				)
+				(justify right)
+			)
+		)
+		(property "Footprint" "Package_TO_SOT_SMD:SC-74-6_1.55x2.9mm_P0.95mm"
+			(at 115.824 36.068 0)
+			(effects
+				(font
+					(size 1.27 1.27)
+					(italic yes)
+				)
+				(hide yes)
+			)
+		)
+		(property "Datasheet" "https://www.onsemi.com/pdf/datasheet/nud3124-d.pdf"
+			(at 121.158 41.148 0)
+			(effects
+				(font
+					(size 1.27 1.27)
+					(italic yes)
+				)
+				(hide yes)
+			)
+		)
+		(property "Description" "Relay Driver (Dual Case)"
+			(at 105.664 33.528 0)
+			(effects
+				(font
+					(size 1.27 1.27)
+				)
+				(hide yes)
+			)
+		)
+		(property "Digi PN" "SZNUD3124DMT1GOSCT-ND"
+			(at 106.934 30.988 0)
+			(effects
+				(font
+					(size 1.27 1.27)
+				)
+				(hide yes)
+			)
+		)
+		(property "Digi URL" "https://www.digikey.com/en/products/detail/onsemi/SZNUD3124DMT1G/3063415"
+			(at 132.842 38.608 0)
+			(effects
+				(font
+					(size 1.27 1.27)
+				)
+				(hide yes)
+			)
+		)
+		(property "MFG" "onsemi"
+			(at 97.028 43.688 0)
+			(effects
+				(font
+					(size 1.27 1.27)
+				)
+				(hide yes)
+			)
+		)
+		(property "MFG PN" "SZNUD3124DMT1G"
+			(at 102.362 28.448 0)
+			(effects
+				(font
+					(size 1.27 1.27)
+				)
+				(hide yes)
+			)
+		)
+		(pin "6"
+		)
+		(pin "1"
+		)
+		(pin "5"
+		)
+		(pin "3"
+		)
+		(pin "4"
+		)
+		(pin "2"
+		)
+		(instances
+			(project ""
+				(path "/ca333741-5826-495c-b860-5422aa5e17fc/fa150f42-0d9b-43a1-bf36-032543240a34"
+					(reference "U8")
 					(unit 1)
 				)
@@
 					(unit 1)
 				)
-			)
-		)
-	)
-	(symbol
-		(lib_id "FS_4_Global_Symbol_Library:SZNUD3124LT1G")
-		(at 88.9 52.07 0)
-		(unit 1)
-		(exclude_from_sim no)
-		(in_bom yes)
-		(on_board yes)
-		(dnp no)
-		(property "Reference" "U16"
-			(at 83.566 43.18 0)
-			(effects
-				(font
-					(size 1.27 1.27)
-				)
-				(justify right)
-			)
-		)
-		(property "Value" "SZNUD3124LT1G"
-			(at 83.566 45.72 0)
-			(effects
-				(font
-					(size 1.27 1.27)
-				)
-				(justify right)
-			)
-		)
-		(property "Footprint" "Package_TO_SOT_SMD:TSOT-23_HandSoldering"
-			(at 115.824 36.068 0)
-			(effects
-				(font
-					(size 1.27 1.27)
-					(italic yes)
-				)
-				(hide yes)
-			)
-		)
-		(property "Datasheet" "https://www.onsemi.com/pdf/datasheet/nud3124-d.pdf"
-			(at 121.158 41.148 0)
-			(effects
-				(font
-					(size 1.27 1.27)
-					(italic yes)
-				)
-				(hide yes)
-			)
-		)
-		(property "Description" "Relay Driver"
-			(at 99.568 33.528 0)
-			(effects
-				(font
-					(size 1.27 1.27)
-				)
-				(hide yes)
-			)
-		)
-		(property "Digi PN" "SZNUD3124LT1GOSCT-ND"
-			(at 106.172 30.988 0)
-			(effects
-				(font
-					(size 1.27 1.27)
-				)
-				(hide yes)
-			)
-		)
-		(property "Digi URL" "https://www.digikey.com/en/products/detail/onsemi/SZNUD3124LT1G/3063416"
-			(at 132.842 38.608 0)
-			(effects
-				(font
-					(size 1.27 1.27)
-				)
-				(hide yes)
-			)
-		)
-		(property "MFG" "onsemi"
-			(at 97.282 43.688 0)
-			(effects
-				(font
-					(size 1.27 1.27)
-				)
-				(hide yes)
-			)
-		)
-		(property "MFG PN" "SZNUD3124LT1G"
-			(at 101.6 28.448 0)
-			(effects
-				(font
-					(size 1.27 1.27)
-				)
-				(hide yes)
-			)
-		)
-		(pin "1"
-		)
-		(pin "3"
-		)
-		(pin "2"
-		)
-		(instances
-			(project "Tractive_Battery_Board"
-				(path "/ca333741-5826-495c-b860-5422aa5e17fc/fa150f42-0d9b-43a1-bf36-032543240a34"
-					(reference "U16")
-					(unit 1)
-				)

Commit message: added nanofit footprints
Parts:
- J5: footprint Connector_Harwin:Harwin_LTek-Male_02_P2.00mm_Vertical -> FS_4_Global_Footprint_Library:CONN_SD-105431-001_02_MOL
- J6: footprint Connector_Harwin:Harwin_LTek-Male_04_P2.00mm_Vertical -> FS_4_Global_Footprint_Library:1054311104
Changed lines of the file:
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@@
 			)
 		)
-		(property "Footprint" "Connector_Harwin:Harwin_LTek-Male_02_P2.00mm_Vertical"
+		(property "Footprint" "FS_4_Global_Footprint_Library:CONN_SD-105431-001_02_MOL"
 			(at 127 58.42 0)
 			(effects
@@
 			)
 		)
-		(property "Footprint" "Connector_Harwin:Harwin_LTek-Male_04_P2.00mm_Vertical"
+		(property "Footprint" "FS_4_Global_Footprint_Library:1054311104"
 			(at 97.79 87.63 0)
 			(effects

Commit message: cleanup + IMD voltage divider fix
Parts:
- removed J6: IRs Power, FS_4_Global_Footprint_Library:1054311104, symbol 1FS_2_Global_Symbol_Library:1053091204
- added J6: IRs Power, FS_4_Global_Footprint_Library:1054311104, symbol Connector_Generic:Conn_01x04
- added R38: 10k, symbol Device:R
- added R54: 100k, symbol Device:R
Connections:
- net GND: now also Q2.3 (S), J6.3 (Pin_3), R54.2; no longer Q2.1 (D)
- net IRs_Final: now also J6.2 (Pin_2), J6.4 (Pin_4)
- net nPreCharge_Control: now also R38.1, R54.1; no longer Q2.2 (G)
- new net: Q2.2 (G), R38.2
- new net: J6.1 (Pin_1), Q2.1 (D)
Other:
- note removed: "using a general nmos, double check if correct"
- moved on the sheet: Q2
