File: GLV_Protection/GLV_Protection_Circuit/GLV_Protection_Circuit.kicad_pcb (KiCad board)
At the start: 2 copper layers, 8 parts, among them Q1 PXP012-30QL, Q2 PXP012-30QL, Q3 SI2302-TP

Commit message: PMOS Update
- Changed the footprint for the PMOS to a higher stocked and less complex PMOS, should not affect logic of circuit
- Made connections to PCB more clear
Parts:
- F1: value Littlefuse 1812L110/33* -> 1812L110/33
- Q1, Q2: value PXP012-30QL -> BSS84; footprint FS_4_Footprint_Library:MLPAK33_SOT8002-1_NEX-M -> FS_4_Footprint_Library:SOT95P240X120-3N
- moved Q2 1.97 mm to (119.5, 44.5)
- moved Q1 1.12 mm to (89.0, 41.5), turned to -90 degrees
- moved Q3 0.50 mm to (119.5, 49.4)
Routing:
- net RPP-: track 0.00 -> 10.3 mm
- net UP-: track 0.00 -> 8.58 mm
- net Net-(Q2-G): track 7.49 -> 8.81 mm
- net UP+: track 7.03 -> 6.17 mm, vias 2 -> 0
- net Net-(D3-A): track 7.48 -> 6.71 mm
Other:
- board outline added: 54 x 17 mm
- board text added: "Input+"
- board text added: "Input-"
- board text added: "Output+"
- board text added: "Output-"
- board text added: "Reverse Polarity"
- board text added: "Undervoltage"
