File: GLV_Protection/GLV_Protection_Circuit/GLV_Protection_Circuit.kicad_sch (KiCad schematic)
At the start: 8 parts, among them Q1 PXP012-30QL, Q2 PXP012-30QL, Q3 SI2302-TP

Commit message: Circuit PCB
- Added/changed footprints
- Circuits made, but may need to replace PMOS with different model for later compression
Parts:
- D3: footprint FS_4_Footprint_Library:DIO_MM3Z9V1T1G -> FS_4_Footprint_Library:SOD-323_1P8X1P35_ONS-M
- Q3: footprint (none) -> FS_4_Footprint_Library:SOT-23_MCC-M
Connections:
- net + renamed UP+
- net UP+: no longer F1.1
- new net RPP+: F1.1
- new net RPP-: D1.1 (A1), Q1.2 (G)
- new net RPPO+: Q1.3 (S)
- new net UP-: Q3.3 (S), R3.1
- new net UPO+: Q2.1 (D)
Other:
- moved on the sheet: D3
Changed lines of the file:
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@@
 	)
 	(rectangle
-		(start 22.86 13.97)
-		(end 83.82 41.91)
+		(start 21.59 13.97)
+		(end 85.09 41.91)
 		(stroke
 			(width 0)
@@
 	(wire
 		(pts
-			(xy 106.68 20.32) (xy 106.68 19.05)
+			(xy 106.68 24.13) (xy 106.68 19.05)
 		)
 		(stroke
@@
 	(wire
 		(pts
-			(xy 106.68 27.94) (xy 106.68 35.56)
+			(xy 106.68 31.75) (xy 106.68 35.56)
 		)
 		(stroke
@@
 	(wire
 		(pts
-			(xy 72.39 21.59) (xy 78.74 21.59)
+			(xy 72.39 21.59) (xy 74.93 21.59)
 		)
 		(stroke
@@
 	(wire
 		(pts
-			(xy 67.31 36.83) (xy 78.74 36.83)
+			(xy 67.31 36.83) (xy 74.93 36.83)
 		)
 		(stroke
@@
 		)
 	)
-	(global_label "+"
+	(global_label "RPP+"
 		(shape input)
 		(at 30.48 21.59 180)
@@
 		)
 		(property "Intersheetrefs" "${INTERSHEET_REFS}"
-			(at 25.9224 21.59 0)
+			(at 22.1124 21.59 0)
 			(show_name yes)
 			(effects
@@
 		)
 	)
-	(global_label ""
+	(global_label "RPPO+"
 		(shape output)
-		(at 78.74 21.59 0)
+		(at 74.93 21.59 0)
 		(fields_autoplaced yes)
 		(effects
@@
 		)
 		(property "Intersheetrefs" "${INTERSHEET_REFS}"
-			(at 81.9792 21.59 0)
+			(at 84.6281 21.59 0)
 			(show_name yes)
 			(effects
@@
 		)
 	)
-	(global_label "-"
+	(global_label "UP-"
 		(shape input)
 		(at 96.52 44.45 180)
@@
 		)
 		(property "Intersheetrefs" "${INTERSHEET_REFS}"
-			(at 91.9624 44.45 0)
+			(at 89.3619 44.45 0)
 			(effects
 				(font
@@
 		)
 	)
-	(global_label ""
+	(global_label "UPO+"
 		(shape output)
 		(at 138.43 19.05 0)
@@
 		)
 		(property "Intersheetrefs" "${INTERSHEET_REFS}"
-			(at 141.6692 19.05 0)
+			(at 146.9186 19.05 0)
 			(show_name yes)
 			(effects
@@
 		)
 	)
-	(global_label ""
+	(global_label "RPPO-"
 		(shape output)
-		(at 78.74 36.83 0)
+		(at 74.93 36.83 0)
 		(fields_autoplaced yes)
 		(effects
@@
 		)
 		(property "Intersheetrefs" "${INTERSHEET_REFS}"
-			(at 81.9792 36.83 0)
+			(at 84.6281 36.83 0)
 			(effects
 				(font
@@
 		)
 	)
-	(global_label "-"
+	(global_label "RPP-"
 		(shape input)
 		(at 30.48 36.83 180)
@@
 		)
 		(property "Intersheetrefs" "${INTERSHEET_REFS}"
-			(at 25.9224 36.83 0)
+			(at 22.1124 36.83 0)
 			(effects
 				(font
@@
 		)
 	)
-	(global_label "+"
+	(global_label "UP+"
 		(shape input)
 		(at 96.52 19.05 180)
@@
 		)
 		(property "Intersheetrefs" "${INTERSHEET_REFS}"
-			(at 91.9624 19.05 0)
+			(at 89.3619 19.05 0)
 			(show_name yes)
 			(effects
@@
 		)
 	)
-	(global_label ""
+	(global_label "UPO-"
 		(shape output)
 		(at 138.43 44.45 0)
@@
 		)
 		(property "Intersheetrefs" "${INTERSHEET_REFS}"
-			(at 141.6692 44.45 0)
+			(at 146.9186 44.45 0)
 			(show_name yes)
 			(effects
@@
 			)
 		)
-		(property "Footprint" ""
+		(property "Footprint" "FS_4_Footprint_Library:SOT-23_MCC-M"
 			(at 135.89 33.02 0)
 			(effects
@@
 	(symbol
 		(lib_id "Diode:1N47xxA")
-		(at 106.68 24.13 270)
+		(at 106.68 27.94 270)
 		(unit 1)
 		(exclude_from_sim no)
@@
 		(dnp no)
 		(property "Reference" "D3"
-			(at 109.22 22.8599 90)
+			(at 109.22 26.6699 90)
 			(effects
 				(font
@@
 		)
 		(property "Value" "MM3Z9V1T1G"
-			(at 108.458 24.892 90)
+			(at 108.458 28.702 90)
 			(effects
 				(font
@@
 			)
 		)
-		(property "Footprint" "FS_4_Footprint_Library:DIO_MM3Z9V1T1G"
-			(at 102.235 24.13 0)
+		(property "Footprint" "FS_4_Footprint_Library:SOD-323_1P8X1P35_ONS-M"
+			(at 102.235 27.94 0)
 			(effects
 				(font
@@
 		)
 		(property "Datasheet" "https://www.vishay.com/docs/85816/1n4728a.pdf"
-			(at 106.68 24.13 0)
+			(at 106.68 27.94 0)
 			(effects
 				(font
@@
 		)
 		(property "Description" "1300mW Silicon planar power Zener diodes, DO-41"
-			(at 106.68 24.13 0)
-			(effects
-				(font
+			(at 106.68 27.94 0)
+			(effects
+				(font

Commit message: PMOS Update
- Changed the footprint for the PMOS to a higher stocked and less complex PMOS, should not affect logic of circuit
- Made connections to PCB more clear
Parts:
- Q1, Q2: value PXP012-30QL -> BSS84; footprint FS_4_Footprint_Library:MLPAK33_SOT8002-1_NEX-M -> FS_4_Footprint_Library:SOT95P240X120-3N
Changed lines of the file:
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@@
 			)
 		)
-		(property "Value" "PXP012-30QL"
+		(property "Value" "BSS84"
 			(at 67.31 17.78 90)
 			(effects
@@
 			)
 		)
-		(property "Footprint" "FS_4_Footprint_Library:MLPAK33_SOT8002-1_NEX-M"
+		(property "Footprint" "FS_4_Footprint_Library:SOT95P240X120-3N"
 			(at 64.77 19.05 0)
 			(effects
@@
 			)
 		)
-		(property "Value" "PXP012-30QL"
+		(property "Value" "BSS84"
 			(at 135.128 26.162 90)
 			(effects
@@
 			)
 		)
-		(property "Footprint" "FS_4_Footprint_Library:MLPAK33_SOT8002-1_NEX-M"
+		(property "Footprint" "FS_4_Footprint_Library:SOT95P240X120-3N"
 			(at 135.89 16.51 0)
 			(effects
