File: BMS/TMPDev/TMPDev.kicad_pcb (KiCad board)
At the start: 2 copper layers, 83.8 x 63.5 mm, 12 parts, among them J1 59453-051110ECHLF, J3 046298703000883+, U1 DS18B20Z+, U1 TMP1075D, U3 TMP1075D

Commit message: Update TMPDev.kicad_pcb
Routing:
- net Net-(U1-GND): track 65.7 -> 66.5 mm
- net Net-(U1-DQ): track 59.1 -> 59.9 mm
Changed lines of the file:
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@@
 	)
 	(segment
-		(start 42.23 43.228)
-		(end 41.840686 43.228)
-		(width 0.254)
-		(layer "B.Cu")
-		(net 7)
-	)
-	(segment
-		(start 42.15 48.97)
-		(end 42.23 48.89)
-		(width 0.254)
-		(layer "B.Cu")
-		(net 7)
-	)
-	(segment
-		(start 42.23 39.272)
-		(end 42.23 39.11429)
-		(width 0.254)
-		(layer "B.Cu")
-		(net 7)
-	)
-	(segment
-		(start 42.555 55.418468)
-		(end 42.548468 55.418468)
-		(width 0.254)
-		(layer "B.Cu")
-		(net 7)
-	)
-	(segment
-		(start 42.15 55.02)
-		(end 42.15 48.97)
+		(start 39.02 39.65)
+		(end 39.02 42.8)
 		(width 0.254)
 		(layer "B.Cu")
@@
 	(segment
 		(start 42.548468 55.418468)
-		(end 42.15 55.02)
-		(width 0.254)
-		(layer "B.Cu")
-		(net 7)
-	)
-	(segment
-		(start 48.255 61.118467)
 		(end 42.555 55.418468)
-		(width 0.254)
-		(layer "B.Cu")
-		(net 7)
-	)
-	(segment
-		(start 41.840686 39.272)
-		(end 42.23 39.272)
-		(width 0.254)
-		(layer "B.Cu")
-		(net 7)
-	)
-	(segment
-		(start 42.23 39.11429)
-		(end 42.114198 38.998488)
-		(width 0.254)
-		(layer "B.Cu")
-		(net 7)
-	)
-	(segment
-		(start 40.682 40.430686)
-		(end 41.840686 39.272)
-		(width 0.254)
-		(layer "B.Cu")
-		(net 7)
-	)
-	(segment
-		(start 40.682 42.069314)
-		(end 40.682 40.430686)
 		(width 0.254)
 		(layer "B.Cu")
@@
 	)
 	(segment
+		(start 42.114198 36.555802)
+		(end 39.02 39.65)
+		(width 0.254)
+		(layer "B.Cu")
+		(net 7)
+	)
+	(segment
 		(start 59.34 66)
 		(end 54.725 61.385)
@@
 	)
 	(segment
-		(start 48.521532 61.385)
-		(end 48.255 61.118467)
+		(start 48.255 61.118467)
+		(end 48.521532 61.385)
 		(width 0.254)
 		(layer "B.Cu")
@@
 	)
 	(segment
-		(start 41.840686 43.228)
-		(end 40.682 42.069314)
+		(start 39.02 42.8)
+		(end 42.391819 46.171819)
 		(width 0.254)
 		(layer "B.Cu")
@@
 	)
 	(segment
-		(start 42.114198 38.998488)
-		(end 42.114198 20.433999)
+		(start 42.391819 46.171819)
+		(end 42.391819 55.261819)
+		(width 0.254)
+		(layer "B.Cu")
+		(net 7)
+	)
+	(segment
+		(start 42.555 55.418468)
+		(end 48.255 61.118467)
 		(width 0.254)
 		(layer "B.Cu")
@@
 	)
 	(segment
-		(start 42.23 48.89)
-		(end 42.23 43.228)
+		(start 42.114198 20.433999)
+		(end 42.114198 36.555802)
+		(width 0.254)
+		(layer "B.Cu")
+		(net 7)
+	)
+	(segment
+		(start 42.391819 55.261819)
+		(end 42.548468 55.418468)
 		(width 0.254)
 		(layer "B.Cu")
@@
 	)
 	(segment
-		(start 48.71 60.93)
-		(end 43.01 55.23)
+		(start 43.01 46.13)
+		(end 46.32 42.82)
 		(width 0.254)
 		(layer "B.Cu")
@@
 	)
 	(segment
-		(start 43.01 55.23)
-		(end 43.01 43.228)
-		(width 0.254)
-		(layer "B.Cu")
-		(net 8)
-	)
-	(segment
-		(start 43.01 43.228)
-		(end 43.479314 43.228)
-		(width 0.254)
-		(layer "B.Cu")
-		(net 8)
-	)
-	(segment
-		(start 44.638 40.430686)
-		(end 43.479314 39.272)
-		(width 0.254)
-		(layer "B.Cu")
-		(net 8)
-	)
-	(segment
-		(start 43.01 34.991596)
-		(end 43.125798 34.875798)
-		(width 0.254)
-		(layer "B.Cu")
-		(net 8)
-	)
-	(segment
-		(start 44.638 42.069314)
-		(end 44.638 40.430686)
-		(width 0.254)
-		(layer "B.Cu")
-		(net 8)
-	)
-	(segment
-		(start 43.479314 43.228)
-		(end 44.638 42.069314)
+		(start 46.32 39.68)
+		(end 43.125798 36.485798)
 		(width 0.254)
 		(layer "B.Cu")
@@
 	)
 	(segment
-		(start 43.479314 39.272)
-		(end 43.01 39.272)
+		(start 43.01 55.23)
+		(end 43.01 46.13)
 		(width 0.254)
 		(layer "B.Cu")
@@
 	)
 	(segment
-		(start 43.125798 34.875798)
+		(start 48.71 60.93)
+		(end 43.01 55.23)
+		(width 0.254)
+		(layer "B.Cu")
+		(net 8)
+	)
+	(segment
+		(start 43.125798 36.485798)
 		(end 43.125798 20.433999)
 		(width 0.254)
@@
 	)
 	(segment
-		(start 43.01 39.272)
-		(end 43.01 34.991596)
+		(start 46.32 42.82)
+		(end 46.32 39.68)
 		(width 0.254)
 		(layer "B.Cu")

Commit message: New board layout, notes sent to Joshua
Parts:
- removed C1, C3: 0.01 uF, Capacitor_SMD:C_0805_2012Metric_Pad1.18x1.45mm_HandSolder
- removed PU_ALRT1, PU_SCL1, PU_SDA1: 5k, Resistor_SMD:R_0805_2012Metric_Pad1.20x1.40mm_HandSolder
- removed REF** (x2): MountingHole_3.2mm_M3, MountingHole:MountingHole_3.2mm_M3
- removed the U1 at (62.2, 41.6)
- removed the U1 at (62.2, 61.6)
- removed U3: TMP1075D, Package_SO:SO-8_3.9x4.9mm_P1.27mm
- added C12: 0.01 uF, Capacitor_SMD:C_0805_2012Metric_Pad1.18x1.45mm_HandSolder, F.Cu at (148.8, 60.2)
- added C14: 0.01 uF, Capacitor_SMD:C_0805_2012Metric_Pad1.18x1.45mm_HandSolder, F.Cu at (168.7, 100.1)
- added PU_ALRT2: 5k, Resistor_SMD:R_0805_2012Metric_Pad1.20x1.40mm_HandSolder, F.Cu at (147.8, 48.3)
- added PU_SDA2: 5k, Resistor_SMD:R_0805_2012Metric_Pad1.20x1.40mm_HandSolder, F.Cu at (147.8, 52.3)
- added RPU_SCL2: 5k, Resistor_SMD:R_0805_2012Metric_Pad1.20x1.40mm_HandSolder, F.Cu at (147.8, 50.3)
- added U1: DS18B20Z+, FS_4_Global_Footprint_Library:21-0041B_8_MXM, F.Cu at (124.7, 106.7)
- added U13: TMP1075D, Package_SO:SO-8_3.9x4.9mm_P1.27mm, F.Cu at (146.8, 66.0)
- added U15: TMP1075D, Package_SO:SO-8_3.9x4.9mm_P1.27mm, F.Cu at (166.4, 106.4)
- J1: footprint formula_slug_footprint_library:AMPHENOL_59453-051110ECHLF -> FS_4_Global_Footprint_Library:AMPHENOL_59453-051110ECHLF; moved to F.Cu
- J3: footprint formula_slug_footprint_library:CONN3_6298_KAV -> FS_4_Global_Footprint_Library:CONN3_6298_KAV; moved to F.Cu
- moved J3 87.2 mm to (127.0, 43.9)
- moved J1 85.5 mm to (145.3, 44.2)
Routing:
- net /SDA: track 121.3 -> 82.6 mm, vias 3 -> 4
- net /ALERT: track 124.7 -> 91.3 mm, vias 3 -> 2
- net +5V: track 113.7 -> 83.3 mm, vias 2 -> 5
- net V-: track 115.1 -> 100.4 mm, vias 19 -> 0
- net /SCL: track 119.1 -> 106.6 mm
- net Net-(U1-GND): track 66.5 -> 64.3 mm, vias 1 -> 0
- net Net-(U1-DQ): track 59.9 -> 61.6 mm, vias 1 -> 0
Other:
- board size 83.8 x 63.5 mm -> 52 x 69.8 mm
- board text removed: "U1"

Commit message: New 5 Pin FPC conn
Parts:
- removed J3: 046298703000883+, FS_4_Global_Footprint_Library:CONN3_6298_KAV
- removed PU_ALRT2, PU_SDA2, RPU_SCL2: 5k, Resistor_SMD:R_0805_2012Metric_Pad1.20x1.40mm_HandSolder
- added J2: 5019510550, formula_slug_footprint_library:CON_5019510550, F.Cu at (126.8, 47.6)
- J1: value 59453-051110ECHLF -> 5019510550; footprint FS_4_Global_Footprint_Library:AMPHENOL_59453-051110ECHLF -> formula_slug_footprint_library:CON_5019510550
- moved J1 3.71 mm to (146.8, 47.6), turned to 0 degrees
Routing:
- net /SCL: track 106.6 -> 85.7 mm
- net /ALERT: track 91.3 -> 79.6 mm
- net /SDA: track 82.6 -> 75.5 mm, vias 4 -> 3
- net V-: track 100.4 -> 95.2 mm
- net Net-(U1-GND): track 64.3 -> 59.8 mm
- net Net-(U1-DQ): track 61.6 -> 58.1 mm
- net +5V: track 83.3 -> 81.8 mm
Other:
- outline, holes or cut-outs redrawn

Commit message: 3D models and some other changes
Parts:
- C12, C14: footprint Capacitor_SMD:C_0805_2012Metric_Pad1.18x1.45mm_HandSolder -> Capacitor_SMD:C_0603_1608Metric_Pad1.08x0.95mm_HandSolder
- moved U15 12.4 mm to (166.8, 94.0), turned to 90 degrees
- moved U1 4.06 mm to (128.8, 106.7)
Routing:
- net Net-(U1-DQ): track 58.1 -> 60.3 mm
- net +5V: track 81.8 -> 83.9 mm
- net /SDA: track 75.5 -> 77.6 mm
- net Net-(U1-GND): track 59.8 -> 58.0 mm
- net /SCL: track 85.7 -> 86.8 mm, vias 3 -> 5
- net V-: track 95.2 -> 96.3 mm
- net /ALERT: track 79.6 -> 80.6 mm, vias 2 -> 4

Commit message: centered the temp sensors on bottom row
Parts:
- moved U15 12.2 mm to (166.8, 106.2), turned to 0 degrees
- moved U1 2.07 mm to (126.8, 106.2)
Routing:
- net V-: track 96.3 -> 92.4 mm
- net /SDA: track 77.6 -> 74.1 mm
- net /ALERT: track 80.6 -> 77.8 mm, vias 4 -> 2
- net +5V: track 83.9 -> 81.8 mm
- net /SCL: track 86.8 -> 84.9 mm, vias 5 -> 3
- net Net-(U1-DQ): track 60.3 -> 58.5 mm

Commit message: increased size for test module
Parts:
- moved U13 55.5 mm to (91.3, 65.4)
- moved C14 55.5 mm to (113.1, 99.5)
- moved J1 55.5 mm to (91.3, 47.0)
- moved C12 55.5 mm to (93.3, 59.6)
- moved J2 55.5 mm to (71.3, 47.0)
- moved U1 55.5 mm to (71.2, 105.6)
- moved U15 55.4 mm to (111.4, 105.6)
Routing:
- net /SCL: track 84.9 -> 81.4 mm
- net +5V: track 81.8 -> 83.5 mm
- net Net-(U1-DQ): track 58.5 -> 59.9 mm
- net Net-(U1-GND): track 57.8 -> 58.9 mm
- net V-: track 92.4 -> 93.5 mm
- net /ALERT: track 77.8 -> 78.4 mm, vias 2 -> 4
Other:
- board size 52 x 69.8 mm -> 92 x 69.8 mm

Commit message: Added silkscreen text
Other:
- board text added: "FS-4 Rev 1.0 Test Module Temp Sense Designed by Joshua Flores"
Changed lines of the file:
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@@
 		(layer "Edge.Cuts")
+	)
+	(gr_text "FS-4 Rev 1.0\nTest Module Temp Sense\nDesigned by Joshua Flores"
+		(at 91.44 104.648 0)
+		(layer "B.SilkS")
+		(effects
+			(font
+				(size 0.55 0.55)
+				(thickness 0.1)
+			)
+			(justify mirror)
+		)
 	)
 	(segment

Commit message: DFM changes :((
Routing:
- net /ALERT: track 78.4 -> 79.4 mm
- net +5V: track 83.5 -> 84.1 mm
