File: VoltageTester/ADC-BalanceBoard/ADC-BalanceBoard.kicad_pcb (KiCad board)
At the start: 2 copper layers, 245 x 245 mm, 235 parts, among them J1 Conn_01x02, U1 MCP3208-CI_SL, U10 MCP3208-CI_SL, U11 MCP3208-CI_SL, U12 MCP3208-CI_SL, U13 MCP3208-CI_SL, U14 NUCLEO-L432KC, U15 FXMAR2104UMX, U16 FXMAR2104UMX, U17 FXMAR2104UMX, U18 FXMAR2104UMX, U2 MCP3208-CI_SL, U3 MCP3208-CI_SL, U4 MCP3208-CI_SL, U5 MCP3208-CI_SL, U6 MCP3208-CI_SL, U7 MCP3208-CI_SL, U8 MCP3208-CI_SL, U9 MCP3208-CI_SL

Commit message: added pin headers to board and library
Parts:
- removed U14: NUCLEO-L432KC, FS_4_Global_Footprint_Library:NUCLEO-L432KC
- added J2: M20-7861546, FS_4_Global_Footprint_Library:HARWIN_M20-7861546, F.Cu at (283.6, 138.6)
- added J3: M20-7861546, FS_4_Global_Footprint_Library:HARWIN_M20-7861546, F.Cu at (268.4, 138.6)
- Cell  22: renamed from REF**
- Cell  23: renamed from REF**
- Cell 1: renamed from REF**
- Cell 10: renamed from REF**
- Cell 100: renamed from REF**
- Cell 11: renamed from REF**
- Cell 12: renamed from REF**
- Cell 13: renamed from REF**
- Cell 14: renamed from REF**
- Cell 15: renamed from REF**
- Cell 16: renamed from REF**
- Cell 17: renamed from REF**
- Cell 18: renamed from REF**
- Cell 19: renamed from REF**
- Cell 2: renamed from REF**
- Cell 20: renamed from REF**
- Cell 21: renamed from REF**
- Cell 24: renamed from REF**
- Cell 25: renamed from REF**
- Cell 26: renamed from REF**
- Cell 27: renamed from REF**
- Cell 28: renamed from REF**
- Cell 29: renamed from REF**
- Cell 3: renamed from REF**
- Cell 30: renamed from REF**
- Cell 31: renamed from REF**
- Cell 32: renamed from REF**
- Cell 33: renamed from REF**
- Cell 34: renamed from REF**
- Cell 35: renamed from REF**
- Cell 36: renamed from REF**
- Cell 37: renamed from REF**
- Cell 38: renamed from REF**
- Cell 39: renamed from REF**
- Cell 4: renamed from REF**
- Cell 40: renamed from REF**
- Cell 41: renamed from REF**
- Cell 42: renamed from REF**
- Cell 43: renamed from REF**
- Cell 44: renamed from REF**
- Cell 45: renamed from REF**
- Cell 46: renamed from REF**
- Cell 47: renamed from REF**
- Cell 48: renamed from REF**
- Cell 49: renamed from REF**
- Cell 5: renamed from REF**
- Cell 50: renamed from REF**
- Cell 51: renamed from REF**
- Cell 52: renamed from REF** (x2)
- Cell 53: renamed from REF**
- Cell 54: renamed from REF**
- Cell 55: renamed from REF**
- Cell 56: renamed from REF**
- Cell 57: renamed from REF**
- Cell 58: renamed from REF**
- Cell 59: renamed from REF**
- Cell 6: renamed from REF**
- Cell 60: renamed from REF**
- Cell 61: renamed from REF**
- Cell 63: renamed from REF**
- Cell 64: renamed from REF**
- Cell 65: renamed from REF**
- Cell 66: renamed from REF**
- Cell 67: renamed from REF**
- Cell 68: renamed from REF**
- Cell 69: renamed from REF**
- Cell 7: renamed from REF**
- Cell 70: renamed from REF**
- Cell 71: renamed from REF**
- Cell 72: renamed from REF**
- Cell 73: renamed from REF**
- Cell 74: renamed from REF**
- Cell 75: renamed from REF**
- Cell 76: renamed from REF**
- Cell 77: renamed from REF**
- Cell 78: renamed from REF**
- Cell 79: renamed from REF**
- Cell 8: renamed from REF**
- Cell 80: renamed from REF**
- Cell 81: renamed from REF**
- Cell 82: renamed from REF**
- Cell 83: renamed from REF**
- Cell 84: renamed from REF**
- Cell 85: renamed from REF**
- Cell 86: renamed from REF**
- Cell 87: renamed from REF**
- Cell 88: renamed from REF**
- Cell 89: renamed from REF**
- Cell 9: renamed from REF**
- Cell 90: renamed from REF**
- Cell 91: renamed from REF**
- Cell 92: renamed from REF**
- Cell 93: renamed from REF**
- Cell 94: renamed from REF**
- Cell 95: renamed from REF**
- Cell 96: renamed from REF**
- Cell 97: renamed from REF**
- Cell 98: renamed from REF**
- Cell 99: renamed from REF**
Routing:
- net B: track 2328.2 -> 3708.2 mm
- net GND: track 1303.3 -> 1237.2 mm, vias 108 -> 110
- net U11_CS_3V3: track 68.5 -> 63.4 mm
- net U10_CS_3V3: track 131.7 -> 127.2 mm, vias 3 -> 4
- net MOSI_3V3: track 93.1 -> 97.0 mm
- net MISO_3V3: track 128.0 -> 125.2 mm, vias 5 -> 6
- net +3V3: track 235.5 -> 238.2 mm, vias 8 -> 10
- net U5_CS_3V3: track 59.6 -> 61.9 mm
- net U7_CS_3V3: track 88.8 -> 91.0 mm
- net U3_CS_3V3: track 54.7 -> 56.4 mm
- net CLK_3V3: track 106.8 -> 107.7 mm
- net U13_CS_3V3: track 57.3 -> 56.4 mm, vias 0 -> 2
- net U12_CS_3V3: track 63.6 -> 62.8 mm, vias 2 -> 0
- net U4_CS_3V3: track 56.8 -> 56.1 mm
- net +5V: track 1069.7 -> 1069.0 mm
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
Commit message: ADC-BalanceBoard PCB v2.0.0 done
Parts:
- removed C6, C7, C8: 1uF, Capacitor_SMD:C_0805_2012Metric_Pad1.18x1.45mm_HandSolder
- removed Cell  22: CPG-23-SMT-TR, FS_4_Global_Footprint_Library:CPG-23-SMT-TR
- removed Cell  23: CPG-23-SMT-TR, FS_4_Global_Footprint_Library:CPG-23-SMT-TR
- removed Cell 100: CPG-23-SMT-TR, FS_4_Global_Footprint_Library:CPG-23-SMT-TR
- removed the Cell 52 at (176.0, 66.0)
- removed the Cell 52 at (198.0, 66.0)
- removed Cell 64: CPG-23-SMT-TR, FS_4_Global_Footprint_Library:CPG-23-SMT-TR
- removed Cell 65: CPG-23-SMT-TR, FS_4_Global_Footprint_Library:CPG-23-SMT-TR
- removed Cell 66: CPG-23-SMT-TR, FS_4_Global_Footprint_Library:CPG-23-SMT-TR
- removed Cell 67: CPG-23-SMT-TR, FS_4_Global_Footprint_Library:CPG-23-SMT-TR
- removed Cell 68: CPG-23-SMT-TR, FS_4_Global_Footprint_Library:CPG-23-SMT-TR
- removed Cell 69: CPG-23-SMT-TR, FS_4_Global_Footprint_Library:CPG-23-SMT-TR
- removed Cell 70: CPG-23-SMT-TR, FS_4_Global_Footprint_Library:CPG-23-SMT-TR
- removed Cell 71: CPG-23-SMT-TR, FS_4_Global_Footprint_Library:CPG-23-SMT-TR
- removed Cell 72: CPG-23-SMT-TR, FS_4_Global_Footprint_Library:CPG-23-SMT-TR
- removed Cell 73: CPG-23-SMT-TR, FS_4_Global_Footprint_Library:CPG-23-SMT-TR
- removed Cell 74: CPG-23-SMT-TR, FS_4_Global_Footprint_Library:CPG-23-SMT-TR
- removed Cell 75: CPG-23-SMT-TR, FS_4_Global_Footprint_Library:CPG-23-SMT-TR
- removed Cell 76: CPG-23-SMT-TR, FS_4_Global_Footprint_Library:CPG-23-SMT-TR
- removed Cell 77: CPG-23-SMT-TR, FS_4_Global_Footprint_Library:CPG-23-SMT-TR
- removed Cell 78: CPG-23-SMT-TR, FS_4_Global_Footprint_Library:CPG-23-SMT-TR
- removed Cell 79: CPG-23-SMT-TR, FS_4_Global_Footprint_Library:CPG-23-SMT-TR
- removed Cell 80: CPG-23-SMT-TR, FS_4_Global_Footprint_Library:CPG-23-SMT-TR
- removed Cell 81: CPG-23-SMT-TR, FS_4_Global_Footprint_Library:CPG-23-SMT-TR
- removed Cell 82: CPG-23-SMT-TR, FS_4_Global_Footprint_Library:CPG-23-SMT-TR
- removed Cell 83: CPG-23-SMT-TR, FS_4_Global_Footprint_Library:CPG-23-SMT-TR
- removed Cell 84: CPG-23-SMT-TR, FS_4_Global_Footprint_Library:CPG-23-SMT-TR
- removed Cell 85: CPG-23-SMT-TR, FS_4_Global_Footprint_Library:CPG-23-SMT-TR
- removed Cell 86: CPG-23-SMT-TR, FS_4_Global_Footprint_Library:CPG-23-SMT-TR
- removed Cell 87: CPG-23-SMT-TR, FS_4_Global_Footprint_Library:CPG-23-SMT-TR
- removed Cell 88: CPG-23-SMT-TR, FS_4_Global_Footprint_Library:CPG-23-SMT-TR
- removed Cell 89: CPG-23-SMT-TR, FS_4_Global_Footprint_Library:CPG-23-SMT-TR
- removed Cell 90: CPG-23-SMT-TR, FS_4_Global_Footprint_Library:CPG-23-SMT-TR
- removed Cell 91: CPG-23-SMT-TR, FS_4_Global_Footprint_Library:CPG-23-SMT-TR
- removed Cell 92: CPG-23-SMT-TR, FS_4_Global_Footprint_Library:CPG-23-SMT-TR
- removed Cell 93: CPG-23-SMT-TR, FS_4_Global_Footprint_Library:CPG-23-SMT-TR
- removed Cell 94: CPG-23-SMT-TR, FS_4_Global_Footprint_Library:CPG-23-SMT-TR
- removed Cell 95: CPG-23-SMT-TR, FS_4_Global_Footprint_Library:CPG-23-SMT-TR
- removed Cell 96: CPG-23-SMT-TR, FS_4_Global_Footprint_Library:CPG-23-SMT-TR
- removed Cell 97: CPG-23-SMT-TR, FS_4_Global_Footprint_Library:CPG-23-SMT-TR
- removed Cell 98: CPG-23-SMT-TR, FS_4_Global_Footprint_Library:CPG-23-SMT-TR
- removed Cell 99: CPG-23-SMT-TR, FS_4_Global_Footprint_Library:CPG-23-SMT-TR
- removed R100, R67, R68, R69, R70, R71, R72, R73, R74, R75, R76, R77, R78, R79, R80, R81, R82, R83, R84, R85, R86, R87, R88, R89, R90, R91, R92, R93, R94, R95, R96, R97, R98, R99: 2, Resistor_SMD:R_0805_2012Metric_Pad1.20x1.40mm_HandSolder
- removed R101, R102, R103, R104: 10k, Resistor_SMD:R_0805_2012Metric_Pad1.20x1.40mm_HandSolder
- removed the REF** at (282.6, 262.2)
- removed the REF** at (282.6, 26.2)
- removed the REF** at (46.6, 26.2)
- removed the REF** at (46.6, 262.2)
- removed U10, U11, U12, U13, U8, U9: MCP3208-CI_SL, FS_4_Global_Footprint_Library:MCP3208-CI_SL
- removed U15, U16, U17, U18: FXMAR2104UMX, FS_4_Global_Footprint_Library:ULTRATHIN_MLP_12L_ONS-L
- added Cell 0: CPG-23-SMT-TR, FS_4_Global_Footprint_Library:CPG-23-SMT-TR, F.Cu at (100.0, 50.0)
- added Cell 22: CPG-23-SMT-TR, FS_4_Global_Footprint_Library:CPG-23-SMT-TR, F.Cu at (144.0, 182.0)
- added Cell 23: CPG-23-SMT-TR, FS_4_Global_Footprint_Library:CPG-23-SMT-TR, F.Cu at (144.0, 204.0)
- added Cell 52: CPG-23-SMT-TR, FS_4_Global_Footprint_Library:CPG-23-SMT-TR, F.Cu at (232.0, 138.0)
- added Cell 62: CPG-23-SMT-TR, FS_4_Global_Footprint_Library:CPG-23-SMT-TR, F.Cu at (254.0, 182.0)
- added REF**: MountingHole_3.5mm, MountingHole:MountingHole_3.5mm, F.Cu at (280.0, 215.0)
- added REF**: MountingHole_3.5mm, MountingHole:MountingHole_3.5mm, F.Cu at (280.0, 25.0)
- added REF**: MountingHole_3.5mm, MountingHole:MountingHole_3.5mm, F.Cu at (90.0, 215.0)
- added REF**: MountingHole_3.5mm, MountingHole:MountingHole_3.5mm, F.Cu at (90.0, 25.0)
- C1, C2, C3, C4, C5: value 1uF -> .1uF
- J1: value Conn_01x02 -> 1054301102; footprint Connector_Molex:Molex_Nano-Fit_105309-xx02_1x02_P2.50mm_Vertical -> FS_4_Global_Footprint_Library:CONN_SD-105430-001_02_MOL
- J2, J3: value M20-7861546 -> HARWIN_M20-7861546
- R65, R66: value 2 -> 10k
- U1, U2, U3, U4: value MCP3208-CI_SL -> ~; footprint FS_4_Global_Footprint_Library:MCP3208-CI_SL -> Package_SO:SSOP-24_5.3x8.2mm_P0.65mm
- U5: value MCP3208-CI_SL -> ADS1015IDGS; footprint FS_4_Global_Footprint_Library:MCP3208-CI_SL -> Package_SO:TSSOP-10_3x3mm_P0.5mm
- U6, U7: value MCP3208-CI_SL -> FXMAR2104UMX; footprint FS_4_Global_Footprint_Library:MCP3208-CI_SL -> FS_4_Global_Footprint_Library:ULTRATHIN_MLP_12L_ONS-L
- moved Cell 40 207.2 mm to (210.0, 50.0)
- moved R49 188.8 mm to (232.0, 45.0)
- moved R50 188.3 mm to (232.0, 67.0)
- moved R9 179.5 mm to (122.0, 45.0)
- moved R10 179.0 mm to (122.0, 67.0)
- moved Cell 48 167.3 mm to (232.0, 50.0)
- moved Cell 49 167.3 mm to (232.0, 72.0)
- moved Cell 50 167.3 mm to (232.0, 94.0)
- moved Cell 31 163.6 mm to (166.0, 204.0)
- moved Cell 10 158.2 mm to (122.0, 94.0)
- moved Cell 8 158.2 mm to (122.0, 50.0)
- moved Cell 9 158.2 mm to (122.0, 72.0)
- moved R58 150.5 mm to (254.0, 67.0)
- moved R59 150.5 mm to (254.0, 89.0)
- moved R57 150.3 mm to (254.0, 45.0)
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Connections:
- J1 pad 2: unconnected-(J1-Pin_2-Pad2) -> VIN
- J2 pad 1: unconnected-(J2-Pad1) -> SCL_3V3
- J2 pad 10: MOSI_3V3 -> (no net)
- J2 pad 11: unconnected-(J2-Pad11) -> (no net)
- J2 pad 12: +5V -> (no net)
- J2 pad 13: unconnected-(J2-Pad13) -> (no net)
- J2 pad 14: GND -> (no net)
- J2 pad 15: unconnected-(J2-Pad15) -> (no net)
- J2 pad 2: +3V3 -> SDA_3V3
- J2 pad 3: unconnected-(J2-Pad3) -> (no net)
- J2 pad 4: U13_CS_3V3 -> GND
- J2 pad 5: CLK_3V3 -> ALERT/RDY_3V3
- J2 pad 6: U12_CS_3V3 -> SA0_3V3
- J2 pad 7: U11_CS_3V3 -> SA1_3V3
- J2 pad 8: unconnected-(J2-Pad8) -> SA2_3V3
- J2 pad 9: unconnected-(J2-Pad9) -> SA3_3V3
- J3 pad 1: U10_CS_3V3 -> VIN
- J3 pad 10: U4_CS_3V3 -> (no net)
- J3 pad 11: U3_CS_3V3 -> (no net)
- J3 pad 12: GND -> (no net)
- J3 pad 13: unconnected-(J3-Pad13) -> (no net)
- J3 pad 14: U2_CS_3V3 -> +3V3
- J3 pad 15: U1_CS_3V3 -> (no net)
- J3 pad 2: U9_CS_3V3 -> GND
- J3 pad 3: MISO_3V3 -> (no net)
- J3 pad 4: U8_CS_3V3 -> +5V
- J3 pad 5: unconnected-(J3-Pad5) -> (no net)
- J3 pad 6: unconnected-(J3-Pad6) -> (no net)
- J3 pad 7: U7_CS_3V3 -> (no net)
- J3 pad 8: U6_CS_3V3 -> (no net)
- J3 pad 9: U5_CS_3V3 -> (no net)
- R1 pad 1: Cell1 -> Cell0
- R10 pad 1: Cell10 -> Cell9
- R11 pad 1: Cell11 -> Cell10
- R12 pad 1: Cell12 -> Cell11
- R13 pad 1: Cell13 -> Cell12
- R14 pad 1: Cell14 -> Cell13
- R15 pad 1: Cell15 -> Cell14
- R16 pad 1: Cell16 -> Cell15
- R17 pad 1: Cell17 -> Cell16
- R18 pad 1: Cell18 -> Cell17
- R19 pad 1: Cell19 -> Cell18
- R2 pad 1: Cell2 -> Cell1
- R20 pad 1: Cell20 -> Cell19
- R21 pad 1: Cell21 -> Cell20
- R22 pad 1: Cell22 -> Cell21
- R23 pad 1: Cell23 -> Cell22
- R24 pad 1: Cell24 -> Cell23
- R25 pad 1: Cell25 -> Cell24
- R26 pad 1: Cell26 -> Cell25
- R27 pad 1: Cell27 -> Cell26
- R28 pad 1: Cell28 -> Cell27
- R29 pad 1: Cell29 -> Cell28
- R3 pad 1: Cell3 -> Cell2
- R30 pad 1: Cell30 -> Cell29
- R31 pad 1: Cell31 -> Cell30
- R32 pad 1: Cell32 -> Cell31
- R33 pad 1: Cell33 -> Cell32
- R34 pad 1: Cell34 -> Cell33
- R35 pad 1: Cell35 -> Cell34
- R36 pad 1: Cell36 -> Cell35
- R37 pad 1: Cell37 -> Cell36
- R38 pad 1: Cell38 -> Cell37
- R39 pad 1: Cell39 -> Cell38
- R4 pad 1: Cell4 -> Cell3
- R40 pad 1: Cell40 -> Cell39
- R41 pad 1: Cell41 -> Cell40
- R42 pad 1: Cell42 -> Cell41
- R43 pad 1: Cell43 -> Cell42
- R44 pad 1: Cell44 -> Cell43
- R45 pad 1: Cell45 -> Cell44
- R46 pad 1: Cell46 -> Cell45
- R47 pad 1: Cell47 -> Cell46
- R48 pad 1: Cell48 -> Cell47
- R49 pad 1: Cell49 -> Cell48
- R5 pad 1: Cell5 -> Cell4
- R50 pad 1: Cell50 -> Cell49
- R51 pad 1: Cell51 -> Cell50
- R52 pad 1: Cell52 -> Cell51
- R53 pad 1: Cell53 -> Cell52
- R54 pad 1: Cell54 -> Cell53
- R55 pad 1: Cell55 -> Cell54
- R56 pad 1: Cell56 -> Cell55
- R57 pad 1: Cell57 -> Cell56
- R58 pad 1: Cell58 -> Cell57
- R59 pad 1: Cell59 -> Cell58
- R6 pad 1: Cell6 -> Cell5
- R60 pad 1: Cell60 -> Cell59
- R61 pad 1: Cell61 -> Cell60
- R62 pad 1: Cell62 -> Cell61
- R63 pad 1: Cell63 -> Cell62
- R64 pad 1: Cell64 -> Cell63
- R65 pad 1: Cell65 -> +3V3
- R65 pad 2: B -> GND
- R66 pad 1: Cell66 -> +3V3
- R66 pad 2: B -> GND
- R7 pad 1: Cell7 -> Cell6
- R8 pad 1: Cell8 -> Cell7
- R9 pad 1: Cell9 -> Cell8
- U1 pad 1: Cell8 -> U1_Common
- U1 pad 10: U1_CS_5V -> SA0_5V
- U1 pad 11: MOSI_5V -> SA1_5V
- U1 pad 12: MISO_5V -> GND
- U1 pad 13: CLK_5V -> SA3_5V
- U1 pad 14: GND -> SA2_5V
- U1 pad 15: +5V -> GND
- U1 pad 16: +5V -> Cell15
- U1 pad 9: GND -> Cell0
- U2 pad 1: Cell18 -> U2_Common
- U2 pad 10: U2_CS_5V -> SA0_5V
- U2 pad 11: MOSI_5V -> SA1_5V
- U2 pad 12: MISO_5V -> GND
- U2 pad 13: CLK_5V -> SA3_5V
- U2 pad 14: GND -> SA2_5V
- U2 pad 15: +5V -> GND
- U2 pad 16: +5V -> Cell31
- U2 pad 2: Cell17 -> Cell23
- U2 pad 3: Cell16 -> Cell22
- U2 pad 4: Cell15 -> Cell21
- U2 pad 5: Cell14 -> Cell20
- U2 pad 6: Cell13 -> Cell19
- U2 pad 7: Cell12 -> Cell18
- U2 pad 8: Cell11 -> Cell17
- U2 pad 9: GND -> Cell16
- U3 pad 1: Cell28 -> U3_Common
- U3 pad 10: U3_CS_5V -> SA0_5V
- U3 pad 11: MOSI_5V -> SA1_5V
- U3 pad 12: MISO_5V -> GND
- U3 pad 13: CLK_5V -> SA3_5V
- U3 pad 14: GND -> SA2_5V
- U3 pad 15: +5V -> GND
- U3 pad 16: +5V -> Cell47
- U3 pad 2: Cell27 -> Cell39
- U3 pad 3: Cell26 -> Cell38
- U3 pad 4: Cell25 -> Cell37
- U3 pad 5: Cell24 -> Cell36
- U3 pad 6: Cell23 -> Cell35
- U3 pad 7: Cell22 -> Cell34
- U3 pad 8: Cell21 -> Cell33
- U3 pad 9: GND -> Cell32
- U4 pad 1: Cell38 -> U4_Common
- U4 pad 10: U4_CS_5V -> SA0_5V
- U4 pad 11: MOSI_5V -> SA1_5V
- U4 pad 12: MISO_5V -> GND
- U4 pad 13: CLK_5V -> SA3_5V
- U4 pad 14: GND -> SA2_5V
- U4 pad 15: +5V -> GND
- U4 pad 16: +5V -> Cell63
- U4 pad 2: Cell37 -> Cell55
- U4 pad 3: Cell36 -> Cell54
- U4 pad 4: Cell35 -> Cell53
- U4 pad 5: Cell34 -> Cell52
- U4 pad 6: Cell33 -> Cell51
- U4 pad 7: Cell32 -> Cell50
- U4 pad 8: Cell31 -> Cell49
- U4 pad 9: GND -> Cell48
- U5 pad 1: Cell48 -> GND
- U5 pad 10: U5_CS_5V -> SCL_5V
- U5 pad 2: Cell47 -> ALERT/RDY_5V
- U5 pad 3: Cell46 -> GND
- U5 pad 4: Cell45 -> U1_Common
- U5 pad 5: Cell44 -> U2_Common
- U5 pad 6: Cell43 -> U3_Common
- U5 pad 7: Cell42 -> U4_Common
- U5 pad 8: Cell41 -> +5V
- U5 pad 9: GND -> SDA_5V
- U6 pad 1: Cell58 -> +5V
- U6 pad 10: U6_CS_5V -> ALERT/RDY_5V
- U6 pad 11: MOSI_5V -> SCL_5V
- U6 pad 12: MISO_5V -> SDA_5V
- U6 pad 2: Cell57 -> +3V3
- U6 pad 3: Cell56 -> SDA_3V3
- U6 pad 4: Cell55 -> SCL_3V3
- U6 pad 5: Cell54 -> ALERT/RDY_3V3
- U6 pad 6: Cell53 -> unconnected-(U6-A3-Pad6)
- U6 pad 7: Cell52 -> GND
- U6 pad 8: Cell51 -> +3V3
- U6 pad 9: GND -> unconnected-(U6-B3-Pad9)
- U7 pad 1: Cell68 -> +5V
- U7 pad 10: U7_CS_5V -> SA2_5V
- U7 pad 11: MOSI_5V -> SA1_5V
- U7 pad 12: MISO_5V -> SA0_5V
- U7 pad 2: Cell67 -> +3V3
- U7 pad 3: Cell66 -> SA0_3V3
- U7 pad 4: Cell65 -> SA1_3V3
- U7 pad 5: Cell64 -> SA2_3V3
- U7 pad 6: Cell63 -> SA3_3V3
- U7 pad 7: Cell62 -> GND
- U7 pad 8: Cell61 -> +3V3
- U7 pad 9: GND -> SA3_5V
Routing:
- net B: track 3708.2 -> 2317.2 mm, vias 100 -> 64
- net MOSI_5V: track 814.5 -> 0.00 mm, vias 4 -> 0
- net MISO_5V: track 809.1 -> 0.00 mm, vias 25 -> 0
- net CLK_5V: track 803.4 -> 0.00 mm, vias 25 -> 0
- net GND: track 1237.2 -> 494.2 mm, vias 110 -> 30
- net +5V: track 1069.0 -> 355.9 mm, vias 28 -> 8
- net U1_CS_5V: track 413.5 -> 0.00 mm, vias 4 -> 0
- net U12_CS_5V: track 249.2 -> 0.00 mm, vias 4 -> 0
- net SA3_5V: track 0.00 -> 245.5 mm, vias 0 -> 8
- net SA2_5V: track 0.00 -> 233.8 mm, vias 0 -> 8
- net U11_CS_5V: track 233.0 -> 0.00 mm, vias 2 -> 0
- net SA1_5V: track 0.00 -> 231.8 mm, vias 0 -> 8
- net SA0_5V: track 0.00 -> 222.5 mm, vias 0 -> 2
- net U2_CS_5V: track 212.0 -> 0.00 mm, vias 16 -> 0
- net U3_CS_5V: track 191.1 -> 0.00 mm, vias 14 -> 0
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- removed copper zone on B.Cu, net GND
- removed copper zone on F.Cu, net GND
Other:
- board size 245 x 245 mm -> 200 x 200 mm
- board text added: "*"

Commit message: Added ground plane
Routing:
- net GND: vias 30 -> 96
- added copper zone on B.Cu, net GND
- added copper zone on F.Cu, net GND

Commit message: changed pin headers
Parts:
- J2, J3: value HARWIN_M20-7861546 -> PinHeader_1x15_P2.54mm_Vertical_SMD_Pin1Right; footprint FS_4_Global_Footprint_Library:HARWIN_M20-7861546 -> Connector_PinHeader_2.54mm:PinHeader_1x15_P2.54mm_Vertical_SMD_Pin1Right
- moved J3 0.16 mm to (278.6, 112.8), turned to 0 degrees
- moved J2 0.16 mm to (263.3, 112.8), turned to 0 degrees

Commit message: pull request changes made
Parts:
- U1, U2, U3, U4: value ~ -> CD74HC4067M96; footprint Package_SO:SSOP-24_5.3x8.2mm_P0.65mm -> FS_4_Global_Footprint_Library:SOIC127P1030X265-24N
- moved C5 4.50 mm to (263.5, 31.0)
- moved U5 4.50 mm to (263.5, 36.0)
- moved U4 3.67 mm to (241.9, 37.0)
- moved U1 3.60 mm to (109.4, 37.0)
- moved U3 3.60 mm to (197.9, 37.0)
- moved U2 3.41 mm to (153.4, 37.0)
Connections:
- net B renamed BalanceNet
Routing:
- net SA1_5V: track 231.8 -> 264.9 mm
- net SA0_5V: track 222.5 -> 254.1 mm
- net GND: track 494.4 -> 523.3 mm
- net SA3_5V: track 245.5 -> 270.9 mm
- net SA2_5V: track 233.8 -> 257.3 mm
- net U4_Common: track 44.2 -> 33.9 mm, vias 4 -> 2
- net U2_Common: track 126.9 -> 119.9 mm, vias 4 -> 2
- net U3_Common: track 83.4 -> 76.4 mm, vias 4 -> 2
- net U1_Common: track 169.8 -> 163.4 mm
- net Cell63: track 172.6 -> 167.6 mm
- net Cell47: track 172.6 -> 167.6 mm
- net Cell15: track 172.6 -> 167.8 mm
- net Cell31: track 172.5 -> 167.8 mm
- net SCL_5V: track 18.2 -> 22.8 mm
- net Cell48: track 19.4 -> 14.8 mm
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
Commit message: Balance net changed to a filled zone
Routing:
- net GND: vias 96 -> 30
- added copper zone on B.Cu, net BalanceNet
- removed copper zone on B.Cu, net GND

Commit message: added silkscreen text
Other:
- board text added: "Formula Slug Rev 1.0 Cell Voltage Checker/Balancer Designed by Karsten Vivian"
Changed lines of the file:
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@@
 		)
 	)
+	(gr_text "Formula Slug Rev 1.0\nCell Voltage Checker/Balancer\nDesigned by Karsten Vivian"
+		(at 251.46 212.09 0)
+		(layer "F.SilkS")
+		(effects
+			(font
+				(size 1 1)
+				(thickness 0.15)
+			)
+		)
+	)
 	(segment
 		(start 277 164.5)
@@
 		(polygon
 			(pts
-				(xy 316.5 201.5) (xy 308 3.5) (xy 71.128 4) (xy 77.224 243.5) (xy 297 241) (xy 316.5 201.5) (xy 316.5 201.5)
-				(xy 316.5 201.5)
+				(xy 316.5 201.5) (xy 308 3.5) (xy 71.128 4) (xy 77.224 243.5) (xy 297 241)
 			)
 		)

Commit message: DFM changes (not as bad as temp sense board thank god)
Routing:
- net GND: track 523.3 -> 525.5 mm
- net U3_Common: track 76.4 -> 75.9 mm
