File: Sample Pack Busbar Board/Sample Pack Busbar Board.kicad_sch (KiCad schematic)
At the start: 10 parts, among them J2 Conn_01x09_MountingPin

Commit message: changes for order
Parts:
- added J1: Conn_01x05_MountingPin, symbol Connector_Generic_MountingPin:Conn_01x05_MountingPin
- J2: footprint (none) -> FS_4_Global_Footprint_Library:CON_5051100992_MOL
Connections:
- no-connect marks 4 -> 11
Changed lines of the file:
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@@
+	)
+	(no_connect
+		(at 101.6 62.23)
 	)
 	(no_connect
@@
 	)
 	(no_connect
+		(at 101.6 64.77)
+	)
+	(no_connect
 		(at 106.68 26.67)
+	)
+	(no_connect
+		(at 101.6 72.39)
 	)
 	(no_connect
 		(at 101.6 39.37)
+	)
+	(no_connect
+		(at 101.6 67.31)
+	)
+	(no_connect
+		(at 101.6 69.85)
+	)
+	(no_connect
+		(at 106.68 77.47)
+	)
+	(no_connect
+		(at 105.41 77.47)
 	)
 	(wire
@@
 			)
 		)
-		(property "Footprint" ""
+		(property "Footprint" "FS_4_Global_Footprint_Library:CON_5051100992_MOL"
 			(at 106.68 41.91 0)
 			(effects
@@
 					(unit 1)
 				)
+			)
+		)
+	)
+	(symbol
+		(lib_id "Connector_Generic_MountingPin:Conn_01x05_MountingPin")
+		(at 106.68 67.31 0)
+		(unit 1)
+		(exclude_from_sim no)
+		(in_bom yes)
+		(on_board yes)
+		(dnp no)
+		(fields_autoplaced yes)
+		(property "Reference" "J1"
+			(at 109.22 66.3955 0)
+			(effects
+				(font
+					(size 1.27 1.27)
+				)
+				(justify left)
+			)
+		)
+		(property "Value" "Conn_01x05_MountingPin"
+			(at 109.22 68.9355 0)
+			(effects
+				(font
+					(size 1.27 1.27)
+				)
+				(justify left)
+			)
+		)
+		(property "Footprint" ""
+			(at 106.68 67.31 0)
+			(effects
+				(font
+					(size 1.27 1.27)
+				)
+				(hide yes)
+			)
+		)
+		(property "Datasheet" "~"
+			(at 106.68 67.31 0)
+			(effects
+				(font
+					(size 1.27 1.27)
+				)
+				(hide yes)
+			)
+		)
+		(property "Description" "Generic connectable mounting pin connector, single row, 01x05, script generated (kicad-library-utils/schlib/autogen/connector/)"
+			(at 106.68 67.31 0)
+			(effects
+				(font
+					(size 1.27 1.27)
+				)
+				(hide yes)
+			)
+		)
+		(pin "4"
+		)
+		(pin "3"
+		)
+		(pin "1"
+		)
+		(pin "2"
+		)
+		(pin "5"
+		)
+		(pin "MP"
+		)
+		(instances
+			(project ""
+				(path "/3e659f42-521e-4c35-9a94-9c44ca4c0cd4"
+					(reference "J1")
+					(unit 1)
+				)

Commit message: fixed track spacing for JLC capabilities
Parts:
- J2: footprint FS_4_Global_Footprint_Library:CON_5051100992_MOL -> Connector_PinHeader_2.00mm:PinHeader_1x06_P2.00mm_Vertical
Connections:
- net V+: now also J2.6 (Pin_6); no longer J2.9 (Pin_9)
Changed lines of the file:
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@@
-	)
-	(no_connect
-		(at 101.6 39.37)
 	)
 	(no_connect
@@
 		(at 105.41 77.47)
 	)
+	(no_connect
+		(at 101.6 31.75)
+	)
 	(wire
 		(pts
@@
 	(wire
 		(pts
-			(xy 88.9 31.75) (xy 101.6 31.75)
-		)
-		(stroke
-			(width 0)
-			(type default)
-		)
-	)
-	(wire
-		(pts
 			(xy 83.82 44.45) (xy 83.82 40.64)
 		)
@@
 	(wire
 		(pts
-			(xy 88.9 31.75) (xy 88.9 20.32)
+			(xy 88.9 20.32) (xy 88.9 39.37)
 		)
 		(stroke
@@
 		(pts
 			(xy 17.78 39.37) (xy 17.78 40.64)
+		)
+		(stroke
+			(width 0)
+			(type default)
+		)
+	)
+	(wire
+		(pts
+			(xy 88.9 39.37) (xy 101.6 39.37)
 		)
 		(stroke
@@
 			)
 		)
-		(property "Footprint" "FS_4_Global_Footprint_Library:CON_5051100992_MOL"
+		(property "Footprint" "Connector_PinHeader_2.00mm:PinHeader_1x06_P2.00mm_Vertical"
 			(at 106.68 41.91 0)
 			(effects
