File: peripheral-boards/peripheral-boards.kicad_sch (KiCad schematic)
At the start: 72 parts, among them J8 FTSH-107-01-F-DV-K-P-TR, SW1 Y97KT23B5NAFP, SW5 A6H-4101, U1 SNG-SPRC-001, U10 D6T-8L-09H, U11 Brake Temp Sense, U12 INA826AIDR, U13 REF35160QDBVR, U14 TCA9406DC, U2 TCA9406DC, U3 STM32G441KBTx, U4 ISO1044DUB, U5 MCP1703AT-5002E/CB, U6 MCP1703AT-3302E/CB, U7 Suspension Travel Sensor, U8 LMV331, U9 D6T-1A-02, Y1 ECS-240-8-37B-CKY-TR

Commit message: fixed Vcca side
Connections:
- net +3V3: now also U14.6 (OE), U14.7 (VCCB), U2.6 (OE), U2.7 (VCCB); no longer U14.3 (VCCA), U2.3 (VCCA)
- net +5V: now also U14.3 (VCCA), U2.3 (VCCA); no longer U14.7 (VCCB), U2.7 (VCCB)
- net 1x1_TireTemp_Sensor_SCL: now also U14.5 (SCL_A); no longer U14.8 (SCL_B)
- net 1x1_TireTemp_Sensor_SDA: now also U14.4 (SDA_A); no longer U14.1 (SDA_B)
- net 1x8_TireTemp_Sensor_SCL: now also U2.5 (SCL_A); no longer U2.8 (SCL_B)
- net 1x8_TireTemp_Sensor_SDA: now also U2.4 (SDA_A); no longer U2.1 (SDA_B)
- new net: J1.24, U2.1 (SDA_B), U9. (GND)
- new net: J1.25, U2.8 (SCL_B), U9. (GND)
- new net: J1.16, U10. (GND), U14.8 (SCL_B)
- new net: J1.17, U10. (GND), U14.1 (SDA_B)
- no-connect marks 10 -> 8
Changed lines of the file:
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@@
 	)
 	(no_connect
-		(at 254 40.64)
-	)
-	(no_connect
 		(at 44.45 240.03)
 	)
@@
 		(at 57.15 229.87)
 	)
-	(no_connect
-		(at 378.46 43.18)
-	)
 	(wire
 		(pts
@@
 	(wire
 		(pts
+			(xy 356.87 43.18) (xy 358.14 43.18)
+		)
+		(stroke
+			(width 0)
+			(type default)
+		)
+	)
+	(wire
+		(pts
 			(xy 236.22 91.44) (xy 232.41 91.44)
 		)
@@
 	(wire
 		(pts
-			(xy 233.68 43.18) (xy 222.25 43.18)
-		)
-		(stroke
-			(width 0)
-			(type default)
-		)
-	)
-	(wire
-		(pts
 			(xy 40.64 90.17) (xy 35.56 90.17)
 		)
@@
 	(wire
 		(pts
+			(xy 222.25 43.18) (xy 233.68 43.18)
+		)
+		(stroke
+			(width 0)
+			(type default)
+		)
+	)
+	(wire
+		(pts
 			(xy 40.64 25.4) (xy 40.64 31.75)
 		)
@@
 	(wire
 		(pts
+			(xy 232.41 40.64) (xy 233.68 40.64)
+		)
+		(stroke
+			(width 0)
+			(type default)
+		)
+	)
+	(wire
+		(pts
 			(xy 283.21 223.52) (xy 288.29 223.52)
 		)
@@
 		(lib_id "Interface:TCA9406DC")
 		(at 368.3 45.72 0)
+		(mirror y)
 		(unit 1)
 		(exclude_from_sim no)
@@
 		(dnp no)
 		(property "Reference" "U2"
-			(at 377.19 54.61 0)
+			(at 375.92 57.15 0)
 			(effects
 				(font
@@
 		)
 		(property "Value" "TCA9406DC"
-			(at 374.65 57.15 0)
+			(at 382.27 59.69 0)
 			(effects
 				(font
@@
 		)
 		(property "Footprint" "Package_SO:SSOP-8_2.95x2.8mm_P0.65mm"
-			(at 358.14 36.83 0)
+			(at 378.46 36.83 0)
 			(effects
 				(font
@@
 		)
 		(property "Datasheet" "www.ti.com/lit/ds/symlink/tca9406.pdf"
-			(at 360.68 34.29 0)
+			(at 375.92 34.29 0)
 			(effects
 				(font
@@
 	)
 	(symbol
+		(lib_id "power:+5V")
+		(at 356.87 43.18 0)
+		(mirror y)
+		(unit 1)
+		(exclude_from_sim no)
+		(in_bom yes)
+		(on_board yes)
+		(dnp no)
+		(property "Reference" "#PWR071"
+			(at 356.87 46.99 0)
+			(effects
+				(font
+					(size 1.27 1.27)
+				)
+				(hide yes)
+			)
+		)
+		(property "Value" "+3V3"
+			(at 356.87 39.37 0)
+			(effects
+				(font
+					(size 1.27 1.27)
+				)
+			)
+		)
+		(property "Footprint" ""
+			(at 356.87 43.18 0)
+			(effects
+				(font
+					(size 1.27 1.27)
+				)
+				(hide yes)
+			)
+		)
+		(property "Datasheet" ""
+			(at 356.87 43.18 0)
+			(effects
+				(font
+					(size 1.27 1.27)
+				)
+				(hide yes)
+			)
+		)
+		(property "Description" "Power symbol creates a global label with name \"+5V\""
+			(at 356.87 43.18 0)
+			(effects
+				(font
+					(size 1.27 1.27)
+				)
+				(hide yes)
+			)
+		)
+		(pin "1"
+		)
+		(instances
+			(project "peripheral-boards"
+				(path "/3ffe4db1-2415-46df-8a68-5537f544061f"
+					(reference "#PWR071")
+					(unit 1)
+				)
+			)
+		)
+	)
+	(symbol
 		(lib_id "power:+3V3")
 		(at 171.45 182.88 0)
@@
 	)
 	(symbol
+		(lib_id "power:+5V")
+		(at 232.41 40.64 0)
+		(mirror y)
+		(unit 1)
+		(exclude_from_sim no)
+		(in_bom yes)
+		(on_board yes)
+		(dnp no)
+		(property "Reference" "#PWR070"
+			(at 232.41 44.45 0)
+			(effects
+				(font
+					(size 1.27 1.27)
+				)
+				(hide yes)
+			)
+		)
+		(property "Value" "+3V3"
+			(at 232.41 36.83 0)
+			(effects
+				(font
+					(size 1.27 1.27)
+				)
+			)
+		)
+		(property "Footprint" ""
+			(at 232.41 40.64 0)
+			(effects
+				(font
+					(size 1.27 1.27)
+				)
+				(hide yes)
+			)
+		)
+		(property "Datasheet" ""
+			(at 232.41 40.64 0)
+			(effects
+				(font
+					(size 1.27 1.27)
+				)
+				(hide yes)
+			)
+		)
+		(property "Description" "Power symbol creates a global label with name \"+5V\""
+			(at 232.41 40.64 0)
+			(effects
+				(font
+					(size 1.27 1.27)
+				)
+				(hide yes)
+			)
+		)
+		(pin "1"
+		)
+		(instances
+			(project "peripheral-boards"
+				(path "/3ffe4db1-2415-46df-8a68-5537f544061f"
+					(reference "#PWR070")
+					(unit 1)
+				)
+			)
+		)
+	)
+	(symbol
 		(lib_id "Device:C")
 		(at 374.65 26.67 270)
@@
 		(lib_id "Interface:TCA9406DC")
 		(at 243.84 43.18 0)
+		(mirror y)
 		(unit 1)
 		(exclude_from_sim no)
@@
 		(on_board yes)
 		(dnp no)
-		(fields_autoplaced yes)
 		(property "Reference" "U14"
-			(at 245.9833 55.88 0)
+			(at 251.46 54.61 0)
 			(effects
 				(font
@@
 		)
 		(property "Value" "TCA9406DC"
-			(at 245.9833 58.42 0)
+			(at 259.08 57.15 0)
 			(effects
 				(font
@@
 		)
 		(property "Footprint" "Package_SO:SSOP-8_2.95x2.8mm_P0.65mm"
-			(at 233.68 34.29 0)
+			(at 254 34.29 0)
 			(effects
 				(font
@@
 		)
 		(property "Datasheet" "www.ti.com/lit/ds/symlink/tca9406.pdf"
-			(at 236.22 31.75 0)
+			(at 251.46 31.75 0)
 			(effects
 				(font
