File: peripheral-boards/peripheral-boards.kicad_pcb (KiCad board)
At the start: 2 copper layers, 41 parts, among them J1 ATS668LSM, J4 Strain Gauge, J8 FTSH-107-01-F-DV-K-P-TR, SW1 Y97KT23B5NAFP, SW2 SW_Nidec_CAS-120A1, SW3 SW_Nidec_CAS-120A1, SW4 SW_Nidec_CAS-120A1, U2 INA125U, U3 STM32G441KBTx, U4 ISO1044DUB, U5 MCP1703AT-5002E/CB, U6 MCP1703AT-3302E/CB, Y1 ECS-240-8-37B-CKY-TR

Commit message: Edited sensor blocks and mock layout, not done
Parts:
- added C6: 100nF, Capacitor_SMD:C_0805_2012Metric_Pad1.18x1.45mm_HandSolder, F.Cu at (180.6, 44.6)
- added D1: 1V, Diode_SMD:D_0805_2012Metric_Pad1.15x1.40mm_HandSolder, F.Cu at (185.4, 49.6)
- added R13: 10K, Resistor_SMD:R_0603_1608Metric_Pad0.98x0.95mm_HandSolder, F.Cu at (185.1, 44.3)
- added R14: 10K, Resistor_SMD:R_0603_1608Metric_Pad0.98x0.95mm_HandSolder, F.Cu at (185.1, 46.8)
- added R16: 4.7k, Resistor_SMD:R_0805_2012Metric_Pad1.20x1.40mm_HandSolder, F.Cu at (175.8, 47.5)
- added R17: 4.7k, Resistor_SMD:R_0805_2012Metric_Pad1.20x1.40mm_HandSolder, F.Cu at (175.8, 50.5)
- added R5: 10K, Capacitor_SMD:C_0805_2012Metric_Pad1.18x1.45mm_HandSolder, F.Cu at (180.6, 47.6)
- added R6: 4.7k, Resistor_SMD:R_0805_2012Metric_Pad1.20x1.40mm_HandSolder, F.Cu at (175.8, 44.6)
- added SW5: A6H-4101, Library:SW_A6H-4101_OMR, F.Cu at (178.1, 39.1)
- added U8: LMV331, Package_TO_SOT_SMD:SOT-23-5, F.Cu at (185.3, 37.5)
- J1: value ATS668LSM -> ~
- R3: value 15K -> 10K
- moved C5 164.0 mm to (36.0, 60.0), turned to 180 degrees
- moved C16 74.3 mm to (217.5, 93.5)
- moved FB1 73.3 mm to (216.0, 103.0)
- moved C14 72.6 mm to (216.5, 84.5)
- moved C15 72.1 mm to (216.5, 82.5)
- moved R12 69.4 mm to (217.4, 90.5)
- moved C18 68.1 mm to (216.5, 80.5)
- moved U3 66.0 mm to (209.5, 93.0)
- moved C7 63.1 mm to (201.5, 94.0)
- moved C10 58.7 mm to (201.5, 83.0)
- moved C13 57.6 mm to (201.5, 80.5)
- moved J8 56.5 mm to (206.9, 105.7)
- moved C17 55.2 mm to (201.5, 85.5)
- moved R4 54.5 mm to (201.5, 90.5)
- moved SW1 54.3 mm to (209.5, 82.5)
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Connections:
- C8 pad 2: +5V -> +3V3
- J1 pad 2: Net-(J1-Pin_2) -> CANL
- J1 pad 3: GND -> CANH
- R1 pad 1: Net-(J1-Pin_2) -> /Wheel_Speed_Out
- R2 pad 1: Net-(J1-Pin_2) -> /Wheel_Speed_Out
- R3 pad 2: unconnected-(R3-Pad2) -> +3V3
- R4 pad 1: Net-(SW4-C) -> Net-(R4-Pad1)
- R4 pad 2: CAN1_RX -> CANH
- R7 pad 1: +3V3 -> /Vrefout
- U2 pad 4: /VrefBG -> /Vrefout
- U3 pad 1: +3V3 -> unconnected-(U3-VDD-Pad1)
- U3 pad 10: unconnected-(U3-PA5-Pad10) -> wheel speed
- U3 pad 11: unconnected-(U3-PA6-Pad11) -> Net-(U3-PA6)
- U3 pad 15: +3V3_A -> unconnected-(U3-VDDA-Pad15)
- U3 pad 17: +3V3 -> unconnected-(U3-VDD-Pad17)
- U3 pad 20: unconnected-(U3-PA10-Pad20) -> Net-(U3-PA10)
- U3 pad 27: unconnected-(U3-PB4-Pad27) -> Net-(U3-PB4)
- U3 pad 28: 1x1_TireTemp_Sensor_SDA -> Net-(U3-PB5)
- U3 pad 29: unconnected-(U3-PB6-Pad29) -> Net-(U3-PB6)
- U3 pad 30: unconnected-(U3-PB7-Pad30) -> 1x1_TireTemp_Sensor_SDA
- U3 pad 5: Net-(SW2-B) -> Net-(U3-PA0)
- U3 pad 6: Net-(SW3-B) -> Net-(U3-PA1)
- U3 pad 9: unconnected-(U3-PA4-Pad9) -> Net-(U3-PA4)
- U4 pad 1: +5V -> +3V3

Commit message: added first layout traces
Parts:
- moved SW5 91.3 mm to (234.1, 111.2)
- moved R13 70.9 mm to (232.2, 97.4)
- moved R14 70.9 mm to (232.2, 99.9)
- moved C5 63.1 mm to (99.0, 62.1)
- moved D1 47.3 mm to (138.4, 44.0), turned to -90 degrees
- moved U8 44.0 mm to (141.3, 39.9)
- moved R5 39.3 mm to (141.6, 42.9), turned to 180 degrees
- moved R3 38.5 mm to (137.1, 37.8), turned to 90 degrees
- moved C6 35.5 mm to (145.6, 38.1)
- moved R2 34.4 mm to (133.9, 39.0)
- moved R1 30.7 mm to (130.3, 40.1), turned to -90 degrees
- moved R4 25.0 mm to (218.3, 109.0)
Routing:
- net +3V3: track 0.00 -> 16.1 mm
- net GND: track 0.00 -> 6.46 mm, vias 0 -> 4
- net Net-(U8-+): track 0.00 -> 5.35 mm
- net /+1V_REF: track 0.00 -> 4.37 mm
- net /Wheel_Speed_Out: track 0.00 -> 2.59 mm

Commit message: Edited layout, very much a rough draft
Parts:
- removed J4: Strain Gauge, Connector_Molex:Molex_Nano-Fit_105309-xx02_1x02_P2.50mm_Vertical
- removed R15: 4.7k, Resistor_SMD:R_0805_2012Metric_Pad1.20x1.40mm_HandSolder
- removed SW2, SW3, SW4: SW_Nidec_CAS-120A1, Button_Switch_SMD:Nidec_Copal_CAS-120A
- removed U2: INA125U, Package_SO:SOIC-16_3.9x9.9mm_P1.27mm
- added C11: 1uF, Capacitor_SMD:C_0603_1608Metric_Pad1.08x0.95mm_HandSolder, F.Cu at (96.1, 125.9)
- added C12: 100nF, Capacitor_SMD:C_0603_1608Metric_Pad1.08x0.95mm_HandSolder, F.Cu at (119.6, 134.4)
- added C19: 1uF, Capacitor_SMD:C_0603_1608Metric_Pad1.08x0.95mm_HandSolder, F.Cu at (96.2, 134.4)
- added C20: 100nF, Capacitor_SMD:C_0603_1608Metric_Pad1.08x0.95mm_HandSolder, F.Cu at (132.3, 127.0)
- added C21: 100nF, Capacitor_SMD:C_0603_1608Metric_Pad1.08x0.95mm_HandSolder, F.Cu at (128.5, 108.7)
- added R18: 309R, Resistor_SMD:R_0603_1608Metric_Pad0.98x0.95mm_HandSolder, F.Cu at (104.9, 134.4)
- added R19: 16K, Resistor_SMD:R_0603_1608Metric_Pad0.98x0.95mm_HandSolder, F.Cu at (96.1, 142.4)
- added R20: 16K, Resistor_SMD:R_0603_1608Metric_Pad0.98x0.95mm_HandSolder, F.Cu at (96.1, 144.9)
- added U12: INA826AIDR, Package_SO:SOIC-8_3.9x4.9mm_P1.27mm, F.Cu at (123.7, 127.3)
- added U13: REF35160QDBVR, Package_TO_SOT_SMD:SOT-23-6, F.Cu at (123.7, 133.1)
- C14: footprint Capacitor_SMD:C_0603_1608Metric_Pad1.08x0.95mm_HandSolder -> Capacitor_SMD:C_0805_2012Metric_Pad1.18x1.45mm_HandSolder
- C5, C6, C8, C9: footprint Capacitor_SMD:C_0805_2012Metric_Pad1.18x1.45mm_HandSolder -> Capacitor_SMD:C_0603_1608Metric_Pad1.08x0.95mm_HandSolder
- D1: footprint Diode_SMD:D_0805_2012Metric_Pad1.15x1.40mm_HandSolder -> Diode_SMD:D_SMA
- J1: footprint Connector_Molex:Molex_Nano-Fit_105309-xx03_1x03_P2.50mm_Vertical -> FS_4_Global_Footprint_Library:ATS13-26PA-BM01
- R1, R2, R3, R5: footprint Capacitor_SMD:C_0805_2012Metric_Pad1.18x1.45mm_HandSolder -> Resistor_SMD:R_0603_1608Metric_Pad0.98x0.95mm_HandSolder
- R10: value Extra -> 16K; footprint Resistor_SMD:R_0805_2012Metric_Pad1.20x1.40mm_HandSolder -> Resistor_SMD:R_0603_1608Metric_Pad0.98x0.95mm_HandSolder
- R11: value 60.4R -> 16K; footprint Resistor_SMD:R_0805_2012Metric_Pad1.20x1.40mm_HandSolder -> Resistor_SMD:R_0603_1608Metric_Pad0.98x0.95mm_HandSolder
- R16, R17, R6, R8: footprint Resistor_SMD:R_0805_2012Metric_Pad1.20x1.40mm_HandSolder -> Resistor_SMD:R_0603_1608Metric_Pad0.98x0.95mm_HandSolder
- R4: value 120 -> 120R
- R7, R9: value 120R -> 360R; footprint Resistor_SMD:R_0805_2012Metric_Pad1.20x1.40mm_HandSolder -> Resistor_SMD:R_0603_1608Metric_Pad0.98x0.95mm_HandSolder
- U4: footprint Package_SO:SOIC-8_3.9x4.9mm_P1.27mm -> FS_4_Global_Footprint_Library:SOIC-8_ISO1044BD
- moved C8 98.9 mm to (145.3, 122.4)
- moved U4 97.0 mm to (148.3, 117.9), turned to 90 degrees
- moved C9 88.0 mm to (146.8, 113.3), turned to 180 degrees
- moved R12 85.7 mm to (142.2, 131.6), turned to 180 degrees
- moved R14 85.3 mm to (155.2, 136.4), turned to 180 degrees
- moved R13 85.1 mm to (155.4, 134.1), turned to 180 degrees
- moved C16 84.1 mm to (144.0, 134.4)
- moved R1 82.9 mm to (136.1, 122.8), turned to 0 degrees
- moved C6 82.7 mm to (141.2, 120.7)
- moved R3 82.5 mm to (132.8, 120.2), turned to 180 degrees
- moved R5 79.9 mm to (139.7, 122.8), turned to 0 degrees
- moved R2 78.8 mm to (132.8, 117.7)
- moved FB1 78.1 mm to (141.5, 126.2)
- moved Y1 77.5 mm to (147.8, 137.2), turned to 180 degrees
- moved C18 77.4 mm to (156.5, 129.3)
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Connections:
- C5 pad 1: +3V3 -> GND
- C5 pad 2: GND -> +3V3
- R10 pad 2: Net-(R10-Pad2) -> STRAIN
- R11 pad 1: Net-(R10-Pad1) -> Net-(J1D-1)
- R11 pad 2: Net-(R10-Pad2) -> SUSPENSION 
- R4 pad 2: CANH -> CANL
- R7 pad 1: /Vrefout -> GND
- RV1 pad 2: /Vin- -> /1V6_Vref
- RV1 pad 3: GND -> /1V6_Vref
- SW5 pad 3: CANL -> Net-(U3-PA1)
- SW5 pad 4: Net-(U3-PA1) -> CANH
- U3 pad 1: unconnected-(U3-VDD-Pad1) -> +3V3
- U3 pad 15: unconnected-(U3-VDDA-Pad15) -> +3V3_A
- U3 pad 17: unconnected-(U3-VDD-Pad17) -> +3V3
Routing:
- net CANH: track 0.00 -> 25.5 mm, vias 0 -> 1
- net 1x1_TireTemp_Sensor_SDA: track 0.00 -> 17.7 mm
- net CANL: track 0.00 -> 9.99 mm
- net Net-(J1D-1): track 0.00 -> 7.94 mm
- net /OSC_IN: track 0.00 -> 6.60 mm
- net GND: track 6.46 -> 0.00 mm, vias 4 -> 16
- net CAN1_TX: track 0.00 -> 5.33 mm
- net CAN1_RX: track 0.00 -> 5.15 mm
- net /OSC_OUT: track 0.00 -> 4.77 mm
- net +12V: track 0.00 -> 3.61 mm
- net +3V3: track 16.1 -> 13.0 mm
- net /Wheel_Speed_Out: track 2.59 -> 0.00 mm
- net +3V3_A: track 0.00 -> 2.12 mm
- net /BOOT0: track 0.00 -> 2.06 mm
- net +5V: track 0.00 -> 1.95 mm
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- added copper zone on F.Cu, net GND
Other:
- board outline added: 55.9 x 40.6 mm

Commit message: More small changes
Parts:
- added H1: MountingHole_Pad, MountingHole:MountingHole_3.2mm_M3_Pad, F.Cu at (172.7, 99.1)
- added H2: MountingHole_Pad, MountingHole:MountingHole_3.2mm_M3_Pad, F.Cu at (116.8, 139.7)
- moved C2 47.7 mm to (168.6, 109.1), turned to 180 degrees
- moved U6 41.7 mm to (164.8, 105.4), turned to 180 degrees
- moved C4 40.7 mm to (160.9, 110.3)
- moved U5 40.1 mm to (164.8, 110.0), turned to 180 degrees
- moved C3 38.6 mm to (163.1, 102.9), turned to -90 degrees
- moved C1 35.0 mm to (162.1, 107.4), turned to -90 degrees
- moved C12 12.2 mm to (119.4, 122.2)
- moved R10 12.2 mm to (129.0, 116.3)
- moved U12 12.2 mm to (123.4, 115.1)
- moved U13 12.2 mm to (123.4, 120.9)
- moved C20 12.2 mm to (132.1, 114.8)
- moved C5 12.2 mm to (129.2, 113.0)
Routing:
- net +12V: track 3.61 -> 17.6 mm
Other:
- board size 55.9 x 40.6 mm -> 66 x 50.8 mm

Commit message: move components significantly
Parts:
- added TP1: PA4, TestPoint:TestPoint_Pad_D1.5mm, F.Cu at (159.0, 155.9)
- added TP2: PA6, TestPoint:TestPoint_Pad_D1.5mm, F.Cu at (160.5, 159.4)
- added TP3: PA10, TestPoint:TestPoint_Pad_D1.5mm, F.Cu at (151.4, 154.9)
- added TP4: PB4, TestPoint:TestPoint_Pad_D1.5mm, F.Cu at (139.7, 155.4)
- added TP5: PB6, TestPoint:TestPoint_Pad_D1.5mm, F.Cu at (151.9, 160.9)
- added TP6: PB7, TestPoint:TestPoint_Pad_D1.5mm, F.Cu at (143.3, 155.4)
- moved C19 69.7 mm to (165.6, 127.5), turned to 90 degrees
- moved R19 67.6 mm to (158.5, 116.3), turned to -90 degrees
- moved C11 67.3 mm to (163.1, 131.6), turned to -90 degrees
- moved R20 64.0 mm to (153.4, 116.3), turned to -90 degrees
- moved R7 59.9 mm to (157.0, 114.3), turned to -90 degrees
- moved R18 53.8 mm to (156.0, 117.3), turned to 180 degrees
- moved R9 51.5 mm to (154.9, 114.3), turned to 90 degrees
- moved C12 48.0 mm to (167.1, 127.5), turned to 90 degrees
- moved U13 43.5 mm to (165.6, 131.6), turned to 90 degrees
- moved R11 36.3 mm to (155.4, 131.1)
- moved C13 36.0 mm to (138.2, 139.7), turned to 90 degrees
- moved C21 33.8 mm to (152.9, 132.1), turned to -90 degrees
- moved U12 33.2 mm to (156.0, 121.9), turned to -90 degrees
- moved SW1 33.1 mm to (133.6, 139.7), turned to 180 degrees
- moved C5 32.1 mm to (159.5, 123.4), turned to -90 degrees
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Connections:
- J1 pad 20: CANH -> CANL
- J1 pad 21: CANL -> CANH
Routing:
- net CANL: track 9.99 -> 41.4 mm, vias 0 -> 1
- net NRST: track 0.00 -> 28.6 mm
- net VCP_UART_RX: track 0.00 -> 24.0 mm, vias 0 -> 2
- net Net-(U3-PA1): track 0.00 -> 22.5 mm, vias 0 -> 4
- net Net-(U3-PA0): track 0.00 -> 21.2 mm
- net VCP_UART_TX: track 0.00 -> 18.4 mm, vias 0 -> 2
- net 1x1_TireTemp_Sensor_SDA: track 17.7 -> 0.00 mm
- net STLINK_SWDIO: track 0.00 -> 14.4 mm, vias 0 -> 2
- net STLINK_SWCLK: track 0.00 -> 13.6 mm, vias 0 -> 2
- net /1V6_Vref: track 0.00 -> 11.8 mm
- net /Vin+: track 0.00 -> 11.1 mm
- net STLINK_SWO: track 0.00 -> 11.0 mm
- net CANH: track 25.5 -> 35.5 mm
- net /Vin-: track 0.00 -> 8.86 mm
- net Net-(J1D-1): track 7.94 -> 0.00 mm
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Other:
- board size 66 x 50.8 mm -> 50.8 x 45.7 mm

Commit message: new layout changes and extra layers
Parts:
- added C22: 100nF, Capacitor_SMD:C_0603_1608Metric_Pad1.08x0.95mm_HandSolder, F.Cu at (122.4, 110.7)
- added C23: 100nF, Capacitor_SMD:C_0603_1608Metric_Pad1.08x0.95mm_HandSolder, F.Cu at (122.4, 112.5)
- added C24: 100nF, Capacitor_SMD:C_0603_1608Metric_Pad1.08x0.95mm_HandSolder, F.Cu at (122.4, 107.2)
- added C25: 100nF, Capacitor_SMD:C_0603_1608Metric_Pad1.08x0.95mm_HandSolder, F.Cu at (122.4, 105.7)
- added U14: TCA9406DC, Package_SO:SSOP-8_2.95x2.8mm_P0.65mm, F.Cu at (127.3, 110.7)
- added U2: TCA9406DC, Package_SO:SSOP-8_2.95x2.8mm_P0.65mm, F.Cu at (127.2, 106.9)
- moved TP4 32.4 mm to (167.9, 139.4)
- moved TP6 27.6 mm to (167.6, 142.5)
- moved TP2 24.2 mm to (167.1, 136.1)
- moved TP5 22.4 mm to (163.8, 142.0)
- moved TP1 20.6 mm to (164.1, 135.9)
- moved TP3 20.4 mm to (164.3, 139.2)
Connections:
- J1 pad 16: 1x1_TireTemp_Sensor_SDA -> Net-(U14-SCL_B)
- J1 pad 17: 1x1_TireTemp_Sensor_SCL -> Net-(U14-SDA_B)
- J1 pad 20: CANL -> CANH
- J1 pad 21: CANH -> CANL
- J1 pad 24: 1x8_TireTemp_Sensor_SDA -> Net-(U2-SDA_B)
- J1 pad 25: 1x8_TireTemp_Sensor_SCL -> Net-(U2-SCL_B)
Routing:
- net +5V: track 2.30 -> 6.89 mm
- net +3V3: vias 0 -> 12
- added copper zone on In2.Cu, net +3V3
- added copper zone on In1.Cu, net GND
Other:
- copper layers 2 -> 4

Commit message: more layout
Parts:
- removed R16, R17, R6, R8: 4.7k, Resistor_SMD:R_0603_1608Metric_Pad0.98x0.95mm_HandSolder
- removed TP1: PA4, TestPoint:TestPoint_Pad_D1.5mm
- removed TP2: PA6, TestPoint:TestPoint_Pad_D1.5mm
- removed TP3: PA10, TestPoint:TestPoint_Pad_D1.5mm
- removed TP4: PB4, TestPoint:TestPoint_Pad_D1.5mm
- removed TP5: PB6, TestPoint:TestPoint_Pad_D1.5mm
- removed TP6: PB7, TestPoint:TestPoint_Pad_D1.5mm
- moved C23 2.54 mm to (122.4, 110.0)
- moved C22 0.76 mm to (122.4, 111.5)
- moved C24 0.51 mm to (122.4, 107.7)
- moved C25 0.51 mm to (122.4, 106.2)
Routing:
- net +3V3: track 9.54 -> 40.3 mm, vias 12 -> 17
- net Net-(U14-SCL_B): track 0.00 -> 26.7 mm
- net +5V: track 6.89 -> 29.1 mm
- net Net-(U14-SDA_B): track 0.00 -> 17.8 mm
- net Net-(U2-SDA_B): track 0.00 -> 15.8 mm
- net /1V6_Vref: track 11.8 -> 23.2 mm
- net +3V3_A: track 0.16 -> 5.80 mm
- net +12V: track 19.0 -> 21.2 mm
- net GND: track 0.00 -> 0.80 mm, vias 0 -> 38
- net 1x8_TireTemp_Sensor_SCL: track 0.00 -> 0.60 mm

Commit message: Prepared peripheral board for order
Parts:
- added G***: , FS_4_Global_Footprint_Library:FORMULA SLUG TITLE, B.Cu at (139.7, 132.1)
- added TP1: PA4, TestPoint:TestPoint_Pad_D1.5mm, B.Cu at (150.1, 130.3)
- added TP2: PA6, TestPoint:TestPoint_Pad_D1.5mm, B.Cu at (150.4, 121.9)
- added TP3: PA10, TestPoint:TestPoint_Pad_D1.5mm, B.Cu at (146.1, 120.1)
- added TP4: PB4, TestPoint:TestPoint_Pad_D1.5mm, B.Cu at (137.2, 121.9)
- added TP5: PB6, TestPoint:TestPoint_Pad_D1.5mm, B.Cu at (140.2, 121.9)
- added TP6: PB7, TestPoint:TestPoint_Pad_D1.5mm, B.Cu at (134.1, 121.9)
- R19, R20: value 16K -> 10k
- SW5: footprint Library:SW_A6H-4101_OMR -> FS_4_Global_Footprint_Library:SW_A6H-4101_OMR
- moved R1 42.3 mm to (164.1, 100.6), turned to 0 degrees
- moved R2 39.4 mm to (164.1, 102.1), turned to 0 degrees
- moved H2 35.7 mm to (127.0, 104.1)
- moved D1 29.9 mm to (165.6, 106.7), turned to 90 degrees
- moved R3 28.5 mm to (165.1, 116.3)
- moved R5 28.3 mm to (165.6, 111.3), turned to 0 degrees
- moved H1 28.1 mm to (162.6, 132.1)
- moved U8 27.2 mm to (165.1, 113.8)
- moved C6 25.9 mm to (162.1, 115.8), turned to -90 degrees
- moved R11 18.2 mm to (149.9, 113.8), turned to 0 degrees
- moved R18 17.4 mm to (149.9, 133.6), turned to -90 degrees
- moved C21 17.0 mm to (149.9, 115.3), turned to 180 degrees
- moved R19 14.1 mm to (152.4, 129.0)
- moved C22 13.9 mm to (127.5, 124.5), turned to 0 degrees
- moved R9 13.5 mm to (159.5, 101.6), turned to -90 degrees
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Connections:
- J1 pad 10: /Wheel_Speed_Out -> CANH
- J1 pad 11: GND -> +5V
- J1 pad 12: +3V3 -> GND
- J1 pad 13: Net-(J1D-1) -> Net-(U14-SDA_B)
- J1 pad 14: GND -> +12V
- J1 pad 15: GND -> +3V3
- J1 pad 16: Net-(U14-SCL_B) -> Net-(J1-Pad16)
- J1 pad 17: Net-(U14-SDA_B) -> GND
- J1 pad 18: +5V -> GND
- J1 pad 19: +5V -> Net-(U2-SCL_B)
- J1 pad 20: CANH -> /Wheel_Speed_Out
- J1 pad 21: CANL -> GND
- J1 pad 22: GND -> /Vin+
- J1 pad 23: GND -> /1V6_Vref
- J1 pad 24: Net-(U2-SDA_B) -> unconnected-(J1-Pad24)
- J1 pad 25: Net-(U2-SCL_B) -> +5V
- J1 pad 26: +5V -> Net-(U2-SDA_B)
- J1 pad 6: unconnected-(J1-Pad6) -> +5V
- J1 pad 7: /1V6_Vref -> Net-(U14-SCL_B)
- J1 pad 8: /Vin+ -> GND
- J1 pad 9: +12V -> CANL
- R11 pad 1: Net-(J1D-1) -> Net-(J1-Pad16)
Routing:
- net 1x8_TireTemp_Sensor_SDA: track 0.00 -> 42.5 mm, vias 0 -> 2
- net 1x8_TireTemp_Sensor_SCL: track 0.60 -> 36.9 mm, vias 0 -> 2
- net /1V6_Vref: track 23.2 -> 54.6 mm
- net /Vin+: track 11.1 -> 41.5 mm, vias 0 -> 2
- net +3V3: track 40.3 -> 64.3 mm, vias 17 -> 14
- net 1x1_TireTemp_Sensor_SDA: track 0.00 -> 23.4 mm
- net +5V: track 29.1 -> 8.66 mm, vias 0 -> 8
- net wheel speed: track 5.57 -> 24.0 mm, vias 0 -> 2
- net CANL: track 41.4 -> 23.8 mm
- net 1x1_TireTemp_Sensor_SCL: track 2.34 -> 19.9 mm
- net Net-(U2-SCL_B): track 0.00 -> 16.5 mm
- net Net-(J1-Pad16): track 0.00 -> 15.5 mm, vias 0 -> 1
- net CANH: track 35.5 -> 21.2 mm, vias 1 -> 0
- net Net-(U8-+): track 3.92 -> 16.7 mm, vias 0 -> 2
- net /Wheel_Speed_Out: track 0.00 -> 11.7 mm
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- added copper zone on In2.Cu, net +5V
Other:
- board size 50.8 x 45.7 mm -> 45.7 x 38.1 mm
- board text added: "*"
- board text added: "A0"
- board text added: "A1"
- board text added: "TRM"
