File: BMS/BMS/BMS.kicad_sch (KiCad schematic)
At the start: 39 parts, among them J1 CON_5019510550, J2 1053131202, J4 1053131202, J5 CON_5019510550, J6 CON_5019510550, J7 CON_5019510550, J8 1053131202, J9 1053131202, Q1 NSV1C201MZ4, SW1 SW_DIP_x04, U1 LTC6810IG-2-TRPBF

Commit message: changes
- replaced 5019510550 connector to 512810598
- schematic cleanup
- added new connector to footprint library
Parts:
- J1, J5, J6, J7: value CON_5019510550 -> 512810598; footprint FS_4_Global_Footprint_Library:CON_5019510550 -> FS_4_Global_Footprint_Library:512810598
- U1: footprint LTC6810IG-2_3ZZTRPBF:SOP50P780X200-44N -> Package_SO:TSSOP-44_4.4x11mm_P0.5mm
Other:
- note added: "E-meter temp sensor low voltage"
- note removed: "Emeter temp sensor low voltage"
- moved on the sheet: J2, J4, J5, J8, J9, R6, R62, R7

Commit message: changes
started layout
Parts:
- J1, J5, J6, J7: DIGI PN 900-5019510550CT-ND -> 900-0512810598CT-ND; DIGI URL https://www.digikey.com/en/products/detail/molex/5019510550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 -> https://www.digikey.com/en/products/detail/molex/0512810598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; MFG PN 5019510550 -> 0512810598
Changed lines of the file:
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@@
 			)
 		)
-		(property "Datasheet" "~"
+		(property "Datasheet" "https://www.molex.com/content/dam/molex/molex-dot-com/products/automated/en-us/salesdrawingpdf/512/51281/512810598_sd.pdf?inline"
 			(at 92.71 107.95 0)
 			(effects
@@
 			)
 		)
-		(property "DIGI PN" "900-5019510550CT-ND"
+		(property "DIGI PN" "900-0512810598CT-ND"
 			(at 92.71 107.95 0)
 			(effects
@@
 			)
 		)
-		(property "DIGI URL" "https://www.digikey.com/en/products/detail/molex/5019510550/13538887"
+		(property "DIGI URL" "https://www.digikey.com/en/products/detail/molex/0512810598/16634006"
 			(at 92.71 107.95 0)
 			(effects
@@
 			)
 		)
-		(property "MFG PN" "5019510550"
+		(property "MFG PN" "0512810598"
 			(at 92.71 107.95 0)
 			(effects
@@
 			)
 		)
-		(property "Datasheet" "~"
+		(property "Datasheet" "https://www.molex.com/content/dam/molex/molex-dot-com/products/automated/en-us/salesdrawingpdf/512/51281/512810598_sd.pdf?inline"
 			(at 212.09 138.43 0)
 			(effects
@@
 			)
 		)
-		(property "DIGI PN" "900-5019510550CT-ND"
+		(property "DIGI PN" "900-0512810598CT-ND"
 			(at 212.09 138.43 0)
 			(effects
@@
 			)
 		)
-		(property "DIGI URL" "https://www.digikey.com/en/products/detail/molex/5019510550/13538887"
+		(property "DIGI URL" "https://www.digikey.com/en/products/detail/molex/0512810598/16634006"
 			(at 212.09 138.43 0)
 			(effects
@@
 			)
 		)
-		(property "MFG PN" "5019510550"
+		(property "MFG PN" "0512810598"
 			(at 212.09 138.43 0)
 			(effects
@@
 			)
 		)
-		(property "Datasheet" "~"
+		(property "Datasheet" "https://www.molex.com/content/dam/molex/molex-dot-com/products/automated/en-us/salesdrawingpdf/512/51281/512810598_sd.pdf?inline"
 			(at 317.5 143.51 0)
 			(effects
@@
 			)
 		)
-		(property "DIGI PN" "900-5019510550CT-ND"
+		(property "DIGI PN" "900-0512810598CT-ND"
 			(at 317.5 143.51 0)
 			(effects
@@
 			)
 		)
-		(property "DIGI URL" "https://www.digikey.com/en/products/detail/molex/5019510550/13538887"
+		(property "DIGI URL" "https://www.digikey.com/en/products/detail/molex/0512810598/16634006"
 			(at 317.5 143.51 0)
 			(effects
@@
 			)
 		)
-		(property "MFG PN" "5019510550"
+		(property "MFG PN" "0512810598"
 			(at 317.5 143.51 0)
 			(effects
@@
 			)
 		)
-		(property "Datasheet" "~"
+		(property "Datasheet" "https://www.molex.com/content/dam/molex/molex-dot-com/products/automated/en-us/salesdrawingpdf/512/51281/512810598_sd.pdf?inline"
 			(at 90.17 59.69 0)
 			(effects
@@
 			)
 		)
-		(property "DIGI PN" "900-5019510550CT-ND"
+		(property "DIGI PN" "900-0512810598CT-ND"
 			(at 90.17 59.69 0)
 			(effects
@@
 			)
 		)
-		(property "DIGI URL" "https://www.digikey.com/en/products/detail/molex/5019510550/13538887"
+		(property "DIGI URL" "https://www.digikey.com/en/products/detail/molex/0512810598/16634006"
 			(at 90.17 59.69 0)
 			(effects
@@
 			)
 		)
-		(property "MFG PN" "5019510550"
+		(property "MFG PN" "0512810598"
 			(at 90.17 59.69 0)
 			(effects

Commit message: layout
Connections:
- net extIsoSPI_N: now also J4.2 (Pin_2); no longer J4.1 (Pin_1)
- net extIsoSPI_P: now also J4.1 (Pin_1); no longer J4.2 (Pin_2)
Changed lines of the file:
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@@
 	)
 	(symbol
+		(lib_name "Conn_01x02_Pin_1")
 		(lib_id "Connector:Conn_01x02_Pin")
 		(at 363.22 87.63 180)
@@
 					(size 1.27 1.27)
 				)
-				(hide yes)
 			)
 		)
@@
 		)
 		(property "Value" "512810598"
-			(at 81.026 51.816 0)
+			(at 78.232 54.102 0)
 			(effects
 				(font

Commit message: layout
Connections:
- net DQ: now also J2.1 (Pin_1); no longer J2.2 (Pin_2)
- net at J5.1 (Pin_1), J9.2 (Pin_2): now also J2.2 (Pin_2); no longer J2.1 (Pin_1)
Changed lines of the file:
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@@
 	)
 	(symbol
+		(lib_name "Conn_01x02_Pin_2")
 		(lib_id "Connector:Conn_01x02_Pin")
 		(at 340.36 132.08 180)

Commit message: layout changes
Connections:
- net BB0/B#: now also J1.4 (Pin_4); no longer J1.2 (Pin_2)
- net BB1/B#+1: now also J1.2 (Pin_2); no longer J1.4 (Pin_4)
- net BB2/B#+1: now also J1.1 (Pin_1); no longer J1.5 (Pin_5)
- net BB3/B#+1: now also J7.5 (Pin_5); no longer J7.1 (Pin_1)
- net BB4/B#+1: now also J7.4 (Pin_4); no longer J7.2 (Pin_2)
- net DQ: now also J9.2 (Pin_2); no longer J9.1 (Pin_1)
- net V-: now also J1.5 (Pin_5); no longer J1.1 (Pin_1)
- net extIsoSPI_N: now also J8.1 (Pin_1); no longer J8.2 (Pin_2)
- net extIsoSPI_P: now also J8.2 (Pin_2); no longer J8.1 (Pin_1)
- net at R2.2, R3.2: now also J7.2 (Pin_2); no longer J7.4 (Pin_4)
- net at J2.2 (Pin_2), J5.1 (Pin_1): now also J9.1 (Pin_1); no longer J9.2 (Pin_2)
Other:
- moved on the sheet: J1, J7
Changed lines of the file:
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@@
 	(symbol
 		(lib_id "Connector_Generic:Conn_01x05")
-		(at 92.71 107.95 180)
+		(at 92.71 107.95 0)
+		(mirror y)
 		(unit 1)
 		(exclude_from_sim no)
@@
 		(dnp no)
 		(property "Reference" "J1"
-			(at 83.566 93.472 0)
+			(at 83.566 122.428 0)
 			(effects
 				(font
@@
 		)
 		(property "Value" "512810598"
-			(at 83.82 98.044 0)
+			(at 83.82 117.856 0)
 			(effects
 				(font
@@
 	)
 	(symbol
+		(lib_name "Conn_01x02_Pin_3")
 		(lib_id "Connector:Conn_01x02_Pin")
 		(at 317.5 129.54 0)
@@
 	(symbol
 		(lib_id "Connector_Generic:Conn_01x05")
-		(at 90.17 59.69 180)
+		(at 90.17 59.69 0)
+		(mirror y)
 		(unit 1)
 		(exclude_from_sim no)
@@
 		(dnp no)
 		(property "Reference" "J7"
-			(at 82.042 48.006 0)
+			(at 82.042 71.374 0)
 			(effects
 				(font
@@
 		)
 		(property "Value" "512810598"
-			(at 78.232 54.102 0)
-			(effects
-				(font
+			(at 78.232 65.278 0)
+			(effects
+				(font

Commit message: layout
added dimensions and made hvlv line dashed
Parts:
- J2, J4, J8, J9: footprint FS_4_Global_Footprint_Library:Nanofit-1054301202-1x2SMD90Deg -> FS_4_Global_Footprint_Library:Nano-Fit_1054301102
Other:
- title: FS-4 BMS Board -> BMS Board
Changed lines of the file:
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@@
 	(paper "B")
 	(title_block
-		(title "FS-4 BMS Board")
+		(title "BMS Board")
 		(date "2026-02-07")
 		(rev "1.1")
@@
 			)
 		)
-		(property "Footprint" "FS_4_Global_Footprint_Library:Nanofit-1054301202-1x2SMD90Deg"
+		(property "Footprint" "FS_4_Global_Footprint_Library:Nano-Fit_1054301102"
 			(at 363.22 87.63 0)
 			(effects
@@
 			)
 		)
-		(property "Footprint" "FS_4_Global_Footprint_Library:Nanofit-1054301202-1x2SMD90Deg"
+		(property "Footprint" "FS_4_Global_Footprint_Library:Nano-Fit_1054301102"
 			(at 363.22 80.01 0)
 			(effects
@@
 			)
 		)
-		(property "Footprint" "FS_4_Global_Footprint_Library:Nanofit-1054301202-1x2SMD90Deg"
+		(property "Footprint" "FS_4_Global_Footprint_Library:Nano-Fit_1054301102"
 			(at 317.5 129.54 0)
 			(effects
@@
 			)
 		)
-		(property "Footprint" "FS_4_Global_Footprint_Library:Nanofit-1054301202-1x2SMD90Deg"
+		(property "Footprint" "FS_4_Global_Footprint_Library:Nano-Fit_1054301102"
 			(at 340.36 132.08 0)
 			(effects

Commit message: Minor BOM changes
Parts:
- C1, C7: DIGI PN 311-3157-1-ND -> (none); DIGI URL https://www.digikey.com/en/products/detail/yageo/AC0805KRX7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 -> (none); Digi PN (none) -> 311-3174-1-ND; Digi URL (none) -> https://www.digikey.com/en/products/detail/yageo/AC0805KRX7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; MFG PN AC0805KRX7R0BB103 -> AC0805KRX7R9BB103
- C2, C3, C4: DIGI PN 13-CC0805KFX7R9BB105CT-ND -> (none); DIGI URL https://www.digikey.com/en/products/detail/yageo/CC0805KFX7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 -> (none); Digi PN (none) -> 13-CC0805KFX7R9BB105CT-ND; Digi URL (none) -> https://www.digikey.com/en/products/detail/yageo/CC0805KFX7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
- C5, C8: DIGI PN 311-2083-1-ND -> (none); DIGI URL https://www.digikey.com/en/products/detail/yageo/CC0805KKX7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 -> (none); Digi PN (none) -> 311-2083-1-ND; Digi URL (none) -> https://www.digikey.com/en/products/detail/yageo/CC0805KKX7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
- C6: DIGI PN 13-CC0805KRNPO9BN150CT-ND -> (none); DIGI URL https://www.digikey.com/en/products/detail/yageo/CC0805KRNP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 -> (none); Digi PN (none) -> 13-CC0805KRNPO9BN150CT-ND; Digi URL (none) -> https://www.digikey.com/en/products/detail/yageo/CC0805KRNP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
- D1, D2: DIGI PN 475-LHR974-LP-1-0-20-R18TR-ND -> (none); DIGI URL https://www.digikey.com/en/products/detail/ams-osram-usa-in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 -> (none); Digi PN (none) -> 475-LSR976-NR-1CT-ND; Digi URL (none) -> https://www.digikey.com/en/products/detail/ams-osram-usa-in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; MFG PN LH R974-LP-1-0-20-R18 -> LS R976-NR-1-0-20-R18
- J1, J5, J6, J7: DIGI PN 900-0512810598CT-ND -> (none); DIGI URL https://www.digikey.com/en/products/detail/molex/0512810598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 -> (none); Digi PN (none) -> 900-0512810598CT-ND; Digi URL (none) -> https://www.digikey.com/en/products/detail/molex/0512810598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
- J2, J4, J8, J9: DIGI PN WM26097CT-ND -> (none); DIGI URL https://www.digikey.com/en/products/detail/molex/1054301202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 -> (none); Digi PN (none) -> WM26097CT-ND; Digi URL (none) -> https://www.digikey.com/en/products/detail/molex/1054301202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
- L1: DIGI PN 553-HM2113ZNL-ND -> (none); DIGI URL https://www.digikey.com/en/products/detail/pulse-electronic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 -> (none); Digi PN (none) -> 553-HM2113ZNLTCT-ND; Digi URL (none) -> https://www.digikey.com/en/products/detail/pulse-electronic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; MFG PN HM2113ZNL -> HM2113ZNLT
- Q1: DIGI PN NSS1C201MZ4T1GOSCT-ND -> (none); DIGI URL https://www.digikey.com/en/products/detail/onsemi/NSS1C201M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 -> (none); Digi PN (none) -> NSS1C201MZ4T1GOSCT-ND; Digi URL (none) -> https://www.digikey.com/en/products/detail/onsemi/NSS1C201M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
- R1: Digi PN (none) -> 311-100CRCT-ND; Digi URL (none) -> https://www.digikey.com/en/products/detail/yageo/RC0805FR-0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; MFG (none) -> YAGEO; MFG PN (none) -> RC0805FR-07100RL
- R10, R9: DIGI PN AF0805FR-0722RL-ND -> (none); DIGI URL https://www.digikey.com/en/products/detail/yageo/AF0805FR-0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 -> (none); Digi PN (none) -> YAG3713CT-ND; Digi URL (none) -> https://www.digikey.com/en/products/detail/yageo/AC0805FR-0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; MFG PN AF0805FR-0722RL -> AC0805FR-0722RL
- R11, R60, R61: DIGI PN 311-10.0KCRCT-ND -> (none); DIGI URL https://www.digikey.com/en/products/detail/yageo/RC0805FR-0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 -> (none); Digi PN (none) -> 311-10.0KCRCT-ND; Digi URL (none) -> https://www.digikey.com/en/products/detail/yageo/RC0805FR-0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
- R2: DIGI PN 13-RC0805FR-1010RLCT-ND -> (none); DIGI URL https://www.digikey.com/en/products/detail/yageo/RC0805FR-1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 -> (none); Digi PN (none) -> 13-RC0805FR-1010RLCT-ND; Digi URL (none) -> https://www.digikey.com/en/products/detail/yageo/RC0805FR-1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
- R3: DIGI PN 311-100CRCT-ND -> (none); DIGI URL https://www.digikey.com/en/products/detail/yageo/RC0805FR-0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 -> (none); Digi PN (none) -> 311-100CRCT-ND; Digi URL (none) -> https://www.digikey.com/en/products/detail/yageo/RC0805FR-0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
- R4, R5: DIGI PN 311-160CRCT-ND -> (none); DIGI URL https://www.digikey.com/en/products/detail/yageo/RC0805FR-0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 -> (none); Digi PN (none) -> 311-160CRCT-ND; Digi URL (none) -> https://www.digikey.com/en/products/detail/yageo/RC0805FR-0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
- R6: DIGI PN YAG5849CT-ND -> (none); DIGI URL https://www.digikey.com/en/products/detail/yageo/SR0805FR-4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 -> (none); Digi PN (none) -> YAG3701CT-ND; Digi URL (none) -> https://www.digikey.com/en/products/detail/yageo/AC0805FR-0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; MFG PN SR0805FR-471K5L -> AC0805FR-071K5L
- R62: DIGI PN 311-200CRCT-ND -> (none); DIGI URL https://www.digikey.com/en/products/detail/yageo/RC0805FR-0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 -> (none); Digi PN (none) -> 311-200CRCT-ND; Digi URL (none) -> https://www.digikey.com/en/products/detail/yageo/RC0805FR-0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
- R66, R67, R68: DIGI PN 13-RC0805FR-134K99LCT-ND -> (none); DIGI URL https://www.digikey.com/en/products/detail/yageo/RC0805FR-1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 -> (none); Digi PN (none) -> 13-RC0805FR-134K99LCT-ND; Digi URL (none) -> https://www.digikey.com/en/products/detail/yageo/RC0805FR-1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
- R7: DIGI PN 311-680CRCT-ND -> (none); DIGI URL https://www.digikey.com/en/products/detail/yageo/RC0805FR-0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 -> (none); Digi PN (none) -> 311-680CRCT-ND; Digi URL (none) -> https://www.digikey.com/en/products/detail/yageo/RC0805FR-0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
- R8: DIGI PN 13-AC0805FR-07402RLCT-ND -> (none); DIGI URL https://www.digikey.com/en/products/detail/yageo/AC0805FR-0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 -> (none); Digi PN (none) -> 13-AC0805FR-07402RLCT-ND; Digi URL (none) -> https://www.digikey.com/en/products/detail/yageo/AC0805FR-0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
- SW1: DIGI PN 39-A6H-4101-ND -> (none); DIGI URL https://www.digikey.com/en/products/detail/omron-electronic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 -> (none); Digi PN (none) -> 39-A6H-4101-ND; Digi URL (none) -> https://www.digikey.com/en/products/detail/omron-electronic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
- U1: DIGI PN 505-LTC6810IG-2#3ZZTRPBFTR-ND -> (none); DIGI URL https://www.digikey.com/en/products/detail/analog-devices-i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 -> (none); Digi PN (none) -> 505-LTC6810IG-2#3ZZPBF-ND; Digi URL (none) -> https://www.digikey.com/en/products/detail/analog-devices-i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; MFG PN LTC6810IG-2#3ZZTRPBF -> LTC6810IG-2#3ZZPBF
