File: BMS/BMS/BalanceSenseBlock.kicad_sch (KiCad schematic)
At the start: 7 parts

Commit message: BMS
updated BMS schematic with new global tags
Parts:
- added C?: 10nF, Capacitor_SMD:C_0805_2012Metric_Pad1.18x1.45mm_HandSolder, symbol Device:C
- added D?: LH R974-LP-1, LED_SMD:LED_0805_2012Metric_Pad1.15x1.40mm_HandSolder, symbol Device:LED_Small
- added Q?: BSS308PE, Package_TO_SOT_SMD:SOT-23, symbol Transistor_FET:BSS84
- added R?: 120, Resistor_SMD:R_0805_2012Metric_Pad1.20x1.40mm_HandSolder, symbol Device:R_Small
- added R?: 100, Resistor_SMD:R_0805_2012Metric_Pad1.20x1.40mm_HandSolder, symbol Device:R
- added R?: 33, Resistor_SMD:R_2512_6332Metric_Pad1.40x3.35mm_HandSolder, symbol Device:R
- added R?: 3.3k, Resistor_SMD:R_0805_2012Metric_Pad1.20x1.40mm_HandSolder, symbol Device:R
Connections:
- net B#: now also D?.1 (K), R?.1
- net B#+1: now also Q?.2 (S), R?.2
- net C#: now also C?.2
- net C#+1: now also C?.1, R?.1
- net S#+1: now also R?.1
- net at Q?.1 (G), R?.2: now also Q?.1 (G), R?.2
- net at Q?.3 (D), R?.1, R?.2: now also Q?.3 (D), R?.1, R?.2
- net at D?.2 (A), R?.2: now also D?.2 (A), R?.2

Commit message: BMS
fixed errors with power flags
Parts:
- gave numbers to parts that had none: 14

Commit message: removed duplicates in balance blocks
Parts:
- removed C8: 10nF, Capacitor_SMD:C_0805_2012Metric_Pad1.18x1.45mm_HandSolder, symbol Device:C
- removed D3: LH R974-LP-1, LED_SMD:LED_0805_2012Metric_Pad1.15x1.40mm_HandSolder, symbol Device:LED_Small
- removed Q3: BSS308PE, Package_TO_SOT_SMD:SOT-23, symbol Transistor_FET:BSS84
- removed R13: 120, Resistor_SMD:R_0805_2012Metric_Pad1.20x1.40mm_HandSolder, symbol Device:R_Small
- removed R14: 33, Resistor_SMD:R_2512_6332Metric_Pad1.40x3.35mm_HandSolder, symbol Device:R
- removed R16: 3.3k, Resistor_SMD:R_0805_2012Metric_Pad1.20x1.40mm_HandSolder, symbol Device:R
- removed R19: 100, Resistor_SMD:R_0805_2012Metric_Pad1.20x1.40mm_HandSolder, symbol Device:R
Other:
- moved on the sheet: C9

Commit message: requested changes made
Parts:
- D4: DIGI PN (none) -> 475-LHR974-LP-1-0-20-R18TR-ND; DIGI URL (none) -> https://www.digikey.com/en/products/detail/ams-osram-usa-in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; MFG (none) -> ams-OSRAM USA INC.; MFG PN (none) -> LH R974-LP-1-0-20-R18
- Q2: DIGI PN (none) -> BSS84CT-ND; DIGI URL (none) -> https://www.digikey.com/en/products/detail/onsemi/BSS84/244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; MFG (none) -> onsemi; MFG PN (none) -> BSS84
- R12: DIGI PN (none) -> 311-120CRCT-ND; DIGI URL (none) -> https://www.digikey.com/en/products/detail/yageo/RC0805FR-0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; MFG (none) -> YAGEO; MFG PN (none) -> RC0805FR-07120RL
- R15: DIGI PN (none) -> 13-RC2512JK-0733RLCT-ND; DIGI URL (none) -> https://www.digikey.com/en/products/detail/yageo/RC2512JK-0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; MFG (none) -> YAGEO; MFG PN (none) -> RC2512JK-0733RL
- R17: DIGI PN (none) -> 13-RC0805FR-133K3LCT-ND; DIGI URL (none) -> https://www.digikey.com/en/products/detail/yageo/RC0805FR-1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; MFG (none) -> YAGEO; MFG PN (none) -> RC0805FR-133K3L
- R18: DIGI PN (none) -> 311-100CRCT-ND; DIGI URL (none) -> https://www.digikey.com/en/products/detail/yageo/RC0805FR-0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; MFG (none) -> YAGEO; MFG PN (none) -> RC0805FR-07100RL
Changed lines of the file:
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@@
 	(generator "eeschema")
 	(generator_version "9.0")
-	(paper "A4")
+	(paper "A")
 	(text "Balance Block"
 		(exclude_from_sim no)
@@
 			)
 		)
+		(property "DIGI PN" "BSS84CT-ND"
+			(at 142.24 99.06 0)
+			(effects
+				(font
+					(size 1.27 1.27)
+				)
+				(hide yes)
+			)
+		)
+		(property "DIGI URL" "https://www.digikey.com/en/products/detail/onsemi/BSS84/244213"
+			(at 142.24 99.06 0)
+			(effects
+				(font
+					(size 1.27 1.27)
+				)
+				(hide yes)
+			)
+		)
+		(property "MFG" "onsemi"
+			(at 142.24 99.06 0)
+			(effects
+				(font
+					(size 1.27 1.27)
+				)
+				(hide yes)
+			)
+		)
+		(property "MFG PN" "BSS84"
+			(at 142.24 99.06 0)
+			(effects
+				(font
+					(size 1.27 1.27)
+				)
+				(hide yes)
+			)
+		)
 		(pin "1"
 		)
@@
 			)
 		)
-		(property "Datasheet" "~"
+		(property "Datasheet" "~https://yageogroup.com/content/datasheet/asset/file/PYU-RC_GROUP_51_ROHS_L"
 			(at 152.4 86.36 0)
 			(effects
@@
 		(property "Description" ""
 			(at 152.4 86.36 0)
+			(effects
+				(font
+					(size 1.27 1.27)
+				)
+				(hide yes)
+			)
+		)
+		(property "DIGI PN" "311-100CRCT-ND"
+			(at 152.4 86.36 90)
+			(effects
+				(font
+					(size 1.27 1.27)
+				)
+				(hide yes)
+			)
+		)
+		(property "DIGI URL" "https://www.digikey.com/en/products/detail/yageo/RC0805FR-07100RL/727543?s=N4IgTCBcDaIMwEYEFoEAY0GEBKmAqyAcgCIgC6AvkA"
+			(at 152.4 86.36 90)
+			(effects
+				(font
+					(size 1.27 1.27)
+				)
+				(hide yes)
+			)
+		)
+		(property "MFG" "YAGEO"
+			(at 152.4 86.36 90)
+			(effects
+				(font
+					(size 1.27 1.27)
+				)
+				(hide yes)
+			)
+		)
+		(property "MFG PN" "RC0805FR-07100RL"
+			(at 152.4 86.36 90)
 			(effects
 				(font
@@
 			)
 		)
-		(property "Datasheet" "~"
+		(property "Datasheet" "~https://yageogroup.com/content/datasheet/asset/file/PYU-RC_GROUP_51_ROHS_L"
 			(at 134.62 104.14 0)
 			(effects
@@
 		(property "Description" ""
 			(at 134.62 104.14 0)
+			(effects
+				(font
+					(size 1.27 1.27)
+				)
+				(hide yes)
+			)
+		)
+		(property "DIGI PN" "311-120CRCT-ND"
+			(at 134.62 104.14 90)
+			(effects
+				(font
+					(size 1.27 1.27)
+				)
+				(hide yes)
+			)
+		)
+		(property "DIGI URL" "https://www.digikey.com/en/products/detail/yageo/RC0805FR-07120RL/727575?s=N4IgTCBcDaIMwEYEFoFgAwGEBKmAqyAcgCIgC6AvkA"
+			(at 134.62 104.14 90)
+			(effects
+				(font
+					(size 1.27 1.27)
+				)
+				(hide yes)
+			)
+		)
+		(property "MFG" "YAGEO"
+			(at 134.62 104.14 90)
+			(effects
+				(font
+					(size 1.27 1.27)
+				)
+				(hide yes)
+			)
+		)
+		(property "MFG PN" "RC0805FR-07120RL"
+			(at 134.62 104.14 90)
 			(effects
 				(font
@@
 			)
 		)
-		(property "Datasheet" "~"
+		(property "Datasheet" "https://look.ams-osram.com/m/1c300b267881b82d/original/LH-R974.pdf"
 			(at 127 107.95 90)
 			(effects
@@
 		(property "Description" ""
 			(at 127 107.95 0)
+			(effects
+				(font
+					(size 1.27 1.27)
+				)
+				(hide yes)
+			)
+		)
+		(property "DIGI PN" "475-LHR974-LP-1-0-20-R18TR-ND"
+			(at 127 107.95 90)
+			(effects
+				(font
+					(size 1.27 1.27)
+				)
+				(hide yes)
+			)
+		)
+		(property "DIGI URL" "https://www.digikey.com/en/products/detail/ams-osram-usa-inc/LH-R974-LP-1-0-20-R18/1227932"
+			(at 127 107.95 90)
+			(effects
+				(font
+					(size 1.27 1.27)
+				)
+				(hide yes)
+			)
+		)
+		(property "MFG" "ams-OSRAM USA INC."
+			(at 127 107.95 90)
+			(effects
+				(font
+					(size 1.27 1.27)
+				)
+				(hide yes)
+			)
+		)
+		(property "MFG PN" "LH R974-LP-1-0-20-R18"
+			(at 127 107.95 90)
 			(effects
 				(font
@@
 			)
 		)
-		(property "Datasheet" "~"
+		(property "Datasheet" "https://yageogroup.com/content/datasheet/asset/file/PYU-RC_GROUP_51_ROHS_L"
 			(at 139.7 107.95 0)
 			(effects
@@
 		(property "Description" ""
 			(at 139.7 107.95 0)
+			(effects
+				(font
+					(size 1.27 1.27)
+				)
+				(hide yes)
+			)
+		)
+		(property "DIGI PN" "13-RC2512JK-0733RLCT-ND"
+			(at 139.7 107.95 90)
+			(effects
+				(font
+					(size 1.27 1.27)
+				)
+				(hide yes)
+			)
+		)
+		(property "DIGI URL" "https://www.digikey.com/en/products/detail/yageo/RC2512JK-0733RL/5922559?s=N4IgTCBcDaIIwGYC0AlAwmArHMApA0kgAwDsCCKAMmgCpIByAIiALoC%2BQA"
+			(at 139.7 107.95 90)
+			(effects
+				(font
+					(size 1.27 1.27)
+				)
+				(hide yes)
+			)
+		)
+		(property "MFG" "YAGEO"
+			(at 139.7 107.95 90)
+			(effects
+				(font
+					(size 1.27 1.27)
+				)
+				(hide yes)
+			)
+		)
+		(property "MFG PN" "RC2512JK-0733RL"
+			(at 139.7 107.95 90)
 			(effects
 				(font
@@
 			)
 		)
-		(property "Datasheet" "~"
+		(property "Datasheet" "https://yageogroup.com/content/datasheet/asset/file/PYU-RC_GROUP_51_ROHS_L"
 			(at 151.13 99.06 0)
 			(effects
@@
 			(effects
 				(font
+					(size 1.27 1.27)
+				)
+				(hide yes)
+			)
+		)
+		(property "DIGI PN" "13-RC0805FR-133K3LCT-ND"
+			(at 151.13 99.06 90)
+			(effects
+				(font
+					(size 1.27 1.27)
+				)
+				(hide yes)
+			)
+		)
+		(property "DIGI URL" "https://www.digikey.com/en/products/detail/yageo/RC0805FR-133K3L/14008213?s=N4IgTCBcDaIIwGYC0AlAwgBgBwYKwDEUlEEBpBAGTQBUkA5AERAF0BfIA"
+			(at 151.13 99.06 90)
+			(effects
+				(font
+					(size 1.27 1.27)
+				)
+				(hide yes)
+			)
+		)
+		(property "MFG" "YAGEO"
+			(at 151.13 99.06 90)
+			(effects
+				(font
+					(size 1.27 1.27)
+				)
+				(hide yes)
+			)
+		)
+		(property "MFG PN" "RC0805FR-133K3L"
+			(at 151.13 99.06 90)
+			(effects
+				(font

Commit message: filled out symbol field
Parts:
- C9: DIGI PN (none) -> 311-3157-1-ND; DIGI URL (none) -> https://www.digikey.com/en/products/detail/yageo/AC0805KRX7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; MFG (none) -> YAGEO; MFG PN (none) -> AC0805KRX7R0BB103
Changed lines of the file:
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@@
 			)
 		)
-		(property "Datasheet" "~"
+		(property "Datasheet" "https://yageogroup.com/content/datasheet/asset/file/UPY-AC_NP0X7RX7S_6_3V-TO-2KV"
 			(at 173.99 100.33 0)
 			(effects
@@
 			(at 173.99 100.33 0)
 			(effects
+				(font
+					(size 1.27 1.27)
+				)
+				(hide yes)
+			)
+		)
+		(property "DIGI PN" "311-3157-1-ND"
+			(at 173.99 100.33 0)
+			(effects
+				(font
+					(size 1.27 1.27)
+				)
+				(hide yes)
+			)
+		)
+		(property "DIGI URL" "https://www.digikey.com/en/products/detail/yageo/AC0805KRX7R0BB103/6643143"
+			(at 173.99 100.33 0)
+			(effects
+				(font
+					(size 1.27 1.27)
+				)
+				(hide yes)
+			)
+		)
+		(property "MFG" "YAGEO"
+			(at 173.99 100.33 0)
+			(effects
+				(font
+					(size 1.27 1.27)
+				)
+				(hide yes)
+			)
+		)
+		(property "MFG PN" "AC0805KRX7R0BB103"
+			(at 173.99 100.33 0)
+			(effects

Commit message: changes made
Parts:
- R15: DIGI PN 13-RC2512JK-0733RLCT-ND -> 13-RC2512FK-0733RLCT-ND; DIGI URL https://www.digikey.com/en/products/detail/yageo/RC2512JK-0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 -> https://www.digikey.com/en/products/detail/yageo/RC2512FK-0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; MFG PN RC2512JK-0733RL -> RC2512FK-0733RL
Changed lines of the file:
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@@
 			)
 		)
-		(property "DIGI PN" "13-RC2512JK-0733RLCT-ND"
+		(property "DIGI PN" "13-RC2512FK-0733RLCT-ND"
 			(at 139.7 107.95 90)
 			(effects
@@
 			)
 		)
-		(property "DIGI URL" "https://www.digikey.com/en/products/detail/yageo/RC2512JK-0733RL/5922559?s=N4IgTCBcDaIIwGYC0AlAwmArHMApA0kgAwDsCCKAMmgCpIByAIiALoC%2BQA"
+		(property "DIGI URL" "https://www.digikey.com/en/products/detail/yageo/RC2512FK-0733RL/5922127"
 			(at 139.7 107.95 90)
 			(effects
@@
 			)
 		)
-		(property "MFG PN" "RC2512JK-0733RL"
+		(property "MFG PN" "RC2512FK-0733RL"
 			(at 139.7 107.95 90)
 			(effects

Commit message: Minor BOM changes
Parts:
- C9: DIGI PN 311-3157-1-ND -> (none); DIGI URL https://www.digikey.com/en/products/detail/yageo/AC0805KRX7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 -> (none); Digi PN (none) -> 311-3174-1-ND; Digi URL (none) -> https://www.digikey.com/en/products/detail/yageo/AC0805KRX7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; MFG PN AC0805KRX7R0BB103 -> AC0805KRX7R9BB103
- D4: DIGI PN 475-LHR974-LP-1-0-20-R18TR-ND -> (none); DIGI URL https://www.digikey.com/en/products/detail/ams-osram-usa-in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 -> (none); Digi PN (none) -> 475-LSR976-NR-1CT-ND; Digi URL (none) -> https://www.digikey.com/en/products/detail/ams-osram-usa-in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; MFG PN LH R974-LP-1-0-20-R18 -> LS R976-NR-1-0-20-R18
- Q2: DIGI PN BSS84CT-ND -> (none); DIGI URL https://www.digikey.com/en/products/detail/onsemi/BSS84/244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 -> (none); Digi PN (none) -> BSS84CT-ND; Digi URL (none) -> https://www.digikey.com/en/products/detail/onsemi/BSS84/244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
- R12: DIGI PN 311-120CRCT-ND -> (none); DIGI URL https://www.digikey.com/en/products/detail/yageo/RC0805FR-0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 -> (none); Digi PN (none) -> 311-120CRCT-ND; Digi URL (none) -> https://www.digikey.com/en/products/detail/yageo/RC0805FR-0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
- R15: DIGI PN 13-RC2512FK-0733RLCT-ND -> (none); DIGI URL https://www.digikey.com/en/products/detail/yageo/RC2512FK-0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 -> (none); Digi PN (none) -> 13-RC2512FK-0733RLCT-ND; Digi URL (none) -> https://www.digikey.com/en/products/detail/yageo/RC2512FK-0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
- R17: DIGI PN 13-RC0805FR-133K3LCT-ND -> (none); DIGI URL https://www.digikey.com/en/products/detail/yageo/RC0805FR-1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 -> (none); Digi PN (none) -> 13-RC0805FR-133K3LCT-ND; Digi URL (none) -> https://www.digikey.com/en/products/detail/yageo/RC0805FR-1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
- R18: DIGI PN 311-100CRCT-ND -> (none); DIGI URL https://www.digikey.com/en/products/detail/yageo/RC0805FR-0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 -> (none); Digi PN (none) -> 311-100CRCT-ND; Digi URL (none) -> https://www.digikey.com/en/products/detail/yageo/RC0805FR-0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
