File: BMS/BMS/BMS.kicad_pcb (KiCad board)
At the start: 2 copper layers, 183.2 x 49.9 mm, 82 parts, among them J1 512810598, J2 1053131202, J4 1053131202, J5 512810598, J6 512810598, J7 512810598, J8 1053131202, J9 1053131202, Q1 NSV1C201MZ4, Q10 BSS308PE, Q12 BSS308PE, Q2 BSS308PE, Q4 BSS308PE, Q6 BSS308PE, Q8 BSS308PE, SW1 SW_DIP_x04, U1 LTC6810IG-2-TRPBF

Commit message: Update BMS.kicad_pcb
some isospi trace improvement
fixed via sizes for trace widths of 20 mils
Routing:
- net IsoSPI_N: track 61.5 -> 46.1 mm
- net V-: track 48.1 -> 50.0 mm
- net IsoSPI_P: track 37.3 -> 36.0 mm
- net Net-(J2-Pin_2): track 63.0 -> 63.7 mm
- net Net-(L1-Pad3): vias 0 -> 2

Commit message: Very slight trace cleanup
Routing:
- net /BB1/B#+1: track 73.3 -> 75.3 mm
- net Net-(J7-Pin_2): track 61.7 -> 61.1 mm
- net V-: track 50.0 -> 49.5 mm

Commit message: BMS rev 2 changes
- I changed pin25 to GPIO4, and replaced the GPIO1 on the temp sense connector and temp sense pullups to GPIO4.
- I added the new busbar connectors

What would we do with the GPIO1 pin? Add the same led that was on GPOI4 previously?
Parts:
- J1, J7: footprint FS_4_Global_Footprint_Library:512810598 -> FS_4_Global_Footprint_Library:849525
- moved J7 3.74 mm to (243.3, 116.7)
- moved J1 3.46 mm to (263.7, 116.7)
Routing:
- net /BB1/B#+1: track 75.3 -> 69.0 mm
- net /BB0/B#: track 94.3 -> 89.7 mm
- net /BB2/B#+1: track 70.5 -> 66.0 mm
- net /BB0/B#+1: track 76.6 -> 72.6 mm
- net /BB3/B#+1: track 56.3 -> 53.1 mm
- net /BB5/B#+1: track 54.2 -> 51.6 mm
- net Net-(J7-Pin_2): track 61.1 -> 59.1 mm
- net /BB4/B#+1: track 56.3 -> 54.4 mm

Commit message: Bump Rev to 2.1
Changed lines of the file:
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@@
 	(title_block
 		(title "BMS Board")
-		(date "2026-02-07")
-		(rev "1.1")
+		(date "2026-04-14")
+		(rev "2.1")
 		(company "Formula Slug")
 		(comment 4 "Sultan Sheikh")
@@
 			(outputformat 1)
 			(mirror no)
-			(drillshape 1)
+			(drillshape 0)
 			(scaleselection 1)
-			(outputdirectory "")
+			(outputdirectory "./out")
 		)
 	)

Commit message: page settings
Parts:
- removed D1: LH R974-LP-1, LED_SMD:LED_0805_2012Metric_Pad1.15x1.40mm_HandSolder
- removed R4: 160, Resistor_SMD:R_0805_2012Metric_Pad1.20x1.40mm_HandSolder
Connections:
- J6 pad 2: 6810_GPIO1 -> 6810_GPIO4
- R66 pad 2: 6810_GPIO1 -> 6810_GPIO4
- U1 pad 18: 6810_GPIO1 -> unconnected-(U1-GPIO1-Pad18)
- U1 pad 25: Net-(D1-K) -> 6810_GPIO4
Routing:
- net 6810_GPIO4: track 0.00 -> 65.8 mm, vias 0 -> 4
- net 6810_GPIO1: track 56.2 -> 0.00 mm, vias 2 -> 0
- net Net-(D1-K): track 4.13 -> 0.00 mm
- net VREG: track 98.9 -> 96.9 mm
- net Net-(D1-A): track 1.79 -> 0.00 mm

Commit message: layout
wired GPIO1 to led in layout
Parts:
- added D1: LH R974-LP-1, LED_SMD:LED_0805_2012Metric_Pad1.15x1.40mm_HandSolder, F.Cu at (172.7, 95.5)
- added R13: 160, Resistor_SMD:R_0805_2012Metric_Pad1.20x1.40mm_HandSolder, F.Cu at (178.8, 96.5)
Connections:
- U1 pad 18: unconnected-(U1-GPIO1-Pad18) -> Net-(D1-K)
Routing:
- net Net-(D1-K): track 0.00 -> 18.8 mm, vias 0 -> 2
- net Net-(D1-A): track 0.00 -> 4.49 mm
- net V-: track 49.9 -> 47.7 mm, vias 16 -> 17
- net VREG: track 96.9 -> 99.0 mm

Commit message: BMS Rev3.0.0: Fix balance block: use NMOS, use datasheet recommended setup
Parts:
- removed Q10, Q12, Q8: BSS308PE, Package_TO_SOT_SMD:SOT-23
- removed the R17 at (199.6, 107.7)
- removed the R25 at (199.6, 112.3)
- removed the R33 at (199.6, 116.8)
- removed the R41 at (199.6, 103.1)
- removed R49, R57: 3.3k, Resistor_SMD:R_0805_2012Metric_Pad1.20x1.40mm_HandSolder
- added D10: 9.1V, Diode_SMD:D_SOD-523, F.Cu at (201.2, 104.5)
- added D12: 9.1V, Diode_SMD:D_SOD-523, F.Cu at (201.2, 99.8)
- added D14: 9.1V, Diode_SMD:D_SOD-523, F.Cu at (201.2, 95.2)
- added D4: 9.1V, Diode_SMD:D_SOD-523, F.Cu at (201.2, 109.0)
- added D6: 9.1V, Diode_SMD:D_SOD-523, F.Cu at (201.2, 113.5)
- added D8: 9.1V, Diode_SMD:D_SOD-523, F.Cu at (201.2, 118.1)
- added Q3: AO3400A, Package_TO_SOT_SMD:SOT-23-3, F.Cu at (204.0, 113.9)
- added Q5: AO3400A, Package_TO_SOT_SMD:SOT-23-3, F.Cu at (204.0, 104.7)
- added Q7: AO3400A, Package_TO_SOT_SMD:SOT-23-3, F.Cu at (204.0, 95.6)
- added R20: 1K, Resistor_SMD:R_0603_1608Metric_Pad0.98x0.95mm_HandSolder, F.Cu at (199.1, 109.0)
- added R24: 1K, Resistor_SMD:R_0603_1608Metric_Pad0.98x0.95mm_HandSolder, F.Cu at (199.1, 113.5)
- added R28: 1K, Resistor_SMD:R_0603_1608Metric_Pad0.98x0.95mm_HandSolder, F.Cu at (199.1, 118.1)
- added R32: 1K, Resistor_SMD:R_0603_1608Metric_Pad0.98x0.95mm_HandSolder, F.Cu at (199.1, 104.4)
- added R36: 1K, Resistor_SMD:R_0603_1608Metric_Pad0.98x0.95mm_HandSolder, F.Cu at (199.1, 99.8)
- added R40: 1K, Resistor_SMD:R_0603_1608Metric_Pad0.98x0.95mm_HandSolder, F.Cu at (199.1, 95.2)
- J1: renamed from J7; value 512810598 -> 84952-5
- J2: renamed from J1; value 512810598 -> 84952-5
- Q2, Q4, Q6: value BSS308PE -> AO3400A; footprint Package_TO_SOT_SMD:SOT-23 -> Package_TO_SOT_SMD:SOT-23-3
- moved Q6 17.7 mm to (204.0, 100.2), turned to -90 degrees
- moved R1 9.91 mm to (196.3, 94.0)
- moved C1 9.40 mm to (188.5, 94.0)
- moved Q4 5.19 mm to (204.0, 118.5), turned to -90 degrees
- moved R41 3.95 mm to (195.8, 97.0), turned to -90 degrees
- moved R37 3.89 mm to (195.8, 101.3), turned to -90 degrees
- moved R33 3.84 mm to (195.8, 105.7), turned to -90 degrees
- moved R21 3.82 mm to (195.8, 110.0), turned to -90 degrees
- moved R29 3.82 mm to (195.8, 118.6), turned to -90 degrees
- moved R25 3.79 mm to (195.8, 114.3), turned to -90 degrees
- moved R26 2.18 mm to (211.1, 119.6), turned to 90 degrees
- moved R30 2.18 mm to (211.1, 105.9), turned to 90 degrees
- moved R34 2.18 mm to (211.1, 101.3), turned to 90 degrees
- moved R38 2.18 mm to (211.1, 96.8), turned to 90 degrees
- moved R18 2.18 mm to (211.1, 110.5), turned to 90 degrees
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- renumbered C11 to C10, C13 to C11, C15 to C12, C17 to C13, C19 to C14, C8 to C2, C2 to C3, C3 to C5, C5 to C6, C6 to C7, C7 to C8, D12 to D11, D14 to D13, D4 to D3, D6 to D5, D8 to D7, D10 to D9, J6 to J3, J9 to J4, J2 to J6, J8 to J7, J4 to J8, R11 to R10, R60 to R11, R67 to R12, R61 to R13, R68 to R14, R9 to R15, R10 to R16, R62 to R17, R12 to R18, R15 to R19, R18 to R21, R20 to R22, R26 to R25, R28 to R26, R31 to R27, R34 to R29, R13 to R3, R36 to R30, R39 to R31, R42 to R33, R44 to R34, R47 to R35, R50 to R37, R52 to R38, R55 to R39, R3 to R4, R58 to R41, R66 to R9
Connections:
- D11 pad 1: /BB0/B#+1 -> Net-(D11-K)
- D13 pad 1: /BB0/B# -> Net-(D13-K)
- D3 pad 1: /BB2/B#+1 -> Net-(D3-K)
- D5 pad 1: /BB3/B#+1 -> Net-(D5-K)
- D7 pad 1: /BB4/B#+1 -> Net-(D7-K)
- D9 pad 1: /BB1/B#+1 -> Net-(D9-K)
- Q2 pad 1: Net-(Q2-G) -> /S4
- Q2 pad 2: /BB3/B#+1 -> /BB2/B#+1
- Q2 pad 3: Net-(Q2-D) -> Net-(D3-K)
- Q4 pad 1: Net-(Q4-G) -> /S6
- Q4 pad 3: Net-(Q4-D) -> Net-(D7-K)
- Q6 pad 1: Net-(Q6-G) -> /S2
- Q6 pad 2: /BB5/B#+1 -> /BB0/B#+1
- Q6 pad 3: Net-(Q6-D) -> Net-(D11-K)
- R18 pad 1: Net-(Q2-D) -> /BB3/B#+1
- R19 pad 1: /BB2/B#+1 -> Net-(D3-K)
- R19 pad 2: Net-(Q2-D) -> /BB3/B#+1
- R22 pad 1: Net-(Q4-D) -> /BB4/B#+1
- R23 pad 1: /BB3/B#+1 -> Net-(D5-K)
- R23 pad 2: Net-(Q4-D) -> /BB4/B#+1
- R26 pad 1: Net-(Q6-D) -> /BB5/B#+1
- R27 pad 1: /BB4/B#+1 -> Net-(D7-K)
- R27 pad 2: Net-(Q6-D) -> /BB5/B#+1
- R30 pad 1: Net-(Q8-D) -> /BB2/B#+1
- R31 pad 1: /BB1/B#+1 -> Net-(D9-K)
- R31 pad 2: Net-(Q8-D) -> /BB2/B#+1
- R34 pad 1: Net-(Q10-D) -> /BB1/B#+1
- R35 pad 1: /BB0/B#+1 -> Net-(D11-K)
- R35 pad 2: Net-(Q10-D) -> /BB1/B#+1
- R38 pad 1: Net-(Q12-D) -> /BB0/B#+1
- R39 pad 1: /BB0/B# -> Net-(D13-K)
- R39 pad 2: Net-(Q12-D) -> /BB0/B#+1
Routing:
- net Net-(D7-K): track 0.00 -> 11.5 mm
- net Net-(D9-K): track 0.00 -> 11.5 mm
- net Net-(D11-K): track 0.00 -> 11.5 mm
- net Net-(D5-K): track 0.00 -> 11.5 mm
- net Net-(D3-K): track 0.00 -> 11.5 mm
- net Net-(D13-K): track 0.00 -> 11.5 mm
- net /C0: track 29.2 -> 17.7 mm
- net /BB0/B#: track 89.7 -> 78.7 mm, vias 3 -> 0
- net Net-(Q4-D): track 8.63 -> 0.00 mm
- net Net-(Q2-D): track 8.63 -> 0.00 mm
- net Net-(Q8-D): track 8.35 -> 0.00 mm
- net Net-(Q6-D): track 8.35 -> 0.00 mm
- net Net-(Q10-D): track 8.35 -> 0.00 mm
- net Net-(Q12-D): track 8.12 -> 0.00 mm
- net /S5: track 13.3 -> 21.2 mm
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