File: fuse-board/fuse-board.kicad_sch (KiCad schematic)
At the start: 13 parts, among them J1 42820-2223, J2 1053141106, J3 ATM15-12PA-BM04

Commit message: rev 1.1 with mini-fit sr
Parts:
- added H2: MountingHole M3, MountingHole:MountingHole_3.2mm_M3, symbol Mechanical:MountingHole
- F1: value TB Fan_A -> 3568; Name (none) -> TB_Fan_A
- F2: value TB Fan_B -> 3568; Name (none) -> TB_Fan_B
- F3: value TB Fan_C -> 3568
- F4: value TBB -> 3568
- F5: value VCU -> 3568
- F6: value Telemetry -> 3568
- F7: value PEB -> 3568; Name (none) -> PEB
- F8: value Shutdown -> 3568; Name (none) -> Shutdown
- F9: value Inverter -> 3568
Connections:
- net 12V_In: now also F1.1, F2.1, F5.2, F6.2, J1.2 (Pin_2); no longer F1.2, F2.2, F5.1, F6.1, J1.1 (Pin_1)
- net GND: now also J1.1 (Pin_1); no longer J1.2 (Pin_2)
- net TBB: now also J3.3 (Pin_3); no longer J3.4 (Pin_4)
- net TB_Fan_A: now also F1.2, J3.6 (Pin_6); no longer F1.1, J3.1 (Pin_1)
- net TB_Fan_B: now also F2.2, J3.5 (Pin_5); no longer F2.1, J3.2 (Pin_2)
- net TB_Fan_C: now also J3.4 (Pin_4); no longer J3.3 (Pin_3)
- net Telemetry: now also F6.1, J3.1 (Pin_1); no longer F6.2, J3.6 (Pin_6)
- net VCU: now also F5.1, J3.2 (Pin_2); no longer F5.2, J3.5 (Pin_5)
Other:
- moved on the sheet: F1, F2, F3, F4, F5, F6, H1, J1

Commit message: v1.2 with ring terminal studs
Parts:
- removed H2: MountingHole M3, MountingHole:MountingHole_3.2mm_M3, symbol Mechanical:MountingHole
- removed J1: 42820-2223, Connector_Molex:Molex_Mini-Fit_Sr_42820-22XX_1x02_P10.00mm_Horizontal, symbol Connector_Generic:Conn_01x02
- added J1, J2: 74651173R, FS_4_Global_Footprint_Library:74651173R, symbol Connector_Generic:Conn_01x01
- renumbered J2 to J3, J3 to J4
Connections:
- net 12V_In: now also J1.1 (Pin_1)
- net GND: now also J3.1 (Pin_1), J3.2 (Pin_2), J3.3 (Pin_3), J2.1 (Pin_1); no longer J3.4 (Pin_4), J3.5 (Pin_5), J3.6 (Pin_6)
- net Inverter: now also J3.6 (Pin_6); no longer J3.3 (Pin_3)
- net PEB: now also J3.4 (Pin_4); no longer J3.1 (Pin_1)
- net Shutdown: now also J3.5 (Pin_5); no longer J3.2 (Pin_2)
Other:
- moved on the sheet: J3

Commit message: v1.3 filled out symbol fields and improved traces
Parts:
- F1, F2, F3, F4, F5, F6, F7, F8, F9: Digi PN (none) -> 36-3568-ND; Digi URL (none) -> https://www.digikey.com/en/products/detail/keystone-electro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; MFG (none) -> Keystone Electronics; MFG PN (none) -> 3568
- J1, J2: Digi PN (none) -> 732-74651173RCT-ND; Digi URL (none) -> https://www.digikey.com/en/products/detail/w%C3%BCrth-elekt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; MFG (none) -> Würth Elektronik; MFG PN (none) -> 74651173R
- J3: symbol Connector_Generic:Conn_02x03_Counter_Clockwise -> Connector_Generic:Conn_02x03_Top_Bottom; Digi PN (none) -> WM16908-ND; Digi URL (none) -> https://www.digikey.com/en/products/detail/molex/1053141106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; MFG (none) -> Molex; MFG PN (none) -> 1053141106
- J4: Digi PN (none) -> 889-3307-ND; Digi URL (none) -> https://www.digikey.com/en/products/detail/amphenol-sine-sy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; MFG (none) -> Amphenol Sine Systems Corp; MFG PN (none) -> ATM15-12PA-BM04
Connections:
- net GND: no longer J3.1 (Pin_1)
- net PEB: now also J3.1 (Pin_1)
Other:
- note added: "10A ATM"
- note added: "5A ATM"
- moved on the sheet: J3

Commit message: v1.4 added note for 12VMP, fixed silkscreen title, fixed chud trace
Other:
- note added: "No return for PEB because the return is on the PEB. Pin 1 gets PEB 12V for use with the 12V measuring point"
Changed lines of the file:
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@@
 		(title "Fuse Board")
 		(date "2026-03-27")
-		(rev "1.3")
+		(rev "1.4")
 		(company "Formula Slug")
 		(comment 4 "Cole Lewis")
@@
 		(effects
 			(font
+				(size 1.27 1.27)
+			)
+			(justify left)
+		)
+	)
+	(text "No return for PEB because the return is on the PEB.\nPin 1 gets PEB 12V for use with the 12V measuring point"
+		(exclude_from_sim no)
+		(at 182.88 43.18 0)
+		(effects
+			(font
