File: BMS Busbar Board/BMS Busbar Board/BMS Busbar Board.kicad_sch (KiCad schematic)
At the start: 17 parts, among them J1 Conn_01x05_MountingPin, J2 Conn_01x05_MountingPin

Commit message: busbar schematic and pcb progress
Parts:
- F8: footprint (none) -> Fuse:Fuse_2010_5025Metric
Changed lines of the file:
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@@
+		)
+	)
+	(netclass_flag ""
+		(length 2.54)
+		(shape round)
+		(at 68.58 116.84 0)
+		(fields_autoplaced yes)
+		(effects
+			(font
+				(size 1.27 1.27)
+			)
+			(justify left bottom)
+		)
+		(property "Netclass" "Power"
+			(at 69.2785 114.3 0)
+			(effects
+				(font
+					(size 1.27 1.27)
+				)
+				(justify left)
+			)
+		)
+		(property "Component Class" ""
+			(at -3.81 0 0)
+			(effects
+				(font
+					(size 1.27 1.27)
+					(italic yes)
+				)
+			)
+		)
+	)
+	(netclass_flag ""
+		(length 2.54)
+		(shape round)
+		(at 116.84 27.94 0)
+		(fields_autoplaced yes)
+		(effects
+			(font
+				(size 1.27 1.27)
+			)
+			(justify left bottom)
+		)
+		(property "Netclass" "Power"
+			(at 117.5385 25.4 0)
+			(effects
+				(font
+					(size 1.27 1.27)
+				)
+				(justify left)
+			)
+		)
+		(property "Component Class" ""
+			(at 44.45 -88.9 0)
+			(effects
+				(font
+					(size 1.27 1.27)
+					(italic yes)
+				)
+			)
+		)
+	)
+	(netclass_flag ""
+		(length 2.54)
+		(shape round)
+		(at 93.98 27.94 0)
+		(fields_autoplaced yes)
+		(effects
+			(font
+				(size 1.27 1.27)
+			)
+			(justify left bottom)
+		)
+		(property "Netclass" "Power"
+			(at 94.6785 25.4 0)
+			(effects
+				(font
+					(size 1.27 1.27)
+				)
+				(justify left)
+			)
+		)
+		(property "Component Class" ""
+			(at 21.59 -88.9 0)
+			(effects
+				(font
+					(size 1.27 1.27)
+					(italic yes)
+				)
+			)
+		)
+	)
+	(netclass_flag ""
+		(length 2.54)
+		(shape round)
+		(at 114.3 129.54 0)
+		(fields_autoplaced yes)
+		(effects
+			(font
+				(size 1.27 1.27)
+			)
+			(justify left bottom)
+		)
+		(property "Netclass" "Power"
+			(at 114.9985 127 0)
+			(effects
+				(font
+					(size 1.27 1.27)
+				)
+				(justify left)
+			)
+		)
+		(property "Component Class" ""
+			(at 41.91 12.7 0)
+			(effects
+				(font
+					(size 1.27 1.27)
+					(italic yes)
+				)
+			)
 		)
 	)
@@
 			)
 		)
-		(property "Footprint" ""
+		(property "Footprint" "Fuse:Fuse_2010_5025Metric"
 			(at 105.41 42.418 90)
 			(effects

Commit message: fuse footprints added
Parts:
- removed F1: Fuse, symbol Device:Fuse
- added F9: Littlefuse 1812L110/33, Fuse:Fuse_1812_4532Metric_Pad1.30x3.40mm_HandSolder, symbol Device:Fuse
- F1: renamed from F9; value Fuse -> Littlefuse 1812L110/33; footprint (none) -> Fuse:Fuse_1812_4532Metric_Pad1.30x3.40mm_HandSolder
- F2, F3, F4, F5, F6, F7: value Fuse -> Littlefuse 1812L110/33; footprint (none) -> Fuse:Fuse_1812_4532Metric_Pad1.30x3.40mm_HandSolder
- F8: value Fuse -> Littlefuse 1812L110/33; footprint Fuse:Fuse_2010_5025Metric -> Fuse:Fuse_1812_4532Metric_Pad1.30x3.40mm_HandSolder
Connections:
- net V-: now also F9.2; no longer F7.2
- net c_sense_cell_2: now also F5.2; no longer F3.2
- net cell_0_minus: now also F8.1, F9.1; no longer F6.1, F7.1
- net cell_0_plus: now also F7.1; no longer F5.1
- net cell_1_plus: now also F6.1; no longer F4.1
- net cell_2_plus: now also F5.1; no longer F3.1
- net cell_3_plus: now also F4.1; no longer F2.1
- net cell_4_plus: now also F3.1
- net cell_5_plus: now also F2.1; no longer F8.1
- net v_sense_cell_0: now also F7.2; no longer F5.2
- net v_sense_cell_1: now also F6.2; no longer F4.2
- net v_sense_cell_3: now also F4.2; no longer F2.2
- net v_sense_cell_4: now also F3.2
- net v_sense_cell_5: now also F2.2; no longer F8.2
- net v_sense_minus: now also F8.2; no longer F6.2

Commit message: pcb wired (drc errors)
Parts:
- J1, J2: footprint (none) -> FS_4_Global_Footprint_Library:CON_5019510550
Connections:
- net V+ renamed V_high
- net V- renamed V_low
Changed lines of the file:
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@@
+		(color 0 0 0 0)
+	)
+	(junction
+		(at 134.62 129.54)
+		(diameter 0)
+		(color 0 0 0 0)
+	)
+	(junction
+		(at 137.16 27.94)
+		(diameter 0)
 		(color 0 0 0 0)
 	)
@@
 		)
 	)
-	(label "V+"
-		(at 127 27.94 0)
-		(effects
-			(font
-				(size 1.27 1.27)
-			)
-			(justify left bottom)
-		)
-	)
 	(label "cell_4_plus"
 		(at 76.2 53.34 0)
@@
 		)
 	)
-	(label "V-"
-		(at 127 129.54 0)
-		(effects
-			(font
-				(size 1.27 1.27)
-			)
-			(justify left bottom)
-		)
-	)
 	(label "v_sense_cell_3"
 		(at 114.3 66.04 0)
@@
 			)
 			(justify left bottom)
-		)
-	)
-	(netclass_flag ""
-		(length 2.54)
-		(shape round)
-		(at 68.58 116.84 0)
-		(fields_autoplaced yes)
-		(effects
-			(font
-				(size 1.27 1.27)
-			)
-			(justify left bottom)
-		)
-		(property "Netclass" "Power"
-			(at 69.2785 114.3 0)
-			(effects
-				(font
-					(size 1.27 1.27)
-				)
-				(justify left)
-			)
-		)
-		(property "Component Class" ""
-			(at -3.81 0 0)
-			(effects
-				(font
-					(size 1.27 1.27)
-					(italic yes)
-				)
-			)
-		)
-	)
-	(netclass_flag ""
-		(length 2.54)
-		(shape round)
-		(at 118.11 27.94 0)
-		(fields_autoplaced yes)
-		(effects
-			(font
-				(size 1.27 1.27)
-			)
-			(justify left bottom)
-		)
-		(property "Netclass" "Power"
-			(at 118.8085 25.4 0)
-			(effects
-				(font
-					(size 1.27 1.27)
-				)
-				(justify left)
-			)
-		)
-		(property "Component Class" ""
-			(at 45.72 -88.9 0)
-			(effects
-				(font
-					(size 1.27 1.27)
-					(italic yes)
-				)
-			)
-		)
-	)
-	(netclass_flag ""
-		(length 2.54)
-		(shape round)
-		(at 67.31 40.64 0)
-		(fields_autoplaced yes)
-		(effects
-			(font
-				(size 1.27 1.27)
-			)
-			(justify left bottom)
-		)
-		(property "Netclass" "Power"
-			(at 68.0085 38.1 0)
-			(effects
-				(font
-					(size 1.27 1.27)
-				)
-				(justify left)
-			)
-		)
-		(property "Component Class" ""
-			(at -5.08 -76.2 0)
-			(effects
-				(font
-					(size 1.27 1.27)
-					(italic yes)
-				)
-			)
-		)
-	)
-	(netclass_flag ""
-		(length 2.54)
-		(shape round)
-		(at 118.11 129.54 0)
-		(fields_autoplaced yes)
-		(effects
-			(font
-				(size 1.27 1.27)
-			)
-			(justify left bottom)
-		)
-		(property "Netclass" "Power"
-			(at 118.8085 127 0)
-			(effects
-				(font
-					(size 1.27 1.27)
-				)
-				(justify left)
-			)
-		)
-		(property "Component Class" ""
-			(at 45.72 12.7 0)
-			(effects
-				(font
-					(size 1.27 1.27)
-					(italic yes)
-				)
-			)
 		)
 	)
@@
 			)
 		)
-		(property "Footprint" ""
+		(property "Footprint" "FS_4_Global_Footprint_Library:CON_5019510550"
 			(at 157.48 96.52 0)
 			(effects
@@
 	)
 	(symbol
+		(lib_id "power:GNDD")
+		(at 134.62 129.54 0)
+		(unit 1)
+		(exclude_from_sim no)
+		(in_bom yes)
+		(on_board yes)
+		(dnp no)
+		(fields_autoplaced yes)
+		(property "Reference" "#PWR02"
+			(at 134.62 135.89 0)
+			(effects
+				(font
+					(size 1.27 1.27)
+				)
+				(hide yes)
+			)
+		)
+		(property "Value" "V_low"
+			(at 134.62 133.35 0)
+			(effects
+				(font
+					(size 1.27 1.27)
+				)
+			)
+		)
+		(property "Footprint" ""
+			(at 134.62 129.54 0)
+			(effects
+				(font
+					(size 1.27 1.27)
+				)
+				(hide yes)
+			)
+		)
+		(property "Datasheet" ""
+			(at 134.62 129.54 0)
+			(effects
+				(font
+					(size 1.27 1.27)
+				)
+				(hide yes)
+			)
+		)
+		(property "Description" "Power symbol creates a global label with name \"GNDD\" , digital ground"
+			(at 134.62 129.54 0)
+			(effects
+				(font
+					(size 1.27 1.27)
+				)
+				(hide yes)
+			)
+		)
+		(pin "1"
+		)
+		(instances
+			(project ""
+				(path "/4a7933dc-894e-4333-8e50-6627480f7b53"
+					(reference "#PWR02")
+					(unit 1)
+				)
+			)
+		)
+	)
+	(symbol
+		(lib_id "power:VAA")
+		(at 137.16 27.94 0)
+		(unit 1)
+		(exclude_from_sim no)
+		(in_bom yes)
+		(on_board yes)
+		(dnp no)
+		(fields_autoplaced yes)
+		(property "Reference" "#PWR01"
+			(at 137.16 31.75 0)
+			(effects
+				(font
+					(size 1.27 1.27)
+				)
+				(hide yes)
+			)
+		)
+		(property "Value" "V_high"
+			(at 137.16 22.86 0)
+			(effects
+				(font
+					(size 1.27 1.27)
+				)
+			)
+		)
+		(property "Footprint" ""
+			(at 137.16 27.94 0)
+			(effects
+				(font
+					(size 1.27 1.27)
+				)
+				(hide yes)
+			)
+		)
+		(property "Datasheet" ""
+			(at 137.16 27.94 0)
+			(effects
+				(font
+					(size 1.27 1.27)
+				)
+				(hide yes)
+			)
+		)
+		(property "Description" "Power symbol creates a global label with name \"VAA\""
+			(at 137.16 27.94 0)
+			(effects
+				(font
+					(size 1.27 1.27)
+				)
+				(hide yes)
+			)
+		)
+		(pin "1"
+		)
+		(instances
+			(project ""
+				(path "/4a7933dc-894e-4333-8e50-6627480f7b53"
+					(reference "#PWR01")
+					(unit 1)
+				)
+			)
+		)
+	)
+	(symbol
 		(lib_id "Connector_Generic_MountingPin:Conn_01x05_MountingPin")
 		(at 157.48 73.66 0)
@@
 			)
 		)
-		(property "Footprint" ""
+		(property "Footprint" "FS_4_Global_Footprint_Library:CON_5019510550"
 			(at 157.48 73.66 0)
 			(effects

Commit message: busbar pcb complete (with violations)
Connections:
- net V_high: now also J1.2 (Pin_2); no longer J1.1 (Pin_1)
- net V_low: now also J2.5 (Pin_5); no longer J2.4 (Pin_4)
- net c_sense_cell_2: now also J2.1 (Pin_1); no longer J1.5 (Pin_5)
- net v_sense_cell_0: now also J2.3 (Pin_3); no longer J2.2 (Pin_2)
- net v_sense_cell_1: now also J2.2 (Pin_2); no longer J2.1 (Pin_1)
- net v_sense_cell_3: now also J1.5 (Pin_5); no longer J1.4 (Pin_4)
- net v_sense_cell_4: now also J1.4 (Pin_4); no longer J1.3 (Pin_3)
- net v_sense_cell_5: now also J1.3 (Pin_3); no longer J1.2 (Pin_2)
- net v_sense_minus: now also J2.4 (Pin_4); no longer J2.3 (Pin_3)
Other:
- moved on the sheet: J1, J2
Changed lines of the file:
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@@
 	)
 	(no_connect
-		(at 157.48 106.68)
+		(at 157.48 104.14)
 	)
 	(no_connect
-		(at 157.48 83.82)
+		(at 157.48 81.28)
 	)
 	(no_connect
-		(at 152.4 101.6)
+		(at 152.4 66.04)
+	)
+	(wire
+		(pts
+			(xy 137.16 68.58) (xy 152.4 68.58)
+		)
+		(stroke
+			(width 0)
+			(type default)
+		)
 	)
 	(wire
@@
 	(wire
 		(pts
-			(xy 152.4 93.98) (xy 129.54 93.98)
+			(xy 134.62 99.06) (xy 152.4 99.06)
 		)
 		(stroke
@@
 	(wire
 		(pts
-			(xy 137.16 68.58) (xy 152.4 68.58)
+			(xy 129.54 93.98) (xy 152.4 93.98)
 		)
 		(stroke
@@
 	(wire
 		(pts
+			(xy 152.4 88.9) (xy 127 88.9)
+		)
+		(stroke
+			(width 0)
+			(type default)
+		)
+	)
+	(wire
+		(pts
+			(xy 109.22 91.44) (xy 152.4 91.44)
+		)
+		(stroke
+			(width 0)
+			(type default)
+		)
+	)
+	(wire
+		(pts
 			(xy 63.5 40.64) (xy 63.5 43.18)
 		)
@@
 	(wire
 		(pts
-			(xy 109.22 78.74) (xy 152.4 78.74)
-		)
-		(stroke
-			(width 0)
-			(type default)
-		)
-	)
-	(wire
-		(pts
 			(xy 93.98 27.94) (xy 93.98 40.64)
 		)
@@
 	(wire
 		(pts
+			(xy 127 88.9) (xy 127 78.74)
+		)
+		(stroke
+			(width 0)
+			(type default)
+		)
+	)
+	(wire
+		(pts
 			(xy 63.5 114.3) (xy 63.5 116.84)
 		)
@@
 	(wire
 		(pts
-			(xy 152.4 99.06) (xy 134.62 99.06)
-		)
-		(stroke
-			(width 0)
-			(type default)
-		)
-	)
-	(wire
-		(pts
 			(xy 134.62 40.64) (xy 109.22 40.64)
 		)
@@
 	(wire
 		(pts
-			(xy 152.4 76.2) (xy 129.54 76.2)
-		)
-		(stroke
-			(width 0)
-			(type default)
-		)
-	)
-	(wire
-		(pts
 			(xy 101.6 129.54) (xy 92.71 129.54)
 		)
@@
 	(wire
 		(pts
-			(xy 152.4 96.52) (xy 132.08 96.52)
-		)
-		(stroke
-			(width 0)
-			(type default)
-		)
-	)
-	(wire
-		(pts
 			(xy 63.5 63.5) (xy 63.5 66.04)
 		)
@@
 	(wire
 		(pts
+			(xy 109.22 78.74) (xy 127 78.74)
+		)
+		(stroke
+			(width 0)
+			(type default)
+		)
+	)
+	(wire
+		(pts
 			(xy 101.6 53.34) (xy 63.5 53.34)
 		)
@@
 	(wire
 		(pts
-			(xy 109.22 91.44) (xy 152.4 91.44)
+			(xy 129.54 76.2) (xy 152.4 76.2)
 		)
 		(stroke
@@
 	(wire
 		(pts
+			(xy 132.08 96.52) (xy 152.4 96.52)
+		)
+		(stroke
+			(width 0)
+			(type default)
+		)
+	)
+	(wire
+		(pts
+			(xy 132.08 73.66) (xy 152.4 73.66)
+		)
+		(stroke
+			(width 0)
+			(type default)
+		)
+	)
+	(wire
+		(pts
 			(xy 137.16 27.94) (xy 137.16 68.58)
 		)
@@
 	(wire
 		(pts
+			(xy 134.62 71.12) (xy 152.4 71.12)
+		)
+		(stroke
+			(width 0)
+			(type default)
+		)
+	)
+	(wire
+		(pts
 			(xy 109.22 104.14) (xy 129.54 104.14)
 		)
@@
 	(wire
 		(pts
-			(xy 132.08 73.66) (xy 152.4 73.66)
-		)
-		(stroke
-			(width 0)
-			(type default)
-		)
-	)
-	(wire
-		(pts
 			(xy 109.22 53.34) (xy 132.08 53.34)
-		)
-		(stroke
-			(width 0)
-			(type default)
-		)
-	)
-	(wire
-		(pts
-			(xy 152.4 71.12) (xy 134.62 71.12)
 		)
 		(stroke
@@
 	(symbol
 		(lib_id "Connector_Generic_MountingPin:Conn_01x05_MountingPin")
-		(at 157.48 96.52 0)
+		(at 157.48 93.98 0)
 		(unit 1)
 		(exclude_from_sim no)
@@
 		(dnp no)
 		(property "Reference" "J2"
+			(at 160.02 93.0655 0)
+			(effects
+				(font
+					(size 1.27 1.27)
+				)
+				(justify left)
+			)
+		)
+		(property "Value" "Conn_01x05_MountingPin"
 			(at 160.02 95.6055 0)
 			(effects
@@
 			)
 		)
-		(property "Value" "Conn_01x05_MountingPin"
-			(at 160.02 98.1455 0)
-			(effects
-				(font
-					(size 1.27 1.27)
-				)
-				(justify left)
-			)
-		)
 		(property "Footprint" "FS_4_Global_Footprint_Library:CON_5019510550"
-			(at 157.48 96.52 0)
+			(at 157.48 93.98 0)
 			(effects
 				(font
@@
 		)
 		(property "Datasheet" "~"
-			(at 157.48 96.52 0)
+			(at 157.48 93.98 0)
 			(effects
 				(font
@@
 		)
 		(property "Description" "Generic connectable mounting pin connector, single row, 01x05, script generated (kicad-library-utils/schlib/autogen/connector/)"
-			(at 157.48 96.52 0)
+			(at 157.48 93.98 0)
 			(effects
 				(font
@@
 	(symbol
 		(lib_id "Connector_Generic_MountingPin:Conn_01x05_MountingPin")
-		(at 157.48 73.66 0)
+		(at 157.48 71.12 0)
 		(unit 1)
 		(exclude_from_sim no)
@@
 		(dnp no)
 		(property "Reference" "J1"
+			(at 160.02 70.2055 0)
+			(effects
+				(font
+					(size 1.27 1.27)
+				)
+				(justify left)
+			)
+		)
+		(property "Value" "Conn_01x05_MountingPin"
 			(at 160.02 72.7455 0)
 			(effects
@@
 			)
 		)
-		(property "Value" "Conn_01x05_MountingPin"
-			(at 160.02 75.2855 0)
-			(effects
-				(font
-					(size 1.27 1.27)
-				)
-				(justify left)
-			)
-		)
 		(property "Footprint" "FS_4_Global_Footprint_Library:CON_5019510550"
-			(at 157.48 73.66 0)
+			(at 157.48 71.12 0)
 			(effects
 				(font
@@
 		)
 		(property "Datasheet" "~"
-			(at 157.48 73.66 0)
+			(at 157.48 71.12 0)
 			(effects
 				(font
@@
 		)
 		(property "Description" "Generic connectable mounting pin connector, single row, 01x05, script generated (kicad-library-utils/schlib/autogen/connector/)"
-			(at 157.48 73.66 0)
-			(effects
-				(font
+			(at 157.48 71.12 0)
+			(effects
+				(font

Commit message: imported and placed new connector
Parts:
- J1, J2: footprint FS_4_Global_Footprint_Library:CON_5019510550 -> FS_4_Global_Footprint_Library:512810598
Changed lines of the file:
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@@
 			)
 		)
-		(property "Footprint" "FS_4_Global_Footprint_Library:CON_5019510550"
+		(property "Footprint" "FS_4_Global_Footprint_Library:512810598"
 			(at 157.48 93.98 0)
 			(effects
@@
 			)
 		)
-		(property "Footprint" "FS_4_Global_Footprint_Library:CON_5019510550"
+		(property "Footprint" "FS_4_Global_Footprint_Library:512810598"
 			(at 157.48 71.12 0)
 			(effects

Commit message: new connector added
Parts:
- removed J1, J2: Conn_01x05_MountingPin, FS_4_Global_Footprint_Library:512810598, symbol Connector_Generic_MountingPin:Conn_01x05_MountingPin
- added J1: 2005280090, FS_4_Global_Footprint_Library:CON_2005280090_MOL, symbol FS_4_Global_Symbol_Library:2005280090
Connections:
- net V_high: now also J1.1
- net V_low: now also J1.9
- net c_sense_cell_2: now also J1.5
- net v_sense_cell_0: now also J1.7
- net v_sense_cell_1: now also J1.6
- net v_sense_cell_3: now also J1.4
- net v_sense_cell_4: now also J1.3
- net v_sense_cell_5: now also J1.2
- net v_sense_minus: now also J1.8
- no-connect marks 3 -> 2
Changed lines of the file:
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@@
 	)
 	(no_connect
-		(at 157.48 104.14)
+		(at 167.64 93.98)
 	)
 	(no_connect
-		(at 157.48 81.28)
-	)
-	(no_connect
-		(at 152.4 66.04)
-	)
-	(wire
-		(pts
-			(xy 137.16 68.58) (xy 152.4 68.58)
+		(at 167.64 91.44)
+	)
+	(wire
+		(pts
+			(xy 160.02 86.36) (xy 167.64 86.36)
+		)
+		(stroke
+			(width 0)
+			(type default)
+		)
+	)
+	(wire
+		(pts
+			(xy 137.16 68.58) (xy 167.64 68.58)
 		)
 		(stroke
@@
 	(wire
 		(pts
-			(xy 134.62 99.06) (xy 152.4 99.06)
+			(xy 134.62 99.06) (xy 162.56 99.06)
 		)
 		(stroke
@@
 	(wire
 		(pts
-			(xy 129.54 93.98) (xy 152.4 93.98)
+			(xy 129.54 93.98) (xy 157.48 93.98)
 		)
 		(stroke
@@
 	(wire
 		(pts
-			(xy 109.22 91.44) (xy 152.4 91.44)
+			(xy 109.22 91.44) (xy 154.94 91.44)
 		)
 		(stroke
@@
 	(wire
 		(pts
+			(xy 157.48 93.98) (xy 157.48 83.82)
+		)
+		(stroke
+			(width 0)
+			(type default)
+		)
+	)
+	(wire
+		(pts
 			(xy 101.6 91.44) (xy 63.5 91.44)
 		)
@@
 	(wire
 		(pts
+			(xy 162.56 99.06) (xy 162.56 88.9)
+		)
+		(stroke
+			(width 0)
+			(type default)
+		)
+	)
+	(wire
+		(pts
 			(xy 63.5 114.3) (xy 63.5 116.84)
 		)
@@
 	(wire
 		(pts
+			(xy 154.94 91.44) (xy 154.94 81.28)
+		)
+		(stroke
+			(width 0)
+			(type default)
+		)
+	)
+	(wire
+		(pts
 			(xy 63.5 88.9) (xy 63.5 91.44)
 		)
@@
 	(wire
 		(pts
+			(xy 152.4 88.9) (xy 152.4 78.74)
+		)
+		(stroke
+			(width 0)
+			(type default)
+		)
+	)
+	(wire
+		(pts
 			(xy 63.5 104.14) (xy 63.5 106.68)
 		)
@@
 	(wire
 		(pts
-			(xy 129.54 76.2) (xy 152.4 76.2)
+			(xy 162.56 88.9) (xy 167.64 88.9)
+		)
+		(stroke
+			(width 0)
+			(type default)
+		)
+	)
+	(wire
+		(pts
+			(xy 129.54 76.2) (xy 167.64 76.2)
 		)
 		(stroke
@@
 	(wire
 		(pts
+			(xy 160.02 96.52) (xy 160.02 86.36)
+		)
+		(stroke
+			(width 0)
+			(type default)
+		)
+	)
+	(wire
+		(pts
 			(xy 132.08 53.34) (xy 132.08 73.66)
 		)
@@
 	(wire
 		(pts
-			(xy 132.08 96.52) (xy 152.4 96.52)
-		)
-		(stroke
-			(width 0)
-			(type default)
-		)
-	)
-	(wire
-		(pts
-			(xy 132.08 73.66) (xy 152.4 73.66)
+			(xy 132.08 96.52) (xy 160.02 96.52)
+		)
+		(stroke
+			(width 0)
+			(type default)
+		)
+	)
+	(wire
+		(pts
+			(xy 132.08 73.66) (xy 167.64 73.66)
 		)
 		(stroke
@@
 	(wire
 		(pts
-			(xy 134.62 71.12) (xy 152.4 71.12)
+			(xy 134.62 71.12) (xy 167.64 71.12)
 		)
 		(stroke
@@
 	(wire
 		(pts
+			(xy 152.4 78.74) (xy 167.64 78.74)
+		)
+		(stroke
+			(width 0)
+			(type default)
+		)
+	)
+	(wire
+		(pts
+			(xy 154.94 81.28) (xy 167.64 81.28)
+		)
+		(stroke
+			(width 0)
+			(type default)
+		)
+	)
+	(wire
+		(pts
 			(xy 63.5 101.6) (xy 63.5 104.14)
 		)
@@
 		(pts
 			(xy 109.22 129.54) (xy 134.62 129.54)
+		)
+		(stroke
+			(width 0)
+			(type default)
+		)
+	)
+	(wire
+		(pts
+			(xy 157.48 83.82) (xy 167.64 83.82)
 		)
 		(stroke
@@
 	)
 	(symbol
-		(lib_id "Connector_Generic_MountingPin:Conn_01x05_MountingPin")
-		(at 157.48 93.98 0)
-		(unit 1)
-		(exclude_from_sim no)
-		(in_bom yes)
-		(on_board yes)
-		(dnp no)
-		(property "Reference" "J2"
-			(at 160.02 93.0655 0)
-			(effects
-				(font
-					(size 1.27 1.27)
-				)
-				(justify left)
-			)
-		)
-		(property "Value" "Conn_01x05_MountingPin"
-			(at 160.02 95.6055 0)
-			(effects
-				(font
-					(size 1.27 1.27)
-				)
-				(justify left)
-			)
-		)
-		(property "Footprint" "FS_4_Global_Footprint_Library:512810598"
-			(at 157.48 93.98 0)
-			(effects
-				(font
-					(size 1.27 1.27)
-				)
-				(hide yes)
-			)
-		)
-		(property "Datasheet" "~"
-			(at 157.48 93.98 0)
-			(effects
-				(font
-					(size 1.27 1.27)
-				)
-				(hide yes)
-			)
-		)
-		(property "Description" "Generic connectable mounting pin connector, single row, 01x05, script generated (kicad-library-utils/schlib/autogen/connector/)"
-			(at 157.48 93.98 0)
-			(effects
-				(font
-					(size 1.27 1.27)
-				)
-				(hide yes)
-			)
-		)
-		(pin "1"
-		)
-		(pin "5"
-		)
-		(pin "4"
-		)
-		(pin "3"
-		)
-		(pin "2"
-		)
-		(pin "MP"
-		)
-		(instances
-			(project "BMS Busbar Board"
-				(path "/4a7933dc-894e-4333-8e50-6627480f7b53"
-					(reference "J2")
-					(unit 1)
-				)
-			)
-		)
-	)
-	(symbol
 		(lib_id "Device:Fuse")
 		(at 105.41 129.54 90)
@@
 	)
 	(symbol
+		(lib_id "FS_4_Global_Symbol_Library:2005280090")
+		(at 167.64 68.58 0)
+		(unit 1)
+		(exclude_from_sim no)
+		(in_bom yes)
+		(on_board yes)
+		(dnp no)
+		(fields_autoplaced yes)
+		(property "Reference" "J1"
+			(at 181.61 80.0099 0)
+			(effects
+				(font
+					(size 1.27 1.27)
+				)
+				(justify left)
+			)
+		)
+		(property "Value" "2005280090"
+			(at 181.61 82.5499 0)
+			(effects
+				(font
+					(size 1.27 1.27)
+				)
+				(justify left)
+			)
+		)
+		(property "Footprint" "FS_4_Global_Footprint_Library:CON_2005280090_MOL"
+			(at 172.974 58.928 0)
+			(effects
+				(font
+					(size 1.27 1.27)
+				)
+				(justify bottom)
+				(hide yes)
+			)
+		)
+		(property "Datasheet" ""
+			(at 167.64 68.58 0)
+			(effects
+				(font
+					(size 1.27 1.27)
+				)
+				(hide yes)
+			)
+		)
+		(property "Description" ""
+			(at 167.64 68.58 0)
+			(effects
+				(font
+					(size 1.27 1.27)
+				)
+				(hide yes)
+			)
+		)
+		(pin "P2"
+		)
+		(pin "8"
+		)
+		(pin "P1"
+		)
+		(pin "2"
+		)
+		(pin "1"
+		)
+		(pin "5"
+		)
+		(pin "6"
+		)
+		(pin "3"
+		)
+		(pin "7"
+		)
+		(pin "9"
+		)
+		(pin "4"
+		)
+		(instances
+			(project ""
+				(path "/4a7933dc-894e-4333-8e50-6627480f7b53"
+					(reference "J1")
+					(unit 1)
+				)
+			)
+		)
+	)
+	(symbol
 		(lib_id "power:GNDD")
 		(at 134.62 129.54 0)
@@
 					(unit 1)
 				)
-			)
-		)
-	)
-	(symbol
-		(lib_id "Connector_Generic_MountingPin:Conn_01x05_MountingPin")
-		(at 157.48 71.12 0)
-		(unit 1)
-		(exclude_from_sim no)
-		(in_bom yes)
-		(on_board yes)
-		(dnp no)
-		(property "Reference" "J1"
-			(at 160.02 70.2055 0)
-			(effects
-				(font
-					(size 1.27 1.27)
-				)
-				(justify left)
-			)
-		)
-		(property "Value" "Conn_01x05_MountingPin"
-			(at 160.02 72.7455 0)
-			(effects
-				(font
-					(size 1.27 1.27)
-				)
-				(justify left)
-			)
-		)
-		(property "Footprint" "FS_4_Global_Footprint_Library:512810598"
-			(at 157.48 71.12 0)
-			(effects
-				(font
-					(size 1.27 1.27)
-				)
-				(hide yes)
-			)
-		)
-		(property "Datasheet" "~"
-			(at 157.48 71.12 0)
-			(effects
-				(font
-					(size 1.27 1.27)
-				)
-				(hide yes)
-			)
-		)
-		(property "Description" "Generic connectable mounting pin connector, single row, 01x05, script generated (kicad-library-utils/schlib/autogen/connector/)"
-			(at 157.48 71.12 0)
-			(effects
-				(font
-					(size 1.27 1.27)
-				)
-				(hide yes)
-			)
-		)
-		(pin "1"
-		)
-		(pin "5"
-		)
-		(pin "4"
-		)
-		(pin "3"
-		)
-		(pin "2"
-		)
-		(pin "MP"
-		)
-		(instances
-			(project ""
-				(path "/4a7933dc-894e-4333-8e50-6627480f7b53"
-					(reference "J1")
-					(unit 1)
-				)
