File: BMS Busbar Board/BMS Busbar Board/BMS Busbar Board.kicad_sch (KiCad schematic)
At the start: 16 parts, among them J1 2005280090

Commit message: changed fuse names
Parts:
- F1, F2, F3, F4, F5, F6, F7, F8, F9: value Littlefuse 1812L110/33 -> Littlefuse 1812L050/30
Changed lines of the file:
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@@
 			)
 		)
-		(property "Value" "Littlefuse 1812L110/33"
+		(property "Value" "Littlefuse 1812L050/30"
 			(at 105.41 74.93 90)
 			(effects
@@
 			)
 		)
-		(property "Value" "Littlefuse 1812L110/33"
+		(property "Value" "Littlefuse 1812L050/30"
 			(at 105.41 125.73 90)
 			(effects
@@
 			)
 		)
-		(property "Value" "Littlefuse 1812L110/33"
+		(property "Value" "Littlefuse 1812L050/30"
 			(at 105.41 49.53 90)
 			(effects
@@
 			)
 		)
-		(property "Value" "Littlefuse 1812L110/33"
+		(property "Value" "Littlefuse 1812L050/30"
 			(at 105.41 24.13 90)
 			(effects
@@
 			)
 		)
-		(property "Value" "Littlefuse 1812L110/33"
+		(property "Value" "Littlefuse 1812L050/30"
 			(at 105.41 36.83 90)
 			(effects
@@
 			)
 		)
-		(property "Value" "Littlefuse 1812L110/33"
+		(property "Value" "Littlefuse 1812L050/30"
 			(at 105.41 87.63 90)
 			(effects
@@
 			)
 		)
-		(property "Value" "Littlefuse 1812L110/33"
+		(property "Value" "Littlefuse 1812L050/30"
 			(at 105.41 62.23 90)
 			(effects
@@
 			)
 		)
-		(property "Value" "Littlefuse 1812L110/33"
+		(property "Value" "Littlefuse 1812L050/30"
 			(at 105.41 113.03 90)
 			(effects
@@
 			)
 		)
-		(property "Value" "Littlefuse 1812L110/33"
+		(property "Value" "Littlefuse 1812L050/30"
 			(at 105.41 100.33 90)
 			(effects

Commit message: changed connector to 5pin version
Parts:
- removed J1: 2005280090, FS_4_Global_Footprint_Library:CON_2005280090_MOL, symbol FS_4_Global_Symbol_Library:2005280090
- added J1, J2: 2005280050, FS_4_Global_Footprint_Library:CON_2005280050_MOL, symbol FS_4_Global_Symbol_Library:2005280050
Connections:
- net V_high: now also J1.5
- net V_low: now also J2.1
- net c_sense_cell_2: now also J1.1
- net v_sense_cell_0: now also J2.3
- net v_sense_cell_1: now also J2.4
- net v_sense_cell_3: now also J1.2
- net v_sense_cell_4: now also J1.3
- net v_sense_cell_5: now also J1.4
- net v_sense_minus: now also J2.2
- no-connect marks 2 -> 5
