File: chargingboard/screen_architecture.kicad_sch (KiCad schematic)
At the start: 15 parts, among them J9 Conn_01x40_MountingPin, U1 BT817Q, U6 AP3019AKTR

Commit message: sum more datasheet
more stuff
Parts:
- J9: Digi PN (none) -> 609-F32D-1A7Y1-21040CT-ND; Digi URL (none) -> https://www.digikey.com/en/products/detail/amphenol-cs-fci/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
- L2: value 22u -> 22uF; Digi PN (none) -> 308-2307-1-ND; Digi URL (none) -> https://www.digikey.com/en/products/detail/sumida-america-i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
- U1: Digi PN (none) -> 2005-BT817Q-RCT-ND; Digi URL (none) -> https://www.digikey.com/en/products/detail/bridgetek-pte-lt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
- U6: Digi PN (none) -> AP3019AKTR-G1DICT-ND; Digi URL (none) -> https://www.digikey.com/en/products/detail/diodes-incorpora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
Changed lines of the file:
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@@
 			)
 		)
-		(property "Datasheet" ""
+		(property "Datasheet" "https://cdn.amphenol-cs.com/media/wysiwyg/files/documentation/datasheet/flex/ffc_fpc_050mm_f32d.pdf"
 			(at 339.09 130.81 0)
 			(effects
@@
 		)
 		(property "Description" "Generic connectable mounting pin connector, single row, 01x40, script generated (kicad-library-utils/schlib/autogen/connector/)"
+			(at 339.09 130.81 0)
+			(effects
+				(font
+					(size 1.27 1.27)
+				)
+				(hide yes)
+			)
+		)
+		(property "Digi PN" "609-F32D-1A7Y1-21040CT-ND"
+			(at 339.09 130.81 0)
+			(effects
+				(font
+					(size 1.27 1.27)
+				)
+				(hide yes)
+			)
+		)
+		(property "Digi URL" "https://www.digikey.com/en/products/detail/amphenol-cs-fci/F32D-1A7Y1-21040/11564657"
 			(at 339.09 130.81 0)
 			(effects
@@
 			)
 		)
+		(property "Digi PN" "2005-BT817Q-RCT-ND"
+			(at 124.46 97.79 0)
+			(effects
+				(font
+					(size 1.27 1.27)
+				)
+				(hide yes)
+			)
+		)
+		(property "Digi URL" "https://www.digikey.com/en/products/detail/bridgetek-pte-ltd/BT817Q-R/13242741"
+			(at 124.46 97.79 0)
+			(effects
+				(font
+					(size 1.27 1.27)
+				)
+				(hide yes)
+			)
+		)
 		(pin "57"
 		)
@@
 		(property "Description" "1.2MHz White LED Boost Drivers with Built-in Schottky, 2.5..16Vin, <30Vout, SOT-23-6"
 			(at 86.36 259.334 0)
+			(effects
+				(font
+					(size 1.27 1.27)
+				)
+				(hide yes)
+			)
+		)
+		(property "Digi PN" "AP3019AKTR-G1DICT-ND"
+			(at 82.55 233.68 0)
+			(effects
+				(font
+					(size 1.27 1.27)
+				)
+				(hide yes)
+			)
+		)
+		(property "Digi URL" "https://www.digikey.com/en/products/detail/diodes-incorporated/AP3019AKTR-G1/4470850"
+			(at 82.55 233.68 0)
 			(effects
 				(font
@@
 			)
 		)
-		(property "Value" "22u"
+		(property "Value" "22uF"
 			(at 64.77 218.44 90)
 			(effects
@@
 			(effects
 				(font
+					(size 1.27 1.27)
+				)
+				(hide yes)
+			)
+		)
+		(property "Digi PN" "308-2307-1-ND"
+			(at 64.77 220.98 90)
+			(effects
+				(font
+					(size 1.27 1.27)
+				)
+				(hide yes)
+			)
+		)
+		(property "Digi URL" "https://www.digikey.com/en/products/detail/sumida-america-inc/CDRH5D28NP-220NC/1059509"
+			(at 64.77 220.98 90)
+			(effects
+				(font

Commit message: some whitespaces fixes
whitespace fixes
Parts:
- C11: MFG (none) -> Samsung Electro-Mechanics; MFG PN (none) -> CL10A106KO8NQNC
- J9: MFG (none) -> Amphenol ICC (FCI); MFG PN (none) -> F32D-1A7Y1-21040
- L2: MFG (none) -> Sumida America Components Inc.; MFG PN (none) -> CDRH5D28NP-220NC
- R2: MFG (none) -> KOA Speer Electronics, Inc.; MFG PN (none) -> RK73H2ETTD4R99F
- U1: MFG (none) -> Bridgetek Pte Ltd.; MFG PN (none) -> BT817Q-R
- U6: MFG (none) -> Diodes Incorporated; MFG PN (none) -> AP3019AKTR-G1
Changed lines of the file:
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@@
 			)
 		)
+		(property "MFG" "Samsung Electro-Mechanics"
+			(at 152.4 76.2 0)
+			(effects
+				(font
+					(size 1.27 1.27)
+				)
+				(hide yes)
+			)
+		)
+		(property "MFG PN" "CL10A106KO8NQNC"
+			(at 152.4 76.2 0)
+			(effects
+				(font
+					(size 1.27 1.27)
+				)
+				(hide yes)
+			)
+		)
 		(pin "1"
 		)
@@
 			)
 		)
+		(property "MFG" "Amphenol ICC (FCI)"
+			(at 339.09 130.81 0)
+			(effects
+				(font
+					(size 1.27 1.27)
+				)
+				(hide yes)
+			)
+		)
+		(property "MFG PN" "F32D-1A7Y1-21040"
+			(at 339.09 130.81 0)
+			(effects
+				(font
+					(size 1.27 1.27)
+				)
+				(hide yes)
+			)
+		)
 		(pin "7"
 		)
@@
 			)
 		)
+		(property "MFG" "Bridgetek Pte Ltd."
+			(at 124.46 97.79 0)
+			(effects
+				(font
+					(size 1.27 1.27)
+				)
+				(hide yes)
+			)
+		)
+		(property "MFG PN" "BT817Q-R"
+			(at 124.46 97.79 0)
+			(effects
+				(font
+					(size 1.27 1.27)
+				)
+				(hide yes)
+			)
+		)
 		(pin "57"
 		)
@@
 			)
 		)
+		(property "MFG" "Diodes Incorporated"
+			(at 82.55 233.68 0)
+			(effects
+				(font
+					(size 1.27 1.27)
+				)
+				(hide yes)
+			)
+		)
+		(property "MFG PN" "AP3019AKTR-G1"
+			(at 82.55 233.68 0)
+			(effects
+				(font
+					(size 1.27 1.27)
+				)
+				(hide yes)
+			)
+		)
 		(pin "5"
 		)
@@
 			)
 		)
+		(property "MFG" "Sumida America Components Inc."
+			(at 64.77 220.98 90)
+			(effects
+				(font
+					(size 1.27 1.27)
+				)
+				(hide yes)
+			)
+		)
+		(property "MFG PN" "CDRH5D28NP-220NC"
+			(at 64.77 220.98 90)
+			(effects
+				(font
+					(size 1.27 1.27)
+				)
+				(hide yes)
+			)
+		)
 		(pin "2"
 		)
@@
 			)
 		)
-		(property "MFG PN" ""
+		(property "MFG PN" "RK73H2ETTD4R99F"
 			(at 100.33 247.65 0)
 			(effects
@@
 			)
 		)
-		(property "MFG" ""
+		(property "MFG" "KOA Speer Electronics, Inc."
 			(at 100.33 247.65 0)
 			(effects

Commit message: more whitespace fixes
more whitespace fixes
Parts:
- C11: Digikey Link https://www.digikey.com/en/products/detail/samsung-electro-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 -> (none); Digikey Part Number 1276-CL10A106KO8NQNCCT-ND -> (none); MFG  Samsung Electro-Mechanics -> (none); Manufacturer Part Number CL10A106KO8NQNC -> (none); Note Min 3.3u as per BT817Q datasheet -> (none)
- C16, C26: Name CL10B105KP8NNNC -> (none)
- L2: Digikey Link https://www.digikey.com/en/produchttps://www.digikey.com/en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 -> (none); Digikey Part Number 308-2307-1-ND -> (none); Manufacturer Part Number CDRH5D28NP-220NC -> (none); Name Sumida CDRH5D28NP-220NC -> (none)
Changed lines of the file:
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@@
-			)
-		)
-		(property "Digikey Part Number" "1276-CL10A106KO8NQNCCT-ND"
-			(at 152.4 76.2 0)
-			(effects
-				(font
-					(size 1.27 1.27)
-				)
-				(hide yes)
-			)
-		)
-		(property "MFG " "Samsung Electro-Mechanics"
-			(at 152.4 76.2 0)
-			(effects
-				(font
-					(size 1.27 1.27)
-				)
-				(hide yes)
-			)
-		)
-		(property "Digikey Link" "https://www.digikey.com/en/products/detail/samsung-electro-mechanics/CL10A106KO8NQNC/10479038"
-			(at 152.4 76.2 0)
-			(effects
-				(font
-					(size 1.27 1.27)
-				)
-				(hide yes)
-			)
-		)
-		(property "Manufacturer Part Number" "CL10A106KO8NQNC"
-			(at 152.4 76.2 0)
-			(effects
-				(font
-					(size 1.27 1.27)
-				)
-				(hide yes)
-			)
-		)
-		(property "Note" "Min 3.3u as per BT817Q datasheet "
-			(at 119.126 69.85 0)
-			(effects
-				(font
-					(size 1.27 1.27)
-				)
-				(justify left top)
-				(hide yes)
 			)
 		)
@@
 			)
 		)
-		(property "Digikey Part Number" ""
-			(at 124.46 97.79 0)
-			(effects
-				(font
-					(size 1.27 1.27)
-				)
-				(hide yes)
-			)
-		)
-		(property "Name" ""
-			(at 124.46 97.79 0)
-			(effects
-				(font
-					(size 1.27 1.27)
-				)
-				(hide yes)
-			)
-		)
-		(property "Digikey Link" ""
-			(at 124.46 97.79 0)
-			(effects
-				(font
-					(size 1.27 1.27)
-				)
-				(hide yes)
-			)
-		)
-		(property "Manufacturer Part Number" ""
-			(at 124.46 97.79 0)
-			(effects
-				(font
-					(size 1.27 1.27)
-				)
-				(hide yes)
-			)
-		)
 		(property "Digi PN" "2005-BT817Q-RCT-ND"
 			(at 124.46 97.79 0)
@@
 			)
 		)
-		(property "Digikey Part Number" "308-2307-1-ND"
-			(at 64.77 220.98 0)
-			(effects
-				(font
-					(size 1.27 1.27)
-				)
-				(hide yes)
-			)
-		)
-		(property "Name" "Sumida CDRH5D28NP-220NC"
-			(at 64.77 220.98 0)
-			(effects
-				(font
-					(size 1.27 1.27)
-				)
-				(hide yes)
-			)
-		)
-		(property "Digikey Link" "https://www.digikey.com/en/produchttps://www.digikey.com/en/products/detail/sumida-america-inc/CDRH5D28NP-220NC/4356377ts/detail/sumida-america-inc/CDRH5D28-220NC/611043"
-			(at 64.77 220.98 0)
-			(effects
-				(font
-					(size 1.27 1.27)
-				)
-				(hide yes)
-			)
-		)
-		(property "Manufacturer Part Number" "CDRH5D28NP-220NC"
-			(at 64.77 220.98 0)
-			(effects
-				(font
-					(size 1.27 1.27)
-				)
-				(hide yes)
-			)
-		)
 		(property "Digi PN" "308-2307-1-ND"
 			(at 64.77 220.98 90)
@@
 			)
 		)
-		(property "Name" "CL10B105KP8NNNC"
-			(at 87.63 213.36 0)
-			(effects
-				(font
-					(size 1.27 1.27)
-				)
-				(hide yes)
-			)
-		)
 		(property "Digi URL" "https://www.digikey.com/en/products/detail/yageo/CC0603KRX5R8BB105/2833610"
 			(at 87.63 213.36 0)
@@
 			(at 168.91 82.55 0)
 			(effects
-				(font
-					(size 1.27 1.27)
-				)
-				(hide yes)
-			)
-		)
-		(property "Name" "CL10B105KP8NNNC"
-			(at 168.91 82.55 0)
-			(effects

Commit message: connector steps
connector steps
Parts:
- J9: footprint Connector_FFC-FPC:Amphenol_F32Q-1A7x1-11040_1x40-1MP_P0.5mm_Horizontal -> FS_4_Global_Footprint_Library:CONN_F32D-1A7Y1-21040_AMP
Changed lines of the file:
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@@
 			)
 		)
-		(property "Footprint" "Connector_FFC-FPC:Amphenol_F32Q-1A7x1-11040_1x40-1MP_P0.5mm_Horizontal"
+		(property "Footprint" "FS_4_Global_Footprint_Library:CONN_F32D-1A7Y1-21040_AMP"
 			(at 339.09 130.81 0)
 			(effects

Commit message: fixes
fixes
Parts:
- removed U1: BT817Q, Package_DFN_QFN:VQFN-64-1EP_9x9mm_P0.5mm_EP7.15x7.15mm, symbol FS_4_Global_Symbol_Library:BT817Q
- added U5: BT817Q, Package_DFN_QFN:VQFN-64-1EP_9x9mm_P0.5mm_EP7.15x7.15mm, symbol FS_4_Global_Footprint_Library:BT817Q
Connections:
- net +1V2: now also U5.2 (VCC1V2), U5.25 (VOUT1V2), U5.57 (VCC1V2)
- net +3V3: now also U5.17 (VCCIO3), U5.24 (VCC), U5.28 (VCCIO2), U5.9 (VCCIO1)
- net GND: now also U5.23 (GND), U5.33 (GND), U5.48 (GND), U5.65 (GND)
- net LCD_Data_Enable: now also U5.35 (DE)
- net LCD_Display_Enable: now also U5.38 (DISP)
- net LCD_Dot_Clock: now also U5.39 (PCLK)
- net LCD_HSync: now also U5.37 (HSYNC)
- net LCD_VSync: now also U5.36 (VSYNC)
- net RGB_B0: now also U5.47 (B0)
- net RGB_B1: now also U5.46 (B1)
- net RGB_B2: now also U5.45 (B2)
- net RGB_B3: now also U5.44 (B3)
- net RGB_B4: now also U5.43 (B4)
- net RGB_B5: now also U5.42 (B5)
- net RGB_B6: now also U5.41 (B6)
- net RGB_B7: now also U5.40 (B7)
- net RGB_G0: now also U5.56 (G0)
- net RGB_G1: now also U5.55 (G1)
- net RGB_G2: now also U5.54 (G2)
- net RGB_G3: now also U5.53 (G3)
- net RGB_G4: now also U5.52 (G4)
- net RGB_G5: now also U5.51 (G5)
- net RGB_G6: now also U5.50 (G6)
- net RGB_G7: now also U5.49 (G7)
- net RGB_R0: now also U5.1 (R0)
- net RGB_R1: now also U5.64 (R1)
- net RGB_R2: now also U5.63 (R2)
- net RGB_R3: now also U5.62 (R3)
- net RGB_R4: now also U5.61 (R4)
- net RGB_R5: now also U5.60 (R5)
- net RGB_R6: now also U5.59 (R6)
- net RGB_R7: now also U5.58 (R7)
- net SPI.CLK: now also U5.3 (SCK)
- net SPI.CS: now also U5.6 (CS_N)
- net SPI.MISO: now also U5.4 (MISO)
- net SPI.MOSI: now also U5.5 (MOSI)
- net driver_power_pin: now also U5.12 (PD_N)
- net at U6.4 (CTRL): now also U5.34 (BACKLIGHT)
Changed lines of the file:
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@@
-	)
-	(symbol
-		(lib_id "FS_4_Global_Symbol_Library:BT817Q")
-		(at 124.46 97.79 0)
-		(unit 1)
-		(exclude_from_sim no)
-		(in_bom yes)
-		(on_board yes)
-		(dnp no)
-		(property "Reference" "U1"
-			(at 152.4 134.366 0)
-			(effects
-				(font
-					(size 1.27 1.27)
-				)
-				(justify left)
-			)
-		)
-		(property "Value" "BT817Q"
-			(at 152.4 136.906 0)
-			(effects
-				(font
-					(size 1.27 1.27)
-				)
-				(justify left)
-			)
-		)
-		(property "Footprint" "Package_DFN_QFN:VQFN-64-1EP_9x9mm_P0.5mm_EP7.15x7.15mm"
-			(at 124.46 97.79 0)
-			(effects
-				(font
-					(size 1.27 1.27)
-				)
-				(hide yes)
-			)
-		)
-		(property "Datasheet" "https://brtchip.com/wp-content/uploads/Support/Documentation/Datasheets/ICs/EVE/DS_BT817_8.pdf"
-			(at 124.46 97.79 0)
-			(effects
-				(font
-					(size 1.27 1.27)
-				)
-				(hide yes)
-			)
-		)
-		(property "Description" "Display Driver IC"
-			(at 124.46 97.79 0)
-			(effects
-				(font
-					(size 1.27 1.27)
-				)
-				(hide yes)
-			)
-		)
-		(property "Digi PN" "2005-BT817Q-RCT-ND"
-			(at 124.46 97.79 0)
-			(effects
-				(font
-					(size 1.27 1.27)
-				)
-				(hide yes)
-			)
-		)
-		(property "Digi URL" "https://www.digikey.com/en/products/detail/bridgetek-pte-ltd/BT817Q-R/13242741"
-			(at 124.46 97.79 0)
-			(effects
-				(font
-					(size 1.27 1.27)
-				)
-				(hide yes)
-			)
-		)
-		(property "MFG" "Bridgetek Pte Ltd."
-			(at 124.46 97.79 0)
-			(effects
-				(font
-					(size 1.27 1.27)
-				)
-				(hide yes)
-			)
-		)
-		(property "MFG PN" "BT817Q-R"
-			(at 124.46 97.79 0)
-			(effects
-				(font
-					(size 1.27 1.27)
-				)
-				(hide yes)
-			)
-		)
-		(pin "57"
-		)
-		(pin "11"
-		)
-		(pin "56"
-		)
-		(pin "39"
-		)
-		(pin "40"
-		)
-		(pin "33"
-		)
-		(pin "10"
-		)
-		(pin "32"
-		)
-		(pin "65"
-		)
-		(pin "2"
-		)
-		(pin "47"
-		)
-		(pin "58"
-		)
-		(pin "16"
-		)
-		(pin "24"
-		)
-		(pin "18"
-		)
-		(pin "64"
-		)
-		(pin "31"
-		)
-		(pin "48"
-		)
-		(pin "54"
-		)
-		(pin "17"
-		)
-		(pin "3"
-		)
-		(pin "51"
-		)
-		(pin "27"
-		)
-		(pin "44"
-		)
-		(pin "25"
-		)
-		(pin "30"
-		)
-		(pin "60"
-		)
-		(pin "13"
-		)
-		(pin "45"
-		)
-		(pin "50"
-		)
-		(pin "46"
-		)
-		(pin "7"
-		)
-		(pin "23"
-		)
-		(pin "1"
-		)
-		(pin "29"
-		)
-		(pin "34"
-		)
-		(pin "41"
-		)
-		(pin "37"
-		)
-		(pin "4"
-		)
-		(pin "8"
-		)
-		(pin "36"
-		)
-		(pin "28"
-		)
-		(pin "59"
-		)
-		(pin "22"
-		)
-		(pin "20"
-		)
-		(pin "6"
-		)
-		(pin "5"
-		)
-		(pin "63"
-		)
-		(pin "62"
-		)
-		(pin "61"
-		)
-		(pin "42"
-		)
-		(pin "26"
-		)
-		(pin "53"
-		)
-		(pin "55"
-		)
-		(pin "35"
-		)
-		(pin "52"
-		)
-		(pin "38"
-		)
-		(pin "21"
-		)
-		(pin "43"
-		)
-		(pin "14"
-		)
-		(pin "15"
-		)
-		(pin "19"
-		)
-		(pin "12"
-		)
-		(pin "49"
-		)
-		(pin "9"
-		)
-		(instances
-			(project "chargingboard"
-				(path "/3b7f9d0d-fe78-4ddc-a74a-12564d0be65c/1fb407b6-2fa5-4dbf-a434-4b5bd0ba4814"
-					(reference "U1")
-					(unit 1)
-				)
-			)
-		)
 	)
 	(symbol
@@
 					(unit 1)
 				)
+			)
+		)
+	)
+	(symbol
+		(lib_id "FS_4_Global_Footprint_Library:BT817Q")
+		(at 124.46 97.79 0)
+		(unit 1)
+		(exclude_from_sim no)
+		(in_bom yes)
+		(on_board yes)
+		(dnp no)
+		(fields_autoplaced yes)
+		(property "Reference" "U5"
+			(at 162.1633 185.42 0)
+			(effects
+				(font
+					(size 1.27 1.27)
+				)
+				(justify left)
+			)
+		)
+		(property "Value" "BT817Q"
+			(at 162.1633 187.96 0)
+			(effects
+				(font
+					(size 1.27 1.27)
+				)
+				(justify left)
+			)
+		)
+		(property "Footprint" "Package_DFN_QFN:VQFN-64-1EP_9x9mm_P0.5mm_EP7.15x7.15mm"
+			(at 124.46 97.79 0)
+			(effects
+				(font
+					(size 1.27 1.27)
+				)
+				(hide yes)
+			)
+		)
+		(property "Datasheet" "https://brtchip.com/wp-content/uploads/Support/Documentation/Datasheets/ICs/EVE/DS_BT817_8.pdf"
+			(at 124.46 97.79 0)
+			(effects
+				(font
+					(size 1.27 1.27)
+				)
+				(hide yes)
+			)
+		)
+		(property "Description" "Display Driver IC"
+			(at 124.46 97.79 0)
+			(effects
+				(font
+					(size 1.27 1.27)
+				)
+				(hide yes)
+			)
+		)
+		(property "Digi PN" "2005-BT817Q-RCT-ND"
+			(at 124.46 97.79 0)
+			(effects
+				(font
+					(size 1.27 1.27)
+				)
+				(hide yes)
+			)
+		)
+		(property "Digi URL" "https://www.digikey.com/en/products/detail/bridgetek-pte-ltd/BT817Q-R/13242741"
+			(at 124.46 97.79 0)
+			(effects
+				(font
+					(size 1.27 1.27)
+				)
+				(hide yes)
+			)
+		)
+		(property "MFG" "Bridgetek Pte Ltd."
+			(at 124.46 97.79 0)
+			(effects
+				(font
+					(size 1.27 1.27)
+				)
+				(hide yes)
+			)
+		)
+		(property "MFG PN" "BT817Q-R"
+			(at 124.46 97.79 0)
+			(effects
+				(font
+					(size 1.27 1.27)
+				)
+				(hide yes)
+			)
+		)
+		(pin "35"
+		)
+		(pin "34"
+		)
+		(pin "11"
+		)
+		(pin "7"
+		)
+		(pin "39"
+		)
+		(pin "38"
+		)
+		(pin "37"
+		)
+		(pin "36"
+		)
+		(pin "32"
+		)
+		(pin "45"
+		)
+		(pin "44"
+		)
+		(pin "15"
+		)
+		(pin "48"
+		)
+		(pin "47"
+		)
+		(pin "46"
+		)
+		(pin "25"
+		)
+		(pin "41"
+		)
+		(pin "40"
+		)
+		(pin "43"
+		)
+		(pin "42"
+		)
+		(pin "28"
+		)
+		(pin "22"
+		)
+		(pin "26"
+		)
+		(pin "8"
+		)
+		(pin "30"
+		)
+		(pin "18"
+		)
+		(pin "13"
+		)
+		(pin "10"
+		)
+		(pin "29"
+		)
+		(pin "27"
+		)
+		(pin "16"
+		)
+		(pin "62"
+		)
+		(pin "1"
+		)
+		(pin "64"
+		)
+		(pin "65"
+		)
+		(pin "17"
+		)
+		(pin "24"
+		)
+		(pin "3"
+		)
+		(pin "63"
+		)
+		(pin "12"
+		)
+		(pin "6"
+		)
+		(pin "52"
+		)
+		(pin "51"
+		)
+		(pin "4"
+		)
+		(pin "20"
+		)
+		(pin "9"
+		)
+		(pin "55"
+		)
+		(pin "54"
+		)
+		(pin "53"
+		)
+		(pin "19"
+		)
+		(pin "50"
+		)
+		(pin "49"
+		)
+		(pin "31"
+		)
+		(pin "61"
+		)
+		(pin "60"
+		)
+		(pin "59"
+		)
+		(pin "58"
+		)
+		(pin "56"
+		)
+		(pin "33"
+		)
+		(pin "14"
+		)
+		(pin "57"
+		)
+		(pin "21"
+		)
+		(pin "2"
+		)
+		(pin "23"
+		)
+		(pin "5"
+		)
+		(instances
+			(project ""
+				(path "/3b7f9d0d-fe78-4ddc-a74a-12564d0be65c/1fb407b6-2fa5-4dbf-a434-4b5bd0ba4814"
+					(reference "U5")
+					(unit 1)
+				)

Commit message: changed 0603
changed 0603
Parts:
- C10, C11, C14, C15, C16, C26, C29, C5, C8, C9: footprint Capacitor_SMD:C_0603_1608Metric -> Capacitor_SMD:C_0603_1608Metric_Pad1.08x0.95mm_HandSolder
- R2: footprint Resistor_SMD:R_1210_3225Metric -> Resistor_SMD:R_1210_3225Metric_Pad1.30x2.65mm_HandSolder
Changed lines of the file:
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@@
 			)
 		)
-		(property "Footprint" "Capacitor_SMD:C_0603_1608Metric"
+		(property "Footprint" "Capacitor_SMD:C_0603_1608Metric_Pad1.08x0.95mm_HandSolder"
 			(at 153.3652 80.01 0)
 			(effects
@@
 			)
 		)
-		(property "Footprint" "Capacitor_SMD:C_0603_1608Metric"
+		(property "Footprint" "Capacitor_SMD:C_0603_1608Metric_Pad1.08x0.95mm_HandSolder"
 			(at 111.4552 82.55 0)
 			(effects
@@
 			)
 		)
-		(property "Footprint" "Capacitor_SMD:C_0603_1608Metric"
+		(property "Footprint" "Capacitor_SMD:C_0603_1608Metric_Pad1.08x0.95mm_HandSolder"
 			(at 107.6452 227.33 0)
 			(effects
@@
 			)
 		)
-		(property "Footprint" "Capacitor_SMD:C_0603_1608Metric"
+		(property "Footprint" "Capacitor_SMD:C_0603_1608Metric_Pad1.08x0.95mm_HandSolder"
 			(at 96.2152 83.82 0)
 			(effects
@@
 			)
 		)
-		(property "Footprint" "Capacitor_SMD:C_0603_1608Metric"
+		(property "Footprint" "Capacitor_SMD:C_0603_1608Metric_Pad1.08x0.95mm_HandSolder"
 			(at 138.1252 82.55 0)
 			(effects
@@
 			)
 		)
-		(property "Footprint" "Capacitor_SMD:C_0603_1608Metric"
+		(property "Footprint" "Capacitor_SMD:C_0603_1608Metric_Pad1.08x0.95mm_HandSolder"
 			(at 86.6648 217.17 0)
 			(effects
@@
 			)
 		)
-		(property "Footprint" "Capacitor_SMD:C_0603_1608Metric"
+		(property "Footprint" "Capacitor_SMD:C_0603_1608Metric_Pad1.08x0.95mm_HandSolder"
 			(at 125.4252 81.28 0)
 			(effects
@@
 			)
 		)
-		(property "Footprint" "Capacitor_SMD:C_0603_1608Metric"
+		(property "Footprint" "Capacitor_SMD:C_0603_1608Metric_Pad1.08x0.95mm_HandSolder"
 			(at 183.8452 85.09 0)
 			(effects
@@
 			)
 		)
-		(property "Footprint" "Capacitor_SMD:C_0603_1608Metric"
+		(property "Footprint" "Capacitor_SMD:C_0603_1608Metric_Pad1.08x0.95mm_HandSolder"
 			(at 167.9448 86.36 0)
 			(effects
@@
 			)
 		)
-		(property "Footprint" "Capacitor_SMD:C_0603_1608Metric"
+		(property "Footprint" "Capacitor_SMD:C_0603_1608Metric_Pad1.08x0.95mm_HandSolder"
 			(at 169.8752 73.66 0)
 			(effects
@@
 			)
 		)
-		(property "Footprint" "Resistor_SMD:R_1210_3225Metric"
+		(property "Footprint" "Resistor_SMD:R_1210_3225Metric_Pad1.30x2.65mm_HandSolder"
 			(at 98.552 247.65 90)
 			(effects
