File: chargingboard/chargingboard.kicad_pcb (KiCad board)
At the start: 2 copper layers, 51 x 94.6 mm, 61 parts, among them J1 Acc SFC, J10 Screen Button, J11 GLVshieldingground, J2 12V Power supply, J3 CAN COTS Charger, J4 Shutdown Button, J5 Reset Button, J6 TSMP to HV, J7 TSMP to Banana Jacks, J8 J1772 Negotiation, J9 Conn_01x40_MountingPin, SW1 Y97KT23B5NAFP, U1 BT817Q, U2 ISO1044BD, U3 STM32G441KBTx, U4 AP63205WU, U6 AP3019AKTR, U7 MIC5504-3.3YM5, Y1 ECS-240-8-37B-CKY-TR

Commit message: new conn
new conn
Parts:
- added C31: 10uF, Capacitor_SMD:C_0603_1608Metric_Pad1.08x0.95mm_HandSolder, F.Cu at (264.1, 34.5)
- added C32: 100nF, Capacitor_SMD:C_0603_1608Metric_Pad1.08x0.95mm_HandSolder, F.Cu at (264.1, 37.0)
- added C33: 100nF, Capacitor_SMD:C_0603_1608Metric_Pad1.08x0.95mm_HandSolder, F.Cu at (264.1, 39.5)
- added C34: 1uF, Capacitor_SMD:C_0603_1608Metric_Pad1.08x0.95mm_HandSolder, F.Cu at (264.1, 42.0)
- added C35: 100nF, Capacitor_SMD:C_0603_1608Metric_Pad1.08x0.95mm_HandSolder, F.Cu at (264.1, 44.5)
- added FB2: FCM 1608KF-601T03, Inductor_SMD:L_0603_1608Metric_Pad1.05x0.95mm_HandSolder, F.Cu at (264.1, 47.0)
- added J13: FTSH-107-01-F-DV-K-P-TR, Connector_PinHeader_1.27mm:PinHeader_2x07_P1.27mm_Vertical_SMD, F.Cu at (239.2, 55.9)
- C10, C14, C15, C5, C8, C9: value 100n -> 100nF
- C11: value 10u -> 10uF
- C16, C17, C26: value 1u -> 1uF
- C29: value 220n -> 220nF
- J1: value Acc SFC -> Conn_02x13_Counter_Clockwise; footprint Connector_Dsub:DSUB-15-HD_Socket_Horizontal_P2.29x1.90mm_EdgePinOffset3.03mm_Housed_MountingHolesOffset4.94mm -> FS_4_Global_Footprint_Library:ATS15-26PB-BM01
- moved J1 11.2 mm to (183.5, 53.0), turned to 0 degrees
Connections:
- net Backlight_PWM renamed Net-(U1-BACKLIGHT)
- C10 pad 1: +3.3VA -> +3V3
- C5 pad 1: +3.3VA -> +3V3
- C8 pad 1: +3.3VA -> +3V3
- U1 pad 17: +3.3VA -> +3V3
- U3 pad 1: +3.3VA -> +3V3

Commit message: rerequest
rerequest
Parts:
- added TP1: TestPoint, TestPoint:TestPoint_Pad_D1.0mm, F.Cu at (226.6, 78.2)
- added TP2: TestPoint, TestPoint:TestPoint_Pad_D1.0mm, F.Cu at (226.6, 81.2)
- added TP3: TestPoint, TestPoint:TestPoint_Pad_D1.0mm, F.Cu at (226.6, 84.3)
- added TP4: TestPoint, TestPoint:TestPoint_Pad_D1.0mm, F.Cu at (226.6, 87.3)
- added TP5: TestPoint, TestPoint:TestPoint_Pad_D1.0mm, F.Cu at (229.7, 78.2)
- added TP6: TestPoint, TestPoint:TestPoint_Pad_D1.0mm, F.Cu at (229.7, 81.2)
- added TP7: TestPoint, TestPoint:TestPoint_Pad_D1.0mm, F.Cu at (229.7, 84.3)
- L2: value 22u -> 22uF
- moved C31 27.1 mm to (245.4, 54.0)
- moved C32 27.1 mm to (245.4, 56.5)
- moved C33 27.1 mm to (245.4, 59.0)
- moved C34 27.1 mm to (245.4, 61.5)
- moved C35 27.1 mm to (245.4, 64.0)
- moved FB2 27.1 mm to (245.4, 66.5)
- moved U6 16.7 mm to (172.5, 73.5)
- moved J13 8.28 mm to (231.1, 54.5)
- moved U3 8.03 mm to (181.8, 61.3)
- moved U1 7.19 mm to (177.9, 80.8)
- moved R2 6.13 mm to (172.5, 69.0)
- moved SW1 4.12 mm to (203.0, 80.5)
- moved J9 0.71 mm to (166.1, 81.2)
Connections:
- U3 pad 13: unconnected-(U3-PB0-Pad13) -> Net-(U3-PB0)
- U3 pad 18: unconnected-(U3-PA8-Pad18) -> Net-(U3-PA8)
- U3 pad 20: unconnected-(U3-PA10-Pad20) -> Net-(U3-PA10)
- U3 pad 25: unconnected-(U3-PA15-Pad25) -> Net-(U3-PA15)
- U3 pad 27: unconnected-(U3-PB4-Pad27) -> Net-(U3-PB4)
- U3 pad 28: unconnected-(U3-PB5-Pad28) -> Net-(U3-PB5)
- U3 pad 29: unconnected-(U3-PB6-Pad29) -> Net-(U3-PB6)
Routing:
- net /Shutdown_Reset: track 61.6 -> 36.2 mm
- net /SH_RESET+: track 63.8 -> 40.7 mm
- net +12V: track 38.1 -> 16.2 mm
- net unconnected-(J1-Pin_16-Pad16): track 0.00 -> 0.79 mm
- net Net-(U4-SW): track 9.21 -> 9.98 mm
Other:
- board text added: "${TITLE} ${REVISION} ${COMPANY} FS-4 Charigng Board Designed by Mihir Bhagatwala Amber Huang Atul Pethe Mathis Delombaerde Teddy Li"
- board text removed: "${TITLE} ${REVISION} ${COMPANY} FS-4 Designed by Mihir Bhagatwala Amber Huang Atul Pethe Mathis Delombaerde Teddy Li"

Commit message: connector steps
connector steps
Parts:
- FB2: value FCM 1608KF-601T03 -> FCM_1608KF-601T03
- J10: value Screen Button -> Screen_Button
- J2: value 12V Power supply -> 12V_Power_supply
- J3: value CAN COTS Charger -> CAN_COTS_Charger
- J4: value Shutdown Button -> Shutdown_Button
- J5: value Reset Button -> Reset_Button
- J6: value TSMP to HV -> TSMP_to_HV
- J7: value TSMP to Banana Jacks -> TSMP_to_Banana Jacks
- J8: value J1772 Negotiation -> J1772_Negotiation
- J9: footprint Connector_FFC-FPC:Amphenol_F32Q-1A7x1-11040_1x40-1MP_P0.5mm_Horizontal -> FS_4_Global_Footprint_Library:CONN_F32D-1A7Y1-21040_AMP
- moved L2 63.8 mm to (179.0, 92.0)
- moved R3 61.2 mm to (204.5, 70.0), turned to 90 degrees
- moved C26 58.1 mm to (197.8, 64.0), turned to 0 degrees
- moved C34 57.9 mm to (191.0, 81.5)
- moved C31 57.9 mm to (191.0, 74.0)
- moved C32 57.9 mm to (191.0, 76.5)
- moved C33 57.9 mm to (191.0, 79.0)
- moved C35 57.9 mm to (191.0, 84.0)
- moved FB2 57.9 mm to (191.0, 86.5)
- moved C5 57.4 mm to (201.5, 69.0), turned to 180 degrees
- moved C8 54.7 mm to (201.5, 66.5), turned to 180 degrees
- moved C14 54.1 mm to (197.5, 69.0), turned to 180 degrees
- moved C10 53.8 mm to (193.8, 64.0), turned to 0 degrees
- moved J13 44.8 mm to (186.4, 58.7)
- moved TP1 42.3 mm to (184.5, 74.0)
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Routing:
- net Net-(U4-SW): track 9.98 -> 0.78 mm
- net +12V: track 16.2 -> 8.61 mm
- net Net-(U4-BST): track 3.24 -> 0.05 mm

Commit message: step file with connectors
step file with connectors
Parts:
- U7: moved to B.Cu
- moved L2 5.50 mm to (184.5, 92.0)
- moved U1 1.20 mm to (176.8, 80.9)
- moved U3 1.05 mm to (176.5, 59.0)
- turned U7 to 0 degrees

Commit message: fixed step
fixed step
Parts:
- moved REF** 1.50 mm to (210.0, 127.5)
- moved U3 0.68 mm to (176.2, 59.6)
- moved REF** 0.50 mm to (167.0, 41.0)
- moved REF** 0.50 mm to (167.0, 127.5)

Commit message: fixes
fixes
Parts:
- removed U4: AP63205WU, Package_TO_SOT_SMD:TSOT-23-6
- added U5: BT817Q, Package_DFN_QFN:VQFN-64-1EP_9x9mm_P0.5mm_EP7.15x7.15mm, F.Cu at (176.9, 82.2)
- U1: value BT817Q -> AP63205WU; footprint Package_DFN_QFN:VQFN-64-1EP_9x9mm_P0.5mm_EP7.15x7.15mm -> Package_TO_SOT_SMD:TSOT-23-6
- U7: moved to F.Cu
- moved U1 38.8 mm to (203.6, 53.0)
- moved Y1 16.0 mm to (195.2, 85.5), turned to 0 degrees
- moved U7 6.02 mm to (204.1, 45.0)
- moved SW1 2.60 mm to (203.1, 77.9)
- moved U2 2.06 mm to (200.0, 59.4)
Connections:
- net /IRs_Final renamed /Shutdown_Acc_Out
- C13 pad 1: Net-(U4-SW) -> Net-(U1-SW)
- C13 pad 2: Net-(U4-BST) -> Net-(U1-BST)
- C2 pad 2: Net-(C2-Pad2) -> GND
- C3 pad 2: Net-(C2-Pad2) -> GND
- C4 pad 1: Net-(C4-Pad1) -> GND
- L1 pad 1: Net-(U4-SW) -> Net-(U1-SW)
- SW1 pad 1: Net-(C4-Pad1) -> GND
- U1 pad 1: /screen_architecture/RGB_R0 -> +5V
- U1 pad 2: +1V2 -> +12V
- U1 pad 3: /SPI.CLK -> +12V
- U1 pad 4: /SPI.MISO -> GND
- U1 pad 5: /SPI.MOSI -> Net-(U1-SW)
- U1 pad 6: /SPI.CS -> Net-(U1-BST)
- U3 pad 15: +3V3 -> +3V3_A
- U6 pad 4: Net-(U1-BACKLIGHT) -> Net-(U5-BACKLIGHT)
- Y1 pad 2: Net-(C2-Pad2) -> GND
Routing:
- net /SH_RESET+: track 40.7 -> 0.00 mm
- net /Shutdown_Reset: track 36.2 -> 0.00 mm
- net +5V: track 15.3 -> 1.96 mm
- net +12V: track 8.61 -> 0.67 mm
- net /CAN_H: track 0.00 -> 6.82 mm
- net /CAN_L: track 3.68 -> 6.82 mm

Commit message: board update
board update
Parts:
- C1, C12, C13, C23, C24: footprint Capacitor_SMD:C_0805_2012Metric_Pad1.18x1.45mm_HandSolder -> Capacitor_SMD:C_0603_1608Metric_Pad1.08x0.95mm_HandSolder
- C10, C11, C14, C15, C16, C17, C26, C29, C5, C8, C9: footprint Capacitor_SMD:C_0603_1608Metric -> Capacitor_SMD:C_0603_1608Metric_Pad1.08x0.95mm_HandSolder
- R10, R11, R12, R13, R3, R7, R8, R9: footprint Resistor_SMD:R_0805_2012Metric_Pad1.20x1.40mm_HandSolder -> Resistor_SMD:R_0603_1608Metric_Pad0.98x0.95mm_HandSolder
- R2: footprint Resistor_SMD:R_1210_3225Metric -> Resistor_SMD:R_1210_3225Metric_Pad1.30x2.65mm_HandSolder
Routing:
- net Net-(U4-SW): track 0.78 -> 0.00 mm
- net (no net): track 0.00 -> 0.78 mm

Commit message: more fixes
more fixes
Parts:
- C6, C7: footprint Capacitor_SMD:C_0805_2012Metric_Pad1.18x1.45mm_HandSolder -> Capacitor_SMD:C_0603_1608Metric_Pad1.08x0.95mm_HandSolder
- moved R2 108.7 mm to (281.1, 67.1)
- moved U3 103.7 mm to (277.8, 79.9)
- moved C6 101.7 mm to (272.3, 129.6)
- moved C7 100.6 mm to (272.3, 132.1)
- moved U2 93.3 mm to (266.3, 125.1)
- moved C11 90.8 mm to (266.1, 29.2)
- moved TP1 90.8 mm to (265.6, 33.2)
- moved TP2 90.8 mm to (265.6, 36.2)
- moved TP5 90.8 mm to (268.7, 33.2)
- moved TP6 90.8 mm to (268.7, 36.2)
- moved TP3 90.8 mm to (265.6, 39.3)
- moved TP4 90.8 mm to (265.6, 42.3)
- moved TP7 90.8 mm to (268.7, 39.3)
- moved C14 84.3 mm to (273.6, 105.3)
- moved C2 84.3 mm to (271.1, 108.8)
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Connections:
- J1 pad 1: +12V -> unconnected-(J1-Pin_1-Pad1)
- J1 pad 19: unconnected-(J1-Pin_19-Pad19) -> GND
- J1 pad 26: unconnected-(J1-Pin_26-Pad26) -> +12V
- J1 pad 6: GND -> unconnected-(J1-Pin_6-Pad6)
Routing:
- net +12V: track 0.67 -> 36.8 mm
- net +5V: track 1.96 -> 19.0 mm
- net GND: track 0.00 -> 8.20 mm
- net Net-(U1-SW): track 0.00 -> 7.43 mm, vias 0 -> 2
- net /Control_Pilot_Filtered: track 0.00 -> 3.98 mm
- net Net-(J10-Pin_2): track 0.00 -> 3.25 mm
- net /Shutdown_Acc_Out: track 0.00 -> 3.00 mm
- net /Proximity_Pilot_Filtered: track 5.33 -> 2.76 mm
- net Net-(U1-BST): track 0.00 -> 2.53 mm
- net +3V3: track 0.00 -> 2.11 mm
- net screen_button: track 0.00 -> 2.06 mm
- net /Control_Pilot_Cutoff: track 6.67 -> 5.84 mm
- net unconnected-(J1-Pin_16-Pad16): track 0.79 -> 0.00 mm
- net (no net): track 0.78 -> 0.00 mm
