File: Power Electronics Board/Power Electronics Board.kicad_pcb (KiCad board)
At the start: 2 copper layers, 109.2 x 94 mm, 71 parts, among them J1 42820-2223, J2 42820-2223, J3 1054301103, J4 1054301103, J5 1054301103, J6 42820-2223, J7 1054301108, K2 AZ2150-1A-12DEF, K3 EW60-1A3-CL12D04,00000, K4 DS1E-ML-DC12V, Q1 AO3400A, Q2 AO3400A, Q3 DMG2301L, U1 MCP6004, U2 LM4040D30QDBZR, U3 MCP1703AT-5002E/CB, U4 CC1R5-1205SR-E, U5 ISOM8111DFSR, U6 MCP6004, U7 LM555xM, U8 SZNUD3124LT1G

Commit message: Updated DRC and traces to meet 2oz copper rules
Parts:
- moved R18 0.89 mm to (169.7, 104.6)
- moved C8 0.38 mm to (169.2, 108.5)
- turned D3 to 180 degrees
Routing:
- net +12V_BAT: track 117.7 -> 122.9 mm
- net +12V_Switched: track 50.7 -> 45.6 mm, vias 0 -> 2
- net TS-: track 86.9 -> 82.8 mm
- net +5V_Isolated: track 51.0 -> 47.5 mm, vias 2 -> 4
- net GND: track 5.38 -> 2.18 mm, vias 21 -> 22
- net Net-(C5-Pad1): track 22.5 -> 19.6 mm
- net +5V_LV: track 44.8 -> 42.8 mm, vias 4 -> 2
- net Net-(J3-Pin_1): track 9.06 -> 7.32 mm
- net Reset_Button_In: track 61.7 -> 60.1 mm
- net TS_Ready: track 43.0 -> 41.6 mm
- net Net-(C6-Pad1): track 15.8 -> 14.7 mm
- net Net-(U7-R): track 37.2 -> 36.1 mm
- net Net-(J3-Pin_3): track 8.85 -> 7.83 mm
- net Net-(J4-Pin_1): track 22.1 -> 21.2 mm
- net Net-(U7-Q): track 37.6 -> 36.7 mm
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
Commit message: Rev 2.0
Added Potentiometer to non inverting pin for LV battery op amp
changed 24.9k resistor to something more standard
Updated both schematic and layout
Parts:
- removed U2: LM4040D30QDBZR, Package_TO_SOT_SMD:SOT-23_Handsoldering
- added RV1: 10K, FS_4_Global_Footprint_Library:TRIM_PV36W103C01B00, F.Cu at (162.8, 115.6)
- R1: value 24.9k -> 39k
- R3: value 100k -> 20k
- TP6: value 3.4V @ 12V ~ 3V @ 10.47V -> 2.45V @ 12V ~ 2.04V @ 10V
- moved R3 18.0 mm to (168.7, 116.5), turned to 90 degrees
- moved R17 0.18 mm to (171.2, 114.6)
- moved Q1 0.12 mm to (173.2, 111.5)
Connections:
- R3 pad 1: +12V_BAT -> Net-(R3-Pad1)
- R3 pad 2: Net-(U1A--) -> GND
Routing:
- net +5V_LV: track 42.8 -> 55.3 mm, vias 2 -> 4
- net +12V_BAT: track 122.9 -> 115.4 mm
- net Net-(U1A--): track 22.9 -> 15.7 mm, vias 4 -> 2
- net Net-(R3-Pad1): track 0.00 -> 4.14 mm

Commit message: Rev 2.1
For some reason on my end my changes werent there, so im not sure if my changes are on github either, so i redid them and am pushing it back onto git
Parts:
- R3: footprint Resistor_SMD:R_0603_1608Metric_Pad0.98x0.95mm_HandSolder -> Resistor_SMD:R_0603_1608Metric
- TP6: value 2.45V @ 12V ~ 2.04V @ 10V -> 3.4V @ 12V ~ 3V @ 10.47V
- moved J4 1.52 mm to (136.1, 66.0)
- moved H3 0.51 mm to (185.9, 63.0)
- moved H4 0.51 mm to (84.3, 63.0)
- moved RV1 0.36 mm to (162.6, 115.3)
- moved R3 0.15 mm to (168.7, 116.3)
Routing:
- net Net-(J4-Pin_3): track 29.3 -> 27.8 mm
- net Net-(J4-Pin_1): track 21.2 -> 21.7 mm
Other:
- board size 109.2 x 94 mm -> 109.2 x 93 mm

Commit message: Rev 2.1.1
just sum light trace edits nun much
Parts:
- moved TP10 9.04 mm to (140.2, 99.1)
- moved U8 0.76 mm to (142.5, 102.1)
Routing:
- net TS_Ready: track 41.6 -> 45.4 mm, vias 4 -> 2
Changed lines of the file:
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@@
 	(footprint "Package_TO_SOT_SMD:TSOT-23_HandSoldering"
 		(layer "F.Cu")
-		(at 142.494 101.346 180)
+		(at 142.494 102.108 180)
 		(descr "5-pin TSOT23 package, http://cds.linear.com/docs/en/packaging/SOT_5_05-08-1635.pdf")
 		(tags "TSOT-23 Hand-soldering")
 		(property "Reference" "U8"
-			(at 2.032 2.286 180)
+			(at 2.286 -2.54 180)
 			(layer "F.SilkS")
 			(effects
@@
 	(footprint "TestPoint:TestPoint_Pad_1.0x1.0mm"
 		(layer "F.Cu")
-		(at 145.796 106.172)
+		(at 140.208 99.06)
 		(descr "SMD rectangular pad as test Point, square 1.0mm side length")
 		(tags "test point SMD pad rectangle square")
 		(property "Reference" "TP10"
-			(at 3.048 0 0)
+			(at 3.048 0.508 0)
 			(layer "F.SilkS")
 			(effects
@@
 	)
 	(segment
-		(start 145.796 106.172)
-		(end 145.796 105.156)
+		(start 144.204 103.058)
+		(end 141.732 100.586)
 		(width 0.254)
 		(layer "F.Cu")
@@
 	)
 	(segment
-		(start 145.796 103.632)
-		(end 153.924 103.632)
+		(start 144.204 103.058)
+		(end 143.697 103.058)
+		(width 0.254)
+		(layer "F.Cu")
+		(net 22)
+	)
+	(segment
+		(start 146.304 103.632)
+		(end 145.796 103.124)
+		(width 0.254)
+		(layer "F.Cu")
+		(net 22)
+	)
+	(segment
+		(start 153.924 103.632)
+		(end 146.304 103.632)
 		(width 0.254)
 		(layer "F.Cu")
@@
 	)
 	(segment
-		(start 144.204 102.296)
-		(end 145.54 103.632)
+		(start 141.224 99.06)
+		(end 140.208 99.06)
 		(width 0.254)
 		(layer "F.Cu")
@@
 	)
 	(segment
-		(start 145.54 103.632)
-		(end 145.796 103.632)
+		(start 141.732 100.586)
+		(end 141.732 99.568)
 		(width 0.254)
 		(layer "F.Cu")
 		(net 22)
 	)
-	(via
-		(at 145.796 105.156)
-		(size 0.508)
-		(drill 0.254)
-		(layers "F.Cu" "B.Cu")
+	(segment
+		(start 141.732 99.568)
+		(end 141.224 99.06)
+		(width 0.254)
+		(layer "F.Cu")
 		(net 22)
 	)
-	(via
-		(at 145.796 103.632)
-		(size 0.508)
-		(drill 0.254)
-		(layers "F.Cu" "B.Cu")
+	(segment
+		(start 145.796 103.124)
+		(end 144.272 103.124)
+		(width 0.254)
+		(layer "F.Cu")
 		(net 22)
 	)
@@
 	)
 	(segment
-		(start 145.796 105.156)
-		(end 145.796 103.632)
-		(width 0.254)
-		(layer "B.Cu")
-		(net 22)
-	)
-	(segment
 		(start 178.816 110.236)
 		(end 177.8 110.236)
@@
 	)
 	(segment
-		(start 135.636 101.346)
-		(end 140.784 101.346)
+		(start 120.904 105.156)
+		(end 118.872 107.188)
 		(width 0.254)
 		(layer "F.Cu")
@@
 	)
 	(segment
-		(start 120.904 105.156)
-		(end 118.872 107.188)
+		(start 133.35 103.632)
+		(end 134.874 102.108)
 		(width 0.254)
 		(layer "F.Cu")
@@
 	)
 	(segment
-		(start 133.35 103.632)
-		(end 135.636 101.346)
+		(start 134.874 102.108)
+		(end 140.784 102.108)
 		(width 0.254)
 		(layer "F.Cu")

Commit message: Rev 2.2
Finished Rev 2 layout, mostly worried about HV side. Need to add more silk screen comments for connectors
Parts:
- removed H4: MountingHole, MountingHole:MountingHole_3.2mm_M3
- removed TP13: GND, TestPoint:TestPoint_Pad_1.0x1.0mm
- added H5: MountingHole_Pad, MountingHole:MountingHole_3.2mm_M3_Pad, F.Cu at (108.7, 80.8)
- J1, J2, J6: value 42820-2223 -> Conn_01x02; footprint FS_4_Global_Footprint_Library:CONN_SDA-42820-0002_02_RC_MOL (42820-2223) -> Connector_Molex:Molex_Mini-Fit_Sr_42819-22XX_1x02_P10.00mm_Vertical
- J4: footprint FS_4_Global_Footprint_Library:1054301103 -> FS_4_Global_Footprint_Library:CONN_SD-105431-001_03_MOL
- J7: footprint FS_4_Global_Footprint_Library:CONN_SD-105430-001_08_MOL -> FS_4_Global_Footprint_Library:Molex-Nano-Fit_2x04_SMD_Vertical
- moved H1 132.1 mm to (53.8, 144.8)
- moved J3 122.0 mm to (192.1, 134.1), turned to 90 degrees
- moved TP8 115.9 mm to (61.5, 146.3)
- moved F4 110.3 mm to (182.4, 138.2), turned to 180 degrees
- moved TP6 105.5 mm to (61.5, 143.8)
- moved F3 102.0 mm to (182.4, 131.1), turned to 0 degrees
- moved R11 101.8 mm to (66.5, 145.3), turned to 90 degrees
- moved R5 101.2 mm to (177.4, 137.2), turned to 0 degrees
- moved R7 99.2 mm to (184.0, 125.5), turned to 180 degrees
- moved R1 99.0 mm to (66.5, 141.7), turned to -90 degrees
- moved R3 96.0 mm to (75.7, 140.2), turned to 0 degrees
- moved R6 95.5 mm to (175.3, 135.1), turned to 0 degrees
- moved TP11 95.0 mm to (88.9, 146.8)
- moved RV1 94.5 mm to (72.6, 144.3)
- moved R2 93.6 mm to (177.4, 131.1), turned to 180 degrees
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Connections:
- J7 pad 8: unconnected-(J7-Pin_8-Pad8) -> GND
- U4 pad 2: unconnected-(U4-On/~{Off}-Pad2) -> GND
Routing:
- net Net-(J5-Pin_3): track 6.46 -> 68.3 mm, vias 0 -> 1
- net Net-(J5-Pin_1): track 17.0 -> 65.6 mm, vias 0 -> 1
- net Net-(D2-K): track 65.3 -> 21.8 mm, vias 4 -> 0
- net +12V_BAT: track 115.4 -> 74.6 mm, vias 3 -> 2
- net +5V_LV: track 55.8 -> 85.1 mm, vias 4 -> 6
- net Shutdown_Final: track 53.4 -> 24.3 mm
- net Reset_Button_In: track 60.1 -> 33.8 mm
- net TS_Ready: track 45.4 -> 21.5 mm, vias 2 -> 0
- net Net-(U7-R): track 36.1 -> 16.0 mm, vias 4 -> 3
- net Net-(U7-Q): track 36.7 -> 18.4 mm
- net Net-(J4-Pin_3): track 27.8 -> 11.9 mm, vias 1 -> 0
- net Net-(J4-Pin_1): track 21.7 -> 36.2 mm
- net Net-(U7-THR): track 20.0 -> 9.38 mm
- net Net-(U1A-+): track 17.5 -> 27.4 mm, vias 0 -> 2
- net +5V_Isolated: track 47.5 -> 38.2 mm
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- removed copper zone on F.Cu, net +5V_LV
Other:
- board size 109.2 x 93 mm -> 149.4 x 71.1 mm
- board text removed: "Discharge"
- board text removed: "GLVMS"
- board text removed: "HV"
- board text removed: "LV"
- board text removed: "LV Input Outputs"
- board text removed: "TSMPS"

Commit message: Rev 2.3
Updated schematic's comments, added labels for connectors
Parts:
- J3: value 1054301103 -> 1054301102; footprint FS_4_Global_Footprint_Library:1054301103 -> FS_4_Global_Footprint_Library:CONN_SD-105430-001_02_MOL
- J4: value 1054301103 -> 1054301102; footprint FS_4_Global_Footprint_Library:CONN_SD-105431-001_03_MOL -> FS_4_Global_Footprint_Library:CONN_SD-105430-001_02_MOL
- J5: value 1054301103 -> 1054311102; footprint FS_4_Global_Footprint_Library:1054301103 -> FS_4_Global_Footprint_Library:CONN_SD-105431-001_02_MOL
- moved G*** 166.1 mm to (64.9, 80.8)
- moved J5 48.8 mm to (143.2, 117.9), turned to 0 degrees
- moved J4 13.9 mm to (167.6, 117.3), turned to 90 degrees
- moved H3 12.2 mm to (182.9, 144.8)
- moved R13 11.9 mm to (144.2, 130.0)
- moved J3 11.8 mm to (180.3, 134.7)
- moved C6 11.7 mm to (149.3, 136.2)
- moved F3 11.7 mm to (170.7, 131.2)
- moved F4 11.7 mm to (170.7, 138.3)
- moved R14 11.7 mm to (144.7, 134.6)
- moved R2 11.7 mm to (165.6, 131.2)
- moved R4 11.7 mm to (149.9, 143.9)
- moved R5 11.7 mm to (165.6, 137.2)
- moved R7 11.7 mm to (172.3, 125.6)
- moved TP12 11.7 mm to (145.7, 136.8)
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Connections:
- F4 pad 1: Net-(J3-Pin_3) -> Net-(J3-Pin_2)
- J3 pad 2: unconnected-(J3-Pin_2-Pad2) -> Net-(J3-Pin_2)
- J4 pad 2: unconnected-(J4-Pin_2-Pad2) -> Net-(J4-Pin_2)
- J5 pad 2: unconnected-(J5-Pin_2-Pad2) -> Net-(J5-Pin_2)
- K4 pad 10: Net-(J5-Pin_1) -> Net-(J4-Pin_1)
- K4 pad 7: Net-(J5-Pin_3) -> Net-(J4-Pin_2)
- R4 pad 1: Net-(J4-Pin_1) -> Net-(J5-Pin_2)
- R4 pad 2: Net-(J3-Pin_3) -> Net-(J3-Pin_2)
- R7 pad 2: Net-(J4-Pin_3) -> Net-(J5-Pin_1)
Routing:
- net Net-(J5-Pin_3): track 68.3 -> 0.00 mm, vias 1 -> 0
- net Net-(J5-Pin_1): track 65.6 -> 12.3 mm, vias 1 -> 0
- net Net-(J4-Pin_2): track 0.00 -> 36.7 mm, vias 0 -> 1
- net Net-(J5-Pin_2): track 0.00 -> 29.4 mm, vias 0 -> 2
- net TS-: track 91.2 -> 62.9 mm, vias 3 -> 4
- net 2V Ref: track 35.3 -> 17.2 mm, vias 0 -> 2
- net Net-(J4-Pin_3): track 11.9 -> 0.00 mm
- net Net-(R14-Pad2): track 30.9 -> 19.2 mm
- net Net-(J3-Pin_2): track 0.00 -> 9.50 mm
- net +5V_Isolated: track 38.2 -> 29.3 mm, vias 4 -> 0
- net Net-(J3-Pin_3): track 8.32 -> 0.00 mm
- net Net-(U6A-+): track 17.2 -> 14.6 mm, vias 0 -> 2
- net Net-(J3-Pin_1): track 7.92 -> 9.50 mm
- net Net-(J4-Pin_1): track 36.2 -> 37.5 mm, vias 0 -> 1
- net Net-(C6-Pad1): track 15.0 -> 14.0 mm
Other:
- board size 149.4 x 71.1 mm -> 137.7 x 71.1 mm
- board text added: "12V"
- board text added: "Discharge"
- board text added: "GLVMS"
- board text added: "GND"
- board text added: "TS+"
- board text added: "TS-"

Commit message: Rev 2.4
Confirmed with @fezboy that layout + schematic were OK. Added 3d models for big important space-relevant components. Still waiting on the OK from @victorkalastirsky mechanically
Parts:
- removed R3: 20k, Resistor_SMD:R_0603_1608Metric
- J1, J2, J6: footprint Connector_Molex:Molex_Mini-Fit_Sr_42819-22XX_1x02_P10.00mm_Vertical -> FS_4_Global_Footprint_Library:Molex_Mini-Fit_Sr_42819-22XX_1x02_P10.00mm_Vertical
- TP6: value 3.4V @ 12V ~ 3V @ 10.47V -> 2.44V @ 12V ~ 2.04V @ 10V
- moved J4 12.7 mm to (180.3, 117.3)
- moved J1 11.2 mm to (54.2, 122.0), turned to 0 degrees
- moved J2 11.1 mm to (54.5, 92.5), turned to 0 degrees
- moved TP4 2.03 mm to (116.3, 109.7)
- moved H5 1.52 mm to (110.2, 80.8)
- moved J6 1.35 mm to (108.5, 102.6)
- moved G*** 1.02 mm to (63.9, 80.8)
Connections:
- J1 pad 1: GND -> +12V_BAT
- J1 pad 2: +12V_BAT -> GND
- J2 pad 1: GND -> Net-(J2-Pin_1)
- J2 pad 2: Net-(J2-Pin_2) -> GND
- K2 pad 1: Net-(J2-Pin_2) -> Net-(J2-Pin_1)
- RV1 pad 3: Net-(R3-Pad1) -> GND
Routing:
- net Net-(J4-Pin_1): track 37.5 -> 50.2 mm
- net Net-(J4-Pin_2): track 36.7 -> 49.4 mm
- net Net-(R3-Pad1): track 4.16 -> 0.00 mm
- net Shutdown_Final: track 24.3 -> 23.3 mm
- net GND: vias 6 -> 8
- added copper zone on F.Cu, net Net-(J2-Pin_1)
- removed copper zone on F.Cu, net Net-(J2-Pin_2)
Other:
- outline, holes or cut-outs redrawn
- board text added: "Discharge+"
- board text added: "Discharge-"
- board text added: "TSMP+"
- board text added: "TSMP-"

Commit message: Rev 2.52
Changed DCDC Connector into studs to save vertical space
Parts:
- removed H5: MountingHole_Pad, MountingHole:MountingHole_3.2mm_M3_Pad
- removed J1, J2: Conn_01x02, FS_4_Global_Footprint_Library:Molex_Mini-Fit_Sr_42819-22XX_1x02_P10.00mm_Vertical
- added J10: Conn_01x02, FS_4_Global_Footprint_Library:Molex_Mini-Fit_Sr_42819-22XX_1x02_P10.00mm_Vertical, F.Cu at (54.2, 123.5)
- added J8: 74651173R, FS_4_Global_Footprint_Library:74651173R, F.Cu at (56.9, 91.9)
- added J9: 74651173R, FS_4_Global_Footprint_Library:74651173R, F.Cu at (56.9, 104.1)
- J6: footprint FS_4_Global_Footprint_Library:Molex_Mini-Fit_Sr_42819-22XX_1x02_P10.00mm_Vertical -> FS_4_Global_Footprint_Library:Molex_Mini-Fit_Sr_42820-22XX_1x02_P10.00mm_Horizontal
- moved J6 18.7 mm to (101.3, 85.4), turned to 0 degrees
- moved TP12 8.27 mm to (153.4, 139.7)
- moved R14 8.17 mm to (152.4, 137.4)
- moved K4 8.08 mm to (127.5, 109.2)
- moved U5 7.84 mm to (131.6, 125.7)
- moved U4 7.84 mm to (135.9, 136.5)
- moved H3 7.77 mm to (190.5, 146.3)
- moved C6 7.66 mm to (156.9, 137.0)
- moved C7 7.66 mm to (166.6, 133.9)
- moved F3 7.66 mm to (178.3, 131.9)
- moved F4 7.66 mm to (178.3, 139.0)
- moved J3 7.66 mm to (187.9, 135.5)
- moved J4 7.66 mm to (188.0, 118.1)
- moved R13 7.66 mm to (151.9, 130.7)
- moved R2 7.66 mm to (173.2, 131.9)
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Connections:
- J6 pad 1: GND -> GLVMS
- J6 pad 2: GLVMS -> GND
Routing:
- net Shutdown_Final: track 23.3 -> 38.8 mm
- net TS_Ready: track 21.5 -> 31.2 mm
- net Net-(K2-Pad3): track 36.7 -> 46.2 mm
- net +12V_Switched: track 54.0 -> 62.2 mm
- net +5V_LV: track 85.1 -> 91.4 mm
- net Net-(U7-R): track 16.0 -> 21.4 mm
- net Net-(J5-Pin_2): track 29.4 -> 32.0 mm
- net Net-(R14-Pad2): track 19.2 -> 21.5 mm
- net +5V_Isolated: track 29.3 -> 31.5 mm
- net Net-(J4-Pin_1): track 50.2 -> 49.4 mm
- net GND: vias 8 -> 10
Other:
- board size 137.7 x 71.1 mm -> 145.3 x 72.6 mm
