File: oven-board/oven-board.kicad_pcb (KiCad board)
At the start: 2 copper layers, 125 x 90.5 mm, 39 parts, among them J1 Temp Sensor Conn, J2 heating element 1, J3 wall outlet, J4 12V Power Supply, J5 heating element 2, J6 wall outlet, J7 switch1, J8 switch1, K1 G2RL-1A-E, K2 G2RL-1A-E, SW1 SW_Push, SW2 SW_Push, SW3 SW_Push, SW4 SW_Push, U1 SZNUD3124LT1G, U2 L78L09_TO92, U3 NUCLEO-L432KC, U4 SZNUD3124LT1G, U5 NHD-C0220BIZ, U6 INA826AIDR, U7 MCP1792x-3302xDB

Commit message: Imported board settings from VCU
Still need to actually change the sizes of traces
Changed lines of the file:
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@@
 			(at 0 -4.15 0)
 			(layer "F.SilkS")
+			(hide yes)
 			(effects
 				(font
@@
 			(at 0 -4.15 0)
 			(layer "F.SilkS")
+			(hide yes)
 			(effects
 				(font
@@
 			(at 0 -4.15 0)
 			(layer "F.SilkS")
+			(hide yes)
 			(effects
 				(font
@@
 			(at 0 -4.15 0)
 			(layer "F.SilkS")
+			(hide yes)
 			(effects
 				(font

Commit message: OvenBoard Layout 2
made all changes requested
Parts:
- moved REF** 0.24 mm to (218.2, 120.7)
- moved REF** 0.23 mm to (218.2, 40.6)
- moved REF** 0.16 mm to (103.3, 120.7)
- moved REF** 0.15 mm to (103.3, 40.6)
Routing:
- net +3.3V: track 94.8 -> 96.8 mm
- net GND: track 0.00 -> 1.71 mm, vias 28 -> 29
- net SDA: track 80.8 -> 81.4 mm
- net Net-(U6-IN-): track 44.8 -> 45.3 mm
- net RELAY_DRVR_2: track 55.6 -> 56.1 mm
Other:
- board text added: "Oven Board Maitreyi Patel"

Commit message: R2.1 Add Revision Info
Other:
- board text added: "Oven Board R${REVISION} Maitreyi Patel"
- board text removed: "Oven Board Maitreyi Patel"
Changed lines of the file:
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@@
 	)
 	(paper "A4")
+	(title_block
+		(title "Oven Board")
+		(date "2026-04-14")
+		(rev "2.1")
+		(company "Formula Slug")
+		(comment 1 "Maitreyi Patel")
+	)
 	(layers
 		(0 "F.Cu" signal)
@@
 		(layer "Edge.Cuts")
 	)
-	(gr_text "Oven Board\nMaitreyi Patel\n"
+	(gr_text "Oven Board R${REVISION}\nMaitreyi Patel\n\n"
 		(at 102.362 108.966 90)
 		(layer "F.SilkS")
