File: oven-board/oven-board.kicad_sch (KiCad schematic)
At the start: 30 parts, among them J1 temp_sensor, J2 heating element, J3 wall outlet, J4 12V Power Supply, K1 G2RL-1A-E, SW1 SW_Push, SW2 SW_Push, SW3 SW_Push, SW4 SW_Push, SW5 SW_Push, U1 MCP6004, U2 MCP6L04-xST, U3 NUCLEO-L432KC, U4 SZNUD3124LT1G, U5 NHD-C0220BIZ

Commit message: OvenBoard Schematic Rev 1.1
Made a few changes to fix schematic, more changes still left
Connections:
- net +12V: no longer U1.4 (V+)
- net +3.3V: now also R11.2, R12.1; no longer R11.1, R12.2
- net SCL: now also R12.2; no longer R11.2
- net SDA: now also R11.1; no longer R12.1
- net SW2: now also U3.CN4_9 (PA4); no longer U3.CN4_11 (PA1)
- net SW3: now also U3.CN4_8 (PA5); no longer U3.CN4_10 (PA3)
- net SW4: now also U3.CN4_7 (PA6); no longer U3.CN4_9 (PA4)
- net Supply_Out: now reaches J4.2 (Pin_2), SW5.2
- net Heating_Out: now reaches J2.1 (Pin_1), K1.13
- new net +5V: U1.4 (V+)
Other:
- moved on the sheet: C1, C2, D1, J1, J2, J3, J4, K1, R10, R11, R12, R4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

Commit message: Schematic Rev 2.0
Need to still add footprints but components selected, other symbol fields filled out
Parts:
- removed R10, R7, R8, R9: 10k, symbol Device:R
- removed U1: MCP6004, symbol Amplifier_Operational:MCP6004
- removed U2: MCP6L04-xST, Package_SO:TSSOP-14_4.4x5mm_P0.65mm, symbol Amplifier_Operational:MCP6L04-xST
- added C3: 0.1uF, symbol Device:C
- added C4: 10nF, symbol Device:C
- added U6: INA826AIDR, D8, symbol INA826AIDR:INA826AIDR
- C1: Digi PN (none) -> 490-1691-1-ND; Digi URL (none) -> https://www.digikey.com/en/products/detail/murata-electroni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; MFG (none) -> Murata; MFG PN (none) -> GRM21BR71C105KA01L
- C2: Digi PN (none) -> 311-1884-1-ND; Digi URL (none) -> https://www.digikey.com/en/products/detail/yageo/CC0805KKX7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; MFG (none) -> Yageo; MFG PN (none) -> CC0805KKX7R8BB225
- J1, J2, J3, J4: Digi PN (none) -> 277-1667-ND; Digi URL (none) -> https://www.digikey.com/en/products/detail/phoenix-contact/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; MFG (none) -> Phoenix Contact; MFG PN (none) -> 1935161
- K1: Digi PN (none) -> Z2924-ND; Digi URL (none) -> https://www.digikey.com/en/products/detail/omron-electronic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; MFG (none) -> Omron Electronics Inc-EMC Div; MFG PN (none) -> G2RL-1A-E DC12
- R1, R2: value 100 -> 1k; Digi PN (none) -> 311-1.0KARCT-ND; Digi URL (none) -> https://www.digikey.com/en/products/detail/yageo/RC0805JR-0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; MFG (none) -> Yageo; MFG PN (none) -> RC0805JR-071KL
- R3: Digi PN (none) -> 311-100ARCT-ND; Digi URL (none) -> https://www.digikey.com/en/products/detail/yageo/RC0805JR-0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; MFG (none) -> Yageo; MFG PN (none) -> RC0805JR-07100RL
- R4: value 10k -> 5.76k; Digi PN (none) -> 311-5.76KHRCT-ND; Digi URL (none) -> https://www.digikey.com/en/products/detail/yageo/RC0603FR-0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; MFG (none) -> Yageo; MFG PN (none) -> RC0603FR-075K76L
- R5: value 4.99k -> 1k; Digi PN (none) -> 311-1.0KARCT-ND; Digi URL (none) -> https://www.digikey.com/en/products/detail/yageo/RC0805JR-0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; MFG (none) -> Yageo; MFG PN (none) -> RC0805JR-071KL
- R6: value 10k -> 1k; Digi PN (none) -> 311-1.0KARCT-ND; Digi URL (none) -> https://www.digikey.com/en/products/detail/yageo/RC0805JR-0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; MFG (none) -> Yageo; MFG PN (none) -> RC0805JR-071KL
- R7: renamed from R12; Digi PN (none) -> 311-4.70KCRCT-ND; Digi URL (none) -> https://www.digikey.com/en/products/detail/yageo/RC0805FR-0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; MFG (none) -> Yageo; MFG PN (none) -> RC0805FR-074K7L
- R8: renamed from R11; Digi PN (none) -> 311-4.70KCRCT-ND; Digi URL (none) -> https://www.digikey.com/en/products/detail/yageo/RC0805FR-0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; MFG (none) -> Yageo; MFG PN (none) -> RC0805FR-074K7L
- SW1, SW2, SW3, SW4, SW5: Digi PN (none) -> EG5398-ND; Digi URL (none) -> www.digikey.com/en/products/detail/e-switch/PB300STQ/6126493; MFG (none) -> E-Switch; MFG PN (none) -> PB300STQ
- U5: Digi PN (none) -> NHD-C0220BIZ-FSW-FBW-3V3M-ND; Digi URL (none) -> https://www.digikey.com/en/products/detail/newhaven-display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; MFG (none) -> Newhaven Display Intl; MFG PN (none) -> NHD-C0220BIZ-FSW-FBW-3V3M
Connections:
- net +12V: now also C3.1, U6.8 (VS+)
- net GND: now also C3.2, U6.5 (VS-), U6.6 (REF)
- net IN_AMP: now also U6.7 (VOUT)
- net v_out1: now also R5.1
- net v_out2: now also R6.1
- net at R4.1: now also U6.2 (RG)
- net at R5.2: now also C4.2, U6.1 (IN-); no longer R6.1
- net at R6.2: now also C4.1, U6.4 (IN+)
- net at R4.2: now also U6.3 (RG); no longer R5.1
Other:
- moved on the sheet: R1, R2, R3

Commit message: Oven Board Rev 2.1
Made all requested changes
Parts:
- added J5: heating element 2, Library:CONN_1890963_PXC, symbol Connector:Conn_01x02_Pin
- added K2: G2RL-1A-E, Library:RELAY_G2RL-1A-E DC5_OMR, symbol Relay:G2RL-1A-E
- added SW6: SW_Push, Library:SW_PB300STQ, symbol Switch:SW_Push
- added TH1: PT100, symbol Sensor_Temperature:PT100
- added U1: SZNUD3124LT1G, Package_TO_SOT_SMD:TSOT-23_HandSoldering, symbol FS_4_Global_Symbol_Library:SZNUD3124LT1G
- C1: footprint (none) -> Library:CAP_GRM21_MUR_1uF
- C2: footprint (none) -> Library:CAP_CC0805_EB_YAG_2.2uF
- C3: footprint (none) -> Library:CC0805N_YAG_0.1uF
- C4: footprint (none) -> Library:CAPC17595_87N_KEM_10nF
- D1: footprint (none) -> Library:LED_LTL-307E_LTO; Digi PN (none) -> 160-1705-ND; Digi URL (none) -> https://www.digikey.com/en/products/detail/liteon/LTL-307E/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; MFG (none) -> Lite-On Inc.; MFG PN (none) -> LTL-307E
- J1: value temp_sensor -> Temp Sensor Conn; footprint (none) -> Library:CONN_1890963_PXC
- J2: value heating element -> heating element 1; footprint (none) -> Library:CONN_1890963_PXC
- J3, J4: footprint (none) -> Library:CONN_1890963_PXC
- K1: footprint Relay_THT:Relay_SPST_Omron_G2RL-1A-E -> Library:RELAY_G2RL-1A-E DC5_OMR
- R1, R2, R5, R6: footprint (none) -> Library:RC0805N_YAG_1K
- R3: footprint (none) -> Library:RC0805N_YAG_100
- R4: footprint (none) -> Library:RC0603N_YAG_5.76K
- R7, R8: footprint (none) -> Library:RES_RC0805_YAG_4.7K
- SW1, SW2, SW3, SW4, SW5: footprint (none) -> Library:SW_PB300STQ
- U3: Digi PN (none) -> 497-16592-ND; Digi URL (none) -> https://www.digikey.com/en/products/detail/stmicroelectroni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; MFG (none) -> STMicroelectronics; MFG PN (none) -> NUCLEO-L432KC
- U5: footprint Display:NHD-C0220BiZ -> Library:NHD-C0220BIZ-FSW-FBW-3V3M_NDI
- U6: footprint D8 -> Library:INA826AIDR
Connections:
- net +12V: now also K2.14, K2.A1, SW6.1
- net GND: now also U1.2
- net RELAY_DRVR: now also U3.CN3_1 (PA9); no longer U3.CN3_6 (PB0)
- net Supply_Out: now also SW6.2
- net RELAY_DRVR_2: now reaches U3.CN3_2 (PA10)
- net RELAY_DRVR_2: now also U1.1
- net Wall_Outlet: now reaches J2.2 (Pin_2), J3.1 (Pin_1)
- net Wall_Outlet: now also J5.2 (Pin_2)
- new net: J5.1 (Pin_1), K2.13
- new net: K2.A2, U1.3
- no-connect marks 20 -> 18
Other:
- moved on the sheet: C1, C2, C3, C4, D1, J1, J2, J3, J4, K1, R1, R2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

Commit message: Oven Board Rev 3.0
made all changes from previous review request, have minimal erc errors (will confirm them tomorrow)
Parts:
- added J6: wall outlet, Library:CONN_1890963_PXC, symbol Connector:Conn_01x02_Pin
- added J7, J8: switch1, Library:CONN_1890963_PXC, symbol Connector:Conn_01x02_Pin
- added R10, R9: R, symbol Device:R
- added R11: 220, Resistor_SMD:R_0805_2012Metric_Pad1.20x1.40mm_HandSolder, symbol Device:R
- added U2: L78L09_TO92, Package_TO_SOT_THT:TO-92_Inline, symbol Regulator_Linear:L78L09_TO92
- added U7: MCP1792x-3302xDB, Package_TO_SOT_SMD:SOT-223-3_TabPin2, symbol Regulator_Linear:MCP1792x-3302xDB
- C1: footprint Library:CAP_GRM21_MUR_1uF -> Capacitor_SMD:C_0805_2012Metric_Pad1.18x1.45mm_HandSolder
- C2: footprint Library:CAP_CC0805_EB_YAG_2.2uF -> Capacitor_SMD:C_0805_2012Metric_Pad1.18x1.45mm_HandSolder
- C3: footprint Library:CC0805N_YAG_0.1uF -> Capacitor_SMD:C_0805_2012Metric_Pad1.18x1.45mm_HandSolder
- C4: footprint Library:CAPC17595_87N_KEM_10nF -> Capacitor_SMD:C_0603_1608Metric_Pad1.08x0.95mm_HandSolder
- K1, K2: footprint Library:RELAY_G2RL-1A-E DC5_OMR -> Relay_THT:Relay_SPST_Omron_G2RL-1A-E
- R1, R2, R5, R6: footprint Library:RC0805N_YAG_1K -> Resistor_SMD:R_0805_2012Metric_Pad1.20x1.40mm_HandSolder
- R3: footprint Library:RC0805N_YAG_100 -> Resistor_SMD:R_0805_2012Metric_Pad1.20x1.40mm_HandSolder
- R4: footprint Library:RC0603N_YAG_5.76K -> Resistor_SMD:R_0603_1608Metric_Pad0.98x0.95mm_HandSolder
- R7, R8: footprint Library:RES_RC0805_YAG_4.7K -> Resistor_SMD:R_0805_2012Metric_Pad1.20x1.40mm_HandSolder
- SW5, SW6: footprint Library:SW_PB300STQ -> (none); Digi PN EG5398-ND -> 2449-RC1123EWC-ND; Digi URL www.digikey.com/en/products/detail/e-switch/PB300STQ/6126493 -> https://www.digikey.com/en/products/detail/cit-relay-and-sw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; MFG E-Switch -> CIT Relay and Switch; MFG PN PB300STQ -> RC1123EWC; now not fitted
Connections:
- net +12V: now also J4.2 (Pin_2), U2.3 (VI), U7.1 (VI); no longer K1.14, K2.14, SW5.1, SW6.1, U3.CN4_1 (VIN)
- net +3.3V: now also U7.3 (VO); no longer U3.CN4_14 (3V3)
- net GND: now also D1.2 (A), U3.CN3_4 (GND), U3.CN4_2 (GND), U2.2 (GND), U7.2 (GND); no longer D1.1 (K)
- net LED: now also R11.2; no longer D1.2 (A)
- net RST: now also U3.CN3_6 (PB0)
- net Live1: now reaches J3.2 (Pin_2)
- net Live1: now also J7.1 (Pin_1)
- removed net Supply_Out: J4.2 (Pin_2), SW5.2, SW6.2
- net Wall_Outlet renamed Neutral1
- net Neutral1: no longer J5.2 (Pin_2)
- new net: D1.1 (K), R11.1
- new net: J8.2 (Pin_2), K2.14
- new net: J7.2 (Pin_2), K1.14
- new net +9V: U2.1 (VO), U3.CN4_1 (VIN)
- new net Live2: J6.2 (Pin_2), J8.1 (Pin_1)
- new net Neutral2: J5.2 (Pin_2), J6.1 (Pin_1)
- no-connect marks 18 -> 16
Other:
- note added: "Linear Regulators"
- moved on the sheet: D1, J2, J3, J4, J5, SW1, SW2, SW3, SW4, U3A

Commit message: Oven Board 3.1
made requested changes, only changed symbol warnings show up on my end
Parts:
- C4: footprint Capacitor_SMD:C_0603_1608Metric_Pad1.08x0.95mm_HandSolder -> Capacitor_SMD:C_0805_2012Metric_Pad1.18x1.45mm_HandSolder
- D1: value LED -> RED_6mA; footprint Library:LED_LTL-307E_LTO -> LED_THT:LED_D5.0mm_IRBlack
- R4: footprint Resistor_SMD:R_0603_1608Metric_Pad0.98x0.95mm_HandSolder -> Resistor_SMD:R_0805_2012Metric_Pad1.20x1.40mm_HandSolder
- U6: footprint Library:INA826AIDR -> Package_SO:SOIC-8_5.3x6.2mm_P1.27mm
Connections:
- net +12V: no longer C3.1, U6.8 (VS+)
- net +3.3V: now also C3.1, U6.8 (VS+)
- net GND: now also D1.1 (K), TH1.2; no longer D1.2 (A)
- net Heating_Out: now also R9.2
- net Live1: now also SW5.2
- net Live2: now also SW6.2
- net Neutral1: now also R9.1
- net Neutral2: now also R10.1
- net v_out2: now also TH1.1
- net at R11.1: now also D1.2 (A); no longer D1.1 (K)
- net at J8.2 (Pin_2), K2.14: now also SW6.1
- net at J5.1 (Pin_1), K2.13: now also R10.2
- net at SW5.1: now also J7.2 (Pin_2), K1.14
Other:
- moved on the sheet: D1

Commit message: OvenBoard Layout Rev 1
Layout Rev 1 complete
Parts:
- U3: footprint FS_3_Global_Footprint_Library:NUCLEO-L432KC -> FS_4_Global_Footprint_Library:NUCLEO-L432KC
Connections:
- net RELAY_DRVR: now also U3.CN3_2 (PA10); no longer U3.CN3_1 (PA9)
- net RELAY_DRVR_2: now also U3.CN3_1 (PA9); no longer U3.CN3_2 (PA10)
- net RST: now also U3.CN3_7 (PB7); no longer U3.CN3_6 (PB0)
- net SCL: now also U3.CN3_6 (PB0); no longer U3.CN3_8 (PB6)
- net SDA: now also U3.CN3_8 (PB6); no longer U3.CN3_7 (PB7)
- net Heating_Out_2: now reaches J5.1 (Pin_1), K2.13, R10.2
- net Heating_Out renamed Heating_Out_1
Changed lines of the file:
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@@
 	(wire
 		(pts
+			(xy 205.74 120.65) (xy 208.28 120.65)
+		)
+		(stroke
+			(width 0)
+			(type default)
+		)
+	)
+	(wire
+		(pts
 			(xy 39.37 76.2) (xy 53.34 76.2)
 		)
@@
 	(wire
 		(pts
+			(xy 205.74 125.73) (xy 208.28 125.73)
+		)
+		(stroke
+			(width 0)
+			(type default)
+		)
+	)
+	(wire
+		(pts
 			(xy 101.6 168.91) (xy 101.6 154.94)
 		)
@@
 		)
 	)
-	(wire
-		(pts
-			(xy 205.74 125.73) (xy 208.28 125.73)
-		)
-		(stroke
-			(width 0)
-			(type default)
-		)
-	)
 	(polyline
 		(pts
@@
 	(wire
 		(pts
-			(xy 205.74 120.65) (xy 208.28 120.65)
-		)
-		(stroke
-			(width 0)
-			(type default)
-		)
-	)
-	(wire
-		(pts
 			(xy 163.83 68.58) (xy 163.83 81.28)
 		)
@@
 	(wire
 		(pts
+			(xy 205.74 123.19) (xy 208.28 123.19)
+		)
+		(stroke
+			(width 0)
+			(type default)
+		)
+	)
+	(wire
+		(pts
 			(xy 76.2 88.9) (xy 86.36 88.9)
 		)
@@
 	(wire
 		(pts
-			(xy 205.74 123.19) (xy 208.28 123.19)
-		)
-		(stroke
-			(width 0)
-			(type default)
-		)
-	)
-	(wire
-		(pts
 			(xy 101.6 96.52) (xy 39.37 96.52)
 		)
@@
 		)
 	)
-	(label "Heating_Out"
+	(label "Heating_Out_1"
 		(at 39.37 96.52 0)
 		(effects
@@
 		)
 	)
+	(label "Heating_Out_2"
+		(at 39.37 168.91 0)
+		(effects
+			(font
+				(size 1.27 1.27)
+			)
+			(justify left bottom)
+		)
+	)
 	(label "GND"
 		(at 39.37 44.45 0)
@@
 	(global_label "SCL"
 		(shape input)
-		(at 205.74 125.73 180)
+		(at 205.74 120.65 180)
 		(fields_autoplaced yes)
 		(effects
@@
 		)
 		(property "Intersheetrefs" "${INTERSHEET_REFS}"
-			(at 199.2472 125.73 0)
+			(at 199.2472 120.65 0)
 			(effects
 				(font
@@
 	(global_label "RST"
 		(shape input)
-		(at 205.74 120.65 180)
+		(at 205.74 123.19 180)
 		(fields_autoplaced yes)
 		(effects
@@
 		)
 		(property "Intersheetrefs" "${INTERSHEET_REFS}"
-			(at 199.3077 120.65 0)
+			(at 199.3077 123.19 0)
 			(effects
 				(font
@@
 	(global_label "RELAY_DRVR"
 		(shape input)
-		(at 208.28 107.95 180)
+		(at 208.28 110.49 180)
 		(fields_autoplaced yes)
 		(effects
@@
 		)
 		(property "Intersheetrefs" "${INTERSHEET_REFS}"
-			(at 193.8043 107.95 0)
+			(at 193.8043 110.49 0)
 			(effects
 				(font
@@
 	(global_label "SDA"
 		(shape input)
-		(at 205.74 123.19 180)
+		(at 205.74 125.73 180)
 		(fields_autoplaced yes)
 		(effects
@@
 		)
 		(property "Intersheetrefs" "${INTERSHEET_REFS}"
-			(at 199.1867 123.19 0)
+			(at 199.1867 125.73 0)
 			(effects
 				(font
@@
 	(global_label "RELAY_DRVR_2"
 		(shape input)
-		(at 208.28 110.49 180)
+		(at 208.28 107.95 180)
 		(fields_autoplaced yes)
 		(effects
@@
 		)
 		(property "Intersheetrefs" "${INTERSHEET_REFS}"
-			(at 191.6272 110.49 0)
+			(at 191.6272 107.95 0)
 			(effects
 				(font
@@
 			)
 		)
-		(property "Footprint" "FS_3_Global_Footprint_Library:NUCLEO-L432KC"
+		(property "Footprint" "FS_4_Global_Footprint_Library:NUCLEO-L432KC"
 			(at 177.8 118.11 0)
 			(effects

Commit message: Imported board settings from VCU
Still need to actually change the sizes of traces
Other:
- moved on the sheet: C1, C2, C3, C4, D1, J1, J2, J3, J4, J5, J6, J7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
