File: BMS/TempSenseBoard/TempSenseBoard.kicad_pcb (KiCad board)
At the start: 4 copper layers, 351 x 131 mm, 27 parts, among them J1 5019510550, J3 5019510550, U1 TMP1075D, U10 TMP1075D, U11 TMP1075D, U12 TMP1075D, U13 DS18B20Z+, U2 TMP1075D, U3 TMP1075D, U4 TMP1075D, U5 TMP1075D, U6 TMP1075D, U7 TMP1075D, U8 TMP1075D, U9 TMP1075D

Commit message: placed components
Parts:
- moved C10 168.7 mm to (69.0, 164.2), turned to -90 degrees
- moved U10 166.9 mm to (64.5, 164.8)
Routing:
- net V-: track 16.7 -> 25.6 mm
- net +5V: track 13.4 -> 15.5 mm
- removed copper zone on In2.Cu, net +5V
- removed copper zone on In1.Cu, net V-
Changed lines of the file:
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@@
 	(footprint "Package_SO:SO-8_3.9x4.9mm_P1.27mm"
 		(layer "F.Cu")
-		(at 230.4887 181.8096)
+		(at 64.5 164.75)
 		(descr "SO, 8 Pin (https://www.nxp.com/docs/en/data-sheet/PCF8523.pdf), generated with kicad-footprint-generator ipc_gullwing_generator.py")
 		(tags "SO SO")
@@
 	(footprint "Capacitor_SMD:C_0603_1608Metric_Pad1.08x0.95mm_HandSolder"
 		(layer "F.Cu")
-		(at 236.8875 181)
+		(at 69 164.25 -90)
 		(descr "Capacitor SMD 0603 (1608 Metric), square (rectangular) end terminal, IPC-7351 nominal with elongated pad for handsoldering. (Body size source: IPC-SM-782 page 76, https://www.pcb-3d.com/wordpress/wp-content/uploads/ipc-sm-782a_amendment_1_and_2.pdf), generated with kicad-footprint-generator")
 		(tags "capacitor handsolder")
 		(property "Reference" "C10"
-			(at 0 -1.43 0)
+			(at 0 -1.43 90)
 			(layer "F.SilkS")
 			(effects
@@
 		)
 		(property "Value" "0.01 uF"
-			(at 0 1.43 0)
+			(at 0 1.43 90)
 			(layer "F.Fab")
 			(effects
@@
 		)
 		(property "Datasheet" "~"
-			(at 0 0 0)
+			(at 0 0 90)
 			(layer "F.Fab")
 			(hide yes)
@@
 		)
 		(property "Description" "Unpolarized capacitor"
-			(at 0 0 0)
+			(at 0 0 90)
 			(layer "F.Fab")
 			(hide yes)
@@
 		(attr smd)
 		(fp_line
-			(start -0.146267 -0.51)
-			(end 0.146267 -0.51)
+			(start -0.146267 0.51)
+			(end 0.146267 0.51)
 			(stroke
 				(width 0.12)
@@
 		)
 		(fp_line
-			(start -0.146267 0.51)
-			(end 0.146267 0.51)
+			(start -0.146267 -0.51)
+			(end 0.146267 -0.51)
 			(stroke
 				(width 0.12)
@@
 		)
 		(fp_line
-			(start -1.65 -0.73)
-			(end 1.65 -0.73)
+			(start -1.65 0.73)
+			(end -1.65 -0.73)
 			(stroke
 				(width 0.05)
@@
 		)
 		(fp_line
-			(start -1.65 0.73)
-			(end -1.65 -0.73)
+			(start 1.65 0.73)
+			(end -1.65 0.73)
 			(stroke
 				(width 0.05)
@@
 		)
 		(fp_line
-			(start 1.65 -0.73)
-			(end 1.65 0.73)
+			(start -1.65 -0.73)
+			(end 1.65 -0.73)
 			(stroke
 				(width 0.05)
@@
 		)
 		(fp_line
-			(start 1.65 0.73)
-			(end -1.65 0.73)
+			(start 1.65 -0.73)
+			(end 1.65 0.73)
 			(stroke
 				(width 0.05)
@@
 		)
 		(fp_line
-			(start -0.8 -0.4)
-			(end 0.8 -0.4)
+			(start -0.8 0.4)
+			(end -0.8 -0.4)
 			(stroke
 				(width 0.1)
@@
 		)
 		(fp_line
-			(start -0.8 0.4)
-			(end -0.8 -0.4)
+			(start 0.8 0.4)
+			(end -0.8 0.4)
 			(stroke
 				(width 0.1)
@@
 		)
 		(fp_line
-			(start 0.8 -0.4)
-			(end 0.8 0.4)
+			(start -0.8 -0.4)
+			(end 0.8 -0.4)
 			(stroke
 				(width 0.1)
@@
 		)
 		(fp_line
-			(start 0.8 0.4)
-			(end -0.8 0.4)
+			(start 0.8 -0.4)
+			(end 0.8 0.4)
 			(stroke
 				(width 0.1)
@@
 		)
 		(fp_text user "${REFERENCE}"
-			(at 0 0 0)
+			(at 0 0 90)
 			(layer "F.Fab")
 			(effects
@@
 		)
 		(pad "1" smd roundrect
-			(at -0.8625 0)
+			(at -0.8625 0 270)
 			(size 1.075 0.95)
 			(layers "F.Cu" "F.Mask" "F.Paste")
@@
 		)
 		(pad "2" smd roundrect
-			(at 0.8625 0)
+			(at 0.8625 0 270)
 			(size 1.075 0.95)
 			(layers "F.Cu" "F.Mask" "F.Paste")
@@
 	)
 	(segment
+		(start 67.075 162.845)
+		(end 68.4575 162.845)
+		(width 0.254)
+		(layer "F.Cu")
+		(net 1)
+	)
+	(segment
 		(start 67.075 84.115)
 		(end 67.075 82.845)
@@
 	)
 	(segment
+		(start 68.4575 162.845)
+		(end 69 163.3875)
+		(width 0.254)
+		(layer "F.Cu")
+		(net 1)
+	)
+	(segment
 		(start 67.075 82.075)
 		(end 67 82)
@@
 	)
 	(segment
+		(start 66.615 165.385)
+		(end 67.075 165.385)
+		(width 0.254)
+		(layer "F.Cu")
+		(net 2)
+	)
+	(segment
 		(start 61.925 87.075)
 		(end 61.5 87.5)
@@
 	)
 	(segment
+		(start 65.345 166.655)
+		(end 66.615 165.385)
+		(width 0.254)
+		(layer "F.Cu")
+		(net 2)
+	)
+	(segment
 		(start 369 85.6125)
 		(end 369 86.25)
@@
 	)
 	(segment
+		(start 67.615 165.385)
+		(end 67.075 165.385)
+		(width 0.254)
+		(layer "F.Cu")
+		(net 2)
+	)
+	(segment
 		(start 67.075 85.385)
 		(end 67.075 86.655)
@@
 	)
 	(segment
+		(start 61.925 166.655)
+		(end 65.345 166.655)
+		(width 0.254)
+		(layer "F.Cu")
+		(net 2)
+	)
+	(segment
 		(start 67.075 86.655)
 		(end 67.075 87.425)
@@
 	)
 	(segment
+		(start 67.075 164.115)
+		(end 67.075 165.385)
+		(width 0.254)
+		(layer "F.Cu")
+		(net 2)
+	)
+	(segment
 		(start 161.925 107.425)
 		(end 162 107.5)
@@
 	)
 	(segment
+		(start 68 165)
+		(end 67.615 165.385)
+		(width 0.254)
+		(layer "F.Cu")
+		(net 2)
+	)
+	(segment
 		(start 361.925 87.425)
 		(end 362 87.5)
@@
 		(net 2)
 	)
+	(segment
+		(start 68.8875 165)
+		(end 68 165)
+		(width 0.254)
+		(layer "F.Cu")
+		(net 2)
+	)
 	(via
 		(at 168.75 106.75)
@@
 			)
 		)
-	)
-	(zone
-		(net 2)
-		(net_name "V-")
-		(layer "In1.Cu")
-		(hatch edge 0.5)
-		(connect_pads
-			(clearance 0.5)
-		)
-		(min_thickness 0.25)
-		(filled_areas_thickness no)
-		(fill yes
-			(thermal_gap 0.5)
-			(thermal_bridge_width 0.5)
-		)
-		(polygon
-			(pts
-				(xy 30 50.59038) (xy 392.75 43.75) (xy 401.75 201.5) (xy 262.75 208) (xy 238.5 174) (xy 178.75 178.5)
-				(xy 160.5 217) (xy 32.5 208)
-			)
-		)
-	)
-	(zone
-		(net 1)
-		(net_name "+5V")
-		(layer "In2.Cu")
-		(name "LV safe zone")
-		(hatch edge 0.5)
-		(priority 1)
-		(connect_pads
-			(clearance 0.5)
-		)
-		(min_thickness 0.25)
-		(filled_areas_thickness no)
-		(fill yes
-			(thermal_gap 0.5)
-			(thermal_bridge_width 0.5)
-		)
-		(polygon
-			(pts
-				(xy 30.5 51.5) (xy 402.25 43.25) (xy 408 205.25) (xy 262 207.5) (xy 238.5 173.25) (xy 182 179) (xy 151.25 212)
-				(xy 34.75 204.5)
-			)
-		)

Commit message: updated placement and traces
Parts:
- moved C9 163.2 mm to (369.0, 164.8), turned to -90 degrees
- moved U9 158.5 mm to (364.5, 164.8)
- moved U5 146.4 mm to (304.5, 124.8)
- moved C5 145.0 mm to (305.0, 121.2), turned to 180 degrees
- moved U6 125.8 mm to (124.5, 124.8)
- moved C3 118.9 mm to (269.0, 104.8), turned to -90 degrees
- moved C6 118.9 mm to (129.0, 124.8), turned to -90 degrees
- moved U3 112.9 mm to (264.5, 104.8)
- moved U12 101.0 mm to (144.5, 185.0)
- moved C12 98.5 mm to (149.0, 184.8), turned to -90 degrees
- moved U7 80.7 mm to (264.5, 144.8)
- moved C8 80.3 mm to (169.0, 144.8), turned to -90 degrees
- moved C7 79.8 mm to (265.5, 141.2), turned to 180 degrees
- moved U8 78.7 mm to (164.5, 144.8)
- moved C11 48.6 mm to (286.2, 181.5), turned to 180 degrees
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Routing:
- net /SDA: track 145.3 -> 244.2 mm, vias 2 -> 6
- net /SCL: track 152.2 -> 246.2 mm
- net V-: track 25.6 -> 93.6 mm, vias 8 -> 2
- net +5V: track 15.5 -> 57.6 mm, vias 4 -> 5
- net /ALERT: track 157.5 -> 149.6 mm
