File: Temporary-Sensor-Board/Temporary-Sensor-Board.kicad_sch (KiCad schematic)
At the start: 23 parts, among them J1 Conn_ST_STDC14, U1 STM32G441KBTx, U2 STM32C092KCU6, U3 TCAN332G, U4 MCP1703Ax-330xxTT, U5 LP2985-1.8, Y2 24MHz

Commit message: .
Parts:
- added TP10: 3.3V, TestPoint:TestPoint_Pad_2.0x2.0mm, symbol Connector:TestPoint
- added TP11: 1.8V, TestPoint:TestPoint_Pad_2.0x2.0mm, symbol Connector:TestPoint
- added TP12: CANH, TestPoint:TestPoint_Pad_2.0x2.0mm, symbol Connector:TestPoint
- added TP13: CANL, TestPoint:TestPoint_Pad_2.0x2.0mm, symbol Connector:TestPoint
- added TP14: SCL, TestPoint:TestPoint_Pad_2.0x2.0mm, symbol Connector:TestPoint
- added TP15: SDA, TestPoint:TestPoint_Pad_2.0x2.0mm, symbol Connector:TestPoint
- added TP3: PB7, TestPoint:TestPoint_Pad_2.0x2.0mm, symbol Connector:TestPoint
- added TP4: PB6, TestPoint:TestPoint_Pad_2.0x2.0mm, symbol Connector:TestPoint
- added TP5: PB5, TestPoint:TestPoint_Pad_2.0x2.0mm, symbol Connector:TestPoint
- added TP6: PB3, TestPoint:TestPoint_Pad_2.0x2.0mm, symbol Connector:TestPoint
- added TP7: PA15, TestPoint:TestPoint_Pad_2.0x2.0mm, symbol Connector:TestPoint
- added TP8: 12VIN, TestPoint:TestPoint_Pad_2.0x2.0mm, symbol Connector:TestPoint
- added TP9: GND, TestPoint:TestPoint_Pad_2.0x2.0mm, symbol Connector:TestPoint
Connections:
- net +12V: now also TP8.1
- net +1V8: now also TP11.1
- net +3.3V: now also TP10.1
- net GND: now also TP9.1
- net I2C_SCL: now also TP14.1
- net I2C_SDA: now also TP15.1
- net PA15: now reaches U1.26 (PB3)
- net PA15: now also U2.26 (PA15), TP7.1
- net PB3: now reaches U1.27 (PB4)
- net PB3: now also U2.27 (PB3), TP6.1
- net PB5: now reaches U1.28 (PB5)
- net PB5: now also U2.29 (PB5), TP5.1
- net PB6: now reaches U1.29 (PB6)
- net PB6: now also U2.30 (PB6), TP4.1
- net PB7: now reaches U1.30 (PB7)
- net PB7: now also U2.31 (PB7), TP3.1
- net at U3.6 (CANL): now also TP13.1
- net at U3.7 (CANH): now also TP12.1
- net PB4: now reaches U2.28 (PB4)
- net PB8: now reaches U2.32 (PB8)
Other:
- moved on the sheet: C1

Commit message: gk
Parts:
- removed R1, R2: 10k, Resistor_SMD:R_0603_1608Metric, symbol Device:R_Small
- removed TP10: 3.3V, TestPoint:TestPoint_Pad_2.0x2.0mm, symbol Connector:TestPoint
- removed TP11: 1.8V, TestPoint:TestPoint_Pad_2.0x2.0mm, symbol Connector:TestPoint
- removed TP12: CANH, TestPoint:TestPoint_Pad_2.0x2.0mm, symbol Connector:TestPoint
- removed TP13: CANL, TestPoint:TestPoint_Pad_2.0x2.0mm, symbol Connector:TestPoint
- removed TP14: SCL, TestPoint:TestPoint_Pad_2.0x2.0mm, symbol Connector:TestPoint
- removed TP15: SDA, TestPoint:TestPoint_Pad_2.0x2.0mm, symbol Connector:TestPoint
- removed TP3: PB7, TestPoint:TestPoint_Pad_2.0x2.0mm, symbol Connector:TestPoint
- removed TP4: PB6, TestPoint:TestPoint_Pad_2.0x2.0mm, symbol Connector:TestPoint
- removed TP5: PB5, TestPoint:TestPoint_Pad_2.0x2.0mm, symbol Connector:TestPoint
- removed TP6: PB3, TestPoint:TestPoint_Pad_2.0x2.0mm, symbol Connector:TestPoint
- removed TP7: PA15, TestPoint:TestPoint_Pad_2.0x2.0mm, symbol Connector:TestPoint
- removed TP8: 12VIN, TestPoint:TestPoint_Pad_2.0x2.0mm, symbol Connector:TestPoint
- removed TP9: GND, TestPoint:TestPoint_Pad_2.0x2.0mm, symbol Connector:TestPoint
- removed U1: STM32G441KBTx, Package_QFP:LQFP-32_7x7mm_P0.8mm, symbol MCU_ST_STM32G4:STM32G441KBTx
- added J2: Conn_01x14_Pin, Connector_PinHeader_1.27mm:PinHeader_1x14_P1.27mm_Vertical, symbol Connector:Conn_01x14_Pin
- added J3: Rightie, Connector_PinHeader_1.27mm:PinHeader_1x12_P1.27mm_Vertical, symbol Connector:Conn_01x12_Socket
- added J4: Cannie, Connector_PinHeader_2.54mm:PinHeader_1x02_P2.54mm_Vertical, symbol Connector:Conn_01x02_Socket
- added J5: Powerie, Connector_PinHeader_2.54mm:PinHeader_1x04_P2.54mm_Vertical, symbol Connector:Conn_01x04_Pin
Connections:
- net +12V: now also J5.4 (Pin_4)
- net +1V8: now also J5.2 (Pin_2)
- net +3.3V: now also J2.14 (Pin_14), J3.12 (Pin_12), J5.3 (Pin_3)
- net GND: now also J2.1 (Pin_1), J3.1 (Pin_1), J5.1 (Pin_1)
- net I2C_SCL: now also J3.4 (Pin_4)
- net I2C_SDA: now also J3.5 (Pin_5)
- net UART_RX: now also J3.2 (Pin_2)
- net UART_TX: now also J3.3 (Pin_3)
- net at U3.6 (CANL): now also J4.2 (Pin_2)
- net at U3.7 (CANH): now also J4.1 (Pin_1)
- net at U2.1 (PB9): now also J3.11 (Pin_11)
- net at U2.10 (PA3): now also J3.9 (Pin_9)
- net at U2.12 (PA5): now also J3.8 (Pin_8)
- net at U2.14 (PA7): now also J3.7 (Pin_7)
- net at U2.17 (PB2): now also J3.6 (Pin_6)
- net at U2.18 (PA8): now also J2.2 (Pin_2)
- net at U2.20 (PC6): now also J2.3 (Pin_3)
- net at U2.21 (PA10): now also J2.4 (Pin_4)
- net at U2.22 (PA11[PA9]): now also J2.5 (Pin_5)
- net at U2.23 (PA12[PA10]): now also J2.6 (Pin_6)
- net at U2.9 (PA2): now also J3.10 (Pin_10)
- net PA15: no longer names the net of U2.26 (PA15)
- net PA15: now also J2.7 (Pin_7)
- net PB3: no longer names the net of U2.27 (PB3)
- net PB3: now also J2.8 (Pin_8)
- net PB4: no longer names the net of U2.28 (PB4)
- net PB4: now also J2.9 (Pin_9)
- net PB5: no longer names the net of U2.29 (PB5)
- net PB5: now also J2.10 (Pin_10)
- net PB6: no longer names the net of U2.30 (PB6)
- net PB6: now also J2.11 (Pin_11)
- net PB7: no longer names the net of U2.31 (PB7)
- net PB7: now also J2.12 (Pin_12)
- net PB8: no longer names the net of U2.32 (PB8)
- net PB8: now also J2.13 (Pin_13)
Other:
- note removed: "Fake"
- moved on the sheet: C1, C2, Y2
