File: LLC Test Bench/LLC Test Bench.kicad_sch (KiCad schematic)
At the start: 17 parts, among them J1 +HV, J2 -HV, J3 +LV, J4 -LV, Q1 NMOS, Q2 NMOS, Q3 NMOS, Q4 NMOS

Commit message: Precharge sheet Added + Fuse
- Added a Precharge sheet to be made
- Modified HV input to HV and HV_PC (PreCharge)
- Added Fuse on positive side of HV, value TBD

Notes:
- Please offer feedback if these will be needed for test bench, safety was in mind while handling a 108V input for testing.
Parts:
- added F1: Fuse, symbol Device:Fuse
Connections:
- net +Vin: no longer J1.1 (Pin_1)
- net GNDPWR: no longer J2.1 (Pin_1)
- new net: F1.1, J1.1 (Pin_1)
- new net Precharge/+HV: F1.2
- new net Precharge/-HV: J2.1 (Pin_1)
Other:
- added sheet Precharge (Precharge.kicad_sch)
- moved on the sheet: J1, J2
Changed lines of the file:
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@@
+	(wire
+		(pts
+			(xy 52.07 133.35) (xy 69.85 133.35)
+		)
+		(stroke
+			(width 0)
+			(type default)
+		)
+	)
 	(wire
 		(pts
@@
 	(wire
 		(pts
+			(xy 19.05 133.35) (xy 20.32 133.35)
+		)
+		(stroke
+			(width 0)
+			(type default)
+		)
+	)
+	(wire
+		(pts
 			(xy 143.51 138.43) (xy 175.26 138.43)
 		)
@@
 	(wire
 		(pts
+			(xy 69.85 133.35) (xy 69.85 123.19)
+		)
+		(stroke
+			(width 0)
+			(type default)
+		)
+	)
+	(wire
+		(pts
 			(xy 130.81 132.08) (xy 134.62 132.08)
 		)
@@
 	(wire
 		(pts
+			(xy 27.94 143.51) (xy 30.48 143.51)
+		)
+		(stroke
+			(width 0)
+			(type default)
+		)
+	)
+	(wire
+		(pts
 			(xy 215.9 157.48) (xy 217.17 157.48)
 		)
@@
 	(wire
 		(pts
+			(xy 69.85 143.51) (xy 69.85 153.67)
+		)
+		(stroke
+			(width 0)
+			(type default)
+		)
+	)
+	(wire
+		(pts
 			(xy 241.3 125.73) (xy 246.38 125.73)
 		)
@@
 	(wire
 		(pts
+			(xy 52.07 143.51) (xy 69.85 143.51)
+		)
+		(stroke
+			(width 0)
+			(type default)
+		)
+	)
+	(wire
+		(pts
 			(xy 262.89 158.75) (xy 262.89 162.56)
 		)
@@
 		(pts
 			(xy 262.89 143.51) (xy 262.89 147.32)
+		)
+		(stroke
+			(width 0)
+			(type default)
+		)
+	)
+	(wire
+		(pts
+			(xy 27.94 133.35) (xy 30.48 133.35)
 		)
 		(stroke
@@
 		(on_board yes)
 		(dnp no)
-		(fields_autoplaced yes)
 		(property "Reference" "#PWR02"
 			(at 71.12 158.75 0)
@@
 		(on_board yes)
 		(dnp no)
-		(fields_autoplaced yes)
 		(property "Reference" "#PWR04"
 			(at 224.79 172.72 0)
@@
 	(symbol
 		(lib_id "Connector:Conn_01x01_Pin")
-		(at 64.77 123.19 0)
+		(at 13.97 133.35 0)
 		(unit 1)
 		(exclude_from_sim no)
@@
 		(on_board yes)
 		(dnp no)
-		(fields_autoplaced yes)
 		(property "Reference" "J1"
-			(at 65.405 118.11 0)
+			(at 14.605 128.27 0)
 			(effects
 				(font
@@
 		)
 		(property "Value" "+HV"
-			(at 65.405 120.65 0)
+			(at 14.732 130.556 0)
 			(effects
 				(font
@@
 		)
 		(property "Footprint" ""
-			(at 64.77 123.19 0)
+			(at 13.97 133.35 0)
 			(effects
 				(font
@@
 		)
 		(property "Datasheet" "~"
-			(at 64.77 123.19 0)
+			(at 13.97 133.35 0)
 			(effects
 				(font
@@
 		)
 		(property "Description" "Generic connector, single row, 01x01, script generated"
-			(at 64.77 123.19 0)
+			(at 13.97 133.35 0)
 			(effects
 				(font
@@
 	(symbol
 		(lib_id "Connector:Conn_01x01_Pin")
-		(at 64.77 153.67 0)
+		(at 22.86 143.51 0)
 		(unit 1)
 		(exclude_from_sim no)
@@
 		(fields_autoplaced yes)
 		(property "Reference" "J2"
-			(at 65.405 148.59 0)
+			(at 23.495 138.43 0)
 			(effects
 				(font
@@
 		)
 		(property "Value" "-HV"
-			(at 65.405 151.13 0)
+			(at 23.495 140.97 0)
 			(effects
 				(font
@@
 		)
 		(property "Footprint" ""
-			(at 64.77 153.67 0)
+			(at 22.86 143.51 0)
 			(effects
 				(font
@@
 		)
 		(property "Datasheet" "~"
-			(at 64.77 153.67 0)
+			(at 22.86 143.51 0)
 			(effects
 				(font
@@
 		)
 		(property "Description" "Generic connector, single row, 01x01, script generated"
-			(at 64.77 153.67 0)
+			(at 22.86 143.51 0)
 			(effects
 				(font
@@
 		)
 	)
+	(symbol
+		(lib_id "Device:Fuse")
+		(at 24.13 133.35 90)
+		(unit 1)
+		(exclude_from_sim no)
+		(in_bom yes)
+		(on_board yes)
+		(dnp no)
+		(fields_autoplaced yes)
+		(property "Reference" "F1"
+			(at 24.13 127 90)
+			(effects
+				(font
+					(size 1.27 1.27)
+				)
+			)
+		)
+		(property "Value" "Fuse"
+			(at 24.13 129.54 90)
+			(effects
+				(font
+					(size 1.27 1.27)
+				)
+			)
+		)
+		(property "Footprint" ""
+			(at 24.13 135.128 90)
+			(effects
+				(font
+					(size 1.27 1.27)
+				)
+				(hide yes)
+			)
+		)
+		(property "Datasheet" "~"
+			(at 24.13 133.35 0)
+			(effects
+				(font
+					(size 1.27 1.27)
+				)
+				(hide yes)
+			)
+		)
+		(property "Description" "Fuse"
+			(at 24.13 133.35 0)
+			(effects
+				(font
+					(size 1.27 1.27)
+				)
+				(hide yes)
+			)
+		)
+		(pin "2"
+		)
+		(pin "1"
+		)
+		(instances
+			(project ""
+				(path "/7abb3fa5-98ae-49c0-a1ab-5c244bba5721"
+					(reference "F1")
+					(unit 1)
+				)
+			)
+		)
+	)
 	(sheet
 		(at 226.06 118.11)
@@
 				)
 			)
+		)
+	)
+	(sheet
+		(at 30.48 130.81)
+		(size 21.59 15.24)
+		(exclude_from_sim no)
+		(in_bom yes)
+		(on_board yes)
+		(dnp no)
+		(fields_autoplaced yes)
+		(stroke
+			(width 0.1524)
+			(type solid)
+		)
+		(fill
+			(color 0 0 0 0.0000)
+		)
+		(property "Sheetname" "Precharge"
+			(at 30.48 130.0984 0)
+			(effects
+				(font
+					(size 1.27 1.27)
+				)
+				(justify left bottom)
+			)
+		)
+		(property "Sheetfile" "Precharge.kicad_sch"
+			(at 30.48 146.6346 0)
+			(effects
+				(font
+					(size 1.27 1.27)
+				)
+				(justify left top)
+			)
+		)
+		(pin "+HV" input
+			(at 30.48 133.35 180)
+			(effects
+				(font
+					(size 1.27 1.27)
+				)
+				(justify left)
+			)
+		)
+		(pin "+HV_PC" output
+			(at 52.07 133.35 0)
+			(effects
+				(font
+					(size 1.27 1.27)
+				)
+				(justify right)
+			)
+		)
+		(pin "-HV" input
+			(at 30.48 143.51 180)
+			(effects
+				(font
+					(size 1.27 1.27)
+				)
+				(justify left)
+			)
+		)
+		(pin "-HV_PC" output
+			(at 52.07 143.51 0)
+			(effects
+				(font
+					(size 1.27 1.27)
+				)
+				(justify right)
+			)
+		)
+		(instances
+			(project "LLC Test Bench"
+				(path "/7abb3fa5-98ae-49c0-a1ab-5c244bba5721"
+					(page "4")
+				)
+			)

Commit message: Implemented OTP(?) + Comments/Minor Symbol Change
- Implemented OTP to trip at 85C
- Changed R symbol in Root to R_US
- Added many comments explaining calculations for OTP

Notes:
- The calculations were derived from a selected component (ERT-JZEG103FA), to be able to trip OTP, a 8kOhm resistor was required. Therefore, a resistor was put in series with the NTC Thermistor to make up the difference the standalone Thermistor could not make.
- From my best understanding of the OVP/OTP pin, the voltage on the pin cannot reach above the OVP trip voltage @ 3.5V. The Thermistor successfully accounts for this by its operation @ 25C setting the pin voltage to 1.65 if this is the case

Please review and check work Thanks
Parts:
- R6, R7: symbol Device:R -> Device:R_US
Changed lines of the file:
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@@
 	)
 	(symbol
-		(lib_id "Device:R")
+		(lib_id "Device:R_US")
 		(at 238.76 157.48 90)
 		(mirror x)
@@
 		)
 		(property "Footprint" ""
-			(at 238.76 155.702 90)
+			(at 239.014 158.496 90)
 			(effects
 				(font
@@
 			)
 		)
-		(property "Description" "Resistor"
+		(property "Description" "Resistor, US symbol"
 			(at 238.76 157.48 0)
 			(effects
@@
 	)
 	(symbol
-		(lib_id "Device:R")
+		(lib_id "Device:R_US")
 		(at 212.09 157.48 90)
 		(mirror x)
@@
 		)
 		(property "Footprint" ""
-			(at 212.09 155.702 90)
+			(at 212.344 158.496 90)
 			(effects
 				(font
@@
 			)
 		)
-		(property "Description" "Resistor"
+		(property "Description" "Resistor, US symbol"
 			(at 212.09 157.48 0)
 			(effects

Commit message: Changed transformer to include tertiary winding
Notes:
- Schematic is not updated for connections (my drag selection does not work on my computer 😡 )
Parts:
- removed TR1: B66368B1020T001, FS_4_Global_Footprint_Library:DIPS4064W80P508L5450H4090Q20N, symbol Transformer:ADT1-1WT-1
- added T1: Transformer_SP_2S, FS_4_Global_Footprint_Library:DIPS4064W80P508L5450H4090Q20N, symbol Device:Transformer_SP_2S
Changed lines of the file:
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@@
+	)
+	(symbol
+		(lib_id "Device:Transformer_SP_2S")
+		(at 194.31 118.11 180)
+		(unit 1)
+		(exclude_from_sim no)
+		(in_bom yes)
+		(on_board yes)
+		(dnp no)
+		(fields_autoplaced yes)
+		(property "Reference" "T1"
+			(at 194.31 102.87 0)
+			(effects
+				(font
+					(size 1.27 1.27)
+				)
+			)
+		)
+		(property "Value" "Transformer_SP_2S"
+			(at 194.31 105.41 0)
+			(effects
+				(font
+					(size 1.27 1.27)
+				)
+			)
+		)
+		(property "Footprint" "FS_4_Global_Footprint_Library:DIPS4064W80P508L5450H4090Q20N"
+			(at 194.31 118.11 0)
+			(effects
+				(font
+					(size 1.27 1.27)
+				)
+				(hide yes)
+			)
+		)
+		(property "Datasheet" "https://www.tdk-electronics.tdk.com/inf/80/db/fer/etd_49_25_16.pdf"
+			(at 194.31 118.11 0)
+			(effects
+				(font
+					(size 1.27 1.27)
+				)
+				(hide yes)
+			)
+		)
+		(property "Description" "BOBBIN COIL FORMER ETD 49X25X16"
+			(at 194.31 118.11 0)
+			(effects
+				(font
+					(size 1.27 1.27)
+				)
+				(hide yes)
+			)
+		)
+		(pin "7"
+		)
+		(pin "1"
+		)
+		(pin "4"
+		)
+		(pin "3"
+		)
+		(pin "2"
+		)
+		(pin "5"
+		)
+		(pin "6"
+		)
+		(instances
+			(project ""
+				(path "/7abb3fa5-98ae-49c0-a1ab-5c244bba5721"
+					(reference "T1")
+					(unit 1)
+				)
+			)
+		)
 	)
 	(symbol
@@
 					(unit 1)
 				)
-			)
-		)
-	)
-	(symbol
-		(lib_id "Transformer:ADT1-1WT-1")
-		(at 201.93 143.51 0)
-		(unit 1)
-		(exclude_from_sim no)
-		(in_bom yes)
-		(on_board yes)
-		(dnp no)
-		(fields_autoplaced yes)
-		(property "Reference" "TR1"
-			(at 201.93 133.35 0)
-			(effects
-				(font
-					(size 1.27 1.27)
-				)
-			)
-		)
-		(property "Value" "B66368B1020T001"
-			(at 201.93 135.89 0)
-			(effects
-				(font
-					(size 1.27 1.27)
-				)
-			)
-		)
-		(property "Footprint" "FS_4_Global_Footprint_Library:DIPS4064W80P508L5450H4090Q20N"
-			(at 201.93 152.4 0)
-			(effects
-				(font
-					(size 1.27 1.27)
-				)
-				(hide yes)
-			)
-		)
-		(property "Datasheet" "https://www.tdk-electronics.tdk.com/inf/80/db/fer/etd_49_25_16.pdf"
-			(at 201.93 143.51 0)
-			(effects
-				(font
-					(size 1.27 1.27)
-				)
-				(hide yes)
-			)
-		)
-		(property "Description" "BOBBIN COIL FORMER ETD 49X25X16"
-			(at 201.93 143.51 0)
-			(effects
-				(font
-					(size 1.27 1.27)
-				)
-				(hide yes)
-			)
-		)
-		(pin "3"
-		)
-		(pin "2"
-		)
-		(pin "1"
-		)
-		(pin "5"
-		)
-		(pin "4"
-		)
-		(pin "6"
-		)
-		(instances
-			(project ""
-				(path "/7abb3fa5-98ae-49c0-a1ab-5c244bba5721"
-					(reference "TR1")
-					(unit 1)
-				)

Commit message: Added Tertiary Winding for VCCP + ISNS
- Added Tertiary Winding for VCCP; used global label to connect to LLC Controller
- Added ISNS to connect to LLC Controller
Parts:
- added C7, C8: C, symbol Device:C
- added D2: D, symbol Device:D
Connections:
- net +Vout: now also T1.2 (PM)
- net GNDPWR: now also T1.4 (OUT1A), T1.6 (OUT2A), C7.2, C8.1
- net VD1: now also T1.1 (IN+)
- net VD2: now also T1.3 (IN-)
- net at T1.5 (OUT1B): now also C2.2
- net at T1.7 (OUT2B): now also D2.2 (A)
- new net ISNS: C8.2
- new net VCCP: C7.1, D2.1 (K)
Other:
- note added: "Select Tertiary winding ratio"
- moved on the sheet: C2, R10, R8, R9, T1

Commit message: Feedback Pin Implementation
- Implemented Feedback Pin on Root Page
- Altered schematic for output side a bit

Notes:
- Select a Vref using the voltage divider for the shunt regulator on Feedback Implementation
- Feedback global labels may be confusing, there is a internal current source that flows out of the FB pin into the BJT of the optocoupler.
Parts:
- added C9: C, symbol Device:C
- added R12, R13, R14: R_US, symbol Device:R_US
- added U3: Optocoupler, symbol Isolator:SFH617A-1
- added U4: TL431D, Package_SO:SOIC-8_3.9x4.9mm_P1.27mm, symbol Reference_Voltage:TL431D
Connections:
- net +Vout: now also Q3.3 (S), Q4.3 (S), R12.1, R13.1; no longer T1.2 (PM)
- net GND: now also T1.2 (PM); no longer Q3.3 (S), Q4.3 (S)
- net GNDPWR: now also U3.3
- new net: C9.1, R13.2, R14.1, U4.8 (REF)
- new net: C9.2, U3.2, U4.1 (K)
- new net: R14.2, U4.2 (A), U4.3 (A), U4.6 (A), U4.7 (A)
- new net: R12.2, U3.1
- new net FB: U3.4
Other:
- note added: "Current flows out of FB pin"
- note added: "Operation Principle: Vout exceeds Vref -> allows Optocoupler to conduct more -> BJT conducts more FB pin voltage drops"
- note added: "Vref: Configure Voltage Divider to program Shunt Regulator"
- moved on the sheet: C4, J3, J4
