File: LLC Test Bench/LLC Test Bench.kicad_sch (KiCad schematic)
At the start: 27 parts, among them J1 +HV, J2 -HV, J3 +LV, J4 -LV, Q1 NMOS, Q2 NMOS, Q3 NMOS, Q4 NMOS, T1 Transformer_SP_2S, U3 Optocoupler, U4 TL431D

Commit message: changed resonant tank values and blk pin
Parts:
- removed R10: 29.4k, symbol Device:R_Small_US
- removed R9: 390, symbol Device:R_Small_US
- added R9: 18k, symbol Device:R_US
- C2: value 500nF -> 1uF
- R8: value 2M -> 1.15M
Connections:
- net GNDPWR: now also R9.2
- net LLC Controller/Gate Driver/BLK: now also R9.1
Other:
- note added: "BLK Start Voltage : 77V BLK Stop Voltage : 65V"
- note added: "Lr = 1.126uH Lm = 6uH"
- note removed: "Hys_Voltage/I_BLK_Hys = 2MOhms"
- note removed: "Hysteresis Voltage Window (may be changed later) = 10V"
- note removed: "I_BLK_Hys = 5uA"
- note removed: "Lr = 2.5uH Lm = 4.8uH Total 7.3uH"
- note removed: "Rlower = 29.79k"
- note removed: "Select Voltage Divider for VBlk"
- note removed: "V_BLK_Start = V_BLK_Stop + V_BLK_StartHys = 1.1V Nom"
- note removed: "V_BLK_Start_Hys = 0.1V Nom"
- note removed: "V_BLK_Stop = 1V Nom"
- note removed: "V_entry = 74.9V V_exit = 84.9"
- note removed: "Vin_min = 75 Select Voltage Divider for 75V -> 1.1V"
Changed lines of the file:
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@@
 		)
 	)
-	(text "Hys_Voltage/I_BLK_Hys = 2MOhms"
-		(exclude_from_sim no)
-		(at 91.948 201.168 0)
-		(effects
-			(font
-				(size 1.27 1.27)
-			)
-		)
-	)
 	(text "n = 4.03 turns ratio"
 		(exclude_from_sim no)
@@
 		)
 	)
-	(text "V_BLK_Start = V_BLK_Stop + V_BLK_StartHys\n= 1.1V Nom"
-		(exclude_from_sim no)
-		(at 97.536 174.244 0)
-		(effects
-			(font
-				(size 1.27 1.27)
-			)
-		)
-	)
 	(text "Vref: Configure Voltage Divider to program Shunt Regulator"
 		(exclude_from_sim no)
@@
 		)
 	)
-	(text "Rlower = 29.79k"
-		(exclude_from_sim no)
-		(at 82.804 205.232 0)
-		(effects
-			(font
-				(size 1.27 1.27)
-			)
-		)
-	)
-	(text "Hysteresis Voltage Window (may be changed later) = 10V"
-		(exclude_from_sim no)
-		(at 103.378 190.5 0)
-		(effects
-			(font
-				(size 1.27 1.27)
-			)
-		)
-	)
-	(text "V_entry = 74.9V\nV_exit = 84.9"
-		(exclude_from_sim no)
-		(at 83.058 210.058 0)
-		(effects
-			(font
-				(size 1.27 1.27)
-			)
-		)
-	)
 	(text "drain voltage\nsense pins\n"
 		(exclude_from_sim no)
@@
 		)
 	)
-	(text "Vin_min = 75\nSelect Voltage Divider for 75V -> 1.1V"
+	(text "BLK Start Voltage : 77V\nBLK Stop Voltage : 65V\n"
 		(exclude_from_sim no)
-		(at 93.726 179.324 0)
+		(at 87.884 118.364 0)
 		(effects
 			(font
@@
 		)
 	)
-	(text "Lr = 2.5uH\nLm = 4.8uH\nTotal 7.3uH\n"
+	(text "Lr = 1.126uH\nLm = 6uH\n"
 		(exclude_from_sim no)
 		(at 176.53 181.864 0)
@@
 		)
 	)
-	(text "I_BLK_Hys = 5uA\n"
-		(exclude_from_sim no)
-		(at 83.312 196.088 0)
-		(effects
-			(font
-				(size 1.27 1.27)
-			)
-		)
-	)
 	(text "Current flows out of FB pin"
 		(exclude_from_sim no)
@@
 		)
 	)
-	(text "Select Voltage Divider for VBlk"
-		(exclude_from_sim no)
-		(at 90.17 161.036 0)
-		(effects
-			(font
-				(size 1.27 1.27)
-			)
-		)
-	)
-	(text "V_BLK_Start_Hys = 0.1V Nom\n"
-		(exclude_from_sim no)
-		(at 89.408 165.1 0)
-		(effects
-			(font
-				(size 1.27 1.27)
-			)
-		)
-	)
 	(text "Use Tertiary winding to supply VCCP\n- will also implement OVP\n"
 		(exclude_from_sim no)
@@
 		)
 	)
-	(text "V_BLK_Stop = 1V Nom\n"
-		(exclude_from_sim no)
-		(at 86.36 169.164 0)
-		(effects
-			(font
-				(size 1.27 1.27)
-			)
-		)
-	)
 	(junction
 		(at 267.97 196.85)
@@
 	(wire
 		(pts
-			(xy 83.82 143.51) (xy 83.82 147.32)
-		)
-		(stroke
-			(width 0)
-			(type default)
-		)
-	)
-	(wire
-		(pts
 			(xy 250.19 191.77) (xy 255.27 191.77)
 		)
@@
 	(wire
 		(pts
-			(xy 83.82 152.4) (xy 83.82 153.67)
+			(xy 83.82 148.59) (xy 83.82 153.67)
 		)
 		(stroke
@@
 	(wire
 		(pts
+			(xy 83.82 135.89) (xy 83.82 140.97)
+		)
+		(stroke
+			(width 0)
+			(type default)
+		)
+	)
+	(wire
+		(pts
 			(xy 251.46 162.56) (xy 251.46 166.37)
 		)
@@
 	(wire
 		(pts
-			(xy 83.82 135.89) (xy 83.82 138.43)
-		)
-		(stroke
-			(width 0)
-			(type default)
-		)
-	)
-	(wire
-		(pts
 			(xy 130.81 142.24) (xy 134.62 142.24)
 		)
@@
 	)
 	(symbol
-		(lib_id "Device:R_Small_US")
-		(at 83.82 140.97 0)
-		(unit 1)
-		(exclude_from_sim no)
-		(in_bom yes)
-		(on_board yes)
-		(dnp no)
-		(fields_autoplaced yes)
-		(property "Reference" "R10"
-			(at 86.36 139.6999 0)
-			(effects
-				(font
-					(size 1.27 1.27)
-				)
-				(justify left)
-			)
-		)
-		(property "Value" "29.4k"
-			(at 86.36 142.2399 0)
-			(effects
-				(font
-					(size 1.27 1.27)
-				)
-				(justify left)
-			)
-		)
-		(property "Footprint" ""
-			(at 83.82 140.97 0)
-			(effects
-				(font
-					(size 1.27 1.27)
-				)
-				(hide yes)
-			)
-		)
-		(property "Datasheet" "~"
-			(at 83.82 140.97 0)
-			(effects
-				(font
-					(size 1.27 1.27)
-				)
-				(hide yes)
-			)
-		)
-		(property "Description" "Resistor, small US symbol"
-			(at 83.82 140.97 0)
-			(effects
-				(font
-					(size 1.27 1.27)
-				)
-				(hide yes)
-			)
-		)
-		(pin "1"
-		)
-		(pin "2"
-		)
-		(instances
-			(project "LLC Test Bench"
-				(path "/7abb3fa5-98ae-49c0-a1ab-5c244bba5721"
-					(reference "R10")
-					(unit 1)
-				)
-			)
-		)
-	)
-	(symbol
 		(lib_id "Device:C")
 		(at 166.37 123.19 0)
@@
 		(on_board yes)
 		(dnp no)
-		(fields_autoplaced yes)
 		(property "Reference" "R8"
 			(at 86.36 128.2699 0)
@@
 			)
 		)
-		(property "Value" "2M"
+		(property "Value" "1.15M"
 			(at 86.36 130.8099 0)
 			(effects
@@
 	(symbol
 		(lib_id "Device:R_US")
-		(at 259.08 175.26 270)
+		(at 83.82 144.78 0)
 		(unit 1)
 		(exclude_from_sim no)
@@
 		(on_board yes)
 		(dnp no)
-		(fields_autoplaced yes)
-		(property "Reference" "R12"
-			(at 259.08 168.91 90)
+		(property "Reference" "R9"
+			(at 86.36 143.5099 0)
 			(effects
 				(font
 					(size 1.27 1.27)
 				)
+				(justify left)
 			)
 		)
-		(property "Value" "R_US"
-			(at 259.08 171.45 90)
+		(property "Value" "18k"
+			(at 86.36 146.0499 0)
 			(effects
 				(font
 					(size 1.27 1.27)
 				)
+				(justify left)
 			)
 		)
 		(property "Footprint" ""
-			(at 258.826 176.276 90)
+			(at 84.836 145.034 90)
 			(effects
 				(font
@@
 		)
 		(property "Datasheet" "~"
-			(at 259.08 175.26 0)
+			(at 83.82 144.78 0)
 			(effects
 				(font
@@
 		)
 		(property "Description" "Resistor, US symbol"
-			(at 259.08 175.26 0)
+			(at 83.82 144.78 0)
 			(effects
 				(font
@@
 			)
 		)
-		(pin "1"
-		)
 		(pin "2"
 		)
+		(pin "1"
+		)
 		(instances
-			(project ""
+			(project "LLC Test Bench"
 				(path "/7abb3fa5-98ae-49c0-a1ab-5c244bba5721"
-					(reference "R12")
+					(reference "R9")
 					(unit 1)
 				)
@@
 	)
 	(symbol
-		(lib_id "power:+48V")
-		(at 233.68 116.84 0)
+		(lib_id "Device:R_US")
+		(at 259.08 175.26 270)
 		(unit 1)
 		(exclude_from_sim no)
@@
 		(on_board yes)
 		(dnp no)
-		(property "Reference" "#PWR012"
-			(at 233.68 120.65 0)
+		(fields_autoplaced yes)
+		(property "Reference" "R12"
+			(at 259.08 168.91 90)
 			(effects
 				(font
 					(size 1.27 1.27)
 				)
-				(hide yes)
 			)
 		)
-		(property "Value" "+Vout"
-			(at 230.378 112.776 0)
+		(property "Value" "R_US"
+			(at 259.08 171.45 90)
 			(effects
 				(font
 					(size 1.27 1.27)
 				)
-				(justify left)
 			)
 		)
 		(property "Footprint" ""
-			(at 233.68 116.84 0)
+			(at 258.826 176.276 90)
 			(effects
 				(font
@@
 			)
 		)
-		(property "Datasheet" ""
-			(at 233.68 116.84 0)
+		(property "Datasheet" "~"
+			(at 259.08 175.26 0)
 			(effects
 				(font
@@
 			)
 		)
-		(property "Description" "Power symbol creates a global label with name \"+48V\""
-			(at 233.68 116.84 0)
+		(property "Description" "Resistor, US symbol"
+			(at 259.08 175.26 0)
 			(effects
 				(font
@@
 		(pin "1"
 		)
+		(pin "2"
+		)
 		(instances
-			(project "LLC Test Bench"
+			(project ""
 				(path "/7abb3fa5-98ae-49c0-a1ab-5c244bba5721"
-					(reference "#PWR012")
+					(reference "R12")
 					(unit 1)
 				)
@@
 	)
 	(symbol
-		(lib_id "Device:R_Small_US")
-		(at 83.82 149.86 0)
+		(lib_id "power:+48V")
+		(at 233.68 116.84 0)
 		(unit 1)
 		(exclude_from_sim no)
@@
 		(on_board yes)
 		(dnp no)
-		(fields_autoplaced yes)
-		(property "Reference" "R9"
-			(at 86.36 148.5899 0)
+		(property "Reference" "#PWR012"
+			(at 233.68 120.65 0)
 			(effects
 				(font
 					(size 1.27 1.27)
 				)
-				(justify left)
+				(hide yes)
 			)
 		)
-		(property "Value" "390"
-			(at 86.36 151.1299 0)
+		(property "Value" "+Vout"
+			(at 230.378 112.776 0)
 			(effects
 				(font
@@
 		)
 		(property "Footprint" ""
-			(at 83.82 149.86 0)
+			(at 233.68 116.84 0)
 			(effects
 				(font
@@
 			)
 		)
-		(property "Datasheet" "~"
-			(at 83.82 149.86 0)
+		(property "Datasheet" ""
+			(at 233.68 116.84 0)
 			(effects
 				(font
@@
 			)
 		)
-		(property "Description" "Resistor, small US symbol"
-			(at 83.82 149.86 0)
+		(property "Description" "Power symbol creates a global label with name \"+48V\""
+			(at 233.68 116.84 0)
 			(effects
 				(font
@@
 		(pin "1"
 		)
-		(pin "2"
-		)
 		(instances
-			(project ""
+			(project "LLC Test Bench"
 				(path "/7abb3fa5-98ae-49c0-a1ab-5c244bba5721"
-					(reference "R9")
+					(reference "#PWR012")
 					(unit 1)
 				)
@@
 			)
 		)
-		(property "Value" "500nF"
+		(property "Value" "1uF"
 			(at 168.91 140.97 90)
 			(effects

Commit message: Changes to ISNS
Parts:
- C8: value C -> 150pF
Connections:
- net GNDPWR: now also C2.1; no longer C8.1, T1.4 (OUT1A)
- net LLC Controller/Gate Driver/HS Return: now also T1.5 (OUT1B); no longer C2.1
- net at C2.2: now also C8.1, T1.4 (OUT1A); no longer T1.5 (OUT1B)
Other:
- moved on the sheet: C2
Changed lines of the file:
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@@
 	(wire
 		(pts
+			(xy 165.1 146.05) (xy 186.69 146.05)
+		)
+		(stroke
+			(width 0)
+			(type default)
+		)
+	)
+	(wire
+		(pts
 			(xy 242.57 157.48) (xy 243.84 157.48)
 		)
@@
 	(wire
 		(pts
-			(xy 143.51 153.67) (xy 180.34 153.67)
+			(xy 143.51 153.67) (xy 160.02 153.67)
 		)
 		(stroke
@@
 	(wire
 		(pts
-			(xy 172.72 146.05) (xy 186.69 146.05)
-		)
-		(stroke
-			(width 0)
-			(type default)
-		)
-	)
-	(wire
-		(pts
 			(xy 267.97 191.77) (xy 267.97 196.85)
 		)
@@
 	(wire
 		(pts
+			(xy 167.64 153.67) (xy 180.34 153.67)
+		)
+		(stroke
+			(width 0)
+			(type default)
+		)
+	)
+	(wire
+		(pts
 			(xy 262.89 191.77) (xy 267.97 191.77)
 		)
@@
 			)
 		)
-		(property "Value" "C"
+		(property "Value" "150pF"
 			(at 184.15 163.8299 0)
 			(effects
@@
 	(symbol
 		(lib_id "Device:C")
-		(at 168.91 146.05 90)
+		(at 163.83 153.67 90)
 		(unit 1)
 		(exclude_from_sim no)
@@
 		(fields_autoplaced yes)
 		(property "Reference" "C2"
-			(at 168.91 138.43 90)
+			(at 163.83 146.05 90)
 			(effects
 				(font
@@
 		)
 		(property "Value" "1uF"
-			(at 168.91 140.97 90)
+			(at 163.83 148.59 90)
 			(effects
 				(font
@@
 		)
 		(property "Footprint" ""
-			(at 172.72 145.0848 0)
+			(at 167.64 152.7048 0)
 			(effects
 				(font
@@
 		)
 		(property "Datasheet" "~"
-			(at 168.91 146.05 0)
+			(at 163.83 153.67 0)
 			(effects
 				(font
@@
 		)
 		(property "Description" "Unpolarized capacitor"
-			(at 168.91 146.05 0)
+			(at 163.83 153.67 0)
 			(effects
 				(font
