File: LLC Test Bench/GateDriver.kicad_sch (KiCad schematic)
At the start: 11 parts, among them U1 UCC256612DDBR

Commit message: TSET Pin
Parts:
- C3: value C_Small -> 2.2uF
- R1: value R_Small_US -> 87k
- R2: value R_Small_US -> 500k
Changed lines of the file:
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@@
 			)
 		)
-		(property "Value" "R_Small_US"
+		(property "Value" "500k"
 			(at 49.53 96.5199 0)
 			(effects
@@
 			)
 		)
-		(property "Value" "R_Small_US"
+		(property "Value" "87k"
 			(at 49.53 109.2199 0)
 			(effects
@@
 			)
 		)
-		(property "Value" "C_Small"
+		(property "Value" "2.2uF"
 			(at 88.646 119.126 90)
 			(effects

Commit message: chose ntc resistor, otp operation confirmed
Parts:
- TH1: value Thermistor_NTC_US -> ERT-JZEG103FA
Changed lines of the file:
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@@
 			)
 		)
-		(property "Value" "Thermistor_NTC_US"
+		(property "Value" "ERT-JZEG103FA"
 			(at 49.53 148.9074 0)
 			(effects
@@
 			)
 		)
-		(property "Datasheet" "~"
+		(property "Datasheet" "https://industrial.panasonic.com/cdbs/www-data/pdf/AUA0000/AUA0000C8.pdf"
 			(at 46.99 146.05 0)
 			(effects

Commit message: Changes to ISNS
Parts:
- R5: value R_Small_US -> 500
Changed lines of the file:
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@@
 			)
 		)
-		(property "Value" "R_Small_US"
+		(property "Value" "500"
 			(at 110.49 110.4899 0)
 			(effects

Commit message: added tertiary winding info, removed precharge + fuse
Parts:
- R1: value 87k -> 99k
- R2: value 500k -> 572k
- R3: value R_Small_US -> 462k
- R4: value R_Small_US -> 179k
Other:
- note added: "LL Pin HFBurstEntry at ~160W i.e ~23% of max load"
- note added: "Vbrkdown = 13V"
Changed lines of the file:
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@@
 	(text "Light Load Entry is determined if FBReplica equals HFBurstEntry"
 		(exclude_from_sim no)
-		(at 46.99 67.564 0)
+		(at 122.682 26.162 0)
+		(effects
+			(font
+				(size 1.27 1.27)
+			)
+		)
+	)
+	(text "Vbrkdown = 13V\n"
+		(exclude_from_sim no)
+		(at 36.322 135.128 0)
+		(effects
+			(font
+				(size 1.27 1.27)
+			)
+		)
+	)
+	(text "LL Pin HFBurstEntry at ~160W i.e ~23% of max load"
+		(exclude_from_sim no)
+		(at 41.656 74.676 0)
 		(effects
 			(font
@@
 	(text "Light Load Activation: say 10% of max load -> 10% of 50A = 5A"
 		(exclude_from_sim no)
-		(at 48.006 64.008 0)
+		(at 121.92 23.114 0)
 		(effects
 			(font
@@
 	(text "FBReplica: 0 to 8V\nGiven by FBReplica = (I_FB-I_OPTO) * R_FBInternal\nwhere I_OPTO is 0 at full load"
 		(exclude_from_sim no)
-		(at 42.672 56.388 0)
+		(at 121.666 18.796 0)
 		(effects
 			(font
@@
 			)
 		)
-		(property "Value" "500k"
+		(property "Value" "572k"
 			(at 49.53 96.5199 0)
 			(effects
@@
 			)
 		)
-		(property "Value" "87k"
+		(property "Value" "99k"
 			(at 49.53 109.2199 0)
 			(effects
@@
 			)
 		)
-		(property "Value" "R_Small_US"
+		(property "Value" "462k"
 			(at 30.48 96.5199 0)
 			(effects
@@
 			)
 		)
-		(property "Value" "R_Small_US"
+		(property "Value" "179k"
 			(at 30.48 109.2199 0)
 			(effects

Commit message: Changes to turns ratio, resistor values, 0603 footprint
Changed turn ratio n=4.03 to 4
Changed resistor values to match E96 values
Assigned Resistors 0603 handsolder footprint
Parts:
- R1: value 99k -> 100k; footprint (none) -> Resistor_SMD:R_0603_1608Metric_Pad0.98x0.95mm_HandSolder
- R11, R5: footprint (none) -> Resistor_SMD:R_0603_1608Metric_Pad0.98x0.95mm_HandSolder
- R2: value 572k -> 576k; footprint (none) -> Resistor_SMD:R_0603_1608Metric_Pad0.98x0.95mm_HandSolder
- R3: value 462k -> 464k; footprint (none) -> Resistor_SMD:R_0603_1608Metric_Pad0.98x0.95mm_HandSolder
- R4: value 179k -> 178k; footprint (none) -> Resistor_SMD:R_0603_1608Metric_Pad0.98x0.95mm_HandSolder
Changed lines of the file:
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@@
 			)
 		)
-		(property "Value" "572k"
+		(property "Value" "576k"
 			(at 49.53 96.5199 0)
 			(effects
@@
 			)
 		)
-		(property "Footprint" ""
+		(property "Footprint" "Resistor_SMD:R_0603_1608Metric_Pad0.98x0.95mm_HandSolder"
 			(at 46.99 95.25 0)
 			(effects
@@
 			)
 		)
-		(property "Footprint" ""
+		(property "Footprint" "Resistor_SMD:R_0603_1608Metric_Pad0.98x0.95mm_HandSolder"
 			(at 107.95 109.22 0)
 			(effects
@@
 			)
 		)
-		(property "Value" "99k"
+		(property "Value" "100k"
 			(at 49.53 109.2199 0)
 			(effects
@@
 			)
 		)
-		(property "Footprint" ""
+		(property "Footprint" "Resistor_SMD:R_0603_1608Metric_Pad0.98x0.95mm_HandSolder"
 			(at 46.99 107.95 0)
 			(effects
@@
 			)
 		)
-		(property "Value" "462k"
+		(property "Value" "464k"
 			(at 30.48 96.5199 0)
 			(effects
@@
 			)
 		)
-		(property "Footprint" ""
+		(property "Footprint" "Resistor_SMD:R_0603_1608Metric_Pad0.98x0.95mm_HandSolder"
 			(at 27.94 95.25 0)
 			(effects
@@
 			)
 		)
-		(property "Value" "179k"
+		(property "Value" "178k"
 			(at 30.48 109.2199 0)
 			(effects
@@
 			)
 		)
-		(property "Footprint" ""
+		(property "Footprint" "Resistor_SMD:R_0603_1608Metric_Pad0.98x0.95mm_HandSolder"
 			(at 27.94 107.95 0)
 			(effects
@@
 			)
 		)
-		(property "Footprint" ""
+		(property "Footprint" "Resistor_SMD:R_0603_1608Metric_Pad0.98x0.95mm_HandSolder"
 			(at 48.006 159.004 90)
 			(effects

Commit message: changes to excel, otp/ovp pin
changes to excel sheet, hopefully fully filled out
changes to otp/ovp pin to complete implementation
- ntc thermistor changed, footprint added 0402 1005metric

note: fatal design flaw? check otp/ovp operation if both happen

refer to FS-Research\DCDC\LTSpice Simulations\150kHz\New LLC Sim.asc
Parts:
- R11: value 6.5k -> 25k
- TH1: value ERT-JZEG103FA -> NTCS0402E3104JHT; footprint (none) -> Resistor_SMD:R_0402_1005Metric_Pad0.72x0.64mm_HandSolder
Connections:
- net GND: now also TH1.2
- net OVP/OTP: now also R11.1
Other:
- note added: "OTP Trip at 85C OVP Trip at 110% of Vout"
- note removed: "100uA Internal Current Source flows out of OVP/OTP pin down to GND"
- note removed: "Calculations with ERT-JZEG103FA NTC Thermistor R @ 25C = 10kOhms B25/85 = 3435k R @ 85C = 1451Ohms Solution: Place R in series to make up the difference Total R = R @ 85C + ~6.5kOhms Normal Operation @ 25 : 16.5kOhms, pin voltage set to 1.65V"
- note removed: "OTP Fault @ 85C"
- note removed: "Target Resistance for OTP trip: 0.8/100uA = 8kOhms"
- moved on the sheet: R11, TH1
Changed lines of the file:
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@@
 	(generator_version "9.0")
 	(paper "A4")
-	(text "100uA Internal Current Source flows out of OVP/OTP pin down to GND"
-		(exclude_from_sim no)
-		(at 48.26 185.928 0)
-		(effects
-			(font
-				(size 1.27 1.27)
-			)
-		)
-	)
 	(text "Light Load Entry is determined if FBReplica equals HFBurstEntry"
 		(exclude_from_sim no)
@@
 		)
 	)
+	(text "OTP Trip at 85C\nOVP Trip at 110% of Vout"
+		(exclude_from_sim no)
+		(at 37.846 166.37 0)
+		(effects
+			(font
+				(size 1.27 1.27)
+			)
+		)
+	)
 	(text "BLK, LL, TSET\nMin V: -0.55V\nMax V: 5.5V\n"
 		(exclude_from_sim no)
@@
 		)
 	)
-	(text "OTP Fault @ 85C"
-		(exclude_from_sim no)
-		(at 22.352 193.04 0)
-		(effects
-			(font
-				(size 1.27 1.27)
-			)
-		)
-	)
 	(text "Cboot\nMin 0.1uF\nCalculate as described in Section 8.3.2\n"
 		(exclude_from_sim no)
@@
 		)
 	)
-	(text "Target Resistance for OTP trip: 0.8/100uA = 8kOhms\n"
-		(exclude_from_sim no)
-		(at 40.132 189.484 0)
-		(effects
-			(font
-				(size 1.27 1.27)
-			)
-		)
-	)
 	(text "Low ESR ceramic 2.2uF decoupling cap\n"
 		(exclude_from_sim no)
@@
 		)
 	)
-	(text "Calculations with ERT-JZEG103FA NTC Thermistor\nR @ 25C = 10kOhms\nB25/85 = 3435k\n\nR @ 85C = 1451Ohms\nSolution: Place R in series to make up the difference\n\nTotal R = R @ 85C + ~6.5kOhms\n\nNormal Operation @ 25 : 16.5kOhms, pin voltage set to 1.65V"
-		(exclude_from_sim no)
-		(at 117.856 184.912 0)
-		(effects
-			(font
-				(size 1.27 1.27)
-			)
-		)
-	)
 	(text "VCCP\n(min based on UVLO specs)\nUVLO Rising : 7.5V nom\nUVLO Falling : 6.8 nom\nnom 15V\nmax 18.5V\n\n"
 		(exclude_from_sim no)
@@
 			)
 		)
+	)
+	(junction
+		(at 36.83 153.67)
+		(diameter 0)
+		(color 0 0 0 0)
 	)
 	(junction
@@
 	)
 	(junction
+		(at 46.99 143.51)
+		(diameter 0)
+		(color 0 0 0 0)
+	)
+	(junction
 		(at 130.81 88.9)
 		(diameter 0)
@@
 	(wire
 		(pts
+			(xy 36.83 143.51) (xy 46.99 143.51)
+		)
+		(stroke
+			(width 0)
+			(type default)
+		)
+	)
+	(wire
+		(pts
 			(xy 107.95 113.03) (xy 107.95 111.76)
 		)
@@
 	(wire
 		(pts
+			(xy 36.83 152.4) (xy 36.83 153.67)
+		)
+		(stroke
+			(width 0)
+			(type default)
+		)
+	)
+	(wire
+		(pts
 			(xy 107.95 104.14) (xy 109.22 104.14)
 		)
@@
 	(wire
 		(pts
-			(xy 46.99 162.56) (xy 46.99 165.1)
-		)
-		(stroke
-			(width 0)
-			(type default)
-		)
-	)
-	(wire
-		(pts
 			(xy 96.52 113.03) (xy 96.52 114.3)
 		)
@@
 	(wire
 		(pts
+			(xy 46.99 152.4) (xy 46.99 153.67)
+		)
+		(stroke
+			(width 0)
+			(type default)
+		)
+	)
+	(wire
+		(pts
 			(xy 27.94 90.17) (xy 27.94 92.71)
 		)
@@
 	(wire
 		(pts
+			(xy 46.99 153.67) (xy 36.83 153.67)
+		)
+		(stroke
+			(width 0)
+			(type default)
+		)
+	)
+	(wire
+		(pts
 			(xy 137.16 88.9) (xy 130.81 88.9)
 		)
@@
 	(wire
 		(pts
+			(xy 46.99 144.78) (xy 46.99 143.51)
+		)
+		(stroke
+			(width 0)
+			(type default)
+		)
+	)
+	(wire
+		(pts
 			(xy 106.68 104.14) (xy 107.95 104.14)
 		)
@@
 	(wire
 		(pts
-			(xy 46.99 151.13) (xy 46.99 154.94)
-		)
-		(stroke
-			(width 0)
-			(type default)
-		)
-	)
-	(wire
-		(pts
 			(xy 46.99 140.97) (xy 46.99 143.51)
 		)
@@
 		(pts
 			(xy 83.82 99.06) (xy 86.36 99.06)
+		)
+		(stroke
+			(width 0)
+			(type default)
+		)
+	)
+	(wire
+		(pts
+			(xy 36.83 144.78) (xy 36.83 143.51)
 		)
 		(stroke
@@
 	(symbol
 		(lib_id "Device:Thermistor_NTC_US")
-		(at 46.99 147.32 0)
+		(at 46.99 148.59 0)
 		(unit 1)
 		(exclude_from_sim no)
@@
 		(fields_autoplaced yes)
 		(property "Reference" "TH1"
-			(at 49.53 146.3674 0)
-			(effects
-				(font
-					(size 1.27 1.27)
-				)
-				(justify left)
-			)
-		)
-		(property "Value" "ERT-JZEG103FA"
-			(at 49.53 148.9074 0)
-			(effects
-				(font
-					(size 1.27 1.27)
-				)
-				(justify left)
-			)
-		)
-		(property "Footprint" ""
-			(at 46.99 146.05 0)
-			(effects
-				(font
-					(size 1.27 1.27)
-				)
-				(hide yes)
-			)
-		)
-		(property "Datasheet" "https://industrial.panasonic.com/cdbs/www-data/pdf/AUA0000/AUA0000C8.pdf"
-			(at 46.99 146.05 0)
+			(at 49.53 147.6374 0)
+			(effects
+				(font
+					(size 1.27 1.27)
+				)
+				(justify left)
+			)
+		)
+		(property "Value" "NTCS0402E3104JHT"
+			(at 49.53 150.1774 0)
+			(effects
+				(font
+					(size 1.27 1.27)
+				)
+				(justify left)
+			)
+		)
+		(property "Footprint" "Resistor_SMD:R_0402_1005Metric_Pad0.72x0.64mm_HandSolder"
+			(at 46.99 147.32 0)
+			(effects
+				(font
+					(size 1.27 1.27)
+				)
+				(hide yes)
+			)
+		)
+		(property "Datasheet" "https://www.vishay.com/docs/29003/ntcs0402e3t.pdf"
+			(at 46.99 147.32 0)
 			(effects
 				(font
@@
 		)
 		(property "Description" "Temperature dependent resistor, negative temperature coefficient, US symbol"
-			(at 46.99 147.32 0)
+			(at 46.99 148.59 0)
 			(effects
 				(font
@@
 	(symbol
 		(lib_id "power:GND")
-		(at 46.99 165.1 0)
+		(at 36.83 153.67 0)
 		(unit 1)
 		(exclude_from_sim no)
@@
 		(fields_autoplaced yes)
 		(property "Reference" "#PWR07"
-			(at 46.99 171.45 0)
+			(at 36.83 160.02 0)
 			(effects
 				(font
@@
 		)
 		(property "Value" "GND"
-			(at 46.99 170.18 0)
+			(at 36.83 158.75 0)
 			(effects
 				(font
@@
 		)
 		(property "Footprint" ""
-			(at 46.99 165.1 0)
+			(at 36.83 153.67 0)
 			(effects
 				(font
@@
 		)
 		(property "Datasheet" ""
-			(at 46.99 165.1 0)
+			(at 36.83 153.67 0)
 			(effects
 				(font
@@
 		)
 		(property "Description" "Power symbol creates a global label with name \"GND\" , ground"
-			(at 46.99 165.1 0)
+			(at 36.83 153.67 0)
 			(effects
 				(font
@@
 	(symbol
 		(lib_id "Device:R_US")
-		(at 46.99 158.75 0)
+		(at 36.83 148.59 0)
 		(unit 1)
 		(exclude_from_sim no)
@@
 		(fields_autoplaced yes)
 		(property "Reference" "R11"
-			(at 49.53 157.4799 0)
-			(effects
-				(font
-					(size 1.27 1.27)
-				)
-				(justify left)
-			)
-		)
-		(property "Value" "6.5k"
-			(at 49.53 160.0199 0)
+			(at 39.37 147.3199 0)
+			(effects
+				(font
+					(size 1.27 1.27)
+				)
+				(justify left)
+			)
+		)
+		(property "Value" "25k"
+			(at 39.37 149.8599 0)
 			(effects
 				(font
@@
 		)
 		(property "Footprint" "Resistor_SMD:R_0603_1608Metric_Pad0.98x0.95mm_HandSolder"
-			(at 48.006 159.004 90)
+			(at 37.846 148.844 90)
 			(effects
 				(font
@@
 		)
 		(property "Datasheet" "~"
-			(at 46.99 158.75 0)
+			(at 36.83 148.59 0)
 			(effects
 				(font
@@
 		)
 		(property "Description" "Resistor, US symbol"
-			(at 46.99 158.75 0)
-			(effects
-				(font
+			(at 36.83 148.59 0)
+			(effects
+				(font

Commit message: changes for eseries, digikey url
changed some resistors to match e series
added digikey url to most resistors + thermistor

modified excel sheet to match e series
Parts:
- R1, R3: DigiKey URL (none) -> https://www.digikey.com/en/products/detail/yageo/RC0603FR-0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
- R11: value 25k -> 29.4k; DigiKey URL (none) -> https://www.digikey.com/en/products/detail/stackpole-electr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
- R2: DigiKey URL (none) -> https://www.digikey.com/en/products/detail/panasonic-indust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
- R4: DigiKey URL (none) -> https://www.digikey.com/en/products/detail/stackpole-electr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
- R5: value 500 -> 510; DigiKey URL (none) -> https://www.digikey.com/en/products/detail/panasonic-indust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
- TH1: DigiKey URL (none) -> https://www.digikey.com/en/products/detail/vishay-beyschlag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
Changed lines of the file:
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@@
+			)
+		)
+		(property "DigiKey URL" "https://www.digikey.com/en/products/detail/panasonic-industry/ERJ-3EKF5763V/196413?_gl=1*mu4021*_up*MQ..*_gs*MQ..&gclid=Cj0KCQjwsMLSBhD9ARIsAIpUTDqn3ZWwTn9PhU43E0MsZzIMmkmM5QxQBzprBcsLf3AYVLb0VQ8Kni0aAovbEALw_wcB&gclsrc=aw.ds"
+			(at 46.99 95.25 0)
+			(effects
+				(font
+					(size 1.27 1.27)
+				)
+				(hide yes)
 			)
 		)
@@
 			)
 		)
+		(property "DigiKey URL" "https://www.digikey.com/en/products/detail/vishay-beyschlag-draloric-bc-components/NTCS0402E3104JHT/1245355"
+			(at 46.99 148.59 0)
+			(effects
+				(font
+					(size 1.27 1.27)
+				)
+				(hide yes)
+			)
+		)
 		(pin "2"
 		)
@@
 			)
 		)
-		(property "Value" "500"
+		(property "Value" "510"
 			(at 110.49 110.4899 0)
 			(effects
@@
 			)
 		)
+		(property "DigiKey URL" "https://www.digikey.com/en/products/detail/panasonic-industry/ERJ-3GEYJ511V/104634?_gl=1*1llcpcq*_up*MQ..*_gs*MQ..&gclid=Cj0KCQjwsMLSBhD9ARIsAIpUTDqn3ZWwTn9PhU43E0MsZzIMmkmM5QxQBzprBcsLf3AYVLb0VQ8Kni0aAovbEALw_wcB&gclsrc=aw.ds"
+			(at 107.95 109.22 0)
+			(effects
+				(font
+					(size 1.27 1.27)
+				)
+				(hide yes)
+			)
+		)
 		(pin "2"
 		)
@@
 			)
 		)
+		(property "DigiKey URL" "https://www.digikey.com/en/products/detail/yageo/RC0603FR-07100KL/726889?_gl=1*113c8wh*_up*MQ..*_gs*MQ..&gclid=Cj0KCQjwsMLSBhD9ARIsAIpUTDqn3ZWwTn9PhU43E0MsZzIMmkmM5QxQBzprBcsLf3AYVLb0VQ8Kni0aAovbEALw_wcB&gclsrc=aw.ds"
+			(at 46.99 107.95 0)
+			(effects
+				(font
+					(size 1.27 1.27)
+				)
+				(hide yes)
+			)
+		)
 		(pin "2"
 		)
@@
 			)
 		)
+		(property "DigiKey URL" "https://www.digikey.com/en/products/detail/yageo/RC0603FR-07464KL/727251?_gl=1*2o5rcl*_up*MQ..*_gs*MQ..&gclid=Cj0KCQjwsMLSBhD9ARIsAIpUTDqn3ZWwTn9PhU43E0MsZzIMmkmM5QxQBzprBcsLf3AYVLb0VQ8Kni0aAovbEALw_wcB&gclsrc=aw.ds"
+			(at 27.94 95.25 0)
+			(effects
+				(font
+					(size 1.27 1.27)
+				)
+				(hide yes)
+			)
+		)
 		(pin "2"
 		)
@@
 			)
 		)
+		(property "DigiKey URL" "https://www.digikey.com/en/products/detail/stackpole-electronics-inc/RMCF0603FT178K/1713674?_gl=1*1bfpx5o*_up*MQ..*_gs*MQ..&gclid=Cj0KCQjwsMLSBhD9ARIsAIpUTDqn3ZWwTn9PhU43E0MsZzIMmkmM5QxQBzprBcsLf3AYVLb0VQ8Kni0aAovbEALw_wcB&gclsrc=aw.ds"
+			(at 27.94 107.95 0)
+			(effects
+				(font
+					(size 1.27 1.27)
+				)
+				(hide yes)
+			)
+		)
 		(pin "2"
 		)
@@
 			)
 		)
-		(property "Value" "25k"
+		(property "Value" "29.4k"
 			(at 39.37 149.8599 0)
 			(effects
@@
 			(at 36.83 148.59 0)
 			(effects
+				(font
+					(size 1.27 1.27)
+				)
+				(hide yes)
+			)
+		)
+		(property "DigiKey URL" "https://www.digikey.com/en/products/detail/stackpole-electronics-inc/RMCF0603FT29K4/1761329?_gl=1*1uwch5s*_up*MQ..*_gs*MQ..&gclid=Cj0KCQjwsMLSBhD9ARIsAIpUTDqn3ZWwTn9PhU43E0MsZzIMmkmM5QxQBzprBcsLf3AYVLb0VQ8Kni0aAovbEALw_wcB&gclsrc=aw.ds"
+			(at 36.83 148.59 0)
+			(effects

Commit message: optocoupler work
Parts:
- added D3: D, symbol Device:D
Connections:
- net VCCP: now also D3.2 (A)
- net at C1.2, U1.14 (HB): now also D3.1 (K)
Other:
- note added: "Low ESR ceramic 2.2uF Decoupling Cap"
- note removed: "LO Return common ground reference"
- note removed: "Low ESR ceramic 2.2uF decoupling cap"
Changed lines of the file:
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@@
-		)
-	)
-	(text "LO Return common ground reference\n"
-		(exclude_from_sim no)
-		(at 136.144 105.41 0)
-		(effects
-			(font
-				(size 1.27 1.27)
-			)
 		)
 	)
 	(text "Cboot\nMin 0.1uF\nCalculate as described in Section 8.3.2\n"
 		(exclude_from_sim no)
-		(at 148.336 93.98 0)
+		(at 165.862 91.694 0)
 		(effects
 			(font
@@
 		)
 	)
-	(text "Low ESR ceramic 2.2uF decoupling cap\n"
+	(text "Low ESR ceramic 2.2uF Decoupling Cap\n"
 		(exclude_from_sim no)
 		(at 88.138 125.984 0)
@@
 	)
 	(junction
-		(at 96.52 80.01)
+		(at 130.81 93.98)
 		(diameter 0)
 		(color 0 0 0 0)
@@
 	(wire
 		(pts
+			(xy 96.52 67.31) (xy 96.52 83.82)
+		)
+		(stroke
+			(width 0)
+			(type default)
+		)
+	)
+	(wire
+		(pts
 			(xy 27.94 101.6) (xy 27.94 105.41)
 		)
@@
 	(wire
 		(pts
+			(xy 130.81 95.25) (xy 130.81 93.98)
+		)
+		(stroke
+			(width 0)
+			(type default)
+		)
+	)
+	(wire
+		(pts
 			(xy 107.95 104.14) (xy 107.95 106.68)
 		)
@@
 	(wire
 		(pts
-			(xy 96.52 83.82) (xy 96.52 80.01)
-		)
-		(stroke
-			(width 0)
-			(type default)
-		)
-	)
-	(wire
-		(pts
 			(xy 46.99 90.17) (xy 46.99 92.71)
 		)
@@
 	(wire
 		(pts
+			(xy 130.81 104.14) (xy 130.81 102.87)
+		)
+		(stroke
+			(width 0)
+			(type default)
+		)
+	)
+	(wire
+		(pts
 			(xy 46.99 140.97) (xy 46.99 143.51)
 		)
@@
 	(wire
 		(pts
-			(xy 96.52 78.74) (xy 96.52 80.01)
-		)
-		(stroke
-			(width 0)
-			(type default)
-		)
-	)
-	(wire
-		(pts
 			(xy 83.82 99.06) (xy 86.36 99.06)
 		)
@@
 	(wire
 		(pts
-			(xy 96.52 80.01) (xy 100.33 80.01)
+			(xy 96.52 67.31) (xy 100.33 67.31)
+		)
+		(stroke
+			(width 0)
+			(type default)
+		)
+	)
+	(wire
+		(pts
+			(xy 133.35 104.14) (xy 130.81 104.14)
 		)
 		(stroke
@@
 	(global_label "VCCP"
 		(shape passive)
-		(at 100.33 80.01 0)
+		(at 100.33 67.31 0)
 		(fields_autoplaced yes)
 		(effects
@@
 		)
 		(property "Intersheetrefs" "${INTERSHEET_REFS}"
-			(at 107.1025 80.01 0)
+			(at 107.1025 67.31 0)
 			(effects
 				(font
@@
 	(global_label "VCCP"
 		(shape passive)
+		(at 133.35 104.14 0)
+		(fields_autoplaced yes)
+		(effects
+			(font
+				(size 1.27 1.27)
+			)
+			(justify left)
+		)
+		(property "Intersheetrefs" "${INTERSHEET_REFS}"
+			(at 140.1225 104.14 0)
+			(effects
+				(font
+					(size 1.27 1.27)
+				)
+				(justify left)
+				(hide yes)
+			)
+		)
+	)
+	(global_label "VCCP"
+		(shape passive)
 		(at 81.28 113.03 180)
 		(fields_autoplaced yes)
@@
 	(hierarchical_label "VCCP"
 		(shape input)
-		(at 96.52 78.74 90)
+		(at 96.52 67.31 90)
 		(effects
 			(font
@@
 					(unit 1)
 				)
+			)
+		)
+	)
+	(symbol
+		(lib_id "Device:D")
+		(at 130.81 99.06 270)
+		(unit 1)
+		(exclude_from_sim no)
+		(in_bom yes)
+		(on_board yes)
+		(dnp no)
+		(fields_autoplaced yes)
+		(property "Reference" "D3"
+			(at 133.35 97.7899 90)
+			(effects
+				(font
+					(size 1.27 1.27)
+				)
+				(justify left)
+			)
+		)
+		(property "Value" "D"
+			(at 133.35 100.3299 90)
+			(effects
+				(font
+					(size 1.27 1.27)
+				)
+				(justify left)
+			)
+		)
+		(property "Footprint" ""
+			(at 130.81 99.06 0)
+			(effects
+				(font
+					(size 1.27 1.27)
+				)
+				(hide yes)
+			)
+		)
+		(property "Datasheet" "~"
+			(at 130.81 99.06 0)
+			(effects
+				(font
+					(size 1.27 1.27)
+				)
+				(hide yes)
+			)
+		)
+		(property "Description" "Diode"
+			(at 130.81 99.06 0)
+			(effects
+				(font
+					(size 1.27 1.27)
+				)
+				(hide yes)
+			)
+		)
+		(property "Sim.Device" "D"
+			(at 130.81 99.06 0)
+			(effects
+				(font
+					(size 1.27 1.27)
+				)
+				(hide yes)
+			)
+		)
+		(property "Sim.Pins" "1=K 2=A"
+			(at 130.81 99.06 0)
+			(effects
+				(font
+					(size 1.27 1.27)
+				)
+				(hide yes)
+			)
+		)
+		(pin "2"
+		)
+		(pin "1"
+		)
+		(instances
+			(project ""
+				(path "/7abb3fa5-98ae-49c0-a1ab-5c244bba5721/8386f46e-cab6-47d2-9440-121b271fbf29"
+					(reference "D3")
+					(unit 1)
+				)
